File: 2x64_Hirose_Circular/test-board/test-board.brd (EAGLE design)
At the start: 40 x 40 mm, 62 parts

Commit message: More work on test board.
Parts:
- removed MECH_E0T, MECH_W0T: DF40HEAD, jonnew:DF40-70HEAD
- removed SWITCH1: DIP_SWITCH_8_POS, josh:DIP_SWITCH_8_POS
- removed TET0: 0, jonnew:TETRODE_128_0.5ID_0.7OD
- removed TET1: 1, jonnew:TETRODE_128_0.5ID_0.7OD
- removed TET10: 10, jonnew:TETRODE_128_0.5ID_0.7OD
- removed TET11: 11, jonnew:TETRODE_128_0.5ID_0.7OD
- removed TET12: 12, jonnew:TETRODE_128_0.5ID_0.7OD
- removed TET13: 13, jonnew:TETRODE_128_0.5ID_0.7OD
- removed TET14: 14, jonnew:TETRODE_128_0.5ID_0.7OD
- removed TET15: 15, jonnew:TETRODE_128_0.5ID_0.7OD
- removed TET2: 2, jonnew:TETRODE_128_0.5ID_0.7OD
- removed TET3: 3, jonnew:TETRODE_128_0.5ID_0.7OD
- removed TET4: 4, jonnew:TETRODE_128_0.5ID_0.7OD
- removed TET5: 5, jonnew:TETRODE_128_0.5ID_0.7OD
- removed TET6: 6, jonnew:TETRODE_128_0.5ID_0.7OD
- removed TET7: 7, jonnew:TETRODE_128_0.5ID_0.7OD
- removed TET8: 8, jonnew:TETRODE_128_0.5ID_0.7OD
- removed TET9: 9, jonnew:TETRODE_128_0.5ID_0.7OD
- added R10, R11, R12, R13, R7, R8, R9: 4609-220k, jonnew:RNX8-0.1
- added S1, S2, S3, S4, S5, S6, S7, S8: (no value), jonnew:ADE008
- added SIG_LEVEL: (no value), jonnew:JP3
Connections:
- removed net N$10: R1.4, SWITCH1.P$5
- removed net N$12: R1.2, SWITCH1.P$7
- removed net N$18: SWITCH1.P$10, SWITCH1.P$11, SWITCH1.P$12, SWITCH1.P$13, SWITCH1.P$14, SWITCH1.P$15, SWITCH1.P$16, SWITCH1.P$9
- removed net N$199: AIN_N0T.33, TET7.3
- removed net N$200: AIN_N0T.32, TET7.2
- removed net N$201: AIN_N0T.31, AIN_N0T.P31, TET7.1
- removed net N$202: AIN_N0T.30, AIN_N0T.P30, TET7.0
- removed net N$203: AIN_N0T.29, AIN_N0T.P29, TET6.3
- removed net N$204: AIN_N0T.28, AIN_N0T.P28, TET6.2
- removed net N$205: AIN_N0T.27, AIN_N0T.P27, TET6.1
- removed net N$215: AIN_N0T.17, AIN_N0T.P17, TET3.3
- removed net N$217: AIN_N0T.15, AIN_N0T.P15, TET3.1
- removed net N$218: AIN_N0T.14, AIN_N0T.P14, TET3.0
- removed net N$220: AIN_N0T.12, AIN_N0T.P12, TET2.2
- removed net N$222: AIN_N0T.10, AIN_N0T.P10, TET2.0
- removed net N$7: R1.7, SWITCH1.P$2
- new net N$26: AIN_N0T.33, R9.1, S4.16
- new net N$27: AIN_N0T.32, R9.2, S4.15
- new net N$28: AIN_N0T.31, AIN_N0T.P31, R9.3, S4.14
- new net N$29: AIN_N0T.30, AIN_N0T.P30, R9.4, S4.13
- new net N$30: AIN_N0T.29, AIN_N0T.P29, R9.5, S4.12
- new net N$31: AIN_N0T.28, AIN_N0T.P28, R9.6, S4.11
- new net N$32: AIN_N0T.27, AIN_N0T.P27, R9.7, S4.10
- new net SIG: R1.C, R10.C, R11.C, R12.C, R13.C, R7.C, R8.C, R9.C, SIG_LEVEL.2
- net -40DB: now also SIG_LEVEL.3
- net -80DB: now also SIG_LEVEL.1
- net GND: now also S1.1, S1.2, S1.3, S1.4, S1.5, S1.6, S1.7, S1.8, S2.1, S2.2, S2.3, S2.4, S2.5, S2.6, S2.7, S2.8, S3.1, S3.2, S3.3, S3.4, S3.5, S3.6, S3.7, S3.8, S4.1, S4.2, S4.3, S4.4, S4.5, S4.6, S4.7, S4.8, S5.1, S5.2, S5.3, S5.4, S5.5, S5.6, S5.7, S5.8, S6.1, S6.2, S6.3, S6.4, S6.5, S6.6, S6.7, S6.8, S7.1, S7.2, S7.3, S7.4, S7.5, S7.6, S7.7, S7.8, S8.1, S8.2, S8.3, S8.4, S8.5, S8.6, S8.7, S8.8
- net N$1000: now also R10.8, S5.9; no longer TET8.0
- net N$11: now also AIN_N0T.12, AIN_N0T.P12, R7.6, S2.11; no longer R1.3, SWITCH1.P$6
- net N$13: now also AIN_N0T.10, AIN_N0T.P10, R7.8, S2.9; no longer R1.1, SWITCH1.P$8
- net N$206: now also R9.8, S4.9; no longer TET6.0
- net N$207: now also R8.1, S3.16; no longer TET5.3
- net N$208: now also R8.2, S3.15; no longer TET5.2
- net N$209: now also R8.3, S3.14; no longer TET5.1
- net N$210: now also R8.4, S3.13; no longer TET5.0
- net N$211: now also R8.5, S3.12; no longer TET4.3
- net N$212: now also R8.6, S3.11; no longer TET4.2
- net N$213: now also R8.7, S3.10; no longer TET4.1
- net N$214: now also R8.8, S3.9; no longer TET4.0
- net N$216: now also R7.2, S2.15; no longer TET3.2
- net N$219: now also R7.5, S2.12; no longer TET2.3
- net N$221: now also R7.7, S2.10; no longer TET2.1
- net N$223: now also R1.1, S1.16; no longer TET1.3
- net N$224: now also R1.2, S1.15; no longer TET1.2
- net N$225: now also R1.3, S1.14; no longer TET1.1
- net N$226: now also R1.4, S1.13; no longer TET1.0
- net N$227: now also R1.5, S1.12; no longer TET0.3
- net N$228: now also R1.6, S1.11; no longer TET0.2
- net N$229: now also R1.7, S1.10; no longer TET0.1
- net N$230: now also R1.8, S1.9; no longer TET0.0
- net N$231: now also R10.7, S5.10; no longer TET8.1
- net N$232: now also R10.6, S5.11; no longer TET8.2
- net N$233: now also R10.5, S5.12; no longer TET8.3
- net N$234: now also R10.4, S5.13; no longer TET9.0
- net N$235: now also R10.3, S5.14; no longer TET9.1
- net N$236: now also R10.2, S5.15; no longer TET9.2
- net N$237: now also R10.1, S5.16; no longer TET9.3
- net N$238: now also R11.8, S6.9; no longer TET10.0
- net N$239: now also R11.7, S6.10; no longer TET10.1
- net N$240: now also R11.6, S6.11; no longer TET10.2
- net N$241: now also R11.5, S6.12; no longer TET10.3
- net N$242: now also R11.4, S6.13; no longer TET11.0
- net N$243: now also R11.3, S6.14; no longer TET11.1
- net N$244: now also R11.2, S6.15; no longer TET11.2
- net N$245: now also R11.1, S6.16; no longer TET11.3
- net N$246: now also R12.8, S7.9; no longer TET12.0
- net N$247: now also R12.7, S7.10; no longer TET12.1
- net N$248: now also R12.6, S7.11; no longer TET12.2
- net N$249: now also R12.5, S7.12; no longer TET12.3
- net N$250: now also R12.4, S7.13; no longer TET13.0
- net N$251: now also R12.3, S7.14; no longer TET13.1
- net N$252: now also R12.2, S7.15; no longer TET13.2
- net N$253: now also R12.1, S7.16; no longer TET13.3
- net N$254: now also R13.8, S8.9; no longer TET14.0
- net N$255: now also R13.7, S8.10; no longer TET14.1
- net N$256: now also R13.6, S8.11; no longer TET14.2
- net N$257: now also R13.5, S8.12; no longer TET14.3
- net N$258: now also R13.4, S8.13; no longer TET15.0
- net N$259: now also R13.3, S8.14; no longer TET15.1
- net N$260: now also R13.2, S8.15; no longer TET15.2
- net N$261: now also R13.1, S8.16; no longer TET15.3
- net N$6: now also AIN_N0T.17, AIN_N0T.P17, R7.1, S2.16; no longer R1.8, SWITCH1.P$1
- net N$8: now also AIN_N0T.15, AIN_N0T.P15, R7.3, S2.14; no longer R1.6, SWITCH1.P$3
- net N$9: now also AIN_N0T.14, AIN_N0T.P14, R7.4, S2.13; no longer R1.5, SWITCH1.P$4
Routing:
- net N$258: track 32.2 -> 3.01 mm
- net N$260: track 35.6 -> 6.47 mm
- net N$256: track 31.5 -> 3.02 mm
- net N$254: track 30.6 -> 3.03 mm
- net N$252: track 29.7 -> 3.04 mm
- net N$250: track 28.7 -> 3.03 mm
- net N$248: track 27.6 -> 3.04 mm
- net N$246: track 26.5 -> 3.05 mm
- net N$244: track 25.3 -> 3.00 mm
- net N$242: track 24.0 -> 3.01 mm
- net N$240: track 22.6 -> 2.97 mm
- net N$238: track 21.2 -> 2.92 mm
- net N$236: track 19.7 -> 2.89 mm
- net N$234: track 18.2 -> 2.85 mm
- net N$232: track 16.6 -> 2.74 mm
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
Commit message: Test board layout.
Parts:
- removed AGND_A0, AGND_A1, REF_A0, REF_A1, SHLD_A0, SHLD_A1: LRG_GP, jonnew:GOLDPIN_0.5ID_0.7OD
- removed SJ_A0, SJ_A1: (no value), jonnew:SJ_2_0402
- added R14, R15: (no value), jonnew:0805
- added REF_GND_LINK, REF_GND_LINK1: (no value), jonnew:JP3
- AIN_N0T: device jonnew:DF40-70HEAD-EIB -> jonnew:DF40-70HEAD
- R2, R3, R4, R5, R6: device jonnew:0603 -> jonnew:0805
- moved R13 271.6 mm to (53.3, 27.9), turned to 90 degrees
- moved R10 249.0 mm to (-53.3, 48.3), turned to 270 degrees
- moved S8 249.0 mm to (63.5, 39.4), turned to 90 degrees
- moved R12 240.0 mm to (53.3, 2.54), turned to 90 degrees
- moved R11 232.3 mm to (-53.3, 22.9), turned to 270 degrees
- moved S7 216.7 mm to (63.5, 14.0), turned to 90 degrees
- moved S4 206.7 mm to (-39.4, 63.5), turned to 180 degrees
- moved R9 206.0 mm to (-27.9, 53.3), turned to 180 degrees
- moved S5 201.2 mm to (-63.5, 36.8), turned to 270 degrees
- moved R8 191.1 mm to (-2.54, 53.3), turned to 180 degrees
- moved S3 188.7 mm to (-14.0, 63.5), turned to 180 degrees
- moved S6 186.0 mm to (-63.5, 11.4), turned to 270 degrees
- moved R7 180.4 mm to (22.9, 53.3), turned to 180 degrees
- moved S2 174.5 mm to (11.4, 63.5), turned to 180 degrees
- moved S1 170.0 mm to (36.8, 63.5), turned to 180 degrees
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Connections:
- removed net AGND_A0: AGND_A0.P$1, AIN_N0T.69, AIN_N0T.70, SJ_A0.2
- removed net AGND_A1: AGND_A1.P$1, AIN_N0T.34, AIN_N0T.35, SJ_A1.2
- removed net N$1000: AIN_N0T.37, AIN_N0T.P37, R10.8, S5.9
- removed net N$208: AIN_N0T.24, AIN_N0T.P24, R8.2, S3.15
- removed net N$209: AIN_N0T.23, AIN_N0T.P23, R8.3, S3.14
- removed net N$211: AIN_N0T.21, AIN_N0T.P21, R8.5, S3.12
- removed net N$213: AIN_N0T.19, AIN_N0T.P19, R8.7, S3.10
- removed net N$223: AIN_N0T.9, AIN_N0T.P9, R1.1, S1.16
- removed net N$224: AIN_N0T.8, AIN_N0T.P8, R1.2, S1.15
- removed net N$225: AIN_N0T.7, AIN_N0T.P7, R1.3, S1.14
- removed net N$226: AIN_N0T.6, AIN_N0T.P6, R1.4, S1.13
- removed net N$227: AIN_N0T.5, AIN_N0T.P5, R1.5, S1.12
- removed net N$228: AIN_N0T.4, AIN_N0T.P4, R1.6, S1.11
- removed net N$229: AIN_N0T.3, AIN_N0T.P3, R1.7, S1.10
- removed net N$232: AIN_N0T.39, AIN_N0T.P39, R10.6, S5.11
- removed net N$234: AIN_N0T.41, AIN_N0T.P41, R10.4, S5.13
- removed net N$236: AIN_N0T.43, AIN_N0T.P43, R10.2, S5.15
- removed net N$240: AIN_N0T.47, AIN_N0T.P47, R11.6, S6.11
- removed net N$244: AIN_N0T.51, AIN_N0T.P51, R11.2, S6.15
- removed net N$246: AIN_N0T.53, AIN_N0T.P53, R12.8, S7.9
- removed net N$26: AIN_N0T.33, R9.1, S4.16
- removed net N$32: AIN_N0T.27, AIN_N0T.P27, R9.7, S4.10
- removed net REF_A0: AIN_N0T.1, REF_A0.P$1
- removed net REF_A1: AIN_N0T.36, REF_A1.P$1
- new net N$10: AIN_N0T.3, R1.2, S1.15
- new net N$12: AIN_N0T.4, R1.3, S1.14
- new net N$18: AIN_N0T.7, R1.6, S1.11
- new net N$19: AIN_N0T.8, R1.7, S1.10
- new net N$20: AIN_N0T.6, R1.5, S1.12
- new net N$21: AIN_N0T.2, R1.1, S1.16
- new net N$22: R15.1, REF_GND_LINK1.1
- new net N$23: AIN_N0T.27, R9.2, S4.15
- new net N$24: AIN_N0T.29, R9.4, S4.13
- new net N$25: AIN_N0T.43, R10.7, S5.10
- new net N$33: AIN_N0T.39, R10.3, S5.14
- new net N$34: AIN_N0T.31, R9.6, S4.11
- new net N$36: AIN_N0T.33, R9.8, S4.9
- new net N$37: AIN_N0T.37, R10.1, S5.16
- new net N$38: AIN_N0T.19, R8.2, S3.15
- new net N$39: AIN_N0T.52, R11.8, S6.9
- new net N$40: AIN_N0T.21, R8.4, S3.13
- new net N$42: AIN_N0T.23, R8.6, S3.11
- new net N$43: AIN_N0T.24, R8.7, S3.10
- new net N$47: AIN_N0T.47, R11.3, S6.14
- new net N$57: AIN_N0T.53, R12.1, S7.16
- new net N$7: AIN_N0T.9, R1.8, S1.9
- new net REF_A: AIN_N0T.1, AIN_N0T.36, REF_GND_LINK.2
- new net REF_B: REF_GND_LINK1.2
- net GND: no longer SJ_A0.1, SJ_A1.1
- net HS_GND: now also AIN_N0T.34, AIN_N0T.35, AIN_N0T.69, AIN_N0T.70
- net N$1: now also R14.1, REF_GND_LINK.1; no longer SHLD_A0.P$1, SJ_A0.COM
- net N$11: now also R7.3, S2.14; no longer AIN_N0T.P12, R7.6, S2.11
- net N$13: now also R7.1, S2.16; no longer AIN_N0T.P10, R7.8, S2.9
- net N$2: now also R14.2, REF_GND_LINK.3; no longer SHLD_A1.P$1, SJ_A1.COM
- net N$206: now also R9.1, S4.16; no longer AIN_N0T.P26, R9.8, S4.9
- net N$207: now also R8.8, S3.9; no longer AIN_N0T.P25, R8.1, S3.16
- net N$210: now also R8.5, S3.12; no longer AIN_N0T.P22, R8.4, S3.13
- net N$212: now also R8.3, S3.14; no longer AIN_N0T.P20, R8.6, S3.11
- net N$214: now also R8.1, S3.16; no longer AIN_N0T.P18, R8.8, S3.9
- net N$216: now also R7.7, S2.10; no longer AIN_N0T.P16, R7.2, S2.15
- net N$219: now also R7.4, S2.13; no longer AIN_N0T.P13, R7.5, S2.12
- net N$221: now also R7.2, S2.15; no longer AIN_N0T.P11, R7.7, S2.10
- net N$230: now also AIN_N0T.5, R1.4, S1.13; no longer AIN_N0T.2, AIN_N0T.P2, R1.8, S1.9
- net N$231: now also R10.2, S5.15; no longer AIN_N0T.P38, R10.7, S5.10
- net N$233: now also R10.4, S5.13; no longer AIN_N0T.P40, R10.5, S5.12
- net N$235: now also R10.6, S5.11; no longer AIN_N0T.P42, R10.3, S5.14
- net N$237: now also R10.8, S5.9; no longer AIN_N0T.P44, R10.1, S5.16
- net N$238: now also R11.1, S6.16; no longer AIN_N0T.P45, R11.8, S6.9
- net N$239: now also R11.2, S6.15; no longer AIN_N0T.P46, R11.7, S6.10
- net N$241: now also R11.4, S6.13; no longer AIN_N0T.P48, R11.5, S6.12
- net N$242: now also R11.5, S6.12; no longer AIN_N0T.P49, R11.4, S6.13
- net N$243: now also R11.6, S6.11; no longer AIN_N0T.P50, R11.3, S6.14
- net N$245: now also AIN_N0T.51, R11.7, S6.10; no longer AIN_N0T.52, AIN_N0T.P52, R11.1, S6.16
- net N$247: now also R12.2, S7.15; no longer AIN_N0T.P54, R12.7, S7.10
- net N$248: now also R12.3, S7.14; no longer AIN_N0T.P55, R12.6, S7.11
- net N$249: now also R12.4, S7.13; no longer AIN_N0T.P56, R12.5, S7.12
- net N$250: now also R12.5, S7.12; no longer AIN_N0T.P57, R12.4, S7.13
- net N$251: now also R12.6, S7.11; no longer AIN_N0T.P58, R12.3, S7.14
- net N$252: now also R12.7, S7.10; no longer AIN_N0T.P59, R12.2, S7.15
- net N$253: now also R12.8, S7.9; no longer AIN_N0T.P60, R12.1, S7.16
- net N$254: now also R13.1, S8.16; no longer AIN_N0T.P61, R13.8, S8.9
- net N$255: now also R13.2, S8.15; no longer AIN_N0T.P62, R13.7, S8.10
- net N$256: now also R13.3, S8.14; no longer AIN_N0T.P63, R13.6, S8.11
- net N$257: now also R13.4, S8.13; no longer AIN_N0T.P64, R13.5, S8.12
- net N$258: now also R13.5, S8.12; no longer R13.4, S8.13
- net N$259: now also R13.6, S8.11; no longer R13.3, S8.14
- net N$260: now also R13.7, S8.10; no longer R13.2, S8.15
- net N$261: now also R13.8, S8.9; no longer R13.1, S8.16
- net N$27: now also R9.7, S4.10; no longer R9.2, S4.15
- net N$28: now also R15.2, REF_GND_LINK1.3; no longer AIN_N0T.31, AIN_N0T.P31, R9.3, S4.14
- net N$29: now also R9.5, S4.12; no longer AIN_N0T.P30, R9.4, S4.13
- net N$30: now also AIN_N0T.41, R10.5, S5.12; no longer AIN_N0T.29, AIN_N0T.P29, R9.5, S4.12
- net N$31: now also R9.3, S4.14; no longer AIN_N0T.P28, R9.6, S4.11
- net N$6: now also R7.8, S2.9; no longer AIN_N0T.P17, R7.1, S2.16
- net N$8: now also R7.6, S2.11; no longer AIN_N0T.P15, R7.3, S2.14
- net N$9: now also R7.5, S2.12; no longer AIN_N0T.P14, R7.4, S2.13
Routing:
- net N$259: track 33.5 -> 0.00 mm, vias 2 -> 0
- net N$261: track 33.3 -> 0.00 mm, vias 1 -> 0
- net N$257: track 31.5 -> 0.00 mm
- net N$255: track 30.7 -> 0.00 mm
- net N$253: track 29.8 -> 0.00 mm
- net N$251: track 28.9 -> 0.00 mm
- net N$249: track 27.8 -> 0.00 mm
- net N$247: track 26.7 -> 0.00 mm
- net N$245: track 25.5 -> 0.00 mm
- net N$243: track 24.1 -> 0.00 mm
- net N$241: track 22.8 -> 0.00 mm
- net N$239: track 21.4 -> 0.00 mm
- net N$237: track 19.9 -> 0.00 mm
- net N$235: track 18.4 -> 0.00 mm
- net N$233: track 16.8 -> 0.00 mm
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- removed copper zone on layer 1, net GND
Other:
- board size 40 x 40 mm -> 152.4 x 165.1 mm
