File: 2x64_Hirose_Circular/test-board/test-board.sch (EAGLE design)
At the start: 61 parts

Commit message: More work on test board.
Parts:
- removed MECH_E0T, MECH_W0T: DF40HEAD, jonnew:PINHD-2X35_DF40HEAD
- removed SWITCH1: DIP_SWITCH_8_POS, josh:DIP_SWITCH_8_POS
- removed TET0: 0, jonnew:TETRODE_128_0.5ID_0.7OD
- removed TET1: 1, jonnew:TETRODE_128_0.5ID_0.7OD
- removed TET10: 10, jonnew:TETRODE_128_0.5ID_0.7OD
- removed TET11: 11, jonnew:TETRODE_128_0.5ID_0.7OD
- removed TET12: 12, jonnew:TETRODE_128_0.5ID_0.7OD
- removed TET13: 13, jonnew:TETRODE_128_0.5ID_0.7OD
- removed TET14: 14, jonnew:TETRODE_128_0.5ID_0.7OD
- removed TET15: 15, jonnew:TETRODE_128_0.5ID_0.7OD
- removed TET2: 2, jonnew:TETRODE_128_0.5ID_0.7OD
- removed TET3: 3, jonnew:TETRODE_128_0.5ID_0.7OD
- removed TET4: 4, jonnew:TETRODE_128_0.5ID_0.7OD
- removed TET5: 5, jonnew:TETRODE_128_0.5ID_0.7OD
- removed TET6: 6, jonnew:TETRODE_128_0.5ID_0.7OD
- removed TET7: 7, jonnew:TETRODE_128_0.5ID_0.7OD
- removed TET8: 8, jonnew:TETRODE_128_0.5ID_0.7OD
- removed TET9: 9, jonnew:TETRODE_128_0.5ID_0.7OD
- added R10, R11, R12, R13, R7, R8, R9: 4609-220k, jonnew:RN1X8
- added S1, S2, S3, S4, S5, S6, S7, S8: (no value), jonnew:DIPSW-008_ADE
- added SIG_LEVEL: (no value), jonnew:JP3E
Connections:
- removed net N$10: R1.4, SWITCH1.E1
- removed net N$12: R1.2, SWITCH1.G1
- removed net N$18: SWITCH1.A2, SWITCH1.B2, SWITCH1.C2, SWITCH1.D2, SWITCH1.E2, SWITCH1.F2, SWITCH1.G2, SWITCH1.H2
- removed net N$199: AIN_N0T.33, TET7.3
- removed net N$200: AIN_N0T.32, TET7.2
- removed net N$201: AIN_N0T.31, TET7.1
- removed net N$202: AIN_N0T.30, TET7.0
- removed net N$203: AIN_N0T.29, TET6.3
- removed net N$204: AIN_N0T.28, TET6.2
- removed net N$205: AIN_N0T.27, TET6.1
- removed net N$215: AIN_N0T.17, TET3.3
- removed net N$217: AIN_N0T.15, TET3.1
- removed net N$218: AIN_N0T.14, TET3.0
- removed net N$220: AIN_N0T.12, TET2.2
- removed net N$222: AIN_N0T.10, TET2.0
- removed net N$7: R1.7, SWITCH1.B1
- new net N$26: AIN_N0T.33, R9.1, S4.16
- new net N$27: AIN_N0T.32, R9.2, S4.15
- new net N$28: AIN_N0T.31, R9.3, S4.14
- new net N$29: AIN_N0T.30, R9.4, S4.13
- new net N$30: AIN_N0T.29, R9.5, S4.12
- new net N$31: AIN_N0T.28, R9.6, S4.11
- new net N$32: AIN_N0T.27, R9.7, S4.10
- new net SIG: R1.C, R10.C, R11.C, R12.C, R13.C, R7.C, R8.C, R9.C, SIG_LEVEL.2
- net -40DB: now also SIG_LEVEL.3
- net -80DB: now also SIG_LEVEL.1
- net GND: now also S1.1, S1.2, S1.3, S1.4, S1.5, S1.6, S1.7, S1.8, S2.1, S2.2, S2.3, S2.4, S2.5, S2.6, S2.7, S2.8, S3.1, S3.2, S3.3, S3.4, S3.5, S3.6, S3.7, S3.8, S4.1, S4.2, S4.3, S4.4, S4.5, S4.6, S4.7, S4.8, S5.1, S5.2, S5.3, S5.4, S5.5, S5.6, S5.7, S5.8, S6.1, S6.2, S6.3, S6.4, S6.5, S6.6, S6.7, S6.8, S7.1, S7.2, S7.3, S7.4, S7.5, S7.6, S7.7, S7.8, S8.1, S8.2, S8.3, S8.4, S8.5, S8.6, S8.7, S8.8
- net N$1000: now also R10.8, S5.9; no longer TET8.0
- net N$11: now also AIN_N0T.12, R7.6, S2.11; no longer R1.3, SWITCH1.F1
- net N$13: now also AIN_N0T.10, R7.8, S2.9; no longer R1.1, SWITCH1.H1
- net N$206: now also R9.8, S4.9; no longer TET6.0
- net N$207: now also R8.1, S3.16; no longer TET5.3
- net N$208: now also R8.2, S3.15; no longer TET5.2
- net N$209: now also R8.3, S3.14; no longer TET5.1
- net N$210: now also R8.4, S3.13; no longer TET5.0
- net N$211: now also R8.5, S3.12; no longer TET4.3
- net N$212: now also R8.6, S3.11; no longer TET4.2
- net N$213: now also R8.7, S3.10; no longer TET4.1
- net N$214: now also R8.8, S3.9; no longer TET4.0
- net N$216: now also R7.2, S2.15; no longer TET3.2
- net N$219: now also R7.5, S2.12; no longer TET2.3
- net N$221: now also R7.7, S2.10; no longer TET2.1
- net N$223: now also R1.1, S1.16; no longer TET1.3
- net N$224: now also R1.2, S1.15; no longer TET1.2
- net N$225: now also R1.3, S1.14; no longer TET1.1
- net N$226: now also R1.4, S1.13; no longer TET1.0
- net N$227: now also R1.5, S1.12; no longer TET0.3
- net N$228: now also R1.6, S1.11; no longer TET0.2
- net N$229: now also R1.7, S1.10; no longer TET0.1
- net N$230: now also R1.8, S1.9; no longer TET0.0
- net N$231: now also R10.7, S5.10; no longer TET8.1
- net N$232: now also R10.6, S5.11; no longer TET8.2
- net N$233: now also R10.5, S5.12; no longer TET8.3
- net N$234: now also R10.4, S5.13; no longer TET9.0
- net N$235: now also R10.3, S5.14; no longer TET9.1
- net N$236: now also R10.2, S5.15; no longer TET9.2
- net N$237: now also R10.1, S5.16; no longer TET9.3
- net N$238: now also R11.8, S6.9; no longer TET10.0
- net N$239: now also R11.7, S6.10; no longer TET10.1
- net N$240: now also R11.6, S6.11; no longer TET10.2
- net N$241: now also R11.5, S6.12; no longer TET10.3
- net N$242: now also R11.4, S6.13; no longer TET11.0
- net N$243: now also R11.3, S6.14; no longer TET11.1
- net N$244: now also R11.2, S6.15; no longer TET11.2
- net N$245: now also R11.1, S6.16; no longer TET11.3
- net N$246: now also R12.8, S7.9; no longer TET12.0
- net N$247: now also R12.7, S7.10; no longer TET12.1
- net N$248: now also R12.6, S7.11; no longer TET12.2
- net N$249: now also R12.5, S7.12; no longer TET12.3
- net N$250: now also R12.4, S7.13; no longer TET13.0
- net N$251: now also R12.3, S7.14; no longer TET13.1
- net N$252: now also R12.2, S7.15; no longer TET13.2
- net N$253: now also R12.1, S7.16; no longer TET13.3
- net N$254: now also R13.8, S8.9; no longer TET14.0
- net N$255: now also R13.7, S8.10; no longer TET14.1
- net N$256: now also R13.6, S8.11; no longer TET14.2
- net N$257: now also R13.5, S8.12; no longer TET14.3
- net N$258: now also R13.4, S8.13; no longer TET15.0
- net N$259: now also R13.3, S8.14; no longer TET15.1
- net N$260: now also R13.2, S8.15; no longer TET15.2
- net N$261: now also R13.1, S8.16; no longer TET15.3
- net N$6: now also AIN_N0T.17, R7.1, S2.16; no longer R1.8, SWITCH1.A1
- net N$8: now also AIN_N0T.15, R7.3, S2.14; no longer R1.6, SWITCH1.C1
- net N$9: now also AIN_N0T.14, R7.4, S2.13; no longer R1.5, SWITCH1.D1
Other:
- moved on the sheet: AGND_B0, AGND_B1, R1, REF_B0, REF_B1, SHLD_B0, SHLD_B1, SJ_B0, SJ_B1, TET16, TET17, TET18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

Commit message: Test board layout.
Parts:
- removed AGND_A0, AGND_A1, REF_A0, REF_A1, SHLD_A0, SHLD_A1: LRG_GP, jonnew:GOLDPIN_0.5ID_0.7OD
- removed SJ_A0, SJ_A1: (no value), jonnew:SJ2_0402
- added R14, R15: (no value), jonnew:R_0805
- added REF_GND_LINK, REF_GND_LINK1: (no value), jonnew:JP3E
- AIN_N0T: device jonnew:PINHD-2X35_DF40HEAD-EIB -> jonnew:PINHD-2X35_DF40HEAD
- R2, R3, R4, R5, R6: device jonnew:R_0603 -> jonnew:R_0805
Connections:
- removed net AGND_A0: AGND_A0.0, AIN_N0T.69, AIN_N0T.70, SJ_A0.2
- removed net AGND_A1: AGND_A1.0, AIN_N0T.34, AIN_N0T.35, SJ_A1.2
- removed net N$1000: AIN_N0T.37, R10.8, S5.9
- removed net N$208: AIN_N0T.24, R8.2, S3.15
- removed net N$209: AIN_N0T.23, R8.3, S3.14
- removed net N$211: AIN_N0T.21, R8.5, S3.12
- removed net N$213: AIN_N0T.19, R8.7, S3.10
- removed net N$223: AIN_N0T.9, R1.1, S1.16
- removed net N$224: AIN_N0T.8, R1.2, S1.15
- removed net N$225: AIN_N0T.7, R1.3, S1.14
- removed net N$226: AIN_N0T.6, R1.4, S1.13
- removed net N$227: AIN_N0T.5, R1.5, S1.12
- removed net N$228: AIN_N0T.4, R1.6, S1.11
- removed net N$229: AIN_N0T.3, R1.7, S1.10
- removed net N$232: AIN_N0T.39, R10.6, S5.11
- removed net N$234: AIN_N0T.41, R10.4, S5.13
- removed net N$236: AIN_N0T.43, R10.2, S5.15
- removed net N$240: AIN_N0T.47, R11.6, S6.11
- removed net N$244: AIN_N0T.51, R11.2, S6.15
- removed net N$246: AIN_N0T.53, R12.8, S7.9
- removed net N$26: AIN_N0T.33, R9.1, S4.16
- removed net N$32: AIN_N0T.27, R9.7, S4.10
- removed net REF_A0: AIN_N0T.1, REF_A0.0
- removed net REF_A1: AIN_N0T.36, REF_A1.0
- new net N$10: AIN_N0T.3, R1.2, S1.15
- new net N$12: AIN_N0T.4, R1.3, S1.14
- new net N$18: AIN_N0T.7, R1.6, S1.11
- new net N$19: AIN_N0T.8, R1.7, S1.10
- new net N$20: AIN_N0T.6, R1.5, S1.12
- new net N$21: AIN_N0T.2, R1.1, S1.16
- new net N$22: R15.1, REF_GND_LINK1.1
- new net N$23: AIN_N0T.27, R9.2, S4.15
- new net N$24: AIN_N0T.29, R9.4, S4.13
- new net N$25: AIN_N0T.43, R10.7, S5.10
- new net N$33: AIN_N0T.39, R10.3, S5.14
- new net N$34: AIN_N0T.31, R9.6, S4.11
- new net N$36: AIN_N0T.33, R9.8, S4.9
- new net N$37: AIN_N0T.37, R10.1, S5.16
- new net N$38: AIN_N0T.19, R8.2, S3.15
- new net N$39: AIN_N0T.52, R11.8, S6.9
- new net N$40: AIN_N0T.21, R8.4, S3.13
- new net N$42: AIN_N0T.23, R8.6, S3.11
- new net N$43: AIN_N0T.24, R8.7, S3.10
- new net N$47: AIN_N0T.47, R11.3, S6.14
- new net N$57: AIN_N0T.53, R12.1, S7.16
- new net N$7: AIN_N0T.9, R1.8, S1.9
- new net REF_A: AIN_N0T.1, AIN_N0T.36, REF_GND_LINK.2
- new net REF_B: REF_GND_LINK1.2
- net GND: no longer SJ_A0.1, SJ_A1.1
- net HS_GND: now also AIN_N0T.34, AIN_N0T.35, AIN_N0T.69, AIN_N0T.70
- net N$1: now also R14.1, REF_GND_LINK.1; no longer SHLD_A0.0, SJ_A0.COM
- net N$11: now also R7.3, S2.14; no longer R7.6, S2.11
- net N$13: now also R7.1, S2.16; no longer R7.8, S2.9
- net N$2: now also R14.2, REF_GND_LINK.3; no longer SHLD_A1.0, SJ_A1.COM
- net N$206: now also R9.1, S4.16; no longer R9.8, S4.9
- net N$207: now also R8.8, S3.9; no longer R8.1, S3.16
- net N$210: now also R8.5, S3.12; no longer R8.4, S3.13
- net N$212: now also R8.3, S3.14; no longer R8.6, S3.11
- net N$214: now also R8.1, S3.16; no longer R8.8, S3.9
- net N$216: now also R7.7, S2.10; no longer R7.2, S2.15
- net N$219: now also R7.4, S2.13; no longer R7.5, S2.12
- net N$221: now also R7.2, S2.15; no longer R7.7, S2.10
- net N$230: now also AIN_N0T.5, R1.4, S1.13; no longer AIN_N0T.2, R1.8, S1.9
- net N$231: now also R10.2, S5.15; no longer R10.7, S5.10
- net N$233: now also R10.4, S5.13; no longer R10.5, S5.12
- net N$235: now also R10.6, S5.11; no longer R10.3, S5.14
- net N$237: now also R10.8, S5.9; no longer R10.1, S5.16
- net N$238: now also R11.1, S6.16; no longer R11.8, S6.9
- net N$239: now also R11.2, S6.15; no longer R11.7, S6.10
- net N$241: now also R11.4, S6.13; no longer R11.5, S6.12
- net N$242: now also R11.5, S6.12; no longer R11.4, S6.13
- net N$243: now also R11.6, S6.11; no longer R11.3, S6.14
- net N$245: now also AIN_N0T.51, R11.7, S6.10; no longer AIN_N0T.52, R11.1, S6.16
- net N$247: now also R12.2, S7.15; no longer R12.7, S7.10
- net N$248: now also R12.3, S7.14; no longer R12.6, S7.11
- net N$249: now also R12.4, S7.13; no longer R12.5, S7.12
- net N$250: now also R12.5, S7.12; no longer R12.4, S7.13
- net N$251: now also R12.6, S7.11; no longer R12.3, S7.14
- net N$252: now also R12.7, S7.10; no longer R12.2, S7.15
- net N$253: now also R12.8, S7.9; no longer R12.1, S7.16
- net N$254: now also R13.1, S8.16; no longer R13.8, S8.9
- net N$255: now also R13.2, S8.15; no longer R13.7, S8.10
- net N$256: now also R13.3, S8.14; no longer R13.6, S8.11
- net N$257: now also R13.4, S8.13; no longer R13.5, S8.12
- net N$258: now also R13.5, S8.12; no longer R13.4, S8.13
- net N$259: now also R13.6, S8.11; no longer R13.3, S8.14
- net N$260: now also R13.7, S8.10; no longer R13.2, S8.15
- net N$261: now also R13.8, S8.9; no longer R13.1, S8.16
- net N$27: now also R9.7, S4.10; no longer R9.2, S4.15
- net N$28: now also R15.2, REF_GND_LINK1.3; no longer AIN_N0T.31, R9.3, S4.14
- net N$29: now also R9.5, S4.12; no longer R9.4, S4.13
- net N$30: now also AIN_N0T.41, R10.5, S5.12; no longer AIN_N0T.29, R9.5, S4.12
- net N$31: now also R9.3, S4.14; no longer R9.6, S4.11
- net N$6: now also R7.8, S2.9; no longer R7.1, S2.16
- net N$8: now also R7.6, S2.11; no longer R7.3, S2.14
- net N$9: now also R7.5, S2.12; no longer R7.4, S2.13
Other:
- moved on the sheet: R1, R10, R11, R12, R13, R7, R8, R9, S1, S2, S3, S4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

Commit message: Intial layout for 2x64 Hirose test board complete
- Silkscree needs work, especially for tetrode and channel labels, which
  will be very important
Parts:
- removed AGND_B0, AGND_B1, REF_B0, REF_B1, SHLD_B0, SHLD_B1: LRG_GP, jonnew:GOLDPIN_0.5ID_0.7OD
- removed REF_GND_LINK, REF_GND_LINK1: (no value), jonnew:JP3E
- removed SJ_B0, SJ_B1: (no value), jonnew:SJ2_0402
- removed TET16: 16, jonnew:TETRODE_128_0.5ID_0.7OD
- removed TET17: 17, jonnew:TETRODE_128_0.5ID_0.7OD
- removed TET18: 18, jonnew:TETRODE_128_0.5ID_0.7OD
- removed TET19: 19, jonnew:TETRODE_128_0.5ID_0.7OD
- removed TET20: 20, jonnew:TETRODE_128_0.5ID_0.7OD
- removed TET21: 21, jonnew:TETRODE_128_0.5ID_0.7OD
- removed TET22: 22, jonnew:TETRODE_128_0.5ID_0.7OD
- removed TET23: 23, jonnew:TETRODE_128_0.5ID_0.7OD
- removed TET24: 24, jonnew:TETRODE_128_0.5ID_0.7OD
- removed TET25: 25, jonnew:TETRODE_128_0.5ID_0.7OD
- removed TET26: 26, jonnew:TETRODE_128_0.5ID_0.7OD
- removed TET27: 27, jonnew:TETRODE_128_0.5ID_0.7OD
- removed TET28: 28, jonnew:TETRODE_128_0.5ID_0.7OD
- removed TET29: 29, jonnew:TETRODE_128_0.5ID_0.7OD
- removed TET30: 30, jonnew:TETRODE_128_0.5ID_0.7OD
- removed TET31: 31, jonnew:TETRODE_128_0.5ID_0.7OD
- added R16, R17, R18, R19, R20: 4609-220k, jonnew:RN1X8
- added REFA_GND_LINK, REFB_GND_LINK: (no value), jonnew:JP3E
- added R_GND, R_RA-GND, R_RB-GND: (no value), jonnew:JP2E_THRU-HOLE
- added S10, S11, S12, S13, S14, S15, S16, S9, SIG_ZONE_SELECT: (no value), jonnew:DIPSW-008_ADE
- added TP1, TP2, TP3, TP4, TP5, TP6: (no value), jonnew:TESTPOINT
- added U$1, U$10, U$11, U$12, U$13, U$14, U$15, U$16, U$17, U$18, U$19, U$20, U$21, U$22, U$23, U$24: (no value), test-board:PINHD-1X9
- AIN_S0T: device jonnew:PINHD-2X35_DF40HEAD-EIB -> jonnew:PINHD-2X35_DF40HEAD
- R14, R15, R6: value (none) -> 4609-220k; device jonnew:R_0805 -> jonnew:RN1X8
Connections:
- removed net AGND_B0: AGND_B0.0, AIN_S0T.69, AIN_S0T.70, SJ_B0.2
- removed net AGND_B1: AGND_B1.0, AIN_S0T.34, AIN_S0T.35, SJ_B1.2
- removed net N$1: R14.1, REF_GND_LINK.1
- removed net N$104: AIN_S0T.46, TET26.2
- removed net N$105: AIN_S0T.47, TET26.1
- removed net N$106: AIN_S0T.48, TET26.0
- removed net N$107: AIN_S0T.49, TET27.3
- removed net N$108: AIN_S0T.50, TET27.2
- removed net N$109: AIN_S0T.51, TET27.1
- removed net N$111: AIN_S0T.53, TET28.3
- removed net N$112: AIN_S0T.54, TET28.2
- removed net N$113: AIN_S0T.55, TET28.1
- removed net N$114: AIN_S0T.56, TET28.0
- removed net N$115: AIN_S0T.57, TET29.3
- removed net N$116: AIN_S0T.58, TET29.2
- removed net N$117: AIN_S0T.59, TET29.1
- removed net N$118: AIN_S0T.60, TET29.0
- removed net N$119: AIN_S0T.61, TET30.3
- removed net N$120: AIN_S0T.62, TET30.2
- removed net N$121: AIN_S0T.63, TET30.1
- removed net N$122: AIN_S0T.64, TET30.0
- removed net N$123: AIN_S0T.65, TET31.3
- removed net N$124: AIN_S0T.66, TET31.2
- removed net N$125: AIN_S0T.67, TET31.1
- removed net N$126: AIN_S0T.68, TET31.0
- removed net N$127: AIN_S0T.2, TET16.3
- removed net N$128: AIN_S0T.37, TET24.3
- removed net N$14: GND_IMP.1, R6.1
- removed net N$16: R4.1
- removed net N$17: R5.1
- removed net N$22: R15.1, REF_GND_LINK1.1
- removed net N$5: U$3.GND
- removed net N$96: AIN_S0T.38, TET24.2
- removed net REF_B0: AIN_S0T.1, REF_B0.0
- removed net REF_B1: AIN_S0T.36, REF_B1.0
- new net N$130: AIN_S0T.62, R20.2, S16.15, U$21.2
- new net N$26: AIN_S0T.7, R6.6, S9.11, U$1.6
- new net N$32: AIN_S0T.9, R6.8, S9.9, U$1.8
- new net N$35: AIN_S0T.10, R14.1, S10.16, U$18.1
- new net N$41: AIN_S0T.11, R14.2, S10.15, U$18.2
- new net N$45: AIN_S0T.14, R14.5, S10.12, U$18.5
- new net N$46: AIN_S0T.15, R14.6, S10.11, U$18.6
- new net N$48: AIN_S0T.16, R14.7, S10.10, U$18.7
- new net N$49: AIN_S0T.19, R15.2, S11.15, U$19.2
- new net N$50: AIN_S0T.20, R15.3, S11.14, U$19.3
- new net N$51: AIN_S0T.21, R15.4, S11.13, U$19.4
- new net N$52: AIN_S0T.22, R15.5, S11.12, U$19.5
- new net N$53: AIN_S0T.23, R15.6, S11.11, U$19.6
- new net N$54: AIN_S0T.24, R15.7, S11.10, U$19.7
- new net N$55: AIN_S0T.25, R15.8, S11.9, U$19.8
- new net N$56: AIN_S0T.26, R16.1, S12.16, U$20.1
- new net N$58: AIN_S0T.27, R16.2, S12.15, U$20.2
- new net N$59: AIN_S0T.28, R16.3, S12.14, U$20.3
- new net N$60: AIN_S0T.29, R16.4, S12.13, U$20.4
- new net N$61: AIN_S0T.30, R16.5, S12.12, U$20.5
- new net N$62: AIN_S0T.31, R16.6, S12.11, U$20.6
- new net N$63: AIN_S0T.32, R16.7, S12.10, U$20.7
- new net N$64: AIN_S0T.33, R16.8, S12.9, U$20.8
- new net SIG_A_15-0: R12.C, R13.C, SIG_ZONE_SELECT.5
- new net SIG_A_31-16: R10.C, R11.C, SIG_ZONE_SELECT.6
- new net SIG_A_47-32: R8.C, R9.C, SIG_ZONE_SELECT.7
- new net SIG_A_63-48: R1.C, R7.C, SIG_ZONE_SELECT.8
- new net SIG_B_15-0: R19.C, R20.C, SIG_ZONE_SELECT.1
- new net SIG_B_31-16: R17.C, R18.C, SIG_ZONE_SELECT.2
- new net SIG_B_47-32: R15.C, R16.C, SIG_ZONE_SELECT.3
- new net SIG_B_63-48: R14.C, R6.C, SIG_ZONE_SELECT.4
- net GND: now also GND_IMP.1, R4.1, R5.1, REFA_GND_LINK.1, REFB_GND_LINK.1, R_GND.2, R_RA-GND.2, R_RB-GND.2, S10.1, S10.2, S10.3, S10.4, S10.5, S10.6, S10.7, S10.8, S11.1, S11.2, S11.3, S11.4, S11.5, S11.6, S11.7, S11.8, S12.1, S12.2, S12.3, S12.4, S12.5, S12.6, S12.7, S12.8, S13.1, S13.2, S13.3, S13.4, S13.5, S13.6, S13.7, S13.8, S14.1, S14.2, S14.3, S14.4, S14.5, S14.6, S14.7, S14.8, S15.1, S15.2, S15.3, S15.4, S15.5, S15.6, S15.7, S15.8, S16.1, S16.2, S16.3, S16.4, S16.5, S16.6, S16.7, S16.8, S9.1, S9.2, S9.3, S9.4, S9.5, S9.6, S9.7, S9.8, TP1.1, TP2.1, U$1.9, U$10.9, U$11.9, U$12.9, U$13.9, U$14.9, U$15.9, U$16.9, U$17.9, U$18.9, U$19.9, U$20.9, U$21.9, U$22.9, U$23.9, U$24.9, U$3.GND; no longer SJ_B0.1, SJ_B1.1
- net HS_GND: now also AIN_S0T.34, AIN_S0T.35; no longer AIN_N0T.34, AIN_N0T.35, AIN_N0T.69, AIN_N0T.70
- net N$10: now also U$13.2
- net N$100: now also AIN_S0T.54, R19.2, S15.15, U$22.2; no longer AIN_S0T.42, TET25.2
- net N$101: now also AIN_S0T.56, R19.4, S15.13, U$22.4; no longer AIN_S0T.43, TET25.1
- net N$102: now also AIN_S0T.58, R19.6, S15.11, U$22.6; no longer AIN_S0T.44, TET25.0
- net N$103: now also AIN_S0T.59, R19.7, S15.10, U$22.7; no longer AIN_S0T.45, TET26.3
- net N$11: now also U$12.3
- net N$110: now also AIN_S0T.13, R14.4, S10.13, U$18.4; no longer AIN_S0T.52, TET27.0
- net N$12: now also U$13.3
- net N$13: now also U$12.1
- net N$15: now also REFA_GND_LINK.3, R_RA-GND.1; no longer GND_IMP.3, R6.2
- net N$18: now also U$13.6
- net N$19: now also U$13.7
- net N$2: now also GND_IMP.3, R_GND.1; no longer R14.2, REF_GND_LINK.3
- net N$20: now also U$13.5
- net N$206: now also U$10.1
- net N$207: now also U$11.8
- net N$21: now also U$13.1
- net N$210: now also U$11.5
- net N$212: now also U$11.3
- net N$214: now also U$11.1
- net N$216: now also U$12.7
- net N$219: now also U$12.4
- net N$221: now also U$12.2
- net N$23: now also U$10.2
- net N$230: now also U$13.4
- net N$231: now also U$14.2
- net N$233: now also U$14.4
- net N$235: now also U$14.6
- net N$237: now also U$14.8
- net N$238: now also U$15.1
- net N$239: now also U$15.2
- net N$24: now also U$10.4
- net N$241: now also U$15.4
- net N$242: now also U$15.5
- net N$243: now also U$15.6
- net N$245: now also U$15.7
- net N$247: now also U$16.2
- net N$248: now also U$16.3
- net N$249: now also U$16.4
- net N$25: now also U$14.7
- net N$250: now also U$16.5
- net N$251: now also U$16.6
- net N$252: now also U$16.7
- net N$253: now also U$16.8
- net N$254: now also U$17.1
- net N$255: now also U$17.2
- net N$256: now also U$17.3
- net N$257: now also U$17.4
- net N$258: now also U$17.5
- net N$259: now also U$17.6
- net N$260: now also U$17.7
- net N$261: now also U$17.8
- net N$27: now also U$10.7
- net N$28: now also REFB_GND_LINK.3, R_RB-GND.1; no longer R15.2, REF_GND_LINK1.3
- net N$29: now also U$10.5
- net N$3: now also AIN_S0T.3, R6.2, S9.15, U$1.2; no longer SHLD_B0.0, SJ_B0.COM
- net N$30: now also U$14.5
- net N$31: now also U$10.3
- net N$33: now also U$14.3
- net N$34: now also U$10.6
- net N$36: now also U$10.8
- net N$37: now also U$14.1
- net N$38: now also U$11.2
- net N$39: now also U$15.8
- net N$4: now also AIN_S0T.5, R6.4, S9.13, U$1.4; no longer SHLD_B1.0, SJ_B1.COM
- net N$40: now also U$11.4
- net N$42: now also U$11.6
- net N$43: now also U$11.7
- net N$47: now also U$15.3
- net N$57: now also U$16.1
- net N$6: now also U$12.8
- net N$65: now also AIN_S0T.8, R6.7, S9.10, U$1.7; no longer AIN_S0T.33, TET23.0
- net N$66: now also AIN_S0T.6, R6.5, S9.12, U$1.5; no longer AIN_S0T.32, TET23.1
- net N$67: now also AIN_S0T.4, R6.3, S9.14, U$1.3; no longer AIN_S0T.31, TET23.2
- net N$68: now also AIN_S0T.2, R6.1, S9.16, U$1.1; no longer AIN_S0T.30, TET23.3
- net N$69: now also AIN_S0T.17, R14.8, S10.9, U$18.8; no longer AIN_S0T.29, TET22.0
- net N$7: now also U$13.8
- net N$70: now also AIN_S0T.12, R14.3, S10.14, U$18.3; no longer AIN_S0T.28, TET22.1
- net N$71: now also AIN_S0T.18, R15.1, S11.16, U$19.1; no longer AIN_S0T.27, TET22.2
- net N$72: now also AIN_S0T.61, R20.1, S16.16, U$21.1; no longer AIN_S0T.26, TET22.3
- net N$73: now also AIN_S0T.60, R19.8, S15.9, U$22.8; no longer AIN_S0T.25, TET21.0
- net N$74: now also AIN_S0T.57, R19.5, S15.12, U$22.5; no longer AIN_S0T.24, TET21.1
- net N$75: now also AIN_S0T.55, R19.3, S15.14, U$22.3; no longer AIN_S0T.23, TET21.2
- net N$76: now also AIN_S0T.53, R19.1, S15.16, U$22.1; no longer AIN_S0T.22, TET21.3
- net N$77: now also AIN_S0T.51, R18.7, S14.10, U$23.7; no longer AIN_S0T.21, TET20.0
- net N$78: now also AIN_S0T.48, R18.4, S14.13, U$23.4; no longer AIN_S0T.20, TET20.1
- net N$79: now also AIN_S0T.46, R18.2, S14.15, U$23.2; no longer AIN_S0T.19, TET20.2
- net N$8: now also U$12.6
- net N$80: now also AIN_S0T.40, R17.4, S13.13, U$24.4; no longer AIN_S0T.18, TET20.3
- net N$81: now also AIN_S0T.52, R18.8, S14.9, U$23.8; no longer AIN_S0T.17, TET19.0
- net N$82: now also AIN_S0T.50, R18.6, S14.11, U$23.6; no longer AIN_S0T.16, TET19.1
- net N$83: now also AIN_S0T.49, R18.5, S14.12, U$23.5; no longer AIN_S0T.15, TET19.2
- net N$84: now also AIN_S0T.47, R18.3, S14.14, U$23.3; no longer AIN_S0T.14, TET19.3
- net N$85: now also AIN_S0T.45, R18.1, S14.16, U$23.1; no longer AIN_S0T.13, TET18.0
- net N$86: now also AIN_S0T.67, R20.7, S16.10, U$21.7; no longer AIN_S0T.12, TET18.1
- net N$87: now also AIN_S0T.65, R20.5, S16.12, U$21.5; no longer AIN_S0T.11, TET18.2
- net N$88: now also AIN_S0T.63, R20.3, S16.14, U$21.3; no longer AIN_S0T.10, TET18.3
- net N$89: now also AIN_S0T.44, R17.8, S13.9, U$24.8; no longer AIN_S0T.9, TET17.0
- net N$9: now also U$12.5
- net N$90: now also AIN_S0T.38, R17.2, S13.15, U$24.2; no longer AIN_S0T.8, TET17.1
- net N$91: now also AIN_S0T.39, R17.3, S13.14, U$24.3; no longer AIN_S0T.7, TET17.2
- net N$92: now also AIN_S0T.42, R17.6, S13.11, U$24.6; no longer AIN_S0T.6, TET17.3
- net N$93: now also AIN_S0T.43, R17.7, S13.10, U$24.7; no longer AIN_S0T.5, TET16.0
- net N$94: now also AIN_S0T.41, R17.5, S13.12, U$24.5; no longer AIN_S0T.4, TET16.1
- net N$95: now also AIN_S0T.37, R17.1, S13.16, U$24.1; no longer AIN_S0T.3, TET16.2
- net N$97: now also AIN_S0T.64, R20.4, S16.13, U$21.4; no longer AIN_S0T.39, TET24.1
- net N$98: now also AIN_S0T.66, R20.6, S16.11, U$21.6; no longer AIN_S0T.40, TET24.0
- net N$99: now also AIN_S0T.68, R20.8, S16.9, U$21.8; no longer AIN_S0T.41, TET25.3
- net REF_A: now also REFA_GND_LINK.2; no longer AIN_N0T.36, REF_GND_LINK.2
- net REF_B: now also AIN_S0T.36, REFB_GND_LINK.2; no longer REF_GND_LINK1.2
- net SIG: now also SIG_ZONE_SELECT.10, SIG_ZONE_SELECT.11, SIG_ZONE_SELECT.12, SIG_ZONE_SELECT.13, SIG_ZONE_SELECT.14, SIG_ZONE_SELECT.15, SIG_ZONE_SELECT.16, SIG_ZONE_SELECT.9; no longer R1.C, R10.C, R11.C, R12.C, R13.C, R7.C, R8.C, R9.C
Other:
- moved on the sheet: GND_IMP, R1, R10, R11, R12, R13, R2, R3, R4, R5, R7, R8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
