File: 2x64_Hirose_Circular/test-board/test-board.sch (EAGLE design)
At the start: 69 parts

Commit message: Pretty much done with layout. Do ERC and gerber verification.
Parts:
- removed REFA_GND_LINK, REFB_GND_LINK, SIG_LEVEL: (no value), jonnew:JP3E
- removed SIG_ZONE_SELECT: (no value), jonnew:DIPSW-008_ADE
- removed U$18, U$19, U$20, U$22, U$23, U$24: (no value), test-board:PINHD-1X9
- added BANK_SELECT: KAT1108E, jonnew:DIPSW-008-SPDT_206-124
- added REFA_TO_GND, REFB_TO_GND, SIG_GAIN: (no value), jonnew:JP3E
- added SIG_IN: 1-1634622-0, josh:BNC_RIGHT_ANGLE
- added TP10, TP11, TP12, TP13: TP_4-40, jonnew:TP_4-40
- added TP7: SIG_IN, jonnew:TPPAD1-20
- added TP8: -40dB, jonnew:TPPAD1-20
- added TP9: -80dB, jonnew:TPPAD1-20
- added U$2, U$4, U$5, U$6, U$7: (no value), test-board:PINHD-1X9
- R1, R10, R11, R12, R13, R14, R15, R16, R6, R7, R8, R9: value 4609-220k -> 4609
- R17, R18: value 4609-220k -> 10k; device jonnew:RN1X8 -> jonnew:R_0805
- R19, R20: value 4609-220k -> 100; device jonnew:RN1X8 -> jonnew:R_0805
- R2, R3: value 10k -> 4609; device jonnew:R_0805 -> jonnew:RN1X8
- R4, R5: value 100 -> 4609; device jonnew:R_0805 -> jonnew:RN1X8
- TP1, TP2, TP3, TP4, TP5, TP6: value (none) -> GND; device jonnew:TESTPOINT -> jonnew:TPPAD1-20
- U$3: value BNC_RIGHT_ANGLE -> (none); device josh:BNC_RIGHT_ANGLE -> test-board:PINHD-1X9
- renumbered U$17 to U$8, U$21 to U$9
Connections:
- removed net SIG_A_15-0: R12.C, R13.C, SIG_ZONE_SELECT.5
- removed net SIG_A_31-16: R10.C, R11.C, SIG_ZONE_SELECT.6
- removed net SIG_A_47-32: R8.C, R9.C, SIG_ZONE_SELECT.7
- removed net SIG_A_63-48: R1.C, R7.C, SIG_ZONE_SELECT.8
- removed net SIG_B_15-0: R19.C, R20.C, SIG_ZONE_SELECT.1
- removed net SIG_B_31-16: R17.C, R18.C, SIG_ZONE_SELECT.2
- removed net SIG_B_47-32: R15.C, R16.C, SIG_ZONE_SELECT.3
- removed net SIG_B_63-48: R14.C, R6.C, SIG_ZONE_SELECT.4
- new net SIG_N_15-0: BANK_SELECT.4, R7.C, R8.C
- new net SIG_N_31-16: BANK_SELECT.3, R5.C, R6.C
- new net SIG_N_47-32: BANK_SELECT.2, R1.C, R2.C
- new net SIG_N_63-48: BANK_SELECT.1, R3.C, R4.C
- new net SIG_S_15-0: BANK_SELECT.8, R10.C, R9.C
- new net SIG_S_31-16: BANK_SELECT.7, R11.C, R12.C
- new net SIG_S_47-32: BANK_SELECT.6, R15.C, R16.C
- new net SIG_S_63-48: BANK_SELECT.5, R13.C, R14.C
- net -40DB: now also R17.2, R18.1, R19.2, SIG_GAIN.3, TP8.TP; no longer R2.2, R3.1, R4.2, SIG_LEVEL.3
- net -80DB: now also R18.2, R20.2, SIG_GAIN.1, TP9.TP; no longer R3.2, R5.2, SIG_LEVEL.1
- net GND: now also BANK_SELECT.-, R19.1, R20.1, REFA_TO_GND.1, REFB_TO_GND.1, SIG_IN.GND, TP1.TP, TP10.TP, TP11.TP, TP12.TP, TP13.TP, TP2.TP, TP3.TP, TP4.TP, TP5.TP, TP6.TP, U$2.9, U$3.9, U$4.9, U$5.9, U$6.9, U$7.9; no longer R4.1, R5.1, REFA_GND_LINK.1, REFB_GND_LINK.1, TP1.1, TP2.1, U$18.9, U$19.9, U$20.9, U$22.9, U$23.9, U$24.9, U$3.GND
- net N$10: now also R4.2, S4.15, U$4.2; no longer R1.2, S1.15, U$13.2
- net N$100: now also R10.2, S10.15, U$10.2; no longer R19.2, S15.15, U$22.2
- net N$101: now also R10.4, S10.13, U$10.4; no longer R19.4, S15.13, U$22.4
- net N$102: now also R10.6, S10.11, U$10.6; no longer R19.6, S15.11, U$22.6
- net N$103: now also R10.7, S10.10, U$10.7; no longer R19.7, S15.10, U$22.7
- net N$11: now also R3.3, S3.14, U$3.3; no longer R7.3, S2.14, U$12.3
- net N$110: now also S14.13, U$14.4; no longer S10.13, U$18.4
- net N$12: now also R4.3, S4.14, U$4.3; no longer R1.3, S1.14, U$13.3
- net N$13: now also R3.1, S3.16, U$3.1; no longer R7.1, S2.16, U$12.1
- net N$130: now also R9.2, S9.15; no longer R20.2, S16.15
- net N$15: now also REFA_TO_GND.3; no longer REFA_GND_LINK.3
- net N$18: now also R4.6, S4.11, U$4.6; no longer R1.6, S1.11, U$13.6
- net N$19: now also R4.7, S4.10, U$4.7; no longer R1.7, S1.10, U$13.7
- net N$20: now also R4.5, S4.12, U$4.5; no longer R1.5, S1.12, U$13.5
- net N$206: now also R1.1, S1.16, U$1.1; no longer R9.1, S4.16, U$10.1
- net N$207: now also R2.8, S2.9, U$2.8; no longer R8.8, S3.9, U$11.8
- net N$21: now also R4.1, S4.16, U$4.1; no longer R1.1, S1.16, U$13.1
- net N$210: now also R2.5, S2.12, U$2.5; no longer R8.5, S3.12, U$11.5
- net N$212: now also R2.3, S2.14, U$2.3; no longer R8.3, S3.14, U$11.3
- net N$214: now also R2.1, S2.16, U$2.1; no longer R8.1, S3.16, U$11.1
- net N$216: now also R3.7, S3.10, U$3.7; no longer R7.7, S2.10, U$12.7
- net N$219: now also R3.4, S3.13, U$3.4; no longer R7.4, S2.13, U$12.4
- net N$221: now also R3.2, S3.15, U$3.2; no longer R7.2, S2.15, U$12.2
- net N$23: now also R1.2, S1.15, U$1.2; no longer R9.2, S4.15, U$10.2
- net N$230: now also R4.4, S4.13, U$4.4; no longer R1.4, S1.13, U$13.4
- net N$231: now also R5.2, U$5.2; no longer R10.2, U$14.2
- net N$233: now also R5.4, U$5.4; no longer R10.4, U$14.4
- net N$235: now also R5.6, U$5.6; no longer R10.6, U$14.6
- net N$237: now also R5.8, U$5.8; no longer R10.8, U$14.8
- net N$238: now also R6.1, U$6.1; no longer R11.1, U$15.1
- net N$239: now also R6.2, U$6.2; no longer R11.2, U$15.2
- net N$24: now also R1.4, S1.13, U$1.4; no longer R9.4, S4.13, U$10.4
- net N$241: now also R6.4, U$6.4; no longer R11.4, U$15.4
- net N$242: now also R6.5, U$6.5; no longer R11.5, U$15.5
- net N$243: now also R6.6, U$6.6; no longer R11.6, U$15.6
- net N$245: now also R6.7, U$6.7; no longer R11.7, U$15.7
- net N$247: now also R7.2, U$7.2; no longer R12.2, U$16.2
- net N$248: now also R7.3, U$7.3; no longer R12.3, U$16.3
- net N$249: now also R7.4, U$7.4; no longer R12.4, U$16.4
- net N$25: now also R5.7, U$5.7; no longer R10.7, U$14.7
- net N$250: now also R7.5, U$7.5; no longer R12.5, U$16.5
- net N$251: now also R7.6, U$7.6; no longer R12.6, U$16.6
- net N$252: now also R7.7, U$7.7; no longer R12.7, U$16.7
- net N$253: now also R7.8, U$7.8; no longer R12.8, U$16.8
- net N$254: now also R8.1; no longer R13.1
- net N$255: now also R8.2; no longer R13.2
- net N$256: now also R8.3; no longer R13.3
- net N$257: now also R8.4; no longer R13.4
- net N$258: now also R8.5; no longer R13.5
- net N$259: now also R8.6; no longer R13.6
- net N$26: now also R13.6, S13.11, U$13.6; no longer R6.6, S9.11, U$1.6
- net N$260: now also R8.7; no longer R13.7
- net N$261: now also R8.8; no longer R13.8
- net N$27: now also R1.7, S1.10, U$1.7; no longer R9.7, S4.10, U$10.7
- net N$28: now also REFB_TO_GND.3; no longer REFB_GND_LINK.3
- net N$29: now also R1.5, S1.12, U$1.5; no longer R9.5, S4.12, U$10.5
- net N$3: now also R13.2, S13.15, U$13.2; no longer R6.2, S9.15, U$1.2
- net N$30: now also R5.5, U$5.5; no longer R10.5, U$14.5
- net N$31: now also R1.3, S1.14, U$1.3; no longer R9.3, S4.14, U$10.3
- net N$32: now also R13.8, S13.9, U$13.8; no longer R6.8, S9.9, U$1.8
- net N$33: now also R5.3, U$5.3; no longer R10.3, U$14.3
- net N$34: now also R1.6, S1.11, U$1.6; no longer R9.6, S4.11, U$10.6
- net N$35: now also S14.16, U$14.1; no longer S10.16, U$18.1
- net N$36: now also R1.8, S1.9, U$1.8; no longer R9.8, S4.9, U$10.8
- net N$37: now also R5.1, U$5.1; no longer R10.1, U$14.1
- net N$38: now also R2.2, S2.15, U$2.2; no longer R8.2, S3.15, U$11.2
- net N$39: now also R6.8, U$6.8; no longer R11.8, U$15.8
- net N$4: now also R13.4, S13.13, U$13.4; no longer R6.4, S9.13, U$1.4
- net N$40: now also R2.4, S2.13, U$2.4; no longer R8.4, S3.13, U$11.4
- net N$41: now also S14.15, U$14.2; no longer S10.15, U$18.2
- net N$42: now also R2.6, S2.11, U$2.6; no longer R8.6, S3.11, U$11.6
- net N$43: now also R2.7, S2.10, U$2.7; no longer R8.7, S3.10, U$11.7
- net N$45: now also S14.12, U$14.5; no longer S10.12, U$18.5
- net N$46: now also S14.11, U$14.6; no longer S10.11, U$18.6
- net N$47: now also R6.3, U$6.3; no longer R11.3, U$15.3
- net N$48: now also S14.10, U$14.7; no longer S10.10, U$18.7
- net N$49: now also S15.15, U$15.2; no longer S11.15, U$19.2
- net N$50: now also S15.14, U$15.3; no longer S11.14, U$19.3
- net N$51: now also S15.13, U$15.4; no longer S11.13, U$19.4
- net N$52: now also S15.12, U$15.5; no longer S11.12, U$19.5
- net N$53: now also S15.11, U$15.6; no longer S11.11, U$19.6
- net N$54: now also S15.10, U$15.7; no longer S11.10, U$19.7
- net N$55: now also S15.9, U$15.8; no longer S11.9, U$19.8
- net N$56: now also S16.16, U$16.1; no longer S12.16, U$20.1
- net N$57: now also R7.1, U$7.1; no longer R12.1, U$16.1
- net N$58: now also S16.15, U$16.2; no longer S12.15, U$20.2
- net N$59: now also S16.14, U$16.3; no longer S12.14, U$20.3
- net N$6: now also R3.8, S3.9, U$3.8; no longer R7.8, S2.9, U$12.8
- net N$60: now also S16.13, U$16.4; no longer S12.13, U$20.4
- net N$61: now also S16.12, U$16.5; no longer S12.12, U$20.5
- net N$62: now also S16.11, U$16.6; no longer S12.11, U$20.6
- net N$63: now also S16.10, U$16.7; no longer S12.10, U$20.7
- net N$64: now also S16.9, U$16.8; no longer S12.9, U$20.8
- net N$65: now also R13.7, S13.10, U$13.7; no longer R6.7, S9.10, U$1.7
- net N$66: now also R13.5, S13.12, U$13.5; no longer R6.5, S9.12, U$1.5
- net N$67: now also R13.3, S13.14, U$13.3; no longer R6.3, S9.14, U$1.3
- net N$68: now also R13.1, S13.16, U$13.1; no longer R6.1, S9.16, U$1.1
- net N$69: now also S14.9, U$14.8; no longer S10.9, U$18.8
- net N$7: now also R4.8, S4.9, U$4.8; no longer R1.8, S1.9, U$13.8
- net N$70: now also S14.14, U$14.3; no longer S10.14, U$18.3
- net N$71: now also S15.16, U$15.1; no longer S11.16, U$19.1
- net N$72: now also R9.1, S9.16; no longer R20.1, S16.16
- net N$73: now also R10.8, S10.9, U$10.8; no longer R19.8, S15.9, U$22.8
- net N$74: now also R10.5, S10.12, U$10.5; no longer R19.5, S15.12, U$22.5
- net N$75: now also R10.3, S10.14, U$10.3; no longer R19.3, S15.14, U$22.3
- net N$76: now also R10.1, S10.16, U$10.1; no longer R19.1, S15.16, U$22.1
- net N$77: now also R11.7, S11.10, U$11.7; no longer R18.7, S14.10, U$23.7
- net N$78: now also R11.4, S11.13, U$11.4; no longer R18.4, S14.13, U$23.4
- net N$79: now also R11.2, S11.15, U$11.2; no longer R18.2, S14.15, U$23.2
- net N$8: now also R3.6, S3.11, U$3.6; no longer R7.6, S2.11, U$12.6
- net N$80: now also R12.4, S12.13, U$12.4; no longer R17.4, S13.13, U$24.4
- net N$81: now also R11.8, S11.9, U$11.8; no longer R18.8, S14.9, U$23.8
- net N$82: now also R11.6, S11.11, U$11.6; no longer R18.6, S14.11, U$23.6
- net N$83: now also R11.5, S11.12, U$11.5; no longer R18.5, S14.12, U$23.5
- net N$84: now also R11.3, S11.14, U$11.3; no longer R18.3, S14.14, U$23.3
- net N$85: now also R11.1, S11.16, U$11.1; no longer R18.1, S14.16, U$23.1
- net N$86: now also R9.7, S9.10; no longer R20.7, S16.10
- net N$87: now also R9.5, S9.12; no longer R20.5, S16.12
- net N$88: now also R9.3, S9.14; no longer R20.3, S16.14
- net N$89: now also R12.8, S12.9, U$12.8; no longer R17.8, S13.9, U$24.8
- net N$9: now also R3.5, S3.12, U$3.5; no longer R7.5, S2.12, U$12.5
- net N$90: now also R12.2, S12.15, U$12.2; no longer R17.2, S13.15, U$24.2
- net N$91: now also R12.3, S12.14, U$12.3; no longer R17.3, S13.14, U$24.3
- net N$92: now also R12.6, S12.11, U$12.6; no longer R17.6, S13.11, U$24.6
- net N$93: now also R12.7, S12.10, U$12.7; no longer R17.7, S13.10, U$24.7
- net N$94: now also R12.5, S12.12, U$12.5; no longer R17.5, S13.12, U$24.5
- net N$95: now also R12.1, S12.16, U$12.1; no longer R17.1, S13.16, U$24.1
- net N$97: now also R9.4, S9.13; no longer R20.4, S16.13
- net N$98: now also R9.6, S9.11; no longer R20.6, S16.11
- net N$99: now also R9.8, S9.9; no longer R20.8, S16.9
- net REF_A: now also REFA_TO_GND.2; no longer REFA_GND_LINK.2
- net REF_B: now also REFB_TO_GND.2; no longer REFB_GND_LINK.2
- net SIG: now also BANK_SELECT.+, SIG_GAIN.2; no longer SIG_LEVEL.2, SIG_ZONE_SELECT.10, SIG_ZONE_SELECT.11, SIG_ZONE_SELECT.12, SIG_ZONE_SELECT.13, SIG_ZONE_SELECT.14, SIG_ZONE_SELECT.15, SIG_ZONE_SELECT.16, SIG_ZONE_SELECT.9
- net SIG_IN: now also R17.1, SIG_IN.SIG, TP7.TP; no longer R2.1, U$3.SIG
Other:
- moved on the sheet: GND_IMP, R1, R10, R11, R12, R13, R6, R7, R8, R9, R_GND, R_RA-GND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

Commit message: Revsion 1.0 of 128 channel test board sent to fab.
Parts:
- removed REFA_TO_GND, REFB_TO_GND: (no value), jonnew:JP3E
- removed R_RA-GND, R_RB-GND: (no value), jonnew:JP2E_THRU-HOLE
- added REF_N_TO_GND, REF_S_TO_GND: (no value), jonnew:JP3E
- added R_REFNORTH, R_REFSOUTH: (no value), jonnew:JP2E_THRU-HOLE
- S1, S10, S11, S12, S13, S14, S15, S16, S2, S3, S4, S5, S6, S7, S8, S9: value (none) -> ADE
Connections:
- removed net REF_A: AIN_N0T.1, REFA_TO_GND.2
- removed net REF_B: AIN_S0T.36, REFB_TO_GND.2
- new net REF_NORTH: AIN_N0T.1, REF_N_TO_GND.2
- new net REF_SOUTH: AIN_S0T.36, REF_S_TO_GND.2
- net GND: now also REF_N_TO_GND.1, REF_S_TO_GND.1, R_REFNORTH.2, R_REFSOUTH.2; no longer REFA_TO_GND.1, REFB_TO_GND.1, R_RA-GND.2, R_RB-GND.2
- net N$15: now also REF_N_TO_GND.3, R_REFNORTH.1; no longer REFA_TO_GND.3, R_RA-GND.1
- net N$28: now also REF_S_TO_GND.3, R_REFSOUTH.1; no longer REFB_TO_GND.3, R_RB-GND.1
Other:
- moved on the sheet: BANK_SELECT, GND_IMP, R1, R10, R11, R12, R13, R14, R15, R16, R2, R3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
