File: 2x64_Hirose_Circular/cable-adapter/cable-adapter-24.brd (EAGLE design)
At the start: 50.8 x 50.8 mm, 48 parts

Commit message: Toward SPI interface board rev 1.2
- Added jumpers for AUX IN breadboard
- Started basic layout
- Changes in SPI cable pinout will need to be reflected in the
  commutator adapter board.
Connections:
- net MISO1+: now also MISO-.P$1, _MISO1-.P$1; no longer MISO+.P$1, _MISO1+.P$1
- net MISO1-: now also MISO+.P$1, _MISO1+.P$1; no longer MISO-.P$1, _MISO1-.P$1
- net MISO2+: now also MISO2-.P$1, _MISO2-.P$1; no longer MISO2+.P$1, _MISO2+.P$1
- net MISO2-: now also MISO2+.P$1, _MISO2+.P$1; no longer MISO2-.P$1, _MISO2-.P$1
- net MOSI+: now also MOSI-.P$1, _MOSI-.P$1; no longer MOSI+.P$1, _MOSI+.P$1
- net MOSI-: now also MOSI+.P$1, _MOSI+.P$1; no longer MOSI-.P$1, _MOSI-.P$1
Routing:
- net MISO2-: track 3.58 -> 6.18 mm
- net MISO2+: track 6.18 -> 3.58 mm
- net MOSI-: track 2.87 -> 4.09 mm
- net MOSI+: track 4.09 -> 2.87 mm
- net MISO1-: track 4.81 -> 4.09 mm
- net MISO1+: track 4.09 -> 4.81 mm
Changed lines of the file:
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@@
 <wire x1="-0.7" y1="-1.8404125" x2="-0.7" y2="-3.4" width="0.3048" layer="1"/>
-</signal>
-<signal name="MOSI+">
-<contactref element="MOSI+" pad="P$1"/>
-<contactref element="_MOSI+" pad="P$1"/>
-<wire x1="-5.207" y1="-1.143" x2="-4.699" y2="-1.651" width="0.127" layer="1"/>
-<wire x1="-4.699" y1="-1.651" x2="-3.35110625" y2="-1.651" width="0.127" layer="1"/>
-<wire x1="-3.35110625" y1="-1.651" x2="-2.7" y2="-2.30210625" width="0.127" layer="1"/>
-<wire x1="-2.7" y1="-2.30210625" x2="-2.7" y2="-3.4" width="0.127" layer="1"/>
 </signal>
 <signal name="LED+2">
@@
 <wire x1="1.935" y1="1.27" x2="1.3" y2="1.905" width="0.127" layer="1"/>
 <wire x1="1.3" y1="1.905" x2="1.3" y2="3.4" width="0.127" layer="1"/>
-</signal>
-<signal name="MISO2+">
-<contactref element="MISO2+" pad="P$1"/>
-<contactref element="_MISO2+" pad="P$1"/>
-<wire x1="1.5" y1="-3.4" x2="1.5" y2="-2.005584375" width="0.127" layer="1"/>
-<wire x1="1.5" y1="-2.005584375" x2="2.235584375" y2="-1.27" width="0.127" layer="1"/>
-<wire x1="2.235584375" y1="-1.27" x2="4.2545" y2="-1.27" width="0.127" layer="1"/>
-<wire x1="4.2545" y1="-1.27" x2="4.5085" y2="-1.016" width="0.127" layer="1"/>
-<wire x1="4.5085" y1="-1.016" x2="4.5085" y2="-0.635" width="0.127" layer="1"/>
-<wire x1="4.5085" y1="-0.635" x2="5.207" y2="0.0635" width="0.127" layer="1"/>
 </signal>
 <signal name="MISO3+">
@@
 </signal>
 <signal name="MOSI-">
-<contactref element="MOSI-" pad="P$1"/>
-<contactref element="_MOSI-" pad="P$1"/>
-<wire x1="-3.81" y1="-0.5715" x2="-3.5248" y2="-0.5715" width="0.127" layer="1"/>
-<wire x1="-3.5248" y1="-0.5715" x2="-1.7" y2="-2.3963" width="0.127" layer="1"/>
-<wire x1="-1.7" y1="-2.3963" x2="-1.7" y2="-2.4" width="0.127" layer="1"/>
+<contactref element="MOSI+" pad="P$1"/>
+<contactref element="_MOSI+" pad="P$1"/>
+<wire x1="-5.207" y1="-1.143" x2="-4.699" y2="-1.651" width="0.127" layer="1"/>
+<wire x1="-4.699" y1="-1.651" x2="-3.35110625" y2="-1.651" width="0.127" layer="1"/>
+<wire x1="-3.35110625" y1="-1.651" x2="-2.7" y2="-2.30210625" width="0.127" layer="1"/>
+<wire x1="-2.7" y1="-2.30210625" x2="-2.7" y2="-3.4" width="0.127" layer="1"/>
 </signal>
 <signal name="MISO1-">
-<contactref element="MISO-" pad="P$1"/>
-<contactref element="_MISO1-" pad="P$1"/>
-<wire x1="-4.02103125" y1="1.3716" x2="-2.335" y2="1.3716" width="0.127" layer="1"/>
-<wire x1="-2.335" y1="1.3716" x2="-1.7" y2="2.1082" width="0.127" layer="1"/>
-<wire x1="-1.7" y1="2.1082" x2="-1.7" y2="2.4" width="0.127" layer="1"/>
-<wire x1="-4.02103125" y1="1.3716" x2="-5.207" y2="0.18563125" width="0.127" layer="1"/>
-<wire x1="-5.207" y1="0.18563125" x2="-5.207" y2="0" width="0.127" layer="1"/>
-</signal>
-<signal name="MISO1+">
 <contactref element="MISO+" pad="P$1"/>
 <contactref element="_MISO1+" pad="P$1"/>
@@
 </signal>
 <signal name="MISO2-">
-<contactref element="MISO2-" pad="P$1"/>
-<contactref element="_MISO2-" pad="P$1"/>
-<wire x1="5.207" y1="-1.0795" x2="4.699" y2="-1.5875" width="0.127" layer="1"/>
-<wire x1="4.699" y1="-1.5875" x2="2.854" y2="-1.5875" width="0.127" layer="1"/>
-<wire x1="2.854" y1="-1.5875" x2="2.6" y2="-1.8415" width="0.127" layer="1"/>
-<wire x1="2.6" y1="-1.8415" x2="2.6" y2="-2.5" width="0.127" layer="1"/>
+<contactref element="MISO2+" pad="P$1"/>
+<contactref element="_MISO2+" pad="P$1"/>
+<wire x1="1.5" y1="-3.4" x2="1.5" y2="-2.005584375" width="0.127" layer="1"/>
+<wire x1="1.5" y1="-2.005584375" x2="2.235584375" y2="-1.27" width="0.127" layer="1"/>
+<wire x1="2.235584375" y1="-1.27" x2="4.2545" y2="-1.27" width="0.127" layer="1"/>
+<wire x1="4.2545" y1="-1.27" x2="4.5085" y2="-1.016" width="0.127" layer="1"/>
+<wire x1="4.5085" y1="-1.016" x2="4.5085" y2="-0.635" width="0.127" layer="1"/>
+<wire x1="4.5085" y1="-0.635" x2="5.207" y2="0.0635" width="0.127" layer="1"/>
 </signal>
 <signal name="MISO4+">
@@
 <wire x1="-5.22576875" y1="2.4" x2="-3.7" y2="2.4" width="0.127" layer="1"/>
 </signal>
+<signal name="MOSI+">
+<contactref element="MOSI-" pad="P$1"/>
+<contactref element="_MOSI-" pad="P$1"/>
+<wire x1="-3.81" y1="-0.5715" x2="-3.5248" y2="-0.5715" width="0.127" layer="1"/>
+<wire x1="-3.5248" y1="-0.5715" x2="-1.7" y2="-2.3963" width="0.127" layer="1"/>
+<wire x1="-1.7" y1="-2.3963" x2="-1.7" y2="-2.4" width="0.127" layer="1"/>
+</signal>
+<signal name="MISO2+">
+<contactref element="MISO2-" pad="P$1"/>
+<contactref element="_MISO2-" pad="P$1"/>
+<wire x1="5.207" y1="-1.0795" x2="4.699" y2="-1.5875" width="0.127" layer="1"/>
+<wire x1="4.699" y1="-1.5875" x2="2.854" y2="-1.5875" width="0.127" layer="1"/>
+<wire x1="2.854" y1="-1.5875" x2="2.6" y2="-1.8415" width="0.127" layer="1"/>
+<wire x1="2.6" y1="-1.8415" x2="2.6" y2="-2.5" width="0.127" layer="1"/>
+</signal>
+<signal name="MISO1+">
+<contactref element="MISO-" pad="P$1"/>
+<contactref element="_MISO1-" pad="P$1"/>
+<wire x1="-4.02103125" y1="1.3716" x2="-2.335" y2="1.3716" width="0.127" layer="1"/>
+<wire x1="-2.335" y1="1.3716" x2="-1.7" y2="2.1082" width="0.127" layer="1"/>
+<wire x1="-1.7" y1="2.1082" x2="-1.7" y2="2.4" width="0.127" layer="1"/>
+<wire x1="-4.02103125" y1="1.3716" x2="-5.207" y2="0.18563125" width="0.127" layer="1"/>
+<wire x1="-5.207" y1="0.18563125" x2="-5.207" y2="0" width="0.127" layer="1"/>
+</signal>
 </signals>
