File: pcie-host/pcie-host.brd (EAGLE design)
At the start: 167.6 x 111.2 mm, 237 parts, among them Q1 BSH103, Q2 BSH103, Q3 NDS351AN, Q4 NDS351AN, Q5 NDS351AN, U100 UEI15-050-Q12P-C, U102 SI8640, U103 SI8642, U104 ISO7240M, U105 ISO7240M, U106 ISO7240M, U107 ISO7240M

Commit message: More PCIe host routing
- Deserializer decoupling is done.
- Im going to get rid of isolation on the immediate digital IO because
  it is not needed.
Parts:
- removed C61, C62, C65: 10uF, jonnew:1206
- removed R13: 1.15k, jonnew:0402
- removed R29: 100k, jonnew:0603
- removed U$8: LT1763CS8-1.8, jonnew:SOIC127P500X400-8N
- added 10K, 13.3K: 9.53k, jonnew:0603
- added C28: 4.7uF, jonnew:0805
- added C30, C32: 0.1uF, jonnew:0603
- added L7: 1uH, jonnew:4020
- C13: value 10nF -> 0.1uF; device jonnew:0402 -> jonnew:0603
- C39: value 10uF -> 22uF; device jonnew:1210 -> jonnew:1206
- C59: value 10uF -> 22uF
- C60: value 1nF -> 0.01uF
- C66: value 100uF -> 47uF
- C67, C71, C82, R43, R44, R45: device jonnew:0603 -> jonnew:0402
- C69: device RHD2000_eval_board:0603 -> jonnew:0402
- C74, C84: device jonnew:0603 -> jonnew:1206
- C77: value 22uF -> 4.7F; device jonnew:0603 -> jonnew:1206
- C80: value 22uF -> 4.7uF; device jonnew:0603 -> jonnew:1206
- C85: value 0.01uF -> 0.1uF
- C86: device RHD2000_eval_board:0603 -> jonnew:0805
- L1: value CIG21L4R7MNE -> 1008PS-472KLB; device jonnew:0805 -> jonnew:1008PS
- L2: value CBC3225T101MR -> SRN6045TA-101M; device jonnew:1210 -> jonnew:SRN6045TA
- L3: value BLM18KG601SN1D -> MPZ2012S102AT000; device jonnew:0603 -> jonnew:0805
- R12: value 3.57k -> 30.1k; device jonnew:0402 -> jonnew:0603
- R46, R47, R48: value DNP -> 0; device jonnew:0603 -> jonnew:0402
- R7: value 220 -> 649k
- U$3: value TPS748_VQFN -> LTM4622_BGA; device jonnew:VQFN20 -> jonnew:BGA_5X5_625X625
- moved TP10 120.8 mm to (137.2, -4.60)
- moved C90 95.1 mm to (-58.1, 17.1), turned to 0 degrees
- moved TP2 93.2 mm to (-61.0, 12.8)
- moved C91 92.8 mm to (-57.7, 19.4)
- moved R37 92.8 mm to (-57.7, 21.6)
- moved R7 81.3 mm to (99.4, 26.1), turned to 90 degrees
- moved C39 59.5 mm to (87.9, 23.2), turned to 0 degrees
- moved C60 58.5 mm to (36.0, 28.1), flipped to the bottom, turned to 180 degrees
- moved C84 26.0 mm to (38.0, 34.7), flipped to the bottom
- moved C3 18.9 mm to (96.8, 14.1), turned to 90 degrees
- moved TP1 18.9 mm to (108.7, 5.13)
- moved C85 17.5 mm to (34.1, 23.1), flipped to the bottom, turned to 270 degrees
- moved C83 14.3 mm to (32.9, 23.1), flipped to the bottom, turned to 270 degrees
- moved R60 14.1 mm to (40.1, 20.0), turned to 180 degrees
- moved C13 13.3 mm to (95.6, 26.1), turned to 270 degrees
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Connections:
- removed net +5V5_ISO: C14.2, C19.+, C61.2, C62.2, C95.+, L3.1, R26.2, R27.2, R29.2, TP15.1, U$3.10, U$3.11, U$3.5, U$3.6, U$3.7, U$3.8, U100.3
- new net +12V_ISO: C14.2, C19.+, C28.2, C3.2, C30.1, C95.+, L3.1, R26.2, R27.2, TP15.1, U$3.A2, U$3.B2, U$3.B3, U$3.D2, U$3.D3, U$3.E2, U100.3
- new net INTVCC: 10K.1, U$3.C3
- new net N$145: R7.1, U$3.C4
- new net VIN: L7.2, U100.1, U100.6
- net +12V_ATX: now also L7.1; no longer C39.1, U100.1, U100.6
- net +1V8_ISO: now also C39.2, U$3.A1, U$3.B1; no longer C13.2, C3.2, U$8.1, U$8.2
- net +3V3_ISO: now also C60.2, U$3.D1, U$3.E1; no longer C65.2, R12.1, R7.1, U$3.1, U$3.18, U$3.19, U$3.20, U$8.5, U$8.8
- net +3V3_ISO_PG_ISO: now also 10K.2, U$3.D4; no longer R29.1, U$3.9
- net GND: no longer C39.2
- net GND_ISO: now also 13.3K.2, C13.1, C28.1, C30.2, C32.1, C39.1, R12.2, R7.2, U$3.B5, U$3.C1, U$3.C2, U$3.C5, U$3.D5; no longer C61.1, C62.1, C65.1, PWR/LOCK.C1, R13.1, U$3.12, U$3.13, U$3.14, U$3.2, U$3.3, U$3.4, U$3.PAD, U$8.3, U$8.6, U$8.7
- net N$10: now also 13.3K.1, U$3.E4; no longer PWR/LOCK.A1, R7.2
- net N$12: now also C32.2, U$3.E3; no longer C60.2, U$3.15
- net N$5: now also R12.1, U$3.A4; no longer R12.2, R13.2, U$3.16
- net N$8: now also C13.2, U$3.A3; no longer C13.1, U$8.4
Routing:
- net V_PROTECT: track 191.4 -> 11.8 mm
- net +12V_ISO: track 0.00 -> 107.6 mm, vias 0 -> 27
- net GPI1_ISO: track 0.00 -> 85.0 mm
- net D9_ISO: track 0.00 -> 82.5 mm
- net D8_ISO: track 0.00 -> 81.1 mm
- net PCLK_ISO: track 0.00 -> 81.0 mm
- net D5_ISO: track 0.00 -> 81.0 mm
- net D4_ISO: track 0.00 -> 80.4 mm
- net D7_ISO: track 0.00 -> 80.1 mm
- net D10_ISO: track 0.00 -> 79.6 mm
- net VSYNC_ISO: track 0.00 -> 79.4 mm
- net D6_ISO: track 0.00 -> 79.3 mm
- net D11_ISO: track 0.00 -> 78.4 mm
- net HSYNC_ISO: track 0.00 -> 78.1 mm
- net D3_ISO: track 0.00 -> 77.4 mm
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- added copper zone on layer 1, net +12V_ISO
- added copper zone on layer 16, net +12V_ISO
- added copper zone on layer 1, net +1V8_ISO
- added copper zone on layer 16, net +1V8_ISO
- added copper zone on layer 16, net +3V3_ISO
- added copper zone on layer 16, net GND_ISO
- added copper zone on layer 1, net N$21
- added copper zone on layer 1, net N$22
- added copper zone on layer 16, net VDDCML0
- added copper zone on layer 16, net VDDCML1
- added copper zone on layer 16, net VDDPLL
- removed copper zone on layer 15, net +3V3
- removed copper zone on layer 1, net +5V5_ISO

Commit message: More PCIe host layout
- Got rid of isolation on immediate IO. It was not needed and all those
  isolator were crowding the board. No need for it to be synchronized
  to pclk either, that I can see.
Parts:
- removed C49, C53, C56: 100nF, RHD2000_eval_board:0603
- removed C51, C52: (no value), jonnew:0402
- removed C7: 0.1uF, RHD2000_eval_board:0603
- removed R12: 30.1k, jonnew:0603
- removed U102: SI8640, jonnew:SOIC_WIDE_16
- removed U103: SI8642, jonnew:SOIC_WIDE_16
- added 30.1K: 9.53k, jonnew:0603
- 13.3K: value 9.53k -> 30.1k
- moved U$11 176.9 mm to (53.3, 62.4), turned to 270 degrees
- moved C6 78.2 mm to (61.6, 94.0)
- moved TP8 78.2 mm to (57.8, 95.5)
- moved D9 78.2 mm to (53.8, 93.0)
- moved R26 78.2 mm to (59.6, 92.0)
- moved R27 78.2 mm to (57.5, 92.0)
- moved U$21 53.7 mm to (84.2, 23.4), turned to 270 degrees
- moved R32 52.6 mm to (69.5, 16.4), turned to 270 degrees
- moved C89 50.4 mm to (68.0, 18.7), turned to 270 degrees
- moved C74 49.9 mm to (73.4, 15.6), turned to 90 degrees
- moved C88 49.5 mm to (69.5, 18.7), turned to 270 degrees
- moved R38 49.2 mm to (82.4, 26.4), turned to 90 degrees
- moved R39 47.5 mm to (81.0, 26.4), turned to 90 degrees
- moved L6 47.3 mm to (71.1, 16.2), turned to 90 degrees
- moved R40 45.9 mm to (79.6, 26.4), turned to 90 degrees
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Connections:
- removed net DAC_LAT_ISO: U$10.6, U102.P11
- removed net DI0_TERM_ISO: Q1.G, R14.2, U102.P14
- removed net DI1_ISO: U$6.1, U103.P4
- removed net DI1_TERM_ISO: Q2.G, R21.2, U102.P13
- removed net DIO_ISO: U$5.1, U103.P3
- removed net DO0_ISO: U$7.2, U$7.5, U103.P5
- removed net DO1_ISO: U$7.12, U$7.9, U103.P6
- new net +12V_FPGA: R26.2, R27.2
- new net +1V8: U$17.3, U$18.3
- new net N$147: R35.2
- net +12V_ISO: no longer R26.2, R27.2
- net +1V8_ISO: now also C59.2, U$3.D1, U$3.E1; no longer C39.2, U$17.3, U$18.3, U$3.A1, U$3.B1
- net +3V3: now also C26.2, C35.2, C36.1, C37.1, C54.2, C55.2, R24.2, R25.2, R69.2, U$10.1, U$10.2, U$5.5, U$6.5, U$7.14; no longer C49.2, C56.2, U102.P1, U103.P10, U103.P16
- net +3V3_ISO: now also C39.2, U$3.A1, U$3.B1; no longer C26.2, C35.2, C36.1, C37.1, C53.2, C54.2, C55.2, C59.2, C7.2, R24.2, R25.2, R35.2, R69.2, U$10.1, U$10.2, U$3.D1, U$3.E1, U$5.5, U$6.5, U$7.14, U102.P10, U102.P16, U103.P1, U103.P7
- net DAC_LAT: now also U$10.6; no longer U102.P6
- net DI0: now also U$5.1; no longer C52.1, U103.P14
- net DI0_TERM: now also Q1.G, R14.2; no longer U102.P3
- net DI1: now also U$6.1; no longer C51.1, U103.P13
- net DI1_TERM: now also Q2.G, R21.2; no longer U102.P4
- net DO0: now also U$7.2, U$7.5; no longer U103.P12
- net DO1: now also U$7.12, U$7.9; no longer U103.P11
- net DO_TEST: no longer U102.P5
- net DO_TEST_ISO: no longer U102.P12
- net GND: no longer C49.1, C51.2, C52.2, C56.1, U102.P2, U102.P8, U103.P15, U103.P9
- net GND_ISO: now also 30.1K.2; no longer C53.1, C7.1, R12.2, U102.P15, U102.P9, U103.P2, U103.P8
- net N$10: now also 30.1K.1; no longer 13.3K.1
- net N$5: now also 13.3K.1; no longer R12.1
- net SCL: now also U$10.7
- net SCL_ISO: no longer U$10.7
- net SDA: now also U$10.8
- net SDA_ISO: no longer U$10.8
Routing:
- net +12V_ISO: track 107.6 -> 3.75 mm, vias 27 -> 22
- net D9_ISO: track 82.5 -> 10.7 mm
- net D10_ISO: track 79.6 -> 11.5 mm
- net GPI1_ISO: track 85.0 -> 19.8 mm
- net D8_ISO: track 81.1 -> 19.0 mm
- net PCLK_ISO: track 81.0 -> 19.9 mm
- net D4_ISO: track 80.4 -> 19.6 mm
- net D7_ISO: track 80.1 -> 19.7 mm
- net D5_ISO: track 81.0 -> 20.9 mm
- net VSYNC_ISO: track 79.4 -> 19.9 mm
- net D3_ISO: track 77.4 -> 18.5 mm
- net HSYNC_ISO: track 78.1 -> 19.6 mm
- net D6_ISO: track 79.3 -> 20.9 mm
- net D11_ISO: track 78.4 -> 20.4 mm
- net D2_ISO: track 75.7 -> 19.2 mm
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- removed copper zone on layer 1, net V_PROTECT

Commit message: Nearly done with PCIe host layout.
Parts:
- removed C90: 0.1uF, jonnew:0402
- removed C91: 0.047uF, jonnew:0402
- removed R37: 49.9, jonnew:0402
- removed TP5: +5V0, jonnew:TESTPOINT_0.035IN
- removed TP_DO0, TP_DO1: MISO1, jonnew:TP09SQ
- added C49, C7: 22uF, jonnew:1210-POL
- added D5: LM4040D25FTA, jonnew:SOT23
- added R12: 100, jonnew:0603
- added U$8: SCREW4, jonnew:SCREW4
- C54: device RHD2000_eval_board:0603 -> jonnew:0805
- moved C96 214.6 mm to (43.4, 61.0), flipped to the bottom, turned to 270 degrees
- moved C97 212.9 mm to (45.0, 60.9), flipped to the bottom, turned to 270 degrees
- moved C99 196.5 mm to (52.4, 60.7), flipped to the bottom, turned to 270 degrees
- moved TP_DI0 190.0 mm to (32.7, 80.9)
- moved TP_DI1 189.6 mm to (32.7, 70.8)
- moved C98 189.3 mm to (51.0, 60.7), flipped to the bottom, turned to 270 degrees
- moved TP2 132.7 mm to (71.6, 18.6)
- moved R9 87.5 mm to (101.2, 34.9), turned to 0 degrees
- moved U$15 87.3 mm to (42.6, 22.2), turned to 90 degrees
- moved C58 87.0 mm to (110.7, 41.9)
- moved R5 85.1 mm to (145.2, 89.5), flipped to the bottom
- moved R10 84.8 mm to (101.2, 36.6), turned to 0 degrees
- moved U$1 78.0 mm to (106.1, 42.9), turned to 270 degrees
- moved R4 77.5 mm to (145.2, 87.6), flipped to the bottom
- moved C57 70.5 mm to (104.8, 47.6), turned to 180 degrees
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Connections:
- removed net +1V8: U$17.3, U$18.3
- removed net DO_TEST_ISO: TP5.1, U$15.P$4
- removed net N$40: C90.1, U$9.32
- removed net N$41: C91.1, U$9.33
- removed net N$42: C91.2, R37.1
- removed net N$43: C90.2
- new net 2V5_REF: D5.1, R12.1, U$17.3, U$18.3
- net +12V_ATX: now also U$8.P$4
- net +3V3: now also R12.2, R6.1, R8.1, U$8.P$2
- net +3V3_ISO: no longer R6.1, R8.1
- net 12V_FPGA: now also C49.+, C7.+, U$8.P$3
- net DO0: now also U$11.26; no longer TP_DO0.TP, U$11.27
- net DO1: now also U$11.27; no longer TP_DO1.TP, U$11.26
- net GND: now also C26.1, C33.2, C34.2, C35.1, C36.2, C37.2, C49.-, C54.1, C55.1, C6.1, C7.-, D1.1, D2.1, D3.1, D4.1, D5.2, D9.A, DI0.GND$1, DI0.GND$2, DI0.GND$3, DI0.GND$4, DI1.GND$1, DI1.GND$2, DI1.GND$3, DI1.GND$4, DO0.GND$1, DO0.GND$2, DO0.GND$3, DO0.GND$4, DO1.GND$1, DO1.GND$2, DO1.GND$3, DO1.GND$4, Q1.S, Q2.S, Q3.S, Q4.S, R11.1, R14.1, R20.1, R21.1, R68.1, R71.1, U$10.5, U$5.2, U$6.2, U$7.7, U$8.P$1
- net GND_ISO: now also U$15.P$4; no longer C26.1, C33.2, C34.2, C35.1, C36.2, C37.2, C54.1, C55.1, C6.1, D1.1, D2.1, D3.1, D4.1, D9.A, DI0.GND$1, DI0.GND$2, DI0.GND$3, DI0.GND$4, DI1.GND$1, DI1.GND$2, DI1.GND$3, DI1.GND$4, DO0.GND$1, DO0.GND$2, DO0.GND$3, DO0.GND$4, DO1.GND$1, DO1.GND$2, DO1.GND$3, DO1.GND$4, Q1.S, Q2.S, Q3.S, Q4.S, R11.1, R14.1, R20.1, R21.1, R37.2, R68.1, R71.1, U$10.5, U$5.2, U$6.2, U$7.7
- net GPI0: now also U$13.7; no longer U$13.6
- net GPI1: now also U$13.6; no longer U$13.7
- net N$2: now also TERM.C2; no longer TERM.C1
- net N$30: now also TERM.A2; no longer TERM.A1
- net N$33: now also TERM.A1; no longer TERM.A2
- net N$7: now also TERM.C1; no longer TERM.C2
Routing:
- net LOCK: track 0.00 -> 64.0 mm, vias 0 -> 2
- net V_PROTECT: track 0.14 -> 60.2 mm, vias 0 -> 4
- net DI0_TERM: track 0.00 -> 56.8 mm, vias 0 -> 1
- net DOUTP_F: track 16.3 -> 71.5 mm
- net DI1_TERM: track 0.00 -> 46.7 mm, vias 0 -> 1
- net SDA_ISO: track 0.00 -> 46.7 mm
- net SCL_ISO: track 0.00 -> 45.2 mm
- net GND: track 14.6 -> 57.5 mm, vias 4 -> 32
- net DO1: track 10.1 -> 48.1 mm, vias 0 -> 3
- net DI0: track 0.00 -> 33.9 mm, vias 0 -> 1
- net DO0: track 7.85 -> 39.1 mm, vias 0 -> 3
- net DI1: track 0.00 -> 25.4 mm, vias 0 -> 1
- net +3V3: track 50.1 -> 75.0 mm, vias 7 -> 19
- net N$7: track 9.35 -> 31.3 mm
- net SEL: track 0.00 -> 19.2 mm, vias 0 -> 2
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- added copper zone on layer 1, net +12V_ATX
- added copper zone on layer 15, net +3V3
- added copper zone on layer 1, net GND
- added copper zone on layer 1, net VIN
