File: pcie-host/pcie-host.sch (EAGLE design)
At the start: 237 parts, among them Q1 NDS351AN, Q2 NDS351AN, Q3 BSH103, Q4 BSH103, Q5 NDS351AN, U1 ISO, U10 LTM4622_BGA, U11 ISO1540DR, U12 UEI15-050-Q12P-C, U13 ISO7240M, U14 ISO7240M, U15 ISO7240M, U16 ISO7240M, U17 ISO7242M, U18 COMM, U19 SN65LVDT388A, U20 SN65LVDS387, U21 SN65LVDS391, U4 SN74LVT125, U5 ADCMP600, U6 ADCMP600, U8 MCP47FEBX2, U9 DS90UB914A-Q1, X1 PCI-MECH_STD-H_HALF-W_FMC-STR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

Commit message: pcie-host board rev. 1.2
- Extra bidirectional isolator added to propogate LOCK and PASS signals from deserializer to host FPGA.
- Immediate non-isolated and isolated SMA IO added.
- Routed HSYNC to normal (LA) differential pins rather than dedicated
clock input which was causing synthesis issues.
Parts:
- removed C82, C84, C86, C88, C91, C92, C93, C95, C97: 0.1uF, jonnew:C_0603
- removed C83, C85, C89, C90, C94, C96, C98: 1nF, jonnew:C_0402
- removed C87: 22uF, jonnew:C-POL_1210
- removed TP28: GND(ISO), jonnew:TP_1MM
- removed TP29: GPIO3, jonnew:TPTP06R
- removed U19: SN65LVDT388A, jonnew:SN65LVDS388A
- removed U20: SN65LVDS387, jonnew:SN65LVDS387_TSSOP
- removed U21: SN65LVDS391, jonnew:SN65LVDS391
- added C41, C64, C65, C68: 10nF, jonnew:C_0402
- added C43, C73, C75: 1nF, jonnew:C_0402
- added C62, C63, C70, C71, C72, C74, C76, C77: 0.1uF, jonnew:C_0603
- added C67: 4.7uF, jonnew:C_1206
- added C69: 0.1uF, jonnew:C_0402
- added C78, C79: 4.7uF, jonnew:C_0805
- added J1, J2: (no value), jonnew:JP3E
- added J3: COMM, jonnew:SCREW4
- added J4: ISO, jonnew:SCREW4
- added J5, J6, J7, J8: (no value), jonnew:COAX_SMA-VERT-SMA
- added R76: 22, jonnew:R_0402
- C1: value 1uF -> 0.1uF; device RHD2000_eval_board:C_0603 -> jonnew:C_0603
- C10, C27, C30, C32, C33: value 10nF -> 0.1uF; device jonnew:C_0402 -> jonnew:C_0603
- C11: value 10nF -> 47uF; device jonnew:C_0402 -> jonnew:C-POL_0807
- C12: value 47nF -> 1uF; device jonnew:C_0402 -> RHD2000_eval_board:C_0603
- C13: value 4.7uF -> 0.1uF; device jonnew:C_0805 -> RHD2000_eval_board:C_0603
- C14: device jonnew:C_0402 -> RHD2000_eval_board:C_0603
- C15: value 0.1uF -> 1uF; device jonnew:C_0402 -> jonnew:C_0805
- C16, C29: device jonnew:C_0402 -> jonnew:C_0603
- C18: value 4.7uF -> 0.1uF; device jonnew:C_1206 -> jonnew:C_0603
- C19: value 4.7F -> 22uF
- C2, C25: device RHD2000_eval_board:C_0603 -> jonnew:C_0603
- C20: value 1uF -> 22uF; device jonnew:C_0805 -> jonnew:C_1206
- C21: value 22uF -> 100uF; device jonnew:C_1206 -> jonnew:C-POL_0807
- C22: value 4.7uF -> 10uF
- C23: value 0.1uF -> 22uF; device jonnew:C_0402 -> jonnew:C-POL_1210
- C24: device jonnew:C_1206 -> jonnew:C-POL_1210
- C26, C28: value 10nF -> 1nF
- C3: value 4.7uF -> 0.1uF; device jonnew:C_0805 -> jonnew:C_0603
- C31: value 10nF -> 10uF; device jonnew:C_0402 -> jonnew:C_1206
- C34, C36: value 0.1uF -> 10nF
- C39: value 0.1uF -> 4.7uF; device jonnew:C_0603 -> jonnew:C_1206
- C4: value 10uF -> 0.1uF
- C40, C51, C53, C56, C57: device jonnew:C_0603 -> jonnew:C_0402
- C42: value 10uF -> 0.1uF; device jonnew:C_1206 -> jonnew:C_0603
- C44: value 100uF -> 0.1uF; device jonnew:C-POL_0807 -> jonnew:C_0603
- C45: value 10uF -> 1nF; device jonnew:C_1206 -> jonnew:C_0402
- C46: value 47uF -> 0.1uF; device jonnew:C-POL_0807 -> jonnew:C_0603
- C47: value 22uF -> 1nF; device jonnew:C-POL_1210 -> jonnew:C_0402
- C48: value 22uF -> 0.1uF; device jonnew:C-POL_1210 -> jonnew:C_0603
- C5, C8: value 0.1uF -> 22uF; device jonnew:C_0603 -> jonnew:C-POL_1210
- C50, C52, C55: value 0.1uF -> 10nF; device jonnew:C_0603 -> jonnew:C_0402
- C54: value 0.1uF -> 4.7F; device jonnew:C_0603 -> jonnew:C_1206
- C58: value 0.1uF -> 47nF; device jonnew:C_0603 -> jonnew:C_0402
- C61: value 0.1uF -> 10uF
- C66: value 22uF -> 0.1uF; device jonnew:C-POL_1210 -> jonnew:C_0402
- L1: value 1008PS-472KLB -> BLM18KG601SN1D; device jonnew:L_1008PS -> jonnew:L_0603
- L2: value SRN6045TA-101M -> BLM18KG601SN1D; device jonnew:L_SRN6045TA -> jonnew:L_0603
- L3: value MPZ2012S102AT000 -> BLM18KG601SN1D; device jonnew:L_0805 -> jonnew:L_0603
- L4: value BLM18KG601SN1D -> MPZ2012S102AT000; device jonnew:L_0603 -> jonnew:L_0805
- L5: value BLM18KG601SN1D -> 1008PS-472KLB; device jonnew:L_0603 -> jonnew:L_1008PS
- L6: value BLM18KG601SN1D -> SRN6045TA-101M; device jonnew:L_0603 -> jonnew:L_SRN6045TA
- Q1, Q2: value NDS351AN -> BSH103
- Q3, Q4: value BSH103 -> NDS351AN
- R1: value 1k -> 100; device cyclops:R_0603 -> jonnew:R_0603
- R10: value 100k -> 100
- R11: value 1k -> 2.2k; device RHD2000_eval_board:R_0603 -> jonnew:R_0603
- R12: value 4.7k -> 10k; device cyclops:R_0603 -> jonnew:R_0603
- R13: value 4.7k -> 150,0.25W; device cyclops:R_0603 -> jonnew:R_1206
- R14, R15: value 10K -> 150,0.25W; device jonnew:R_0402 -> jonnew:R_1206
- R16: value 150,0.25W -> 1k; device jonnew:R_1206 -> jonnew:R_0603
- R17: value 150,0.25W -> 1k; device jonnew:R_1206 -> RHD2000_eval_board:R_0603
- R18: value 10K -> 100k; device jonnew:R_0402 -> jonnew:R_0603
- R19: value 10K -> 4.7k; device jonnew:R_0402 -> cyclops:R_0603
- R2: value 1k -> 2.2k; device cyclops:R_0603 -> jonnew:R_0603
- R20: value 1K -> 1k; device jonnew:R_0603 -> cyclops:R_0603
- R21, R22, R24: value 150,0.25W -> 2.2k; device jonnew:R_1206 -> jonnew:R_0603
- R23: value 150,0.25W -> 100k; device jonnew:R_1206 -> cyclops:R_0603
- R25: value 10K -> 2.2k; device jonnew:R_0402 -> jonnew:R_0603
- R26: value 10k -> 4.7k; device jonnew:R_0603 -> cyclops:R_0603
- R27: value 10k -> 100
- R28: value 100 -> 1k; device jonnew:R_0603 -> cyclops:R_0603
- R29, R67: value 100 -> 100k; device jonnew:R_0603 -> cyclops:R_0603
- R3, R34: value 100k -> 10k; device cyclops:R_0603 -> jonnew:R_0603
- R30: value 49.9 -> 1k; device jonnew:R_0402 -> jonnew:R_0603
- R31, R32: value 2.2k -> 1k
- R33: device cyclops:R_0603 -> jonnew:R_0603
- R35: value 22 -> 9.53k; device jonnew:R_0402 -> jonnew:R_0603
- R36: value 22 -> 1k; device jonnew:R_0402 -> cyclops:R_0603
- R37: value 22 -> 30.1k; device jonnew:R_0402 -> jonnew:R_0603
- R38: value 22 -> 649k; device jonnew:R_0402 -> jonnew:R_0603
- R39: value 22 -> 13.3k; device jonnew:R_0402 -> jonnew:R_0603
- R4: value 100k -> 150,0.25W; device cyclops:R_0603 -> jonnew:R_1206
- R42: value 22 -> 49.9
- R46: value 1k -> 22; device cyclops:R_0603 -> jonnew:R_0402
- R5, R6: value 2.2k -> 150,0.25W; device jonnew:R_0603 -> jonnew:R_1206
- R55: value 30.1k -> 22; device jonnew:R_0603 -> jonnew:R_0402
- R56: value 10k -> 10K; device jonnew:R_0603 -> jonnew:R_0402
- R57, R60: value 10K -> 22
- R58: value 0 -> 22
- R59: value 13.3k -> 22; device jonnew:R_0603 -> jonnew:R_0402
- R61, R63: value 0 -> 10K
- R64: value 649k -> 10K; device jonnew:R_0603 -> jonnew:R_0402
- R65, R66: device jonnew:R_0603 -> cyclops:R_0603
- R68: value 9.53k -> 1K
- R69: value 2.2k -> 1K
- R7: value 1K -> 1k
- R70: value 2.2k -> 10K; device jonnew:R_0603 -> jonnew:R_0402
- R71, R72: value 1k -> 10K; device jonnew:R_0603 -> jonnew:R_0402
- R73, R74: value 1k -> 0; device jonnew:R_0603 -> jonnew:R_0402
- R75: value 1k -> 0; device cyclops:R_0603 -> jonnew:R_0402
- R8: value 100k -> 1k
- R9: value 1k -> 100k
- TP1: value GND(ISO) -> DI1; device jonnew:TP_1MM -> jonnew:TPTP09SQ
- TP10: value GND -> +3.3V
- TP14: value GND -> VPROTECT(+4.3V); device jonnew:TP_2MM -> jonnew:TP_0.035IN
- TP15: value GND -> SCL(ISO); device jonnew:TP_2MM -> jonnew:TP_1MM
- TP16: value GND -> SDA(ISO); device jonnew:TP_2MM -> jonnew:TP_1MM
- TP17, TP21: value GND -> GND(ISO); device jonnew:TP_2MM -> jonnew:TP_1MM
- TP18: value GND(ISO) -> GND
- TP19: value GND(ISO) -> SDA
- TP2: value +1.8V(ISO) -> DI0; device jonnew:TP_1MM -> jonnew:TPTP09SQ
- TP20: value GND(ISO) -> SCL
- TP22: value +3.3V -> +1.8V(ISO); device jonnew:TP_2MM -> jonnew:TP_1MM
- TP23: value GND -> +3.3V(ISO); device jonnew:TP_1MM -> jonnew:TP_2MM
- TP24: value SDA -> +5.5V(ISO); device jonnew:TP_1MM -> jonnew:TP_2MM
- TP25: value SCL -> GND(ISO)
- TP26: value SCL(ISO) -> GND(ISO)
- TP27: value SDA(ISO) -> GND(ISO)
- TP3: value +3.3V(ISO) -> GND; device jonnew:TP_2MM -> jonnew:TP_0.035IN
- TP4: value +5.5V(ISO) -> GND
- TP5: value PASS -> GND; device jonnew:TPTP06R -> jonnew:TP_2MM
- TP6: value DI1 -> GND; device jonnew:TPTP09SQ -> jonnew:TP_2MM
- TP7: value DI0 -> GND; device jonnew:TPTP09SQ -> jonnew:TP_2MM
- TP8: device jonnew:TP_0.035IN -> jonnew:TP_2MM
- TP9: value VPROTECT(+4.3V) -> GND; device jonnew:TP_0.035IN -> jonnew:TP_2MM
- U1: value ISO -> ADCMP600; device jonnew:SCREW4 -> jonnew:COMPARITOR_ADCMP600
- U10: value LTM4622_BGA -> ISO7740; device jonnew:LTM4622_BGA -> jonnew:DIGISO-4-0
- U11: value ISO1540DR -> SN65LVDS387; device jonnew:DIGISO-I2C_SOIC -> jonnew:SN65LVDS387_TSSOP
- U12: value UEI15-050-Q12P-C -> DS90UB914A-Q1; device jonnew:DC-DC-CONVERTER-ADJ_UEI15 -> jonnew:DS90UB914A-Q1
- U13, U14: value ISO7240M -> ISO7740
- U15: value ISO7240M -> (none); device jonnew:DIGISO-4-0 -> jonnew:DIPSW-004_SMD-0.05IN
- U16: value ISO7240M -> SN65LVDS391; device jonnew:DIGISO-4-0 -> jonnew:SN65LVDS391
- U17: value ISO7242M -> ISO7742; device jonnew:DIGISO-2-2 -> jonnew:DIGISO-4-0
- U18: value COMM -> ISO7741; device jonnew:SCREW4 -> jonnew:DIGISO-3-1
- U2: value (none) -> ADCMP600; device jonnew:JP3E -> jonnew:COMPARITOR_ADCMP600
- U3: value (none) -> SN74LVT125; device jonnew:JP3E -> jonnew:QUAD-LINE-DRIVER_SOIC
- U4: value SN74LVT125 -> MCP47FEBX2; device jonnew:QUAD-LINE-DRIVER_SOIC -> jonnew:MCP47FEBX2
- U5: value ADCMP600 -> ISO1540DR; device jonnew:COMPARITOR_ADCMP600 -> jonnew:DIGISO-I2C_SOIC
- U6: value ADCMP600 -> UEI15-050-Q12P-C; device jonnew:COMPARITOR_ADCMP600 -> jonnew:DC-DC-CONVERTER-ADJ_UEI15
- U7: value (none) -> LTM4622_BGA; device jonnew:DIPSW-004_SMD-0.05IN -> jonnew:LTM4622_BGA
- U8: value MCP47FEBX2 -> SN65LVDT388A; device jonnew:MCP47FEBX2 -> jonnew:SN65LVDS388A
- U9: value DS90UB914A-Q1 -> ISO7740; device jonnew:DS90UB914A-Q1 -> jonnew:DIGISO-4-0
Connections:
- removed net DAC_LAT: U19.B1Y, U8.LAT/HVC
- removed net DO_TEST: U19.B2Y
- removed net GPI0: U17.VOB, U21.4A
- removed net GPI0_ISO: R40.1, U17.VIB
- removed net GPI1: U17.VOA, U21.3A
- removed net GPI1_ISO: R48.1, U17.VIA
- removed net GPO0: U17.VID, U19.D1Y
- removed net GPO1: U17.VIC, U19.D2Y
- removed net GPO1_ISO: R47.1, U17.VOC
- removed net N$1: R39.1, U17.VOD
- new net DES_GPIO0: U17.VID, U8.D2Y
- new net DES_GPIO0_ISO: R60.1, U17.VOD
- new net DES_GPIO1: U17.VIC, U8.D1Y
- new net DES_GPIO1_ISO: R59.1, U17.VOC
- new net DES_GPIO2: U17.VIB, U8.C2Y
- new net DES_GPIO2_ISO: R58.1, U17.VOB
- new net DES_GPIO3: U17.VIA, U8.C1Y
- new net DES_GPIO3_ISO: R57.1, U17.VOA
- new net LOCK_ISO: R66.2, U12.LOCK, U18.VIA
- new net N$56: R76.1, U18.VIC
- new net PASS_ISO: R76.2, U12.PASS
- new net SMA_IN: FMC_LPCG$1.LA27_P, J6.1, U18.VOB
- new net SMA_IN_ISO: J5.1, U18.VIB
- new net SMA_OUT: FMC_LPCG$1.LA27_N, J8.1, U18.VID
- new net SMA_OUT_ISO: J7.1, U18.VOD
- net $N1: now also D2.COMM, R10.1, R11.2, R13.2, R14.2, R15.2; no longer D4.COMM, R17.2, R22.2, R24.2, R29.1, R6.2
- net $N101: now also D3.COMM, R19.2, U3.1Y, U3.2Y; no longer D1.COMM, R13.2, U4.1Y, U4.2Y
- net $N2: now also D4.COMM, R26.2, U3.3Y, U3.4Y; no longer D2.COMM, R12.2, U4.3Y, U4.4Y
- net $N3: now also D1.COMM, R1.1, R2.2, R4.2, R6.2; no longer D3.COMM, R16.2, R21.2, R23.2, R28.1
- net +12V_ATX: now also C11.+, C21.+; no longer C44.+, C46.+
- net +12V_FPGA: now also C5.+, C6.2, C7.2, J3.3, R24.2, R25.2; no longer C66.+, C80.2, C82.2, R69.2, R70.2, U18.3
- net +1V8_ISO: now also C20.2, C34.2, C50.2, C51.2, C55.2, C56.2, J4.2, L1.2, L2.1, L3.2, R70.1, R71.1, R72.1, TP22.TP, U12.VDDD, U12.VDDR, U12.VDDSSCG, U7.VOUT1; no longer C24.2, C31.2, C32.2, C33.2, C36.2, C37.2, L4.2, L5.2, L6.1, R57.1, R60.1, R62.1, TP2.TP, U1.2, U10.VOUT1, U9.VDDD, U9.VDDR, U9.VDDSSCG
- net +3V3: now also C1.1, C10.2, C12.2, C13.2, C14.2, C15.2, C18.2, C26.2, C27.2, C28.2, C3.1, C33.2, C42.2, C43.2, C44.2, C45.2, C46.2, C47.2, C49.2, C63.2, C71.2, C72.2, C73.2, C74.2, C75.2, C8.+, C9.2, J3.2, R20.2, R21.2, R22.2, R27.2, R28.2, R33.2, TP10.TP, U10.EN2, U10.VDD2, U11.ENA, U11.ENB, U11.ENC, U11.END, U11.VCC, U16.EN1,2, U16.EN3,4, U16.VCC, U17.VDD1, U18.EN2, U18.VDD2, U1G$2.V+, U2G$2.V+, U3.VCC, U4.REFA, U4.VDD, U5.VDD1, U8.DVCC, U8.ENA, U8.ENB, U8.ENC, U8.END, U8.VCC, U9.EN2, U9.VDD2; no longer C1.2, C2.2, C20.2, C56.2, C57.2, C58.2, C59.2, C61.2, C8.1, C83.2, C84.2, C85.2, C86.2, C87.+, C88.2, C89.2, C9.1, C90.2, C91.2, C92.2, C93.2, C94.2, C95.2, C96.2, C97.2, C98.2, R1.2, R2.2, R31.2, R67.2, R71.2, R72.2, TP22.TP, U11.VDD1, U15.EN2, U15.VDD2, U16.EN2, U16.VDD2, U17.EN2, U17.VDD2, U18.2, U19.DVCC, U19.ENA, U19.ENB, U19.ENC, U19.END, U19.VCC, U20.ENA, U20.ENB, U20.ENC, U20.END, U20.VCC, U21.EN1,2, U21.EN3,4, U21.VCC, U4.VCC, U5G$2.V+, U6G$2.V+, U8.REFA, U8.VDD
- net +3V3_ISO: now also C17.2, C19.2, C32.2, C48.2, C59.2, C62.2, C64.2, C65.2, C66.2, C67.2, C68.2, C69.2, C70.2, C80.2, J4.3, R30.2, R31.2, R36.2, R56.1, R61.2, R62.2, R63.2, R64.2, TP23.TP, U10.VDD1, U12.VDDIO1, U12.VDDIO2, U12.VDDIO3, U17.EN2, U17.VDD2, U18.EN1, U18.VDD1, U5.VDD2, U7.VOUT2, U9.VDD1; no longer C21.2, C27.2, C28.2, C29.2, C30.2, C34.2, C38.2, C49.2, C50.2, C51.2, C52.2, C53.2, C54.2, R14.2, R15.2, R18.2, R19.2, R25.1, R46.2, R66.2, R75.2, TP3.TP, U1.3, U10.VOUT2, U11.VDD2, U15.VDD1, U16.VDD1, U17.VDD1, U9.VDDIO1, U9.VDDIO2, U9.VDDIO3
- net +3V3_ISO_PG: now also U11.D4A, U14.VOD; no longer U16.VOD, U20.D4A
- net +3V3_ISO_PG_ISO: now also R34.2, U14.VID, U7.PGOOD1; no longer R56.2, U10.PGOOD1, U16.VID
- net +3V3_ISO_PG_N: now also FMC_LPCG$1.LA26_N, U11.D4Z; no longer FMC_LPCG$1.LA01_N_CC, U20.D4Z
- net +3V3_ISO_PG_P: now also FMC_LPCG$1.LA26_P, U11.D4Y; no longer FMC_LPCG$1.LA01_P_CC, U20.D4Y
- net +5.5V_ISO: now also C22.2, C23.+, C24.+, C31.2, C77.1, C79.2, L4.1, TP24.TP, U6.+VO, U7.RUN1, U7.RUN2, U7.VIN; no longer C13.2, C17.1, C42.2, C45.2, C47.+, C48.+, L3.1, TP4.TP, U10.RUN1, U10.RUN2, U10.VIN, U12.+VO
- net 2V5_REF: now also J1.3, J2.3, R27.1; no longer R67.1, U2.3, U3.3
- net BIAS_DI0: now also J1.1, U4.VOUT0; no longer U2.1, U8.VOUT0
- net BIAS_DI1: now also J2.1, U4.VOUT1; no longer U3.1, U8.VOUT1
- net BISTEN: now also R64.1, U12.BISTEN, U15.1; no longer R19.1, U7.1, U9.BISTEN
- net D0: now also U11.A1A, U9.VOA; no longer U13.VOA, U20.A1A
- net D0_ISO: now also R55.1, U9.VIA; no longer R54.1, U13.VIA
- net D0_N: now also U11.A1Z; no longer U20.A1Z
- net D0_P: now also U11.A1Y; no longer U20.A1Y
- net D1: now also U11.A2A, U9.VOB; no longer U13.VOB, U20.A2A
- net D10: now also U11.C3A, U13.VOC; no longer U15.VOC, U20.C3A
- net D10_ISO: now also R45.1, U13.VIC; no longer R35.1, U15.VIC
- net D10_N: now also U11.C3Z; no longer U20.C3Z
- net D10_P: now also U11.C3Y; no longer U20.C3Y
- net D11: now also U11.C4A, U13.VOD; no longer U15.VOD, U20.C4A
- net D11_ISO: now also R44.1, U13.VID; no longer R42.1, U15.VID
- net D11_N: now also U11.C4Z; no longer U20.C4Z
- net D11_P: now also U11.C4Y; no longer U20.C4Y
- net D1_ISO: now also R54.1, U9.VIB; no longer R38.1, U13.VIB
- net D1_N: now also U11.A2Z; no longer U20.A2Z
- net D1_P: now also U11.A2Y; no longer U20.A2Y
- net D2: now also U11.A3A, U9.VOC; no longer U13.VOC, U20.A3A
- net D2_ISO: now also R53.1, U9.VIC; no longer R45.1, U13.VIC
- net D2_N: now also U11.A3Z; no longer U20.A3Z
- net D2_P: now also U11.A3Y; no longer U20.A3Y
- net D3: now also U11.A4A, U9.VOD; no longer U13.VOD, U20.A4A
- net D3_ISO: now also R52.1, U9.VID; no longer R53.1, U13.VID
- net D3_N: now also U11.A4Z; no longer U20.A4Z
- net D3_P: now also U11.A4Y; no longer U20.A4Y
- net D4: now also U10.VOA, U11.B1A; no longer U14.VOA, U20.B1A
- net D4_ISO: now also R51.1, U10.VIA; no longer R37.1, U14.VIA
- net D4_N: now also U11.B1Z; no longer U20.B1Z
- net D4_P: now also U11.B1Y; no longer U20.B1Y
- net D5: now also U10.VOB, U11.B2A; no longer U14.VOB, U20.B2A
- net D5_ISO: now also R50.1, U10.VIB; no longer R44.1, U14.VIB
- net D5_N: now also U11.B2Z; no longer U20.B2Z
- net D5_P: now also U11.B2Y; no longer U20.B2Y
- net D6: now also U10.VOC, U11.B3A; no longer U14.VOC, U20.B3A
- net D6_ISO: now also R49.1, U10.VIC; no longer R52.1, U14.VIC
- net D6_N: now also U11.B3Z; no longer U20.B3Z
- net D6_P: now also U11.B3Y; no longer U20.B3Y
- net D7: now also U10.VOD, U11.B4A; no longer U14.VOD, U20.B4A
- net D7_ISO: now also R48.1, U10.VID; no longer R36.1, U14.VID
- net D7_N: now also U11.B4Z; no longer U20.B4Z
- net D7_P: now also U11.B4Y; no longer U20.B4Y
- net D8: now also U11.C1A, U13.VOA; no longer U15.VOA, U20.C1A
- net D8_ISO: now also R47.1, U13.VIA; no longer R43.1, U15.VIA
- net D8_N: now also U11.C1Z; no longer U20.C1Z
- net D8_P: now also U11.C1Y; no longer U20.C1Y
- net D9: now also U11.C2A, U13.VOB; no longer U15.VOB, U20.C2A
- net D9_ISO: now also R46.1, U13.VIB; no longer R51.1, U15.VIB
- net D9_N: now also U11.C2Z; no longer U20.C2Z
- net D9_P: now also U11.C2Y; no longer U20.C2Y
- net DAC_LAT_N: now also U8.B1B; no longer U19.B1B
- net DAC_LAT_P: now also U8.B1A; no longer U19.B1A
- net DI0: now also TP2.TP, U16.1A, U1G$1.OUT; no longer TP7.TP, U21.1A, U5G$1.OUT
- net DI0_N: now also U16.1Z; no longer U21.1Z
- net DI0_P: now also U16.1Y; no longer U21.1Y
- net DI0_TERM: now also R7.1, R8.1, U8.A1Y; no longer R73.1, R9.1, U19.A1Y
- net DI0_TERM_N: now also U8.A1B; no longer U19.A1B
- net DI0_TERM_P: now also U8.A1A; no longer U19.A1A
- net DI1: now also TP1.TP, U16.2A, U2G$1.OUT; no longer TP6.TP, U21.2A, U6G$1.OUT
- net DI1_N: now also U16.2Z; no longer U21.2Z
- net DI1_P: now also U16.2Y; no longer U21.2Y
- net DI1_TERM: now also R16.1, R17.1, U8.A2Y; no longer R11.1, R74.1, U19.A2Y
- net DI1_TERM_N: now also U8.A2B; no longer U19.A2B
- net DI1_TERM_P: now also U8.A2A; no longer U19.A2A
- net DO0: now also U3.1A, U3.2A, U8.B2Y; no longer U19.C2Y, U4.1A, U4.2A
- net DO0_N: now also U8.C1B; no longer U19.C1B
- net DO0_P: now also U8.C1A; no longer U19.C1A
- net DO1: now also U3.3A, U3.4A, U8.B1Y; no longer U19.C1Y, U4.3A, U4.4A
- net DO1_N: now also U8.C2B; no longer U19.C2B
- net DO1_P: now also U8.C2A; no longer U19.C2A
- net DOUTP_F: now also C57.2, L5.2, R68.2; no longer C16.2, L1.2, R7.2
- net DO_TEST_N: now also U8.B2B; no longer U19.B2B
- net DO_TEST_P: now also U8.B2A; no longer U19.B2A
- net GND: now also C1.2, C10.1, C11.-, C12.1, C13.1, C14.1, C15.1, C16.1, C18.1, C2.2, C21.-, C26.1, C27.1, C28.1, C3.2, C33.1, C4.2, C42.1, C43.1, C44.1, C45.1, C46.1, C47.1, C49.1, C5.-, C6.1, C63.1, C7.1, C71.1, C72.1, C73.1, C74.1, C75.1, C8.-, C9.1, J3.1, J3.4, J6.2, J8.2, R11.1, R18.1, R2.1, R23.1, R29.1, R9.1, TP18.TP, TP3.TP, TP4.TP, TP5.TP, TP6.TP, TP7.TP, TP9.TP, U10.GND2, U11.GND, U16.GND, U17.GND1, U18.GND2, U1G$2.V-, U2G$2.V-, U3.GND, U4.AVSS, U4.LAT/HVC, U5.GND1, U6.GND, U8.AGND, U8.DGND, U8.GND, U9.GND2; no longer C1.1, C2.1, C20.1, C44.-, C46.-, C55.1, C56.1, C57.1, C58.1, C59.1, C6.2, C61.1, C66.-, C7.2, C8.2, C80.1, C82.1, C83.1, C84.1, C85.1, C86.1, C87.-, C88.1, C89.1, C9.2, C90.1, C91.1, C92.1, C93.1, C94.1, C95.1, C96.1, C97.1, C98.1, R10.1, R3.1, R4.1, R5.1, R6.1, R8.1, TP10.TP, TP14.TP, TP15.TP, TP16.TP, TP17.TP, TP21.TP, TP23.TP, U11.GND1, U12.GND, U15.GND2, U16.GND2, U17.GND2, U18.1, U18.4, U19.AGND, U19.DGND, U19.GND, U20.GND, U21.GND, U4.GND, U5G$2.V-, U6G$2.V-, U8.AVSS
- net GND_ISO: now also C17.1, C20.1, C23.-, C24.-, C41.1, C48.1, C55.1, C56.1, C59.1, C61.1, C62.1, C64.1, C65.1, C66.1, C67.1, C68.1, C69.1, C70.1, C76.2, C77.2, C78.1, C79.1, C80.1, J4.1, J4.4, J5.2, J7.2, R35.2, R37.2, R38.2, R39.2, R42.2, R67.1, R73.2, R74.2, R75.2, TP17.TP, TP21.TP, TP25.TP, TP26.TP, TP27.TP, U10.GND1, U12.DAP, U12.RES, U12.TESTEN, U15.5, U15.6, U15.7, U15.8, U17.GND2, U18.GND1, U5.GND2, U6.-VO, U7.GND, U7.SYNC/MODE, U9.GND1; no longer C10.1, C11.1, C13.1, C14.1, C15.1, C17.2, C18.1, C21.1, C23.1, C24.1, C26.1, C27.1, C28.1, C3.1, C33.1, C4.1, C42.1, C45.1, C47.-, C48.-, C49.1, C5.2, R30.2, R34.1, R55.2, R58.2, R59.2, R61.2, R63.2, R64.2, R68.2, TP1.TP, TP18.TP, TP19.TP, TP20.TP, TP28.TP, U1.1, U1.4, U10.GND, U10.SYNC/MODE, U11.GND2, U12.-VO, U15.GND1, U16.GND1, U17.GND1, U7.5, U7.6, U7.7, U7.8, U9.DAP, U9.RES, U9.TESTEN
- net GPI0_N: now also U16.4Z; no longer U21.4Z
- net GPI0_P: now also U16.4Y; no longer U21.4Y
- net GPI1_N: now also U16.3Z; no longer U21.3Z
- net GPI1_P: now also U16.3Y; no longer U21.3Y
- net GPO0_N: now also U8.D1B; no longer U19.D1B
- net GPO0_P: now also U8.D1A; no longer U19.D1A
- net GPO1_N: now also U8.D2B; no longer U19.D2B
- net GPO1_P: now also U8.D2A; no longer U19.D2A
- net HSYNC: now also U11.D1A, U14.VOA; no longer U16.VOA, U20.D1A
- net HSYNC_ISO: now also R43.1, U14.VIA; no longer R50.1, U16.VIA
- net HSYNC_N: now also FMC_LPCG$1.LA01_N_CC, U11.D1Z; no longer FMC_LPCG$1.GBTCLK0_M2C_N, U20.D1Z
- net HSYNC_P: now also FMC_LPCG$1.LA01_P_CC, U11.D1Y; no longer FMC_LPCG$1.GBTCLK0_M2C_P, U20.D1Y
- net IDX0: now also R70.2, R73.1, U12.IDX0; no longer R57.2, R58.1, U9.IDX0
- net IDX1: now also R71.2, R74.1, U12.IDX1; no longer R60.2, R61.1, U9.IDX1
- net INTVCC: now also R34.1, U7.INTVCC; no longer R56.1, U10.INTVCC
- net LOCK: now also U16.3A, U18.VOA; no longer R33.2, U9.LOCK
- net MODE: now also R72.2, R75.1, U12.MODE; no longer R62.2, R63.1, U9.MODE
- net N$10: now also R37.1, U7.FB1; no longer R55.1, U10.FB1
- net N$12: now also C30.2, U7.TRACK/SS1; no longer C40.2, U10.TRACK/SS1
- net N$13: now also U12.VSYNC; no longer U9.VSYNC
- net N$136: now also J1.2, R3.1; no longer R26.1, U2.2
- net N$145: now also R38.1, U7.FREQ; no longer R64.1, U10.FREQ
- net N$15: now also R65.1; no longer R46.1
- net N$16: now also R43.2, U12.HSYNC; no longer R50.2, U9.HSYNC
- net N$18: now also C2.1, R3.2, U1G$1.-IN; no longer C6.1, R26.2, U5G$1.-IN
- net N$19: now also R10.2, U2G$1.+IN; no longer R29.2, U6G$1.+IN
- net N$2: now also Q1.D, R4.1, R5.1, R6.1; no longer Q3.D, R16.1, R21.1, R23.1
- net N$20: now also C4.1, R12.2, U2G$1.-IN; no longer C7.1, R27.2, U6G$1.-IN
- net N$21: now also L5.1, L6.2, R68.1, R69.2; no longer L1.1, L2.2, R20.2, R7.1
- net N$22: now also C76.1, C78.2, L4.2, L6.1, R69.1; no longer C3.2, C5.1, L2.1, L3.2, R20.1
- net N$23: now also R20.1; no longer R1.1
- net N$24: now also R21.1, U3.~1G, U3.~2G; no longer R31.1, U4.~1G, U4.~2G
- net N$25: now also R22.1, U3.~3G, U3.~4G; no longer R32.1, U4.~3G, U4.~4G
- net N$26: now also R35.1, U6.TRIM; no longer R68.1, U12.TRIM
- net N$27: now also C57.1, U12.RIN0+; no longer C16.1, U9.RIN0+
- net N$28: now also C58.1, U12.RIN0-; no longer C12.1, U9.RIN0-
- net N$3: now also R1.2, U1G$1.+IN; no longer R28.2, U5G$1.+IN
- net N$30: now also R8.2; no longer R9.2
- net N$31: now also R28.1; no longer R2.1
- net N$32: now also C58.2, R42.1; no longer C12.2, R30.1
- net N$33: now also R36.1; no longer R75.1
- net N$34: now also Q2.G, R16.2, R18.2; no longer Q4.G, R74.2, R8.2
- net N$35: now also Q3.D; no longer Q1.D
- net N$36: now also J2.2, R12.1; no longer R27.1, U3.2
- net N$37: now also Q1.G, R7.2, R9.2; no longer Q3.G, R10.2, R73.2
- net N$38: now also R57.2, U12.GPIO3; no longer TP29.TP, U9.GPIO3
- net N$39: now also Q3.G, R19.1, R23.2; no longer Q1.G, R13.1, R3.2
- net N$4: now also R40.2, U12.PCLK; no longer R49.2, U9.PCLK
- net N$44: now also R46.2, U12.ROUT9; no longer R51.2, U9.ROUT9
- net N$45: now also R47.2, U12.ROUT8; no longer R43.2, U9.ROUT8
- net N$46: now also R48.2, U12.ROUT7; no longer R36.2, U9.ROUT7
- net N$47: now also R49.2, U12.ROUT6; no longer R52.2, U9.ROUT6
- net N$48: now also R50.2, U12.ROUT5; no longer R44.2, U9.ROUT5
- net N$49: now also R51.2, U12.ROUT4; no longer R37.2, U9.ROUT4
- net N$5: now also R39.1, U7.FB2; no longer R59.1, U10.FB2
- net N$50: now also R52.2, U12.ROUT3; no longer R53.2, U9.ROUT3
- net N$51: now also R53.2, U12.ROUT2; no longer R45.2, U9.ROUT2
- net N$52: now also R54.2, U12.ROUT1; no longer R38.2, U9.ROUT1
- net N$53: now also R55.2, U12.ROUT0; no longer R54.2, U9.ROUT0
- net N$54: now also R44.2, U12.ROUT11; no longer R42.2, U9.ROUT11
- net N$55: now also R45.2, U12.ROUT10; no longer R35.2, U9.ROUT10
- net N$57: now also R58.2, U12.GPIO2; no longer R47.2, U9.GPIO2
- net N$58: now also R59.2, U12.GPIO1; no longer R40.2, U9.GPIO1
- net N$59: now also R60.2, U12.GPIO0; no longer R48.2, U9.GPIO0
- net N$60: now also Q4.D; no longer Q2.D
- net N$61: now also Q4.G, R26.1, R29.2; no longer Q2.G, R12.1, R4.2
- net N$62: now also R66.1, R67.2; no longer R33.1, R34.2
- net N$7: now also Q2.D, R13.1, R14.1, R15.1; no longer Q4.D, R17.1, R22.1, R24.1
- net N$8: now also C29.2, U7.TRACK/SS2; no longer C39.2, U10.TRACK/SS2
- net N$9: now also R17.2; no longer R11.2
- net OEN: now also R63.1, U12.OEN, U15.2; no longer R15.1, U7.2, U9.OEN
- net OSS_SEL: now also R62.1, U12.OSS_SEL, U15.3; no longer R18.1, U7.3, U9.OSS_SEL
- net PASS: now also U16.4A, U18.VOC; no longer R39.2, TP5.TP, U9.PASS
- net PCLK: now also U11.D3A, U14.VOC; no longer U16.VOC, U20.D3A
- net PCLK_ISO: now also R40.1, U14.VIC; no longer R49.1, U16.VIC
- net PCLK_N: now also U11.D3Z; no longer U20.D3Z
- net PCLK_P: now also U11.D3Y; no longer U20.D3Y
- net PDN: now also C61.2, R56.2, U12.PDN; no longer C4.2, R25.2, U9.PDN
- net SCL: now also R33.1, TP20.TP, U4.SCL, U5.SCL1; no longer R72.1, TP25.TP, U11.SCL1, U8.SCL
- net SCL_ISO: now also R30.1, TP15.TP, U12.SCL, U5.SCL2; no longer R65.1, TP26.TP, U11.SCL2, U9.SCL
- net SDA: now also R32.1, TP19.TP, U4.SDA, U5.SDA1; no longer R71.1, TP24.TP, U11.SDA1, U8.SDA
- net SDA_ISO: now also R31.1, TP16.TP, U12.SDA, U5.SDA2; no longer R66.1, TP27.TP, U11.SDA2, U9.SDA
- net SEL: now also R61.1, U12.SEL, U15.4; no longer R14.1, U7.4, U9.SEL
- net VDDCML0: now also C52.2, C53.2, C54.2, L3.1, U12.VDDCML0; no longer C11.2, C15.2, C19.2, L5.1, U9.VDDCML0
- net VDDCML1: now also C36.2, C37.2, C38.2, L1.1, U12.VDDCML1; no longer C10.2, C14.2, C18.2, L4.1, U9.VDDCML1
- net VDDPLL: now also C39.2, C40.2, C41.2, L2.2, U12.VDDPLL; no longer C22.2, C23.2, C26.2, L6.2, U9.VDDPLL
- net VIN: now also U6.EN, U6.VIN; no longer U12.EN, U12.VIN
- net VSYNC: now also U11.D2A, U14.VOB; no longer U16.VOB, U20.D2A
- net VSYNC_ISO: now also U14.VIB; no longer U16.VIB
- net VSYNC_N: now also U11.D2Z; no longer U20.D2Z
- net VSYNC_P: now also U11.D2Y; no longer U20.D2Y
- net V_PROTECT: now also C16.2, R24.1, R25.1, TP14.TP; no longer C55.2, R69.1, R70.1, TP9.TP
Other:
- note added: "DI0, DI1, PASS, LOCK"
- note added: "DNP"
- note added: "Seeed 4 layer stackup: 1.4 mil trace 8 mil prepeg 0.7 mil trace XX mil FR4 core 0.7 mil trace 8 mil prepeg 1.4 mil trace"
- note removed: "Seeed 4 layer stackup: 1.4 mil trace 8 mill prepeg 0.7 mil trace XX mil FR4 core 0.7 mil trace 8 mil prepeg 1.4 mil trace"
- moved on the sheet: C1, C10, C11, C12, C13, C14, C15, C16, C17, C18, C19, C2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

Commit message: Added path the deserializer PDN input on host board
- Tactile switch on panel
- Path from host FPGA
- Allows hard reset of deserializer
Parts:
- removed TP25: GND(ISO), jonnew:TP_1MM
- added Q6: NDS351AN, jonnew:N-MOSFET_SOT23-GSD
- added R77: 1k, jonnew:R_0402
- added R78: 100k, jonnew:R_0402
- added R79, R80: 0, jonnew:R_0402
- added S1: (no value), jonnew:SPST_TACT2_EVQPF
- J4: device jonnew:SCREW4 -> jonnew:PINHD-1X4
Connections:
- removed net PDN: C61.2, R56.2, U12.PDN
- new net N$1: Q6.G, R77.1, R78.2
- new net N$40: J7.1, R80.1
- new net PDN_ISO: C61.2, Q6.D, R56.2, R77.2, R79.2, S1.S, U12.PDN
- net GND_ISO: now also Q6.S, R78.1, S1.P; no longer TP25.TP
- net SMA_OUT_ISO: now also R79.1, R80.2; no longer J7.1
Other:
- moved on the sheet: C61, J4, J5, J7, LINK, R56, R61, R62, R63, R64

Commit message: Minor fixes to pcie-host board during BOM updated
- BOM simplification and correction
- Some minor layout fixes
Parts:
- removed TP27: GND(ISO), jonnew:TP_1MM
- added TP25: GND(ISO), jonnew:TP_1MM
- C12: device RHD2000_eval_board:C_0603 -> jonnew:C_0805
- C54: value 4.7F -> 4.7uF
- C61: device jonnew:C_0603 -> jonnew:C_1206
- C78, C79: device jonnew:C_0805 -> jonnew:C_1206
- L5: value 1008PS-472KLB -> 1008PS-472
- L6: value SRN6045TA-101M -> SRNxx-101M
- Q5: value NDS351AN -> NDS351
- R56, R61, R62, R63, R72: value 10K -> 10k
- R64, R70, R71: value 10K -> 1k; device jonnew:R_0402 -> jonnew:R_0603
- R65: value 1k -> 10k; device cyclops:R_0603 -> jonnew:R_0402
- R67: device cyclops:R_0603 -> jonnew:R_0603
- R68: value 1K -> 1k; device jonnew:R_0603 -> cyclops:R_0603
- R69: value 1K -> 100k; device jonnew:R_0603 -> cyclops:R_0603
- R73, R74: value 0 -> 10k
- R76: value 22 -> 0
- R77: value 1k -> 3k
- R78: value 100k -> 22
- U17: value ISO7742 -> ISO7740
Connections:
- net +1V8_ISO: now also R73.1, R74.1; no longer R70.1, R71.1
- net +3V3_ISO: now also R66.2; no longer R64.2
- net BISTEN: now also R65.1; no longer R64.1
- net DOUTP_F: now also R70.2; no longer R68.2
- net GND_ISO: now also R69.1, R76.2, R77.2, TP25.TP; no longer R73.2, R74.2, R78.1, TP27.TP
- net IDX0: now also R72.2, R75.1; no longer R70.2, R73.1
- net IDX1: now also R73.2, R76.1; no longer R71.2, R74.1
- net LOCK_ISO: now also R68.2; no longer R66.2
- net MODE: now also R74.2, R77.1; no longer R72.2, R75.1
- net N$1: now also Q5.G, R64.1, R67.2; no longer Q6.G, R77.1, R78.2
- net N$15: now also R66.1; no longer R65.1
- net N$21: now also R70.1, R71.2; no longer R68.1, R69.2
- net N$22: now also R71.1; no longer R69.1
- net N$29: now also Q6.D; no longer Q5.D
- net N$40: now also R79.1; no longer R80.1
- net N$56: now also R78.1; no longer R76.1
- net N$62: now also Q6.G, R68.1, R69.2; no longer Q5.G, R66.1, R67.2
- net PASS_ISO: now also R78.2; no longer R76.2
- net PDN_ISO: now also Q5.D, R64.2, R80.2; no longer Q6.D, R77.2, R79.2
- net SMA_OUT_ISO: now also R79.2, R80.1; no longer R79.1, R80.2
Other:
- moved on the sheet: Q5, Q6, R64, R65, R66, R67, R68, R69, R70, R71, R72, R73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
