File: headstage/headstage.sch (EAGLE design)
At the start: 43 parts, among them U1 ADXL335, U2 74HC4053

Commit message: Headstage Rev 1.2
- New digital interface matches the updated SPI interface board
- Accelerometer turned to be normal with direction of head
- Accelerometer jumpered in using 0 ohm resistors
- All 6 AUX inputs and a single output are pinned out through the
  digital interface and via testpoints on the headstage module.
Parts:
- removed R11, R12, R13: 0, jonnew:R_0201
- added A1, A2, A3, B1, B2, B3, BOUT: (no value), jonnew:TESTPOINT_SMALL
- renumbered PLT to PLATE
Connections:
- removed net DGND_THRU: DTHRU_BNA.1, DTHRU_BNA.2, DTHRU_BNA.3, DTHRU_BNA.5, DTHRU_BNA.6, DTHRU_BNA.7, DTHRU_TNA.1, DTHRU_TNA.2, DTHRU_TNA.3, DTHRU_TNA.5, DTHRU_TNA.6, DTHRU_TNA.7
- removed net VDD_THRU: DTHRU_BNA.10, DTHRU_BNA.8, DTHRU_BNA.9, DTHRU_TNA.10, DTHRU_TNA.8, DTHRU_TNA.9
- removed net XOUT2: R11.2
- removed net YOUT2: R12.2
- removed net ZOUT2: R13.2
- new net AUXIN1_A_THRU: DTHRU_BNA.1, DTHRU_TNA.1
- new net AUXIN1_B_THRU: DTHRU_BNA.5, DTHRU_TNA.5
- new net AUXIN2_A_THRU: DTHRU_BNA.2, DTHRU_TNA.2
- new net AUXIN2_B_THRU: DTHRU_BNA.6, DTHRU_TNA.6
- new net AUXIN3_A_THRU: DTHRU_BNA.3, DTHRU_TNA.3
- new net AUXIN3_B_THRU: DTHRU_BNA.7, DTHRU_TNA.7
- new net GND_THRU: DTHRU_BNA.8, DTHRU_BNA.9, DTHRU_TNA.8, DTHRU_TNA.9
- new net VCC_THRU: DTHRU_BNA.10, DTHRU_TNA.10
- net AUXIN1_A: now also A1.1; no longer R11.1
- net AUXIN1_B: now also B1.1
- net AUXIN2_A: now also A2.1; no longer R12.1
- net AUXIN2_B: now also B2.1
- net AUXIN3_A: now also A3.1; no longer R13.1
- net AUXIN3_B: now also B3.1
- net AUXOUT_B: now also BOUT.1
- net GND: now also U1.NC1, U1.NC2, U1.NC6
Other:
- note added: "Solderable Pins"
- note removed: "GYRO"
- moved on the sheet: C3

Commit message: Updates to 128-channel headstage module
- More grounding vias
- Top and bottom ground pours
- Stop ring around top periphery to attach faraday cange for next gen
  drives
Parts:
- removed REF2: REF, jonnew:TESTPOINT_SMALL
- ATHRU_TEB, ATHRU_TWB, MECH_TNB, MECH_TSB: device jonnew:PINHD-2X35_DF40HEAD -> jonnew:PINHD-2X35+4_DF40-70HEAD
- DIO_TEA, DTHRU_TNA: device jonnew:PINHD-2X10_DF40-20HEAD -> jonnew:PINHD-2X10+4_DF40-HEAD
- R1, R10, R2, R3, R8, R9: device jonnew:R_0201 -> jonnew:R_0402
Connections:
- net GND: now also ATHRU_TEB.M1, ATHRU_TEB.M2, ATHRU_TEB.M3, ATHRU_TEB.M4, ATHRU_TWB.M1, ATHRU_TWB.M2, ATHRU_TWB.M3, ATHRU_TWB.M4, DIO_TEA.M1, DIO_TEA.M2, DIO_TEA.M3, DIO_TEA.M4, DTHRU_TNA.M1, DTHRU_TNA.M2, DTHRU_TNA.M3, DTHRU_TNA.M4, MECH_TNB.M1, MECH_TNB.M2, MECH_TNB.M3, MECH_TNB.M4, MECH_TSB.M1, MECH_TSB.M2, MECH_TSB.M3, MECH_TSB.M4
- net REF: no longer REF2.1
Other:
- moved on the sheet: A1, A2, A3, AMP_A, AMP_B, B1, B2, B3, BOUT, C1, C2, C3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
