File: eib-256/eib-256-nanoz-adapter.sch (EAGLE design)
At the start: 42 parts, among them U1 DG4052E_MQFN, U10 DG4052E_MQFN, U11 DG4052E_MQFN, U12 DG4052E_MQFN, U13 DG4052E_MQFN, U14 DG4052E_MQFN, U15 DG4052E_MQFN, U16 DG4052E_MQFN, U17 DG4052E_MQFN, U18 DG4052E_MQFN, U19 DG4052E_MQFN, U2 DG4052E_MQFN, U20 DG4052E_MQFN, U21 DG4052E_MQFN, U22 DG4052E_MQFN, U23 DG4052E_MQFN, U24 DG4052E_MQFN, U25 DG4052E_MQFN, U26 DG4052E_MQFN, U27 DG4052E_MQFN, U28 DG4052E_MQFN, U29 DG4052E_MQFN, U3 DG4052E_MQFN, U30 DG4052E_MQFN, U31 DG4052E_MQFN, U32 DG4052E_MQFN, U4 DG4052E_MQFN, U5 DG4052E_MQFN, U6 DG4052E_MQFN, U7 DG4052E_MQFN, U8 DG4052E_MQFN, U9 DG4052E_MQFN

Commit message: More work on eib-245 nanoz adapter board
- Hard routing done
- Needs user pinout for power, ref, etc
- Needs reverse polarity protection
Parts:
- added $1_8_$1: (no value), jonnew:PINHD-4X10_MOLC-THRU
- added C10, C15, C16, C17, C18, C5, C6, C9: 1uF, jonnew:C_0603
- added C11, C12: 10uF, jonnew:C-POL_1210
- added C13, C14, C3, C4, C7, C8: 0.1uF, jonnew:C_0402
- added D1, D2: (no value), jonnew:LED_0603
- added R3, R4: 1k, jonnew:R_0603
- added TP1, TP2, TP3, TP4: (no value), jonnew:TESTPOINT
- added U101, U33: (no value), jonnew:JP3E
- added U102: SCREW4, jonnew:SCREW4
- C1, C2: value (none) -> 0.1uF
Connections:
- removed net N$106: $1_8_$G$1.17
- removed net N$107: $1_8_$G$2.2
- removed net N$108: $1_8_$G$2.3
- removed net N$109: $1_8_$G$2.4
- removed net N$111: U21.Y, U22.Y, U23.Y
- removed net NC: $1_8_$G$1.18
- new net N$449: D1.A, R3.1
- new net N$451: D2.A, R4.1
- new net TT34: $1_8_$1G$2.9, U10.X
- new net TT35: $1_8_$1G$2.12, U10.Y
- new net TT36: $1_8_$1G$2.8, U11.X
- new net TT37: $1_8_$1G$2.13, U11.Y
- new net TT38: $1_8_$1G$2.7, U12.X
- new net TT39: $1_8_$1G$2.14, U12.Y
- new net TT40: $1_8_$1G$2.19, U13.X
- new net TT41: $1_8_$1G$2.20, U13.Y
- new net TT42: $1_8_$1G$2.17, U14.X
- new net TT43: $1_8_$1G$2.18, U14.Y
- new net TT44: $1_8_$1G$2.5, U15.X
- new net TT45: $1_8_$1G$2.16, U15.Y
- new net TT46: $1_8_$1G$2.6, U16.X
- new net TT47: $1_8_$1G$2.15, U16.Y
- new net TT48: $1_8_$1G$1.1, U17.X
- new net TT49: $1_8_$1G$1.2, U17.Y
- new net TT50: $1_8_$1G$1.3, U18.X
- new net TT51: $1_8_$1G$1.4, U18.Y
- new net TT52: $1_8_$1G$1.5, U19.X
- new net TT53: $1_8_$1G$1.16, U19.Y
- new net TT54: $1_8_$1G$1.6, U20.X
- new net TT55: $1_8_$1G$1.15, U20.Y
- new net TT56: $1_8_$1G$1.10, U21.X
- new net TT57: $1_8_$1G$1.11, U21.Y
- new net TT58: $1_8_$1G$1.9, U22.X
- new net TT59: $1_8_$1G$1.12, U22.Y
- new net TT60: $1_8_$1G$1.8, U23.X
- new net TT61: $1_8_$1G$1.13, U23.Y
- new net TT62: $1_8_$1G$1.7, U24.X
- new net TT63: $1_8_$1G$1.14, U24.Y
- new net VCC_HEAD: U101.1
- new net VCC_PRE: TP1.1, U101.2, U101.3
- new net VSS_HEAD: U33.1
- new net VSS_PRE: TP2.1, U33.2, U33.3
- net A: now also U1.A, U2.A, U3.A, U32.A, U4.A, U5.A, U6.A, U7.A
- net B: now also U1.B, U2.B, U3.B, U32.B, U4.B, U5.B, U6.B, U7.B
- net GND: now also C10.2, C11.-, C12.+, C13.2, C14.2, C15.2, C16.2, C17.2, C18.2, C3.2, C4.2, C5.2, C6.2, C7.2, C8.2, C9.2, D1.C, R4.2, TP4.1, U1.!EN, U1.GND, U102.3, U2.!EN, U2.GND, U26.!EN, U3.!EN, U3.GND, U30.!EN, U32.!EN, U32.GND, U4.!EN, U4.GND, U5.!EN, U5.GND, U6.!EN, U6.GND, U7.!EN, U7.GND
- net N$1: no longer U9.X3
- net N$10: no longer U10.X0
- net N$105: no longer U16.Y1
- net N$11: no longer U10.X1
- net N$112: no longer U32.X0
- net N$113: no longer U32.X1
- net N$114: no longer U32.X2
- net N$115: no longer U32.Y0
- net N$116: no longer U32.Y2
- net N$117: no longer U32.Y3
- net N$12: no longer U10.X2
- net N$13: no longer U10.Y0
- net N$14: no longer U10.Y2
- net N$141: no longer U32.Y1
- net N$142: no longer U31.X3
- net N$143: no longer U31.X0
- net N$144: no longer U31.X1
- net N$145: no longer U31.X2
- net N$146: no longer U31.Y0
- net N$147: no longer U31.Y2
- net N$148: no longer U31.Y3
- net N$149: no longer U31.Y1
- net N$15: no longer U10.Y3
- net N$150: no longer U30.X3
- net N$151: no longer U30.X0
- net N$152: no longer U30.X1
- net N$153: no longer U30.X2
- net N$154: no longer U30.Y0
- net N$155: no longer U30.Y2
- net N$156: no longer U30.Y3
- net N$157: no longer U30.Y1
- net N$158: no longer U29.X3
- net N$159: no longer U29.X0
- net N$16: no longer U10.Y1
- net N$160: no longer U29.X1
- net N$161: no longer U29.X2
- net N$162: no longer U29.Y0
- net N$163: no longer U29.Y2
- net N$164: no longer U29.Y3
- net N$165: no longer U29.Y1
- net N$166: no longer U28.X3
- net N$167: no longer U28.X0
- net N$168: no longer U28.X1
- net N$169: no longer U28.X2
- net N$17: no longer U11.X3
- net N$170: no longer U28.Y0
- net N$171: no longer U28.Y2
- net N$172: no longer U28.Y3
- net N$173: no longer U28.Y1
- net N$174: no longer U27.X3
- net N$175: no longer U27.X0
- net N$176: no longer U27.X1
- net N$177: no longer U27.X2
- net N$178: no longer U27.Y0
- net N$179: no longer U27.Y2
- net N$18: no longer U11.X0
- net N$180: no longer U27.Y3
- net N$181: no longer U27.Y1
- net N$182: no longer U26.X3
- net N$183: no longer U26.X0
- net N$184: no longer U26.X1
- net N$185: no longer U26.X2
- net N$186: no longer U26.Y0
- net N$187: no longer U26.Y2
- net N$188: no longer U26.Y3
- net N$189: no longer U26.Y1
- net N$19: no longer U11.X1
- net N$190: no longer U25.Y0
- net N$191: no longer U25.Y2
- net N$192: no longer U25.Y3
- net N$193: no longer U25.Y1
- net N$194: no longer U25.X3
- net N$195: no longer U25.X0
- net N$196: no longer U25.X1
- net N$197: no longer U25.X2
- net N$198: no longer U24.X3
- net N$199: no longer U24.X0
- net N$2: no longer U9.X0
- net N$20: no longer U11.X2
- net N$200: no longer U24.X1
- net N$201: no longer U24.X2
- net N$202: no longer U24.Y0
- net N$203: no longer U24.Y2
- net N$204: no longer U24.Y3
- net N$205: no longer U24.Y1
- net N$206: no longer U23.X3
- net N$207: no longer U23.X0
- net N$208: no longer U23.X1
- net N$209: no longer U23.X2
- net N$21: no longer U11.Y0
- net N$210: no longer U23.Y0
- net N$211: no longer U23.Y2
- net N$212: no longer U23.Y3
- net N$213: no longer U23.Y1
- net N$214: no longer U22.X3
- net N$215: no longer U22.X0
- net N$216: no longer U22.X1
- net N$217: no longer U22.X2
- net N$218: no longer U22.Y0
- net N$219: no longer U22.Y2
- net N$22: no longer U11.Y2
- net N$220: no longer U22.Y3
- net N$221: no longer U22.Y1
- net N$222: no longer U21.X3
- net N$223: no longer U21.X0
- net N$224: no longer U21.X1
- net N$225: no longer U21.X2
- net N$226: no longer U21.Y0
- net N$227: no longer U21.Y2
- net N$228: no longer U21.Y3
- net N$229: no longer U21.Y1
- net N$23: no longer U11.Y3
- net N$230: no longer U20.X3
- net N$231: no longer U20.X0
- net N$232: no longer U20.X1
- net N$233: no longer U20.X2
- net N$234: no longer U20.Y0
- net N$235: no longer U20.Y2
- net N$236: no longer U20.Y3
- net N$237: no longer U20.Y1
- net N$238: no longer U19.X3
- net N$239: no longer U19.X0
- net N$24: no longer U11.Y1
- net N$240: no longer U19.X1
- net N$241: no longer U19.X2
- net N$242: no longer U19.Y0
- net N$243: no longer U19.Y2
- net N$244: no longer U19.Y3
- net N$245: no longer U19.Y1
- net N$246: no longer U18.X3
- net N$247: no longer U18.X0
- net N$248: no longer U18.X1
- net N$249: no longer U18.X2
- net N$25: no longer U12.X3
- net N$250: no longer U18.Y0
- net N$251: no longer U18.Y2
- net N$252: no longer U18.Y3
- net N$253: no longer U18.Y1
- net N$254: no longer U17.X3
- net N$255: no longer U17.X0
- net N$256: no longer U17.X1
- net N$257: no longer U17.X2
- net N$258: no longer U17.Y0
- net N$259: no longer U17.Y2
- net N$26: no longer U12.X0
- net N$260: no longer U17.Y3
- net N$261: no longer U17.Y1
- net N$27: no longer U12.X1
- net N$28: no longer U12.X2
- net N$29: no longer U12.Y0
- net N$3: no longer U9.X1
- net N$30: no longer U12.Y2
- net N$31: no longer U12.Y3
- net N$32: no longer U32.X3
- net N$33: no longer U12.Y1
- net N$34: no longer U13.X3
- net N$35: no longer U13.X0
- net N$36: no longer U13.X1
- net N$37: no longer U13.X2
- net N$38: no longer U13.Y0
- net N$39: no longer U13.Y2
- net N$4: no longer U9.X2
- net N$40: no longer U13.Y3
- net N$41: no longer U13.Y1
- net N$42: no longer U14.X3
- net N$43: no longer U14.X0
- net N$44: no longer U14.X1
- net N$45: no longer U14.X2
- net N$46: no longer U14.Y0
- net N$47: no longer U14.Y2
- net N$48: no longer U14.Y3
- net N$49: no longer U14.Y1
- net N$5: no longer U9.Y0
- net N$50: no longer U15.X3
- net N$51: no longer U15.X0
- net N$52: no longer U15.X1
- net N$53: no longer U15.X2
- net N$54: no longer U15.Y0
- net N$55: no longer U15.Y2
- net N$56: no longer U15.Y3
- net N$57: no longer U15.Y1
- net N$58: no longer U16.X3
- net N$59: no longer U16.X0
- net N$6: no longer U9.Y2
- net N$60: no longer U16.X1
- net N$61: no longer U16.X2
- net N$62: no longer U16.Y0
- net N$63: no longer U16.Y2
- net N$64: no longer U16.Y3
- net N$7: no longer U9.Y3
- net N$8: no longer U9.Y1
- net N$9: no longer U10.X3
- net REF: now also $1_8_$1G$1.20, $1_8_$1G$2.1, $1_8_$1G$2.2, $1_8_$G$2.2, TP3.1, U102.4; no longer $1_8_$G$1.19
- net TT00: now also $1_8_$G$1.1; no longer U9.X
- net TT01: now also $1_8_$G$1.2; no longer U9.Y
- net TT02: now also $1_8_$G$1.3; no longer U10.X
- net TT03: now also $1_8_$G$1.4; no longer U10.Y
- net TT04: now also $1_8_$G$1.5; no longer U11.X
- net TT05: now also $1_8_$G$1.16; no longer U11.Y
- net TT06: now also $1_8_$G$1.6; no longer U12.X
- net TT07: now also $1_8_$G$1.15; no longer U12.Y
- net TT08: now also $1_8_$G$1.10; no longer U13.X
- net TT09: now also $1_8_$G$1.11; no longer U13.Y
- net TT10: now also $1_8_$G$1.9; no longer U14.X
- net TT11: now also $1_8_$G$1.12; no longer U14.Y
- net TT12: now also $1_8_$G$1.8; no longer U15.X
- net TT13: now also $1_8_$G$1.13; no longer U15.Y
- net TT14: now also $1_8_$G$1.7; no longer U16.X
- net TT15: now also $1_8_$G$1.14; no longer U16.Y
- net TT16: now also $1_8_$G$2.10; no longer U17.X
- net TT17: now also $1_8_$G$2.11; no longer U17.Y
- net TT18: now also $1_8_$G$2.9; no longer U18.X
- net TT19: now also $1_8_$G$2.12; no longer U18.Y
- net TT20: now also $1_8_$G$2.8; no longer U19.X
- net TT21: now also $1_8_$G$2.13; no longer U19.Y
- net TT22: now also $1_8_$G$2.7; no longer U20.X
- net TT23: now also $1_8_$G$2.14; no longer U20.Y
- net TT24: now also $1_8_$G$2.19; no longer U21.X, U22.X, U23.X
- net TT25: now also $1_8_$G$2.20
- net TT26: now also $1_8_$G$2.17
- net TT27: now also $1_8_$G$2.18
- net TT28: now also $1_8_$G$2.5
- net TT29: now also $1_8_$G$2.16
- net TT30: now also $1_8_$G$2.6
- net TT31: now also $1_8_$G$2.15
- net TT32: now also $1_8_$1G$2.10, U9.X; no longer U24.Y
- net TT33: now also $1_8_$1G$2.11, U9.Y; no longer U24.X
- net VCC: now also C11.+, C13.1, C15.1, C17.1, C3.1, C5.1, C7.1, C9.1, R3.2, U1.V+, U102.1, U2.V+, U26.V+, U3.V+, U32.V+, U4.V+, U5.V+, U6.V+, U7.V+
- net VSS: now also C10.1, C12.-, C14.1, C16.1, C18.1, C4.1, C6.1, C8.1, D2.C, U1.V-, U102.2, U2.V-, U26.V-, U3.V-, U30.V-, U32.V-, U4.V-, U5.V-, U6.V-, U7.V-
Other:
- moved on the sheet: C1, C2, R1, R2, S1, U10, U11, U12, U13, U14, U15, U16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

Commit message: Finished rat EIB nanoz adapter board
- Repo needs some reorganization since this board can be used for both
256 and 128 channel EIBs
Parts:
- removed TP1, TP2, TP3, TP4: (no value), jonnew:TESTPOINT
- removed U101, U33: (no value), jonnew:JP3E
- removed U102: SCREW4, jonnew:SCREW4
- added C19, C21, C24, C26, C27, C28, C31, C32: 0.1uF, jonnew:C_0402
- added C20, C22, C23, C25, C29, C30, C33, C34: 1uF, jonnew:C_0603
- added D3, D4: (no value), jonnew:LED_0603
- added J1, J2, J3, J4, J5: (no value), jonnew:JP3E_SMD
- added J6: (no value), jonnew:SCREW4
- added Q1: DMN3404L, jonnew:N-MOSFET_SOT23-GSD
- added Q2: DMP3056L, jonnew:P-MOSFET_SOT23-GSD
- added R5, R6: 1k, jonnew:R_0603
- C1, C13, C2: value 0.1uF -> 1uF; device jonnew:C_0402 -> jonnew:C_0603
- C11: value 10uF -> 0.1uF; device jonnew:C-POL_1210 -> jonnew:C_0402
- C12: value 10uF -> 1uF; device jonnew:C-POL_1210 -> jonnew:C_0603
- C16, C9: value 1uF -> 0.1uF; device jonnew:C_0603 -> jonnew:C_0402
- C17, C18: value 1uF -> 10uF; device jonnew:C_0603 -> jonnew:C-POL_1210
- D1, D2: value (none) -> UDZ10B-7; device jonnew:LED_0603 -> jonnew:Z-DIODE_SOD-323; PARTNO (none) -> UDZ10B-7
- R1, R2: value 10k -> 1k
- R3, R4: value 1k -> 10k
- S1: value (none) -> 219-2MSTR
- renumbered $1_8_$ to J8, $1_8_$1 to J7
Connections:
- new net GND1: U13.GND
- new net GND2: U23.GND
- new net GND4: U31.GND
- new net GND_HEAD: J3.3, J7G$1.17
- new net GPIO0_HEAD: J1.1, J7G$2.3
- new net GPIO1_HEAD: J2.1, J7G$2.4
- new net GPIO2_HEAD: J8G$2.3
- new net GPIO3_HEAD: J8G$2.4
- new net N$450: D1.A, Q2.G, R1.2
- new net N$452: U13.!EN
- new net N$453: U23.!EN
- new net N$454: D2.C, Q1.G, R2.1
- new net N$456: U31.!EN
- new net N$457: J1.3, S1.4
- new net N$460: J2.3, S1.3
- new net VCC_LOCAL: J5.1, J6.1
- new net VSS_LOCAL: J4.1, J6.2
- net A: now also J1.2, R3.1, U10.A, U11.A, U12.A, U13.A, U14.A, U15.A, U16.A, U17.A, U18.A, U19.A, U20.A, U21.A, U22.A, U23.A, U24.A, U25.A, U26.A, U27.A, U28.A, U29.A, U30.A, U31.A, U9.A; no longer R2.1, S1.4
- net B: now also J2.2, R4.1, U10.B, U11.B, U12.B, U13.B, U14.B, U15.B, U16.B, U17.B, U18.B, U19.B, U20.B, U21.B, U22.B, U23.B, U24.B, U25.B, U26.B, U27.B, U28.B, U29.B, U30.B, U31.B, U9.B; no longer R1.1, S1.3
- net GND: now also C11.2, C12.2, C17.-, C18.+, C19.2, C20.2, C21.2, C22.2, C23.2, C24.2, C25.2, C26.2, C27.2, C28.2, C29.2, C30.2, C31.2, C32.2, C33.2, C34.2, D3.C, D4.A, J3.1, J3.2, J6.3, R1.1, R2.2, U10.!EN, U10.GND, U11.!EN, U11.GND, U12.!EN, U12.GND, U14.!EN, U14.GND, U15.!EN, U15.GND, U16.!EN, U16.GND, U17.!EN, U17.GND, U18.!EN, U18.GND, U19.!EN, U19.GND, U20.!EN, U20.GND, U21.!EN, U21.GND, U22.!EN, U22.GND, U24.!EN, U24.GND, U25.!EN, U25.GND, U26.GND, U27.!EN, U27.GND, U28.!EN, U28.GND, U29.!EN, U29.GND, U30.GND, U9.!EN, U9.GND; no longer C11.-, C12.+, C17.2, C18.2, D1.C, R4.2, TP4.1, U102.3
- net N$100: now also U8.X3; no longer U5.X3
- net N$101: now also U7.Y1; no longer U6.Y1
- net N$102: now also U7.Y3; no longer U6.Y3
- net N$103: now also U7.Y2; no longer U6.Y2
- net N$104: now also U7.Y0; no longer U6.Y0
- net N$110: now also U7.X2; no longer U6.X2
- net N$118: now also U8.Y1; no longer U5.Y1
- net N$119: now also U8.Y3; no longer U5.Y3
- net N$120: now also U8.Y2; no longer U5.Y2
- net N$121: now also U8.Y0; no longer U5.Y0
- net N$122: now also U7.X1; no longer U6.X1
- net N$123: now also U7.X0; no longer U6.X0
- net N$124: now also U7.X3; no longer U6.X3
- net N$125: now also U6.Y1; no longer U7.Y1
- net N$126: now also U6.Y3; no longer U7.Y3
- net N$127: now also U6.Y2; no longer U7.Y2
- net N$128: now also U6.Y0; no longer U7.Y0
- net N$129: now also U6.X2; no longer U7.X2
- net N$130: now also U6.X1; no longer U7.X1
- net N$131: now also U6.X0; no longer U7.X0
- net N$132: now also U6.X3; no longer U7.X3
- net N$133: now also U5.Y1; no longer U8.Y1
- net N$134: now also U5.Y3; no longer U8.Y3
- net N$135: now also U5.Y2; no longer U8.Y2
- net N$136: now also U5.Y0; no longer U8.Y0
- net N$137: now also U5.X2; no longer U8.X2
- net N$138: now also U5.X1; no longer U8.X1
- net N$139: now also U5.X0; no longer U8.X0
- net N$140: now also U5.X3; no longer U8.X3
- net N$449: now also D3.A, R5.1; no longer D1.A, R3.1
- net N$451: now also D4.C, R6.2; no longer D2.A, R4.1
- net N$97: now also U8.X2; no longer U5.X2
- net N$98: now also U8.X1; no longer U5.X1
- net N$99: now also U8.X0; no longer U5.X0
- net REF: now also J6.4; no longer TP3.1, U102.4
- net TT00: now also U24.X; no longer U25.X
- net TT01: now also U24.Y; no longer U25.Y
- net TT02: now also U23.X; no longer U26.X
- net TT03: now also U23.Y; no longer U26.Y
- net TT04: now also U21.X; no longer U27.X
- net TT05: now also U21.Y; no longer U27.Y
- net TT06: now also U19.X; no longer U28.X
- net TT07: now also U19.Y; no longer U28.Y
- net TT08: now also U11.X; no longer U29.X
- net TT09: now also U11.Y; no longer U29.Y
- net TT10: now also U13.X; no longer U30.X
- net TT11: now also U13.Y; no longer U30.Y
- net TT12: now also U15.X; no longer U31.X
- net TT13: now also U15.Y; no longer U31.Y
- net TT14: now also U17.X; no longer U32.X
- net TT15: now also U17.Y; no longer U32.Y
- net TT24: now also U8.X; no longer U5.X
- net TT25: now also U8.Y; no longer U5.Y
- net TT26: now also U7.X; no longer U6.X
- net TT27: now also U7.Y; no longer U6.Y
- net TT28: now also U6.X; no longer U7.X
- net TT29: now also U6.Y; no longer U7.Y
- net TT30: now also U5.X; no longer U8.X
- net TT31: now also U5.Y; no longer U8.Y
- net TT36: now also U12.X; no longer U11.X
- net TT37: now also U12.Y; no longer U11.Y
- net TT38: now also U14.X; no longer U12.X
- net TT39: now also U14.Y; no longer U12.Y
- net TT40: now also U22.X; no longer U13.X
- net TT41: now also U22.Y; no longer U13.Y
- net TT42: now also U20.X; no longer U14.X
- net TT43: now also U20.Y; no longer U14.Y
- net TT44: now also U18.X; no longer U15.X
- net TT45: now also U18.Y; no longer U15.Y
- net TT48: now also U32.X; no longer U17.X
- net TT49: now also U32.Y; no longer U17.Y
- net TT50: now also U31.X; no longer U18.X
- net TT51: now also U31.Y; no longer U18.Y
- net TT52: now also U30.X; no longer U19.X
- net TT53: now also U30.Y; no longer U19.Y
- net TT54: now also U29.X; no longer U20.X
- net TT55: now also U29.Y; no longer U20.Y
- net TT56: now also U25.X; no longer U21.X
- net TT57: now also U25.Y; no longer U21.Y
- net TT58: now also U26.X; no longer U22.X
- net TT59: now also U26.Y; no longer U22.Y
- net TT60: now also U27.X; no longer U23.X
- net TT61: now also U27.Y; no longer U23.Y
- net TT62: now also U28.X; no longer U24.X
- net TT63: now also U28.Y; no longer U24.Y
- net VCC: now also C10.1, C16.1, C17.+, C19.1, C2.1, C20.1, C25.1, C26.1, C31.1, C32.1, C33.1, C34.1, C4.1, D1.C, Q2.S, R4.2, R5.2, U10.V+, U11.V+, U12.V+, U13.V+, U14.V+, U15.V+, U16.V+, U17.V+, U18.V+, U19.V+, U20.V+, U21.V+, U22.V+, U23.V+, U24.V+, U25.V+, U27.V+, U28.V+, U29.V+, U30.V+, U31.V+, U9.V+; no longer C11.+, C13.1, C17.1, C5.1, C7.1, R1.2, R2.2, U102.1
- net VCC_HEAD: now also J5.3, J7G$1.19; no longer U101.1
- net VCC_PRE: now also J5.2, Q2.D; no longer TP1.1, U101.2, U101.3
- net VSS: now also C11.1, C12.1, C13.1, C18.-, C21.1, C22.1, C23.1, C24.1, C27.1, C28.1, C29.1, C30.1, C5.1, C7.1, D2.A, Q1.S, R6.1, U10.V-, U11.V-, U12.V-, U13.V-, U14.V-, U15.V-, U16.V-, U17.V-, U18.V-, U19.V-, U20.V-, U21.V-, U22.V-, U23.V-, U24.V-, U25.V-, U27.V-, U28.V-, U29.V-, U31.V-, U9.V-; no longer C10.1, C12.-, C16.1, C18.1, C2.1, C4.1, D2.C, U102.2
- net VSS_HEAD: now also J4.3, J7G$1.18; no longer U33.1
- net VSS_PRE: now also J4.2, Q1.D; no longer TP2.1, U33.2, U33.3
Other:
- moved on the sheet: C1, C10, C11, C12, C13, C14, C15, C16, C17, C18, C2, C3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
