File: eib-128/eib-128_panel.brd (EAGLE design)
At the start: 130 x 130 mm, 477 parts

Commit message: Updated eib-128 to match next-gen drive form factor.
Parts:
- removed AGND_A0, AGND_A1, AGND_A10, AGND_A11, AGND_A12, AGND_A13, AGND_A14, AGND_A15, AGND_A16, AGND_A17, AGND_A2, AGND_A3, AGND_A4, AGND_A5, AGND_A6, AGND_A7, AGND_A8, AGND_A9, AGND_B0, AGND_B1, AGND_B10, AGND_B11, AGND_B12, AGND_B13, AGND_B14, AGND_B15, AGND_B16, AGND_B17, AGND_B2, AGND_B3, AGND_B4, AGND_B5, AGND_B6, AGND_B7, AGND_B8, AGND_B9, REF_A12, REF_A13, REF_A14, REF_A15, REF_A16, REF_A17, REF_B12, REF_B13, REF_B14, REF_B15, REF_B16, REF_B17, SHLD_A0, SHLD_A12, SHLD_A13, SHLD_A14, SHLD_A15, SHLD_A16, SHLD_A17, SHLD_B0, SHLD_B12, SHLD_B13, SHLD_B14, SHLD_B15, SHLD_B16, SHLD_B17: LRG_GP, jonnew:GOLDPIN_0.5ID_0.7OD
- removed AIN_N0T, AIN_N0T1, AIN_N0T2, AIN_N0T3, AIN_N0T4, AIN_N0T5, AIN_N0T6, AIN_N0T7, AIN_N0T8, AIN_S0T, AIN_S0T1, AIN_S0T2, AIN_S0T3, AIN_S0T4, AIN_S0T5, AIN_S0T6, AIN_S0T7, AIN_S0T8: DF40HEAD, jonnew:DF40-70HEAD-EIB
- removed MECH_E0T, MECH_E0T1, MECH_E0T2, MECH_E0T3, MECH_E0T4, MECH_E0T5, MECH_E0T6, MECH_E0T7, MECH_E0T8, MECH_W0T, MECH_W0T1, MECH_W0T2, MECH_W0T3, MECH_W0T4, MECH_W0T5, MECH_W0T6, MECH_W0T7, MECH_W0T8: DF40HEAD, jonnew:DF40-70HEAD
- removed SJ_A0, SJ_A1, SJ_A10, SJ_A11, SJ_A12, SJ_A13, SJ_A14, SJ_A15, SJ_A16, SJ_A17, SJ_A2, SJ_A3, SJ_A4, SJ_A5, SJ_A6, SJ_A7, SJ_A8, SJ_A9, SJ_B0, SJ_B1, SJ_B10, SJ_B11, SJ_B12, SJ_B13, SJ_B14, SJ_B15, SJ_B16, SJ_B17, SJ_B2, SJ_B3, SJ_B4, SJ_B5, SJ_B6, SJ_B7, SJ_B8, SJ_B9: (no value), jonnew:SJ_2_0402
- added A, A1, A10, A11, A2, A3, A4, A5, A6, A7, A8, A9, B, B1, B10, B11, B2, B3, B4, B5, B6, B7, B8, B9: DF40HEAD, jonnew:DF40-70HEAD
- added AN_A, AN_A1, AN_A10, AN_A11, AN_A2, AN_A3, AN_A4, AN_A5, AN_A6, AN_A7, AN_A8, AN_A9, AN_B, AN_B1, AN_B10, AN_B11, AN_B2, AN_B3, AN_B4, AN_B5, AN_B6, AN_B7, AN_B8, AN_B9, CAT0_A, CAT0_A1, CAT0_A10, CAT0_A11, CAT0_A2, CAT0_A3, CAT0_A4, CAT0_A5, CAT0_A6, CAT0_A7, CAT0_A8, CAT0_A9, CAT0_B, CAT0_B1, CAT0_B10, CAT0_B11, CAT0_B2, CAT0_B3, CAT0_B4, CAT0_B5, CAT0_B6, CAT0_B7, CAT0_B8, CAT0_B9, CAT1_A, CAT1_A1, CAT1_A10, CAT1_A11, CAT1_A2, CAT1_A3, CAT1_A4, CAT1_A5, CAT1_A6, CAT1_A7, CAT1_A8, CAT1_A9, CAT1_B, CAT1_B1, CAT1_B10, CAT1_B11, CAT1_B2, CAT1_B3, CAT1_B4, CAT1_B5, CAT1_B6, CAT1_B7, CAT1_B8, CAT1_B9, ESTIM_A, ESTIM_A1, ESTIM_A10, ESTIM_A11, ESTIM_A2, ESTIM_A3, ESTIM_A4, ESTIM_A5, ESTIM_A6, ESTIM_A7, ESTIM_A8, ESTIM_A9, ESTIM_B, ESTIM_B1, ESTIM_B10, ESTIM_B11, ESTIM_B2, ESTIM_B3, ESTIM_B4, ESTIM_B5, ESTIM_B6, ESTIM_B7, ESTIM_B8, ESTIM_B9, GND0, GND1, GND10, GND11, GND12, GND13, GND14, GND15, GND16, GND17, GND18, GND19, GND2, GND20, GND21, GND22, GND23, GND24, GND25, GND26, GND27, GND28, GND29, GND3, GND30, GND31, GND32, GND33, GND34, GND35, GND36, GND37, GND38, GND39, GND4, GND40, GND41, GND42, GND43, GND44, GND45, GND46, GND47, GND5, GND6, GND7, GND8, GND9, SHLD_A, SHLD_B: LRG_GP, jonnew:GOLDPIN_0.5ID_0.7OD
- added TET288, TET320, TET352: 0, jonnew:TETRODE_128_0.5ID_0.7OD
- added TET289, TET321, TET353: 1, jonnew:TETRODE_128_0.5ID_0.7OD
- added TET290, TET322, TET354: 2, jonnew:TETRODE_128_0.5ID_0.7OD
- added TET291, TET323, TET355: 3, jonnew:TETRODE_128_0.5ID_0.7OD
- added TET292, TET324, TET356: 4, jonnew:TETRODE_128_0.5ID_0.7OD
- added TET293, TET325, TET357: 5, jonnew:TETRODE_128_0.5ID_0.7OD
- added TET294, TET326, TET358: 6, jonnew:TETRODE_128_0.5ID_0.7OD
- added TET295, TET327, TET359: 7, jonnew:TETRODE_128_0.5ID_0.7OD
- added TET296, TET328, TET360: 8, jonnew:TETRODE_128_0.5ID_0.7OD
- added TET297, TET329, TET361: 9, jonnew:TETRODE_128_0.5ID_0.7OD
- added TET298, TET330, TET362: 10, jonnew:TETRODE_128_0.5ID_0.7OD
- added TET299, TET331, TET363: 11, jonnew:TETRODE_128_0.5ID_0.7OD
- added TET300, TET332, TET364: 12, jonnew:TETRODE_128_0.5ID_0.7OD
- added TET301, TET333, TET365: 13, jonnew:TETRODE_128_0.5ID_0.7OD
- added TET302, TET334, TET366: 14, jonnew:TETRODE_128_0.5ID_0.7OD
- added TET303, TET335, TET367: 15, jonnew:TETRODE_128_0.5ID_0.7OD
- added TET304, TET336, TET368: 16, jonnew:TETRODE_128_0.5ID_0.7OD
- added TET305, TET337, TET369: 17, jonnew:TETRODE_128_0.5ID_0.7OD
- added TET306, TET338, TET370: 18, jonnew:TETRODE_128_0.5ID_0.7OD
- added TET307, TET339, TET371: 19, jonnew:TETRODE_128_0.5ID_0.7OD
- added TET308, TET340, TET372: 20, jonnew:TETRODE_128_0.5ID_0.7OD
- added TET309, TET341, TET373: 21, jonnew:TETRODE_128_0.5ID_0.7OD
- added TET310, TET342, TET374: 22, jonnew:TETRODE_128_0.5ID_0.7OD
- added TET311, TET343, TET375: 23, jonnew:TETRODE_128_0.5ID_0.7OD
- added TET312, TET344, TET376: 24, jonnew:TETRODE_128_0.5ID_0.7OD
- added TET313, TET345, TET377: 25, jonnew:TETRODE_128_0.5ID_0.7OD
- added TET314, TET346, TET378: 26, jonnew:TETRODE_128_0.5ID_0.7OD
- added TET315, TET347, TET379: 27, jonnew:TETRODE_128_0.5ID_0.7OD
- added TET316, TET348, TET380: 28, jonnew:TETRODE_128_0.5ID_0.7OD
- added TET317, TET349, TET381: 29, jonnew:TETRODE_128_0.5ID_0.7OD
- added TET318, TET350, TET382: 30, jonnew:TETRODE_128_0.5ID_0.7OD
- added TET319, TET351, TET383: 31, jonnew:TETRODE_128_0.5ID_0.7OD
- added U$10, U$11, U$12: (no value), jonnew:EIB_MOUNT_A
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Connections:
- removed net AGND_A0: AGND_A0.P$1, AIN_N0T.69, AIN_N0T.70, SJ_A0.2
- removed net AGND_A1: AGND_A1.P$1, AIN_N0T.34, AIN_N0T.35, SJ_A1.2
- removed net AGND_A10: AGND_A11.P$1, AIN_N0T5.69, AIN_N0T5.70, SJ_A10.2
- removed net AGND_A11: AGND_A10.P$1, AIN_N0T5.34, AIN_N0T5.35, SJ_A11.2
- removed net AGND_A12: AGND_A13.P$1, AIN_N0T6.69, AIN_N0T6.70, SJ_A12.2
- removed net AGND_A13: AGND_A12.P$1, AIN_N0T6.34, AIN_N0T6.35, SJ_A13.2
- removed net AGND_A14: AGND_A15.P$1, AIN_N0T7.69, AIN_N0T7.70, SJ_A14.2
- removed net AGND_A15: AGND_A14.P$1, AIN_N0T7.34, AIN_N0T7.35, SJ_A15.2
- removed net AGND_A16: AGND_A17.P$1, AIN_N0T8.69, AIN_N0T8.70, SJ_A16.2
- removed net AGND_A17: AGND_A16.P$1, AIN_N0T8.34, AIN_N0T8.35, SJ_A17.2
- removed net AGND_A2: AGND_A3.P$1, AIN_N0T1.69, AIN_N0T1.70, SJ_A2.2
- removed net AGND_A3: AGND_A2.P$1, AIN_N0T1.34, AIN_N0T1.35, SJ_A3.2
- removed net AGND_A4: AGND_A5.P$1, AIN_N0T2.69, AIN_N0T2.70, SJ_A4.2
- removed net AGND_A5: AGND_A4.P$1, AIN_N0T2.34, AIN_N0T2.35, SJ_A5.2
- removed net AGND_A6: AGND_A7.P$1, AIN_N0T3.69, AIN_N0T3.70, SJ_A6.2
- removed net AGND_A7: AGND_A6.P$1, AIN_N0T3.34, AIN_N0T3.35, SJ_A7.2
- removed net AGND_A8: AGND_A9.P$1, AIN_N0T4.69, AIN_N0T4.70, SJ_A8.2
- removed net AGND_A9: AGND_A8.P$1, AIN_N0T4.34, AIN_N0T4.35, SJ_A9.2
- removed net AGND_B0: AGND_B0.P$1, AIN_S0T.69, AIN_S0T.70, SJ_B0.2
- removed net AGND_B1: AGND_B1.P$1, AIN_S0T.34, AIN_S0T.35, SJ_B1.2
- removed net AGND_B10: AGND_B11.P$1, AIN_S0T5.34, AIN_S0T5.35, SJ_B11.2
- removed net AGND_B11: AGND_B10.P$1, AIN_S0T5.69, AIN_S0T5.70, SJ_B10.2
- removed net AGND_B12: AGND_B13.P$1, AIN_S0T6.34, AIN_S0T6.35, SJ_B13.2
- removed net AGND_B13: AGND_B12.P$1, AIN_S0T6.69, AIN_S0T6.70, SJ_B12.2
- removed net AGND_B14: AGND_B15.P$1, AIN_S0T7.34, AIN_S0T7.35, SJ_B15.2
- removed net AGND_B15: AGND_B14.P$1, AIN_S0T7.69, AIN_S0T7.70, SJ_B14.2
- removed net AGND_B16: AGND_B17.P$1, AIN_S0T8.34, AIN_S0T8.35, SJ_B17.2
- removed net AGND_B17: AGND_B16.P$1, AIN_S0T8.69, AIN_S0T8.70, SJ_B16.2
- removed net AGND_B2: AGND_B3.P$1, AIN_S0T1.34, AIN_S0T1.35, SJ_B3.2
- removed net AGND_B3: AGND_B2.P$1, AIN_S0T1.69, AIN_S0T1.70, SJ_B2.2
- removed net AGND_B4: AGND_B5.P$1, AIN_S0T2.34, AIN_S0T2.35, SJ_B5.2
- removed net AGND_B5: AGND_B4.P$1, AIN_S0T2.69, AIN_S0T2.70, SJ_B4.2
- removed net AGND_B6: AGND_B7.P$1, AIN_S0T3.34, AIN_S0T3.35, SJ_B7.2
- removed net AGND_B7: AGND_B6.P$1, AIN_S0T3.69, AIN_S0T3.70, SJ_B6.2
- removed net AGND_B8: AGND_B9.P$1, AIN_S0T4.34, AIN_S0T4.35, SJ_B9.2
- removed net AGND_B9: AGND_B8.P$1, AIN_S0T4.69, AIN_S0T4.70, SJ_B8.2
- removed net GND1: SJ_A2.1, SJ_A3.1, SJ_B2.1, SJ_B3.1
- removed net GND2: SJ_A4.1, SJ_A5.1, SJ_B4.1, SJ_B5.1
- removed net GND3: SJ_A6.1, SJ_A7.1, SJ_B6.1, SJ_B7.1
- removed net GND4: SJ_A8.1, SJ_A9.1, SJ_B8.1, SJ_B9.1
- removed net GND5: SJ_A10.1, SJ_A11.1, SJ_B10.1, SJ_B11.1
- removed net GND6: SJ_A12.1, SJ_A13.1, SJ_B12.1, SJ_B13.1
- removed net GND7: SJ_A14.1, SJ_A15.1, SJ_B14.1, SJ_B15.1
- removed net GND8: SJ_A16.1, SJ_A17.1, SJ_B16.1, SJ_B17.1
- removed net REF_A0: AIN_N0T.1, REF_A0.P$1
- removed net REF_A12: AIN_N0T6.1, REF_A12.P$1
- removed net REF_A13: AIN_N0T6.36, REF_A13.P$1
- removed net REF_A14: AIN_N0T7.1, REF_A14.P$1
- removed net REF_A15: AIN_N0T7.36, REF_A15.P$1
- removed net REF_A16: AIN_N0T8.1, REF_A16.P$1
- removed net REF_A17: AIN_N0T8.36, REF_A17.P$1
- removed net REF_B0: AIN_S0T.1, REF_B0.P$1
- removed net REF_B12: AIN_S0T6.36, REF_B12.P$1
- removed net REF_B13: AIN_S0T6.1, REF_B13.P$1
- removed net REF_B14: AIN_S0T7.36, REF_B14.P$1
- removed net REF_B15: AIN_S0T7.1, REF_B15.P$1
- removed net REF_B16: AIN_S0T8.36, REF_B16.P$1
- removed net REF_B17: AIN_S0T8.1, REF_B17.P$1
- new net AN_A: A.36, AN_A.P$1
- new net AN_A1: A1.36, AN_A1.P$1
- new net AN_A10: A10.36, AN_A10.P$1
- new net AN_A11: A11.36, AN_A11.P$1
- new net AN_A2: A2.36, AN_A2.P$1
- new net AN_A3: A3.36, AN_A3.P$1
- new net AN_A4: A4.36, AN_A4.P$1
- new net AN_A5: A5.36, AN_A5.P$1
- new net AN_A6: A6.36, AN_A6.P$1
- new net AN_A7: A7.36, AN_A7.P$1
- new net AN_A8: A8.36, AN_A8.P$1
- new net AN_A9: A9.36, AN_A9.P$1
- new net AN_B: AN_B.P$1, B.36
- new net AN_B1: AN_B1.P$1, B1.36
- new net AN_B10: AN_B10.P$1, B10.36
- new net AN_B11: AN_B11.P$1, B11.36
- new net AN_B2: AN_B2.P$1, B2.36
- new net AN_B3: AN_B3.P$1, B3.36
- new net AN_B4: AN_B4.P$1, B4.36
- new net AN_B5: AN_B5.P$1, B5.36
- new net AN_B6: AN_B6.P$1, B6.36
- new net AN_B7: AN_B7.P$1, B7.36
- new net AN_B8: AN_B8.P$1, B8.36
- new net AN_B9: AN_B9.P$1, B9.36
- new net CAT0_A: A.34, CAT0_A.P$1
- new net CAT0_A1: A1.34, CAT0_A1.P$1
- new net CAT0_A10: A10.34, CAT0_A10.P$1
- new net CAT0_A11: A11.34, CAT0_A11.P$1
- new net CAT0_A2: A2.34, CAT0_A2.P$1
- new net CAT0_A3: A3.34, CAT0_A3.P$1
- new net CAT0_A4: A4.34, CAT0_A4.P$1
- new net CAT0_A5: A5.34, CAT0_A5.P$1
- new net CAT0_A6: A6.34, CAT0_A6.P$1
- new net CAT0_A7: A7.34, CAT0_A7.P$1
- new net CAT0_A8: A8.34, CAT0_A8.P$1
- new net CAT0_A9: A9.34, CAT0_A9.P$1
- new net CAT0_B: B.34, CAT0_B.P$1
- new net CAT0_B1: B1.34, CAT0_B1.P$1
- new net CAT0_B10: B10.34, CAT0_B10.P$1
- new net CAT0_B11: B11.34, CAT0_B11.P$1
- new net CAT0_B2: B2.34, CAT0_B2.P$1
- new net CAT0_B3: B3.34, CAT0_B3.P$1
- new net CAT0_B4: B4.34, CAT0_B4.P$1
- new net CAT0_B5: B5.34, CAT0_B5.P$1
- new net CAT0_B6: B6.34, CAT0_B6.P$1
- new net CAT0_B7: B7.34, CAT0_B7.P$1
- new net CAT0_B8: B8.34, CAT0_B8.P$1
- new net CAT0_B9: B9.34, CAT0_B9.P$1
- new net CAT1_A: A.35, CAT1_A.P$1
- new net CAT1_A1: A1.35, CAT1_A1.P$1
- new net CAT1_A10: A10.35, CAT1_A10.P$1
- new net CAT1_A11: A11.35, CAT1_A11.P$1
- new net CAT1_A2: A2.35, CAT1_A2.P$1
- new net CAT1_A3: A3.35, CAT1_A3.P$1
- new net CAT1_A4: A4.35, CAT1_A4.P$1
- new net CAT1_A5: A5.35, CAT1_A5.P$1
- new net CAT1_A6: A6.35, CAT1_A6.P$1
- new net CAT1_A7: A7.35, CAT1_A7.P$1
- new net CAT1_A8: A8.35, CAT1_A8.P$1
- new net CAT1_A9: A9.35, CAT1_A9.P$1
- new net CAT1_B: B.35, CAT1_B.P$1
- new net CAT1_B1: B1.35, CAT1_B1.P$1
- new net CAT1_B10: B10.35, CAT1_B10.P$1
- new net CAT1_B11: B11.35, CAT1_B11.P$1
- new net CAT1_B2: B2.35, CAT1_B2.P$1
- new net CAT1_B3: B3.35, CAT1_B3.P$1
- new net CAT1_B4: B4.35, CAT1_B4.P$1
- new net CAT1_B5: B5.35, CAT1_B5.P$1
- new net CAT1_B6: B6.35, CAT1_B6.P$1
- new net CAT1_B7: B7.35, CAT1_B7.P$1
- new net CAT1_B8: B8.35, CAT1_B8.P$1
- new net CAT1_B9: B9.35, CAT1_B9.P$1
- new net ESTIM_A: A.69, ESTIM_A.P$1
- new net ESTIM_A1: A1.69, ESTIM_A1.P$1
- new net ESTIM_A10: A10.69, ESTIM_A10.P$1
- new net ESTIM_A11: A11.69, ESTIM_A11.P$1
- new net ESTIM_A2: A2.69, ESTIM_A2.P$1
- new net ESTIM_A3: A3.69, ESTIM_A3.P$1
- new net ESTIM_A4: A4.69, ESTIM_A4.P$1
- new net ESTIM_A5: A5.69, ESTIM_A5.P$1
- new net ESTIM_A6: A6.69, ESTIM_A6.P$1
- new net ESTIM_A7: A7.69, ESTIM_A7.P$1
- new net ESTIM_A8: A8.69, ESTIM_A8.P$1
- new net ESTIM_A9: A9.69, ESTIM_A9.P$1
- new net ESTIM_B: B.69, ESTIM_B.P$1
- new net ESTIM_B1: B1.69, ESTIM_B1.P$1
- new net ESTIM_B10: B10.69, ESTIM_B10.P$1
- new net ESTIM_B11: B11.69, ESTIM_B11.P$1
- new net ESTIM_B2: B2.69, ESTIM_B2.P$1
- new net ESTIM_B3: B3.69, ESTIM_B3.P$1
- new net ESTIM_B4: B4.69, ESTIM_B4.P$1
- new net ESTIM_B5: B5.69, ESTIM_B5.P$1
- new net ESTIM_B6: B6.69, ESTIM_B6.P$1
- new net ESTIM_B7: B7.69, ESTIM_B7.P$1
- new net ESTIM_B8: B8.69, ESTIM_B8.P$1
- new net ESTIM_B9: B9.69, ESTIM_B9.P$1
- new net N$1189: A9.43, TET297.2
- new net N$1190: A9.44, TET297.3
- new net N$1191: A9.45, TET298.0
- new net N$1192: A9.46, TET298.1
- new net N$1193: A9.47, TET298.2
- new net N$1194: A9.48, TET298.3
- new net N$1195: A9.49, TET299.0
- new net N$1196: A9.50, TET299.1
- new net N$1197: A9.51, TET299.2
- new net N$1198: A9.52, TET299.3
- new net N$1199: A9.53, TET300.0
- new net N$1200: A9.54, TET300.1
- new net N$1201: A9.55, TET300.2
- new net N$1202: A9.56, TET300.3
- new net N$1203: A9.57, TET301.0
- new net N$1204: A9.58, TET301.1
- new net N$1205: A9.59, TET301.2
- new net N$1206: A9.60, TET301.3
- new net N$1207: A9.61, TET302.0
- new net N$1208: A9.62, TET302.1
- new net N$1209: A9.63, TET302.2
- new net N$1210: A9.64, TET302.3
- new net N$1211: A9.65, TET303.0
- new net N$1212: A9.66, TET303.1
- new net N$1213: A9.67, TET303.2
- new net N$1214: A9.68, TET303.3
- new net N$1215: A9.2, TET288.0
- new net N$1216: A9.37, TET296.0
- new net N$1217: B9.33, TET311.0
- new net N$1218: B9.32, TET311.1
- new net N$1219: B9.31, TET311.2
- new net N$1220: B9.30, TET311.3
- new net N$1221: B9.29, TET310.0
- new net N$1222: B9.28, TET310.1
- new net N$1223: B9.27, TET310.2
- new net N$1224: B9.26, TET310.3
- new net N$1225: B9.25, TET309.0
- new net N$1226: B9.24, TET309.1
- new net N$1227: B9.23, TET309.2
- new net N$1228: B9.22, TET309.3
- new net N$1229: B9.21, TET308.0
- new net N$1230: B9.20, TET308.1
- new net N$1231: B9.19, TET308.2
- new net N$1232: B9.18, TET308.3
- new net N$1233: B9.17, TET307.0
- new net N$1234: B9.16, TET307.1
- new net N$1235: B9.15, TET307.2
- new net N$1236: B9.14, TET307.3
- new net N$1237: B9.13, TET306.0
- new net N$1238: B9.12, TET306.1
- new net N$1239: B9.11, TET306.2
- new net N$1240: B9.10, TET306.3
- new net N$1241: B9.9, TET305.0
- new net N$1242: B9.8, TET305.1
- new net N$1243: B9.7, TET305.2
- new net N$1244: B9.6, TET305.3
- new net N$1245: B9.5, TET304.0
- new net N$1246: B9.4, TET304.1
- new net N$1247: B9.3, TET304.2
- new net N$1248: B9.38, TET312.2
- new net N$1249: B9.39, TET312.1
- new net N$1250: B9.40, TET312.0
- new net N$1251: B9.41, TET313.3
- new net N$1252: B9.42, TET313.2
- new net N$1253: B9.43, TET313.1
- new net N$1254: B9.44, TET313.0
- new net N$1255: B9.45, TET314.3
- new net N$1256: B9.46, TET314.2
- new net N$1257: B9.47, TET314.1
- new net N$1258: B9.48, TET314.0
- new net N$1259: B9.49, TET315.3
- new net N$1260: B9.50, TET315.2
- new net N$1261: B9.51, TET315.1
- new net N$1262: B9.52, TET315.0
- new net N$1263: B9.53, TET316.3
- new net N$1264: B9.54, TET316.2
- new net N$1265: B9.55, TET316.1
- new net N$1266: B9.56, TET316.0
- new net N$1267: B9.57, TET317.3
- new net N$1268: B9.58, TET317.2
- new net N$1269: B9.59, TET317.1
- new net N$1270: B9.60, TET317.0
- new net N$1271: B9.61, TET318.3
- new net N$1272: B9.62, TET318.2
- new net N$1273: B9.63, TET318.1
- new net N$1274: B9.64, TET318.0
- new net N$1275: B9.65, TET319.3
- new net N$1276: B9.66, TET319.2
- new net N$1277: B9.67, TET319.1
- new net N$1278: B9.68, TET319.0
- new net N$1279: B9.2, TET304.3
- new net N$1280: B9.37, TET312.3
- new net N$1281: A10.33, TET327.3
- new net N$1282: A10.32, TET327.2
- new net N$1283: A10.31, TET327.1
- new net N$1284: A10.30, TET327.0
- new net N$1285: A10.29, TET326.3
- new net N$1286: A10.28, TET326.2
- new net N$1287: A10.27, TET326.1
- new net N$1288: A10.26, TET326.0
- new net N$1289: A10.25, TET325.3
- new net N$1290: A10.24, TET325.2
- new net N$1291: A10.23, TET325.1
- new net N$1292: A10.22, TET325.0
- new net N$1293: A10.21, TET324.3
- new net N$1294: A10.20, TET324.2
- new net N$1295: A10.19, TET324.1
- new net N$1296: A10.18, TET324.0
- new net N$1297: A10.17, TET323.3
- new net N$1298: A10.16, TET323.2
- new net N$1299: A10.15, TET323.1
- new net N$1300: A10.14, TET323.0
- new net N$1301: A10.13, TET322.3
- new net N$1302: A10.12, TET322.2
- new net N$1303: A10.11, TET322.1
- new net N$1304: A10.10, TET322.0
- new net N$1305: A10.9, TET321.3
- new net N$1306: A10.8, TET321.2
- new net N$1307: A10.7, TET321.1
- new net N$1308: A10.6, TET321.0
- new net N$1309: A10.5, TET320.3
- new net N$1310: A10.4, TET320.2
- new net N$1311: A10.3, TET320.1
- new net N$1312: A10.38, TET328.1
- new net N$1313: A10.39, TET328.2
- new net N$1314: A10.40, TET328.3
- new net N$1315: A10.41, TET329.0
- new net N$1316: A10.42, TET329.1
- new net N$1317: A10.43, TET329.2
- new net N$1318: A10.44, TET329.3
- new net N$1319: A10.45, TET330.0
- new net N$1320: A10.46, TET330.1
- new net N$1321: A10.47, TET330.2
- new net N$1322: A10.48, TET330.3
- new net N$1323: A10.49, TET331.0
- new net N$1324: A10.50, TET331.1
- new net N$1325: A10.51, TET331.2
- new net N$1326: A10.52, TET331.3
- new net N$1327: A10.53, TET332.0
- new net N$1328: A10.54, TET332.1
- new net N$1329: A10.55, TET332.2
- new net N$1330: A10.56, TET332.3
- new net N$1331: A10.57, TET333.0
- new net N$1332: A10.58, TET333.1
- new net N$1333: A10.59, TET333.2
- new net N$1334: A10.60, TET333.3
- new net N$1335: A10.61, TET334.0
- new net N$1336: A10.62, TET334.1
- new net N$1337: A10.63, TET334.2
- new net N$1338: A10.64, TET334.3
- new net N$1339: A10.65, TET335.0
- new net N$1340: A10.66, TET335.1
- new net N$1341: A10.67, TET335.2
- new net N$1342: A10.68, TET335.3
- new net N$1343: A10.2, TET320.0
- new net N$1344: A10.37, TET328.0
- new net N$1345: B10.33, TET343.0
- new net N$1346: B10.32, TET343.1
- new net N$1347: B10.31, TET343.2
- new net N$1348: B10.30, TET343.3
- new net N$1349: B10.29, TET342.0
- new net N$1350: B10.28, TET342.1
- new net N$1351: B10.27, TET342.2
- new net N$1352: B10.26, TET342.3
- new net N$1353: B10.25, TET341.0
- new net N$1354: B10.24, TET341.1
- new net N$1355: B10.23, TET341.2
- new net N$1356: B10.22, TET341.3
- new net N$1357: B10.21, TET340.0
- new net N$1358: B10.20, TET340.1
- new net N$1359: B10.19, TET340.2
- new net N$1360: B10.18, TET340.3
- new net N$1361: B10.17, TET339.0
- new net N$1362: B10.16, TET339.1
- new net N$1363: B10.15, TET339.2
- new net N$1364: B10.14, TET339.3
- new net N$1365: B10.13, TET338.0
- new net N$1366: B10.12, TET338.1
- new net N$1367: B10.11, TET338.2
- new net N$1368: B10.10, TET338.3
- new net N$1369: B10.9, TET337.0
- new net N$1370: B10.8, TET337.1
- new net N$1371: B10.7, TET337.2
- new net N$1372: B10.6, TET337.3
- new net N$1373: B10.5, TET336.0
- new net N$1374: B10.4, TET336.1
- new net N$1375: B10.3, TET336.2
- new net N$1376: B10.38, TET344.2
- new net N$1377: B10.39, TET344.1
- new net N$1378: B10.40, TET344.0
- new net N$1379: B10.41, TET345.3
- new net N$1380: B10.42, TET345.2
- new net N$1381: B10.43, TET345.1
- new net N$1382: B10.44, TET345.0
- new net N$1383: B10.45, TET346.3
- new net N$1384: B10.46, TET346.2
- new net N$1385: B10.47, TET346.1
- new net N$1386: B10.48, TET346.0
- new net N$1387: B10.49, TET347.3
- new net N$1388: B10.50, TET347.2
- new net N$1389: B10.51, TET347.1
- new net N$1390: B10.52, TET347.0
- new net N$1391: B10.53, TET348.3
- new net N$1392: B10.54, TET348.2
- new net N$1393: B10.55, TET348.1
- new net N$1394: B10.56, TET348.0
- new net N$1395: B10.57, TET349.3
- new net N$1396: B10.58, TET349.2
- new net N$1397: B10.59, TET349.1
- new net N$1398: B10.60, TET349.0
- new net N$1399: B10.61, TET350.3
- new net N$1400: B10.62, TET350.2
- new net N$1401: B10.63, TET350.1
- new net N$1402: B10.64, TET350.0
- new net N$1403: B10.65, TET351.3
- new net N$1404: B10.66, TET351.2
- new net N$1405: B10.67, TET351.1
- new net N$1406: B10.68, TET351.0
- new net N$1407: B10.2, TET336.3
- new net N$1408: B10.37, TET344.3
- new net N$1409: A11.33, TET359.3
- new net N$1410: A11.32, TET359.2
- new net N$1411: A11.31, TET359.1
- new net N$1412: A11.30, TET359.0
- new net N$1413: A11.29, TET358.3
- new net N$1414: A11.28, TET358.2
- new net N$1415: A11.27, TET358.1
- new net N$1416: A11.26, TET358.0
- new net N$1417: A11.25, TET357.3
- new net N$1418: A11.24, TET357.2
- new net N$1419: A11.23, TET357.1
- new net N$1420: A11.22, TET357.0
- new net N$1421: A11.21, TET356.3
- new net N$1422: A11.20, TET356.2
- new net N$1423: A11.19, TET356.1
- new net N$1424: A11.18, TET356.0
- new net N$1425: A11.17, TET355.3
- new net N$1426: A11.16, TET355.2
- new net N$1427: A11.15, TET355.1
- new net N$1428: A11.14, TET355.0
- new net N$1429: A11.13, TET354.3
- new net N$1430: A11.12, TET354.2
- new net N$1431: A11.11, TET354.1
- new net N$1432: A11.10, TET354.0
- new net N$1433: A11.9, TET353.3
- new net N$1434: A11.8, TET353.2
- new net N$1435: A11.7, TET353.1
- new net N$1436: A11.6, TET353.0
- new net N$1437: A11.5, TET352.3
- new net N$1438: A11.4, TET352.2
- new net N$1439: A11.3, TET352.1
- new net N$1440: A11.38, TET360.1
- new net N$1441: A11.39, TET360.2
- new net N$1442: A11.40, TET360.3
- new net N$1443: A11.41, TET361.0
- new net N$1444: A11.42, TET361.1
- new net N$1445: A11.43, TET361.2
- new net N$1446: A11.44, TET361.3
- new net N$1447: A11.45, TET362.0
- new net N$1448: A11.46, TET362.1
- new net N$1449: A11.47, TET362.2
- new net N$1450: A11.48, TET362.3
- new net N$1451: A11.49, TET363.0
- new net N$1452: A11.50, TET363.1
- new net N$1453: A11.51, TET363.2
- new net N$1454: A11.52, TET363.3
- new net N$1455: A11.53, TET364.0
- new net N$1456: A11.54, TET364.1
- new net N$1457: A11.55, TET364.2
- new net N$1458: A11.56, TET364.3
- new net N$1459: A11.57, TET365.0
- new net N$1460: A11.58, TET365.1
- new net N$1461: A11.59, TET365.2
- new net N$1462: A11.60, TET365.3
- new net N$1463: A11.61, TET366.0
- new net N$1464: A11.62, TET366.1
- new net N$1465: A11.63, TET366.2
- new net N$1466: A11.64, TET366.3
- new net N$1467: A11.65, TET367.0
- new net N$1468: A11.66, TET367.1
- new net N$1469: A11.67, TET367.2
- new net N$1470: A11.68, TET367.3
- new net N$1471: A11.2, TET352.0
- new net N$1472: A11.37, TET360.0
- new net N$1473: B11.33, TET375.0
- new net N$1474: B11.32, TET375.1
- new net N$1475: B11.31, TET375.2
- new net N$1476: B11.30, TET375.3
- new net N$1477: B11.29, TET374.0
- new net N$1478: B11.28, TET374.1
- new net N$1479: B11.27, TET374.2
- new net N$1480: B11.26, TET374.3
- new net N$1481: B11.25, TET373.0
- new net N$1482: B11.24, TET373.1
- new net N$1483: B11.23, TET373.2
- new net N$1484: B11.22, TET373.3
- new net N$1485: B11.21, TET372.0
- new net N$1486: B11.20, TET372.1
- new net N$1487: B11.19, TET372.2
- new net N$1488: B11.18, TET372.3
- new net N$1489: B11.17, TET371.0
- new net N$1490: B11.16, TET371.1
- new net N$1491: B11.15, TET371.2
- new net N$1492: B11.14, TET371.3
- new net N$1493: B11.13, TET370.0
- new net N$1494: B11.12, TET370.1
- new net N$1495: B11.11, TET370.2
- new net N$1496: B11.10, TET370.3
- new net N$1497: B11.9, TET369.0
- new net N$1498: B11.8, TET369.1
- new net N$1499: B11.7, TET369.2
- new net N$1500: B11.6, TET369.3
- new net N$1501: B11.5, TET368.0
- new net N$1502: B11.4, TET368.1
- new net N$1503: B11.3, TET368.2
- new net N$1504: B11.38, TET376.2
- new net N$1505: B11.39, TET376.1
- new net N$1506: B11.40, TET376.0
- new net N$1507: B11.41, TET377.3
- new net N$1508: B11.42, TET377.2
- new net N$1509: B11.43, TET377.1
- new net N$1510: B11.44, TET377.0
- new net N$1511: B11.45, TET378.3
- new net N$1512: B11.46, TET378.2
- new net N$1513: B11.47, TET378.1
- new net N$1514: B11.48, TET378.0
- new net N$1515: B11.49, TET379.3
- new net N$1516: B11.50, TET379.2
- new net N$1517: B11.51, TET379.1
- new net N$1518: B11.52, TET379.0
- new net N$1519: B11.53, TET380.3
- new net N$1520: B11.54, TET380.2
- new net N$1521: B11.55, TET380.1
- new net N$1522: B11.56, TET380.0
- new net N$1523: B11.57, TET381.3
- new net N$1524: B11.58, TET381.2
- new net N$1525: B11.59, TET381.1
- new net N$1526: B11.60, TET381.0
- new net N$1527: B11.61, TET382.3
- new net N$1528: B11.62, TET382.2
- new net N$1529: B11.63, TET382.1
- new net N$1530: B11.64, TET382.0
- new net N$1531: B11.65, TET383.3
- new net N$1532: B11.66, TET383.2
- new net N$1533: B11.67, TET383.1
- new net N$1534: B11.68, TET383.0
- new net N$1535: B11.2, TET368.3
- new net N$1536: B11.37, TET376.3
- new net REF_A: A.1, REF_A0.P$1
- new net REF_B: B.1, REF_B0.P$1
- net GND: now also A.70, A.M1, A.M2, A.M3, A.M4, A1.70, A1.M1, A1.M2, A1.M3, A1.M4, A10.70, A10.M1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; no longer SJ_A0.1, SJ_A1.1, SJ_B0.1, SJ_B1.1
- net N$1: now also A1.33, TET39.3; no longer SHLD_A0.P$1, SJ_A0.COM
- net N$10: now also A1.24, TET37.2; no longer AIN_N0T1.28, AIN_N0T1.P28, TET38.2
- net N$100: now also B.42; no longer AIN_S0T.42, AIN_S0T.P42
- net N$1000: now also A.37; no longer AIN_N0T.37, AIN_N0T.P37
- net N$1001: now also B7.47, TET250.1; no longer AIN_S0T7.21, AIN_S0T7.P21, TET244.0
- net N$1002: now also B7.48, TET250.0; no longer AIN_S0T7.20, AIN_S0T7.P20, TET244.1
- net N$1003: now also B7.49, TET251.3; no longer AIN_S0T7.19, AIN_S0T7.P19, TET244.2
- net N$1004: now also B7.50, TET251.2; no longer AIN_S0T7.18, AIN_S0T7.P18, TET244.3
- net N$1005: now also B7.51, TET251.1; no longer AIN_S0T7.17, AIN_S0T7.P17, TET243.0
- net N$1006: now also B7.52, TET251.0; no longer AIN_S0T7.16, AIN_S0T7.P16, TET243.1
- net N$1007: now also B7.53, TET252.3; no longer AIN_S0T7.15, AIN_S0T7.P15, TET243.2
- net N$1008: now also B7.54, TET252.2; no longer AIN_S0T7.14, AIN_S0T7.P14, TET243.3
- net N$1009: now also B7.55, TET252.1; no longer AIN_S0T7.13, AIN_S0T7.P13, TET242.0
- net N$101: now also B.43; no longer AIN_S0T.43, AIN_S0T.P43
- net N$1010: now also B7.56, TET252.0; no longer AIN_S0T7.12, AIN_S0T7.P12, TET242.1
- net N$1011: now also B7.57, TET253.3; no longer AIN_S0T7.11, AIN_S0T7.P11, TET242.2
- net N$1012: now also B7.58, TET253.2; no longer AIN_S0T7.10, AIN_S0T7.P10, TET242.3
- net N$1013: now also B7.59, TET253.1; no longer AIN_S0T7.9, AIN_S0T7.P9, TET241.0
- net N$1014: now also B7.60, TET253.0; no longer AIN_S0T7.8, AIN_S0T7.P8, TET241.1
- net N$1015: now also B7.61, TET254.3; no longer AIN_S0T7.7, AIN_S0T7.P7, TET241.2
- net N$1016: now also B7.62, TET254.2; no longer AIN_S0T7.6, AIN_S0T7.P6, TET241.3
- net N$1017: now also B7.63, TET254.1; no longer AIN_S0T7.5, AIN_S0T7.P5, TET240.0
- net N$1018: now also B7.64, TET254.0; no longer AIN_S0T7.4, AIN_S0T7.P4, TET240.1
- net N$1019: now also B7.65, TET255.3; no longer AIN_S0T7.3, AIN_S0T7.P3, TET240.2
- net N$102: now also B.44; no longer AIN_S0T.44, AIN_S0T.P44
- net N$1020: now also B7.66, TET255.2; no longer AIN_S0T7.38, AIN_S0T7.P38, TET248.2
- net N$1021: now also B7.67, TET255.1; no longer AIN_S0T7.39, AIN_S0T7.P39, TET248.1
- net N$1022: now also B7.68, TET255.0; no longer AIN_S0T7.40, AIN_S0T7.P40, TET248.0
- net N$1023: now also B7.2, TET240.3; no longer AIN_S0T7.41, AIN_S0T7.P41, TET249.3
- net N$1024: now also B7.37, TET248.3; no longer AIN_S0T7.42, AIN_S0T7.P42, TET249.2
- net N$1025: now also A8.33, TET263.3; no longer AIN_S0T7.43, AIN_S0T7.P43, TET249.1
- net N$1026: now also A8.32, TET263.2; no longer AIN_S0T7.44, AIN_S0T7.P44, TET249.0
- net N$1027: now also A8.31, TET263.1; no longer AIN_S0T7.45, AIN_S0T7.P45, TET250.3
- net N$1028: now also A8.30, TET263.0; no longer AIN_S0T7.46, AIN_S0T7.P46, TET250.2
- net N$1029: now also A8.29, TET262.3; no longer AIN_S0T7.47, AIN_S0T7.P47, TET250.1
- net N$103: now also B.45; no longer AIN_S0T.45, AIN_S0T.P45
- net N$1030: now also A8.28, TET262.2; no longer AIN_S0T7.48, AIN_S0T7.P48, TET250.0
- net N$1031: now also A8.27, TET262.1; no longer AIN_S0T7.49, AIN_S0T7.P49, TET251.3
- net N$1032: now also A8.26, TET262.0; no longer AIN_S0T7.50, AIN_S0T7.P50, TET251.2
- net N$1033: now also A8.25, TET261.3; no longer AIN_S0T7.51, AIN_S0T7.P51, TET251.1
- net N$1034: now also A8.24, TET261.2; no longer AIN_S0T7.52, AIN_S0T7.P52, TET251.0
- net N$1035: now also A8.23, TET261.1; no longer AIN_S0T7.53, AIN_S0T7.P53, TET252.3
- net N$1036: now also A8.22, TET261.0; no longer AIN_S0T7.54, AIN_S0T7.P54, TET252.2
- net N$1037: now also A8.21, TET260.3; no longer AIN_S0T7.55, AIN_S0T7.P55, TET252.1
- net N$1038: now also A8.20, TET260.2; no longer AIN_S0T7.56, AIN_S0T7.P56, TET252.0
- net N$1039: now also A8.19, TET260.1; no longer AIN_S0T7.57, AIN_S0T7.P57, TET253.3
- net N$104: now also B.46; no longer AIN_S0T.46, AIN_S0T.P46
- net N$1040: now also A8.18, TET260.0; no longer AIN_S0T7.58, AIN_S0T7.P58, TET253.2
- net N$1041: now also A8.17, TET259.3; no longer AIN_S0T7.59, AIN_S0T7.P59, TET253.1
- net N$1042: now also A8.16, TET259.2; no longer AIN_S0T7.60, AIN_S0T7.P60, TET253.0
- net N$1043: now also A8.15, TET259.1; no longer AIN_S0T7.61, AIN_S0T7.P61, TET254.3
- net N$1044: now also A8.14, TET259.0; no longer AIN_S0T7.62, AIN_S0T7.P62, TET254.2
- net N$1045: now also A8.13, TET258.3; no longer AIN_S0T7.63, AIN_S0T7.P63, TET254.1
- net N$1046: now also A8.12, TET258.2; no longer AIN_S0T7.64, AIN_S0T7.P64, TET254.0
- net N$1047: now also A8.11, TET258.1; no longer AIN_S0T7.65, TET255.3
- net N$1048: now also A8.10, TET258.0; no longer AIN_S0T7.66, TET255.2
- net N$1049: now also A8.9, TET257.3; no longer AIN_S0T7.67, TET255.1
- net N$105: now also B.47; no longer AIN_S0T.47, AIN_S0T.P47
- net N$1050: now also A8.8, TET257.2; no longer AIN_S0T7.68, TET255.0
- net N$1051: now also A8.7, TET257.1; no longer AIN_S0T7.2, AIN_S0T7.P2, TET240.3
- net N$1052: now also A8.6, TET257.0; no longer AIN_S0T7.37, AIN_S0T7.P37, TET248.3
- net N$1053: now also A8.5, TET256.3; no longer SHLD_A14.P$1, SJ_A14.COM
- net N$1054: now also A8.4, TET256.2; no longer SHLD_A15.P$1, SJ_A15.COM
- net N$1055: now also A8.3, TET256.1; no longer SHLD_B14.P$1, SJ_B14.COM
- net N$1056: now also A8.38, TET264.1; no longer SHLD_B15.P$1, SJ_B15.COM
- net N$1057: now also A8.39, TET264.2; no longer AIN_N0T8.33, TET263.3
- net N$1058: now also A8.40, TET264.3; no longer AIN_N0T8.32, TET263.2
- net N$1059: now also A8.41, TET265.0; no longer AIN_N0T8.31, AIN_N0T8.P31, TET263.1
- net N$106: now also B.48; no longer AIN_S0T.48, AIN_S0T.P48
- net N$1060: now also A8.42, TET265.1; no longer AIN_N0T8.30, AIN_N0T8.P30, TET263.0
- net N$1061: now also A8.43, TET265.2; no longer AIN_N0T8.29, AIN_N0T8.P29, TET262.3
- net N$1062: now also A8.44, TET265.3; no longer AIN_N0T8.28, AIN_N0T8.P28, TET262.2
- net N$1063: now also A8.45, TET266.0; no longer AIN_N0T8.27, AIN_N0T8.P27, TET262.1
- net N$1064: now also A8.46, TET266.1; no longer AIN_N0T8.26, AIN_N0T8.P26, TET262.0
- net N$1065: now also A8.47, TET266.2; no longer AIN_N0T8.25, AIN_N0T8.P25, TET261.3
- net N$1066: now also A8.48, TET266.3; no longer AIN_N0T8.24, AIN_N0T8.P24, TET261.2
- net N$1067: now also A8.49, TET267.0; no longer AIN_N0T8.23, AIN_N0T8.P23, TET261.1
- net N$1068: now also A8.50, TET267.1; no longer AIN_N0T8.22, AIN_N0T8.P22, TET261.0
- net N$1069: now also A8.51, TET267.2; no longer AIN_N0T8.21, AIN_N0T8.P21, TET260.3
- net N$107: now also B.49; no longer AIN_S0T.49, AIN_S0T.P49
- net N$1070: now also A8.52, TET267.3; no longer AIN_N0T8.20, AIN_N0T8.P20, TET260.2
- net N$1071: now also A8.53, TET268.0; no longer AIN_N0T8.19, AIN_N0T8.P19, TET260.1
- net N$1072: now also A8.54, TET268.1; no longer AIN_N0T8.18, AIN_N0T8.P18, TET260.0
- net N$1073: now also A8.55, TET268.2; no longer AIN_N0T8.17, AIN_N0T8.P17, TET259.3
- net N$1074: now also A8.56, TET268.3; no longer AIN_N0T8.16, AIN_N0T8.P16, TET259.2
- net N$1075: now also A8.57, TET269.0; no longer AIN_N0T8.15, AIN_N0T8.P15, TET259.1
- net N$1076: now also A8.58, TET269.1; no longer AIN_N0T8.14, AIN_N0T8.P14, TET259.0
- net N$1077: now also A8.59, TET269.2; no longer AIN_N0T8.13, AIN_N0T8.P13, TET258.3
- net N$1078: now also A8.60, TET269.3; no longer AIN_N0T8.12, AIN_N0T8.P12, TET258.2
- net N$1079: now also A8.61, TET270.0; no longer AIN_N0T8.11, AIN_N0T8.P11, TET258.1
- net N$108: now also B.50; no longer AIN_S0T.50, AIN_S0T.P50
- net N$1080: now also A8.62, TET270.1; no longer AIN_N0T8.10, AIN_N0T8.P10, TET258.0
- net N$1081: now also A8.63, TET270.2; no longer AIN_N0T8.9, AIN_N0T8.P9, TET257.3
- net N$1082: now also A8.64, TET270.3; no longer AIN_N0T8.8, AIN_N0T8.P8, TET257.2
- net N$1083: now also A8.65, TET271.0; no longer AIN_N0T8.7, AIN_N0T8.P7, TET257.1
- net N$1084: now also A8.66, TET271.1; no longer AIN_N0T8.6, AIN_N0T8.P6, TET257.0
- net N$1085: now also A8.67, TET271.2; no longer AIN_N0T8.5, AIN_N0T8.P5, TET256.3
- net N$1086: now also A8.68, TET271.3; no longer AIN_N0T8.4, AIN_N0T8.P4, TET256.2
- net N$1087: now also A8.2, TET256.0; no longer AIN_N0T8.3, AIN_N0T8.P3, TET256.1
- net N$1088: now also A8.37, TET264.0; no longer AIN_N0T8.38, AIN_N0T8.P38, TET264.1
- net N$1089: now also B8.33, TET279.0; no longer AIN_N0T8.39, AIN_N0T8.P39, TET264.2
- net N$109: now also B.51; no longer AIN_S0T.51, AIN_S0T.P51
- net N$1090: now also B8.32, TET279.1; no longer AIN_N0T8.40, AIN_N0T8.P40, TET264.3
- net N$1091: now also B8.31, TET279.2; no longer AIN_N0T8.41, AIN_N0T8.P41, TET265.0
- net N$1092: now also B8.30, TET279.3; no longer AIN_N0T8.42, AIN_N0T8.P42, TET265.1
- net N$1093: now also B8.29, TET278.0; no longer AIN_N0T8.43, AIN_N0T8.P43, TET265.2
- net N$1094: now also B8.28, TET278.1; no longer AIN_N0T8.44, AIN_N0T8.P44, TET265.3
- net N$1095: now also B8.27, TET278.2; no longer AIN_N0T8.45, AIN_N0T8.P45, TET266.0
- net N$1096: now also B8.26, TET278.3; no longer AIN_N0T8.46, AIN_N0T8.P46, TET266.1
- net N$1097: now also B8.25, TET277.0; no longer AIN_N0T8.47, AIN_N0T8.P47, TET266.2
- net N$1098: now also B8.24, TET277.1; no longer AIN_N0T8.48, AIN_N0T8.P48, TET266.3
- net N$1099: now also B8.23, TET277.2; no longer AIN_N0T8.49, AIN_N0T8.P49, TET267.0
- net N$11: now also A1.23, TET37.1; no longer AIN_N0T1.27, AIN_N0T1.P27, TET38.1
- net N$110: now also B.52; no longer AIN_S0T.52, AIN_S0T.P52
- net N$1100: now also B8.22, TET277.3; no longer AIN_N0T8.50, AIN_N0T8.P50, TET267.1
- net N$1101: now also B8.21, TET276.0; no longer AIN_N0T8.51, AIN_N0T8.P51, TET267.2
- net N$1102: now also B8.20, TET276.1; no longer AIN_N0T8.52, AIN_N0T8.P52, TET267.3
- net N$1103: now also B8.19, TET276.2; no longer AIN_N0T8.53, AIN_N0T8.P53, TET268.0
- net N$1104: now also B8.18, TET276.3; no longer AIN_N0T8.54, AIN_N0T8.P54, TET268.1
- net N$1105: now also B8.17, TET275.0; no longer AIN_N0T8.55, AIN_N0T8.P55, TET268.2
- net N$1106: now also B8.16, TET275.1; no longer AIN_N0T8.56, AIN_N0T8.P56, TET268.3
- net N$1107: now also B8.15, TET275.2; no longer AIN_N0T8.57, AIN_N0T8.P57, TET269.0
- net N$1108: now also B8.14, TET275.3; no longer AIN_N0T8.58, AIN_N0T8.P58, TET269.1
- net N$1109: now also B8.13, TET274.0; no longer AIN_N0T8.59, AIN_N0T8.P59, TET269.2
- net N$111: now also B.53; no longer AIN_S0T.53, AIN_S0T.P53
- net N$1110: now also B8.12, TET274.1; no longer AIN_N0T8.60, AIN_N0T8.P60, TET269.3
- net N$1111: now also B8.11, TET274.2; no longer AIN_N0T8.61, AIN_N0T8.P61, TET270.0
- net N$1112: now also B8.10, TET274.3; no longer AIN_N0T8.62, AIN_N0T8.P62, TET270.1
- net N$1113: now also B8.9, TET273.0; no longer AIN_N0T8.63, AIN_N0T8.P63, TET270.2
- net N$1114: now also B8.8, TET273.1; no longer AIN_N0T8.64, AIN_N0T8.P64, TET270.3
- net N$1115: now also B8.7, TET273.2; no longer AIN_N0T8.65, TET271.0
- net N$1116: now also B8.6, TET273.3; no longer AIN_N0T8.66, TET271.1
- net N$1117: now also B8.5, TET272.0; no longer AIN_N0T8.67, TET271.2
- net N$1118: now also B8.4, TET272.1; no longer AIN_N0T8.68, TET271.3
- net N$1119: now also B8.3, TET272.2; no longer AIN_N0T8.2, AIN_N0T8.P2, TET256.0
- net N$112: now also B.54; no longer AIN_S0T.54, AIN_S0T.P54
- net N$1120: now also B8.38, TET280.2; no longer AIN_N0T8.37, AIN_N0T8.P37, TET264.0
- net N$1121: now also B8.39, TET280.1; no longer AIN_S0T8.33, TET279.0
- net N$1122: now also B8.40, TET280.0; no longer AIN_S0T8.32, TET279.1
- net N$1123: now also B8.41, TET281.3; no longer AIN_S0T8.31, AIN_S0T8.P31, TET279.2
- net N$1124: now also B8.42, TET281.2; no longer AIN_S0T8.30, AIN_S0T8.P30, TET279.3
- net N$1125: now also B8.43, TET281.1; no longer AIN_S0T8.29, AIN_S0T8.P29, TET278.0
- net N$1126: now also B8.44, TET281.0; no longer AIN_S0T8.28, AIN_S0T8.P28, TET278.1
- net N$1127: now also B8.45, TET282.3; no longer AIN_S0T8.27, AIN_S0T8.P27, TET278.2
- net N$1128: now also B8.46, TET282.2; no longer AIN_S0T8.26, AIN_S0T8.P26, TET278.3
- net N$1129: now also B8.47, TET282.1; no longer AIN_S0T8.25, AIN_S0T8.P25, TET277.0
- net N$113: now also B.55; no longer AIN_S0T.55, AIN_S0T.P55
- net N$1130: now also B8.48, TET282.0; no longer AIN_S0T8.24, AIN_S0T8.P24, TET277.1
- net N$1131: now also B8.49, TET283.3; no longer AIN_S0T8.23, AIN_S0T8.P23, TET277.2
- net N$1132: now also B8.50, TET283.2; no longer AIN_S0T8.22, AIN_S0T8.P22, TET277.3
- net N$1133: now also B8.51, TET283.1; no longer AIN_S0T8.21, AIN_S0T8.P21, TET276.0
- net N$1134: now also B8.52, TET283.0; no longer AIN_S0T8.20, AIN_S0T8.P20, TET276.1
- net N$1135: now also B8.53, TET284.3; no longer AIN_S0T8.19, AIN_S0T8.P19, TET276.2
- net N$1136: now also B8.54, TET284.2; no longer AIN_S0T8.18, AIN_S0T8.P18, TET276.3
- net N$1137: now also B8.55, TET284.1; no longer AIN_S0T8.17, AIN_S0T8.P17, TET275.0
- net N$1138: now also B8.56, TET284.0; no longer AIN_S0T8.16, AIN_S0T8.P16, TET275.1
- net N$1139: now also B8.57, TET285.3; no longer AIN_S0T8.15, AIN_S0T8.P15, TET275.2
- net N$114: now also B.56; no longer AIN_S0T.56, AIN_S0T.P56
- net N$1140: now also B8.58, TET285.2; no longer AIN_S0T8.14, AIN_S0T8.P14, TET275.3
- net N$1141: now also B8.59, TET285.1; no longer AIN_S0T8.13, AIN_S0T8.P13, TET274.0
- net N$1142: now also B8.60, TET285.0; no longer AIN_S0T8.12, AIN_S0T8.P12, TET274.1
- net N$1143: now also B8.61, TET286.3; no longer AIN_S0T8.11, AIN_S0T8.P11, TET274.2
- net N$1144: now also B8.62, TET286.2; no longer AIN_S0T8.10, AIN_S0T8.P10, TET274.3
- net N$1145: now also B8.63, TET286.1; no longer AIN_S0T8.9, AIN_S0T8.P9, TET273.0
- net N$1146: now also B8.64, TET286.0; no longer AIN_S0T8.8, AIN_S0T8.P8, TET273.1
- net N$1147: now also B8.65, TET287.3; no longer AIN_S0T8.7, AIN_S0T8.P7, TET273.2
- net N$1148: now also B8.66, TET287.2; no longer AIN_S0T8.6, AIN_S0T8.P6, TET273.3
- net N$1149: now also B8.67, TET287.1; no longer AIN_S0T8.5, AIN_S0T8.P5, TET272.0
- net N$115: now also B.57; no longer AIN_S0T.57, AIN_S0T.P57
- net N$1150: now also B8.68, TET287.0; no longer AIN_S0T8.4, AIN_S0T8.P4, TET272.1
- net N$1151: now also B8.2, TET272.3; no longer AIN_S0T8.3, AIN_S0T8.P3, TET272.2
- net N$1152: now also B8.37, TET280.3; no longer AIN_S0T8.38, AIN_S0T8.P38, TET280.2
- net N$1153: now also A9.33, TET295.3; no longer AIN_S0T8.39, AIN_S0T8.P39, TET280.1
- net N$1154: now also A9.32, TET295.2; no longer AIN_S0T8.40, AIN_S0T8.P40, TET280.0
- net N$1155: now also A9.31, TET295.1; no longer AIN_S0T8.41, AIN_S0T8.P41, TET281.3
- net N$1156: now also A9.30, TET295.0; no longer AIN_S0T8.42, AIN_S0T8.P42, TET281.2
- net N$1157: now also A9.29, TET294.3; no longer AIN_S0T8.43, AIN_S0T8.P43, TET281.1
- net N$1158: now also A9.28, TET294.2; no longer AIN_S0T8.44, AIN_S0T8.P44, TET281.0
- net N$1159: now also A9.27, TET294.1; no longer AIN_S0T8.45, AIN_S0T8.P45, TET282.3
- net N$116: now also B.58; no longer AIN_S0T.58, AIN_S0T.P58
- net N$1160: now also A9.26, TET294.0; no longer AIN_S0T8.46, AIN_S0T8.P46, TET282.2
- net N$1161: now also A9.25, TET293.3; no longer AIN_S0T8.47, AIN_S0T8.P47, TET282.1
- net N$1162: now also A9.24, TET293.2; no longer AIN_S0T8.48, AIN_S0T8.P48, TET282.0
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Routing:
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- added copper zone on layer 15, net GND
- added copper zone on layer 2, net GND
- removed copper zone on layer 1, net GND1
- removed copper zone on layer 16, net GND1
- removed copper zone on layer 1, net GND2
- removed copper zone on layer 16, net GND2
- removed copper zone on layer 1, net GND3
- removed copper zone on layer 16, net GND3
- removed copper zone on layer 1, net GND4
- removed copper zone on layer 16, net GND4
- removed copper zone on layer 1, net GND5
- removed copper zone on layer 16, net GND5
- removed copper zone on layer 1, net GND6
- removed copper zone on layer 16, net GND6
- removed copper zone on layer 1, net GND7
- removed copper zone on layer 16, net GND7
- removed copper zone on layer 1, net GND8
- removed copper zone on layer 16, net GND8
Other:
- board size 130 x 130 mm -> 210 x 160 mm
- board text added: "ANA"
- board text added: "ANB"
- board text added: "B"
- board text added: "C0A"
- board text added: "C0B"
- board text added: "C1A"
- board text added: "C1B"
- board text added: "ESA"
- board text added: "ESB"
- board text added: "G"
- board text added: "Rev. 1.2 CERN OHL 1.2 JPN, MWL@MIT 2017"
- board text removed: "A-S-G"
- board text removed: "AIN_N0T"
- board text removed: "AIN_S0T"
- board text removed: "G-S-A"
- board text removed: "MECH_E0T"
- board text removed: "MECH_W0T"
- board text removed: "Rev. 1.1 CC BY-SA-NC-4.0 JPN, MWL@MIT 2016-02"
- board text removed: "S"
