File: test-board-128-256/test-board-128-256.sch (EAGLE design)
At the start: 76 parts

Commit message: Added estim and optostim test circuits to test-board-128-256
- Allows user to test electrical stimulation and optical stimulation of
headstage-128-256
Parts:
- removed REF_N_TO_GND: (no value), jonnew:JP3E
- removed R_REFNORTH: (no value), jonnew:JP2E_THRU-HOLE
- added CDL_A, CDL_B, D1_EXT_A, D1_EXT_B, D2_EXT_A, D2_EXT_B, RS_A, RS_B: (no value), jonnew:JP2E_THRU-HOLE
- added D1, D3: LXZ1-PB01, jonnew:LED_LXZ1
- added D2, D4: LXZ1-PL01, jonnew:LED_LXZ1
- added LED_SELECT_A, LED_SELECT_B: (no value), jonnew:JP3E
- added TP14: V_ISTIM_A, jonnew:TPPAD1-20
- added TP15: V_ISTIM_B, jonnew:TPPAD1-20
- AIN_N0T, AIN_S0T: device jonnew:PINHD-2X35_DF40HEAD -> jonnew:PINHD-2X35+4_DF40-70HEAD
- renumbered REF_S_TO_GND to REF_TO_GND, R_REFSOUTH to R_REF
Connections:
- removed net N$15: REF_N_TO_GND.3, R_REFNORTH.1
- removed net REF_NORTH: AIN_N0T.1, REF_N_TO_GND.2
- removed net REF_SOUTH: AIN_S0T.36, REF_TO_GND.2
- new net AN_A: AIN_N0T.36, LED_SELECT_A.2
- new net AN_B: AIN_S0T.36, LED_SELECT_B.2
- new net AN_INT: D1.A, D2.A, LED_SELECT_A.3
- new net AN_INT1: D3.A, D4.A, LED_SELECT_B.3
- new net CAT0_A: AIN_N0T.34, D1.C, D2_EXT_A.1
- new net CAT0_B: AIN_S0T.34, D2_EXT_B.1, D3.C
- new net CAT1_A: AIN_N0T.35, D1_EXT_A.1, D2.C
- new net CAT1_B: AIN_S0T.35, D1_EXT_B.1, D4.C
- new net ISTIM_A: AIN_N0T.69, CDL_A.2, TP14.TP
- new net ISTIM_B: AIN_S0T.69, CDL_B.2, TP15.TP
- new net N$1: CDL_A.1, RS_A.2
- new net N$14: CDL_B.1, RS_B.2
- new net N$16: D1_EXT_B.2, D2_EXT_B.2, LED_SELECT_B.1
- new net N$5: D1_EXT_A.2, D2_EXT_A.2, LED_SELECT_A.1
- new net REF: AIN_N0T.1, AIN_S0T.1, REF_TO_GND.2, RS_A.1, RS_B.1
- net GND: no longer REF_N_TO_GND.1, R_REFNORTH.2
- net HS_GND: now also AIN_N0T.70, AIN_S0T.70; no longer AIN_S0T.34, AIN_S0T.35
Other:
- note added: "Stim LEDs"
- note added: "Stimulation Electrode ~200 uM diameter: 110nF in series with 3.5k (Noorsal, 2012)"

Commit message: Lots of small fixes and cleanup
- Taking care of little issues that have been bothering me
- Dediated serdes interface board moved to deprecated
- Non-serialized headstage moved to deprecated
- Deleted top-level datasheets directory which does not really
apply to anything anymore
- Added pdfs versions of board schematics so that eagle is not
needed to see them.
- Small fixes to test-boards: High power LEDs moved to bottom to prevent
blinding ppl. Silkscreen improved. License updated. Etc. Gerbers
updated.
- Removed random deprecated design files where I found them.
Parts:
- renumbered AIN_N0T to A-OR-D, AIN_S0T to B-OR-C
