File: headstage-256/expansion-board/hs-256-expansion.sch (EAGLE design)
At the start: 16 parts, among them J2 PINHD-2X5_DF40-REC, J4 PINHD-2X5_DF40-REC, J5 PINHD-2X6, J6 PINHD-2X4

Commit message: Fix errors in headstage-256 expansion boards
- Headers were too close to receptacles in debug board
- Some components did not have values
- Added BOM to the google sheet based on this design
Parts:
- C3: value 1uF -> 10uF; device jonnew:C_0402 -> jonnew:C-POL_0805
- C4: value (none) -> 0.1uF; device jonnew:C-POL_0805 -> jonnew:C_0402
- C5: value (none) -> 0.1uF
- C6: value 0.1uF -> 1uF
- J3: value (none) -> PINHD-2X5_DF40-REC; device jonnew:PINHD-2X10_DF40-20REC -> jonnew:PINHD-2X5_DF40-REC
- J4: value PINHD-2X5_DF40-REC -> (none); device jonnew:PINHD-2X5_DF40-REC -> jonnew:PINHD-2X10_DF40-20REC
- J5: value PINHD-2X6 -> PINHD-2X4; device jonnew:PINHD-2X6 -> jonnew:PINHD-2X4
- J6: value PINHD-2X4 -> PINHD-2X6; device jonnew:PINHD-2X4 -> jonnew:PINHD-2X6
- U1: value (none) -> REF3318; device jonnew:MICROPHONE-PCM_SPH -> jonnew:VREF_SOT
- U2: value (none) -> SPM0408LE5H-TB-6
- U3: value (none) -> SPH0641LU4H-1; device jonnew:VREF_SOT -> jonnew:MICROPHONE-PCM_SPH
Connections:
- net +3V3: now also C4.1, J3.6, J3.8, J4.17, J4.18, J6.12, U1.VIN, U3.SELECT, U3.VDD; no longer C2.1, J3.17, J3.18, J4.6, J4.8, J5.12, U1.SELECT, U1.VDD, U3.VIN
- net A/D_IN1: now also J4.5; no longer J3.5
- net A/D_VREF: now also J4.6; no longer J3.6
- net ANOUT: now also C3.-; no longer C4.-
- net CLK: now also U3.CLK; no longer U1.CLK
- net DATA: now also U3.DATA; no longer U1.DATA
- net EXP1: now also J4.13, J6.3; no longer J3.13, J5.3
- net EXP10: now also J3.7, J5.3; no longer J4.7, J6.3
- net EXP11: now also J3.3, J5.5; no longer J4.3, J6.5
- net EXP12: now also J3.1, J5.6; no longer J4.1, J6.6
- net EXP13: now also J3.5, J5.4; no longer J4.5, J6.4
- net EXP14: now also J3.10, J5.2; no longer J4.10, J6.2
- net EXP2: now also J4.2, J6.10; no longer J3.2, J5.10
- net EXP3: now also J4.8, J6.6; no longer J3.8, J5.6
- net EXP4: now also J4.10, J6.4; no longer J3.10, J5.4
- net EXP5/VMEAS: now also J4.1, J6.9; no longer J3.1, J5.9
- net EXP6: now also J4.14, J6.5; no longer J3.14, J5.5
- net EXP7: now also J4.3, J6.8; no longer J3.3, J5.8
- net EXP8: now also J4.15, J6.7; no longer J3.15, J5.7
- net EXP9: now also J3.9, J5.1; no longer J4.9, J6.1
- net GND: now also C4.2, J3.2, J4.11, J4.12, J4.16, J4.7, J4.9, J5.7, J5.8, J6.1, J6.2; no longer C3.2, J3.11, J3.12, J3.16, J3.7, J3.9, J4.2, J5.1, J5.2, J6.7, J6.8
- net N$1: now also C6.1; no longer C3.1
- net N$5: now also C3.+; no longer C4.+
- net VCOAX: now also J4.19, J4.20, J6.11; no longer J3.19, J3.20, J5.11
- net VREF: now also C2.1, U1.VOUT; no longer C6.1, U3.VOUT
Other:
- moved on the sheet: C1, C2, C3, C4, C5, C6
