File: lesion-256/lesion-256.sch (EAGLE design)
At the start: 9 parts

Commit message: Added another breakout for electrolesioning with eib-64
- I just put it as breakaway board on the existing lesion-256 board
- I will change the name of this directory and all files after this
commit
Parts:
- added J1: DF40C-70DP-0.4V(51), jonnew:PINHD-2X35+4DF40-70HEAD-LESS-SILK
- added J4: (no value), jonnew:PINHD-2X8_SMD_0.5"
- added J7: (no value), jonnew:JP3E_SMD-0.05
Connections:
- new net N$1: J1.53, J1.54, J1.55, J1.56, J4.10
- new net N$10: J1.26, J1.27, J1.28, J1.29, J4.3
- new net N$11: J1.30, J1.31, J1.32, J1.33, J4.1
- new net N$12: J1.37, J1.38, J1.39, J1.40, J4.2
- new net N$13: J1.41, J1.42, J1.43, J1.44, J4.4
- new net N$14: J1.45, J1.46, J1.47, J1.48, J4.6
- new net N$15: J1.49, J1.50, J1.51, J1.52, J4.8
- new net N$2: J1.57, J1.58, J1.59, J1.60, J4.12
- new net N$3: J1.61, J1.62, J1.63, J1.64, J4.14
- new net N$32: J1.6, J1.7, J1.8, J1.9, J4.13
- new net N$4: J1.2, J1.3, J1.4, J1.5, J4.15
- new net N$5: J1.65, J1.66, J1.67, J1.68, J4.16
- new net N$6: J1.10, J1.11, J1.12, J1.13, J4.11
- new net N$7: J1.14, J1.15, J1.16, J1.17, J4.9
- new net N$8: J1.18, J1.19, J1.20, J1.21, J4.7
- new net N$9: J1.22, J1.23, J1.24, J1.25, J4.5
- net AGND: now also J1.1, J1.69, J1.M1, J1.M2, J1.M3, J1.M4, J7.1, J7.2, J7.3
Other:
- note added: "FOR EIB-128 & EIB-256"
- note added: "FOR EIB-64"
