File: lesion-breakout/lesion-breakout.sch (EAGLE design)
At the start: 12 parts, among them J1 DF40C-70DP-0.4V(51)

Commit message: Improved lesion-breakout layout
- Moved recepticals to available space on periphery
Parts:
- removed JA1, JA3, JA5, JA7: DF40C(2.0)-70DS-0.4V(51), jonnew:PINHD-2X35_DF40REC
- added J10, J12: (no value), jonnew:PINHD-2X8_SMD_0.5"
- added J11, J9: DF40C(2.0)-70DS-0.4V(51), jonnew:PINHD-2X35_DF40REC
- added TP1, TP2, TP3, TP4: (no value), jonnew:TP_1MM
- J1: value DF40C-70DP-0.4V(51) -> DF40C(2.0)-70DS-0.4V(51); device jonnew:PINHD-2X35+4DF40-70HEAD-LESS-SILK -> jonnew:PINHD-2X35_DF40REC
- J3: value (none) -> DF40C(2.0)-70DS-0.4V(51); device jonnew:PINHD-2X8_SMD_0.5" -> jonnew:PINHD-2X35_DF40REC
- J4: value (none) -> DF40C-70DP-0.4V(51); device jonnew:PINHD-2X8_SMD_0.5" -> jonnew:PINHD-2X35+4DF40-70HEAD-LESS-SILK
- J5: device jonnew:JP3E_SMD-0.05 -> jonnew:PINHD-2X8_SMD_0.5"
- J6: device jonnew:PINHD-2X8_SMD_0.5" -> jonnew:JP3E_SMD-0.05
Connections:
- removed net N$100: J8.7, JA7.14, JA7.15, JA7.16, JA7.17
- removed net N$101: J8.9, JA7.18, JA7.19, JA7.20, JA7.21
- removed net N$102: J8.11, JA7.22, JA7.23, JA7.24, JA7.25
- removed net N$103: J8.13, JA7.26, JA7.27, JA7.28, JA7.29
- removed net N$104: J8.15, JA7.30, JA7.31, JA7.32, JA7.33
- removed net N$105: J8.16, JA7.37, JA7.38, JA7.39, JA7.40
- removed net N$106: J8.14, JA7.41, JA7.42, JA7.43, JA7.44
- removed net N$107: J8.12, JA7.45, JA7.46, JA7.47, JA7.48
- removed net N$108: J8.10, JA7.49, JA7.50, JA7.51, JA7.52
- removed net N$109: J8.8, JA7.53, JA7.54, JA7.55, JA7.56
- removed net N$110: J8.6, JA7.57, JA7.58, JA7.59, JA7.60
- removed net N$111: J8.4, JA7.61, JA7.62, JA7.63, JA7.64
- removed net N$112: J8.2, JA7.65, JA7.66, JA7.67, JA7.68
- removed net N$16: J2.1, JA1.2, JA1.3, JA1.4, JA1.5
- removed net N$17: J2.3, JA1.6, JA1.7, JA1.8, JA1.9
- removed net N$18: J2.5, JA1.10, JA1.11, JA1.12, JA1.13
- removed net N$19: J2.7, JA1.14, JA1.15, JA1.16, JA1.17
- removed net N$20: J2.9, JA1.18, JA1.19, JA1.20, JA1.21
- removed net N$21: J2.11, JA1.22, JA1.23, JA1.24, JA1.25
- removed net N$22: J2.13, JA1.26, JA1.27, JA1.28, JA1.29
- removed net N$23: J2.15, JA1.30, JA1.31, JA1.32, JA1.33
- removed net N$24: J2.16, JA1.37, JA1.38, JA1.39, JA1.40
- removed net N$25: J2.14, JA1.41, JA1.42, JA1.43, JA1.44
- removed net N$26: J2.12, JA1.45, JA1.46, JA1.47, JA1.48
- removed net N$27: J2.10, JA1.49, JA1.50, JA1.51, JA1.52
- removed net N$28: J2.8, JA1.53, JA1.54, JA1.55, JA1.56
- removed net N$29: J2.6, JA1.57, JA1.58, JA1.59, JA1.60
- removed net N$30: J2.4, JA1.61, JA1.62, JA1.63, JA1.64
- removed net N$31: J2.2, JA1.65, JA1.66, JA1.67, JA1.68
- removed net N$65: J6.1, JA5.2, JA5.3, JA5.4, JA5.5
- removed net N$66: J6.3, JA5.6, JA5.7, JA5.8, JA5.9
- removed net N$67: J6.5, JA5.10, JA5.11, JA5.12, JA5.13
- removed net N$68: J6.7, JA5.14, JA5.15, JA5.16, JA5.17
- removed net N$69: J6.9, JA5.18, JA5.19, JA5.20, JA5.21
- removed net N$70: J6.11, JA5.22, JA5.23, JA5.24, JA5.25
- removed net N$71: J6.13, JA5.26, JA5.27, JA5.28, JA5.29
- removed net N$72: J6.15, JA5.30, JA5.31, JA5.32, JA5.33
- removed net N$73: J6.16, JA5.37, JA5.38, JA5.39, JA5.40
- removed net N$74: J6.14, JA5.41, JA5.42, JA5.43, JA5.44
- removed net N$75: J6.12, JA5.45, JA5.46, JA5.47, JA5.48
- removed net N$76: J6.10, JA5.49, JA5.50, JA5.51, JA5.52
- removed net N$77: J6.8, JA5.53, JA5.54, JA5.55, JA5.56
- removed net N$78: J6.6, JA5.57, JA5.58, JA5.59, JA5.60
- removed net N$79: J6.4, JA5.61, JA5.62, JA5.63, JA5.64
- removed net N$80: J6.2, JA5.65, JA5.66, JA5.67, JA5.68
- removed net N$97: J8.1, JA7.2, JA7.3, JA7.4, JA7.5
- removed net N$98: J8.3, JA7.6, JA7.7, JA7.8, JA7.9
- removed net N$99: J8.5, JA7.10, JA7.11, JA7.12, JA7.13
- new net N$113: J11.2, J11.3, J11.4, J11.5, J12.1
- new net N$114: J11.6, J11.7, J11.8, J11.9, J12.3
- new net N$115: J11.10, J11.11, J11.12, J11.13, J12.5
- new net N$116: J11.14, J11.15, J11.16, J11.17, J12.7
- new net N$117: J11.18, J11.19, J11.20, J11.21, J12.9
- new net N$118: J11.22, J11.23, J11.24, J11.25, J12.11
- new net N$119: J11.26, J11.27, J11.28, J11.29, J12.13
- new net N$120: J11.30, J11.31, J11.32, J11.33, J12.15
- new net N$121: J11.37, J11.38, J11.39, J11.40, J12.16
- new net N$122: J11.41, J11.42, J11.43, J11.44, J12.14
- new net N$123: J11.45, J11.46, J11.47, J11.48, J12.12
- new net N$124: J11.49, J11.50, J11.51, J11.52, J12.10
- new net N$125: J11.53, J11.54, J11.55, J11.56, J12.8
- new net N$126: J11.57, J11.58, J11.59, J11.60, J12.6
- new net N$127: J11.61, J11.62, J11.63, J11.64, J12.4
- new net N$128: J11.65, J11.66, J11.67, J11.68, J12.2
- new net N$49: J3.2, J3.3, J3.4, J3.5, J5.1
- new net N$50: J3.6, J3.7, J3.8, J3.9, J5.3
- new net N$51: J3.10, J3.11, J3.12, J3.13, J5.5
- new net N$52: J3.14, J3.15, J3.16, J3.17, J5.7
- new net N$53: J3.18, J3.19, J3.20, J3.21, J5.9
- new net N$54: J3.22, J3.23, J3.24, J3.25, J5.11
- new net N$55: J3.26, J3.27, J3.28, J3.29, J5.13
- new net N$56: J3.30, J3.31, J3.32, J3.33, J5.15
- new net N$57: J3.37, J3.38, J3.39, J3.40, J5.16
- new net N$58: J3.41, J3.42, J3.43, J3.44, J5.14
- new net N$59: J3.45, J3.46, J3.47, J3.48, J5.12
- new net N$60: J3.49, J3.50, J3.51, J3.52, J5.10
- new net N$61: J3.53, J3.54, J3.55, J3.56, J5.8
- new net N$62: J3.57, J3.58, J3.59, J3.60, J5.6
- new net N$63: J3.61, J3.62, J3.63, J3.64, J5.4
- new net N$64: J3.65, J3.66, J3.67, J3.68, J5.2
- new net N$81: J10.1, J9.2, J9.3, J9.4, J9.5
- new net N$82: J10.3, J9.6, J9.7, J9.8, J9.9
- new net N$83: J10.5, J9.10, J9.11, J9.12, J9.13
- new net N$84: J10.7, J9.14, J9.15, J9.16, J9.17
- new net N$85: J10.9, J9.18, J9.19, J9.20, J9.21
- new net N$86: J10.11, J9.22, J9.23, J9.24, J9.25
- new net N$87: J10.13, J9.26, J9.27, J9.28, J9.29
- new net N$88: J10.15, J9.30, J9.31, J9.32, J9.33
- new net N$89: J10.16, J9.37, J9.38, J9.39, J9.40
- new net N$90: J10.14, J9.41, J9.42, J9.43, J9.44
- new net N$91: J10.12, J9.45, J9.46, J9.47, J9.48
- new net N$92: J10.10, J9.49, J9.50, J9.51, J9.52
- new net N$93: J10.8, J9.53, J9.54, J9.55, J9.56
- new net N$94: J10.6, J9.57, J9.58, J9.59, J9.60
- new net N$95: J10.4, J9.61, J9.62, J9.63, J9.64
- new net N$96: J10.2, J9.65, J9.66, J9.67, J9.68
- net AGND: now also J1.70, J11.1, J11.70, J3.1, J3.70, J4.1, J4.69, J4.M1, J4.M2, J4.M3, J4.M4, J6.1, J6.2, J6.3, J9.1, J9.70, TP1.TP, TP2.TP, TP3.TP, TP4.TP; no longer J1.69, J1.M1, J1.M2, J1.M3, J1.M4, J5.1, J5.2, J5.3, JA1.1, JA1.70, JA3.1, JA3.70, JA5.1, JA5.70, JA7.1, JA7.70
- net N$1: now also J4.53, J4.54, J4.55, J4.56, J8.10; no longer J1.53, J1.54, J1.55, J1.56, J4.10
- net N$10: now also J4.26, J4.27, J4.28, J4.29, J8.3; no longer J1.26, J1.27, J1.28, J1.29, J4.3
- net N$11: now also J4.30, J4.31, J4.32, J4.33, J8.1; no longer J1.30, J1.31, J1.32, J1.33, J4.1
- net N$12: now also J4.37, J4.38, J4.39, J4.40, J8.2; no longer J1.37, J1.38, J1.39, J1.40, J4.2
- net N$13: now also J4.41, J4.42, J4.43, J4.44, J8.4; no longer J1.41, J1.42, J1.43, J1.44, J4.4
- net N$14: now also J4.45, J4.46, J4.47, J4.48, J8.6; no longer J1.45, J1.46, J1.47, J1.48, J4.6
- net N$15: now also J4.49, J4.50, J4.51, J4.52, J8.8; no longer J1.49, J1.50, J1.51, J1.52, J4.8
- net N$2: now also J4.57, J4.58, J4.59, J4.60, J8.12; no longer J1.57, J1.58, J1.59, J1.60, J4.12
- net N$3: now also J4.61, J4.62, J4.63, J4.64, J8.14; no longer J1.61, J1.62, J1.63, J1.64, J4.14
- net N$32: now also J4.6, J4.7, J4.8, J4.9, J8.13; no longer J1.6, J1.7, J1.8, J1.9, J4.13
- net N$33: now also J1.2, J1.3, J1.4, J1.5, J2.1; no longer J3.1, JA3.2, JA3.3, JA3.4, JA3.5
- net N$34: now also J1.6, J1.7, J1.8, J1.9, J2.3; no longer J3.3, JA3.6, JA3.7, JA3.8, JA3.9
- net N$35: now also J1.10, J1.11, J1.12, J1.13, J2.5; no longer J3.5, JA3.10, JA3.11, JA3.12, JA3.13
- net N$36: now also J1.14, J1.15, J1.16, J1.17, J2.7; no longer J3.7, JA3.14, JA3.15, JA3.16, JA3.17
- net N$37: now also J1.18, J1.19, J1.20, J1.21, J2.9; no longer J3.9, JA3.18, JA3.19, JA3.20, JA3.21
- net N$38: now also J1.22, J1.23, J1.24, J1.25, J2.11; no longer J3.11, JA3.22, JA3.23, JA3.24, JA3.25
- net N$39: now also J1.26, J1.27, J1.28, J1.29, J2.13; no longer J3.13, JA3.26, JA3.27, JA3.28, JA3.29
- net N$4: now also J4.2, J4.3, J4.4, J4.5, J8.15; no longer J1.2, J1.3, J1.4, J1.5, J4.15
- net N$40: now also J1.30, J1.31, J1.32, J1.33, J2.15; no longer J3.15, JA3.30, JA3.31, JA3.32, JA3.33
- net N$41: now also J1.37, J1.38, J1.39, J1.40, J2.16; no longer J3.16, JA3.37, JA3.38, JA3.39, JA3.40
- net N$42: now also J1.41, J1.42, J1.43, J1.44, J2.14; no longer J3.14, JA3.41, JA3.42, JA3.43, JA3.44
- net N$43: now also J1.45, J1.46, J1.47, J1.48, J2.12; no longer J3.12, JA3.45, JA3.46, JA3.47, JA3.48
- net N$44: now also J1.49, J1.50, J1.51, J1.52, J2.10; no longer J3.10, JA3.49, JA3.50, JA3.51, JA3.52
- net N$45: now also J1.53, J1.54, J1.55, J1.56, J2.8; no longer J3.8, JA3.53, JA3.54, JA3.55, JA3.56
- net N$46: now also J1.57, J1.58, J1.59, J1.60, J2.6; no longer J3.6, JA3.57, JA3.58, JA3.59, JA3.60
- net N$47: now also J1.61, J1.62, J1.63, J1.64, J2.4; no longer J3.4, JA3.61, JA3.62, JA3.63, JA3.64
- net N$48: now also J1.65, J1.66, J1.67, J1.68, J2.2; no longer J3.2, JA3.65, JA3.66, JA3.67, JA3.68
- net N$5: now also J4.65, J4.66, J4.67, J4.68, J8.16; no longer J1.65, J1.66, J1.67, J1.68, J4.16
- net N$6: now also J4.10, J4.12, J4.13, J8.11; no longer J1.10, J1.11, J1.12, J1.13
- net N$7: now also J4.14, J4.15, J4.16, J4.17, J8.9; no longer J1.14, J1.15, J1.16, J1.17, J4.9
- net N$8: now also J4.18, J4.19, J4.20, J4.21, J8.7; no longer J1.18, J1.19, J1.20, J1.21, J4.7
- net N$9: now also J4.22, J4.23, J4.24, J4.25, J8.5; no longer J1.22, J1.23, J1.24, J1.25, J4.5
Other:
- moved on the sheet: J2, J7, J8
