File: lighthouse-booster/lighthouse-booster.sch (EAGLE design)
At the start: 326 parts, among them J1 AYF532835, Q1 BSZ034N04LSATMA1, Q2 BSZ034N04LSATMA1, Q3 BSZ034N04LSATMA1, Q4 BSZ034N04LSATMA1, Q5 BSZ034N04LSATMA1, Q6 BSZ034N04LSATMA1, Q7 BSZ034N04LSATMA1, Q8 BSZ034N04LSATMA1, U1 UCC27517DBVR, U2 UCC27517DBVR, U3 UCC27517DBVR, U4 UCC27517DBVR, U5 UCC27517DBVR, U6 UCC27517DBVR, U7 UCC27517DBVR, U8 UCC27517DBVR

Commit message: Lighthouse-booster Rev. 1.1
- Minor fixes to version 1.0 after testing
- Replaced 0 ohm jumpers between gate driver and gate with 47 kOhm
pulldowns to prevent possible DC damage to LEDs when board is not
driven
- Decrease current limit resistors to 360 mOhm. This should give us 5
Amps per LED string after empirical testing
- Fixed mis-aligned guide hole placement
Parts:
- C1, C10, C11, C12, C13, C14, C15, C16, C17, C18, C19, C2, C20, C21, C22, C23, C24, C25, C26, C27, C28, C29, C3, C30, C37, C38, C39, C4, C40, C41, C42, C43, C44, C45, C46, C47, C48, C49, C5, C50, C51, C52, C53, C54, C55, C56, C57, C58, C59, C6, C60, C61, C62, C63, C64, C65, C66, C7, C73, C74, C75, C76, C77, C78, C79, C8, C80, C81, C82, C83, C84, C85, C86, C87, C88, C89, C9, C90, C91, C92: value 6.8uF -> 22uF
- R1, R10, R11, R12, R13, R14, R15, R16, R17, R18, R19, R2, R20, R21, R22, R23, R24, R25, R26, R27, R28, R29, R3, R30, R34, R35, R36, R37, R38, R39, R4, R40, R41, R42, R43, R44, R45, R46, R47, R48, R49, R5, R50, R51, R52, R53, R54, R55, R56, R57, R58, R59, R6, R60, R61, R62, R63, R67, R68, R69, R7, R70, R71, R72, R73, R74, R75, R76, R77, R78, R79, R8, R80, R81, R82, R83, R84, R85, R86, R9: value 0.75 -> 0.36
- R31, R32, R33, R64, R65, R66, R87, R88: value 0 -> 47k
Connections:
- removed net N$120: Q5.G, R65.2
- removed net N$143: Q6.G, R66.2
- removed net N$166: Q8.G, R88.2
- removed net N$22: Q4.G, R64.2
- removed net N$5: Q7.G, R87.2
- removed net N$51: Q1.G, R31.2
- removed net N$74: Q2.G, R32.2
- removed net N$97: Q3.G, R33.2
- net GND: now also R31.2, R32.2, R33.2, R64.2, R65.2, R66.2, R87.2, R88.2
- net N$110: now also Q3.G
- net N$133: now also Q5.G
- net N$156: now also Q6.G
- net N$179: now also Q8.G
- net N$23: now also Q7.G
- net N$41: now also Q4.G
- net N$64: now also Q1.G
- net N$87: now also Q2.G
Other:
- moved on the sheet: R31, R32, R33, R64, R65, R66, R87, R88

Commit message: lighthouse-booster rev 1.1
- Updates after testing revision 1.0
- Added sychrnonous load switch to decouple the array from main 12V
power during pulses so that the motor rail is loaded
- Some keepout fixes so it actually fits flat on the platform
- Other small stuff
Parts:
- removed R20: 0.36, jonnew:R_0805T
- added C101, C102: 22uF, jonnew:C_0805T
- added Q9: BSZ034N04LSATMA1, jonnew:N-MOSFET_TSDSON-8
- added R89, R90: 0.36, jonnew:R_0805T
- added TP1, TP2: (no value), jonnew:TPTP12R
- added U9: UCC27517DBVR, jonnew:UCC27517_SOT
- C100, C32, C68, C98: value 10nF -> 22uF; device jonnew:C_0402T -> jonnew:C_0805T
- C11: value 22uF -> 4.7uF; device jonnew:C_0805T -> jonnew:C_0603T
- C14, C3, C4: value 22uF -> 0.1uF; device jonnew:C_0805T -> jonnew:C_0402T
- C25, C28, C29, C30: value 22uF -> 2.2mF; device jonnew:C_0805T -> jonnew:C-POL_C5MMA-SMD
- C31, C33, C67, C69, C97, C99: value 0.1uF -> 22uF; device jonnew:C_0402T -> jonnew:C_0805T
- C34, C36, C70, C72: value 10nF -> 0.1uF
- C40, C41, C42, C7, C76, C77, C78, C8: value 22uF -> 10nF; device jonnew:C_0805T -> jonnew:C_0402T
- C93, C94, C95, C96: value 47uF -> 22uF; device jonnew:C_1210 -> jonnew:C_0805T
- D25: value (none) -> LTST-C19HE1WT; device jonnew:LED_LUXEON-3.7MM -> jonnew:LED-RGB_LTST
- D91: value LTST-C19HE1WT -> (none); device jonnew:LED-RGB_LTST -> jonnew:LED_LUXEON-3.7MM
- Q1: value BSZ034N04LSATMA1 -> Si7655ADN; device jonnew:N-MOSFET_TSDSON-8 -> jonnew:P-MOSFET_POWERPACK-1212-8
- R18, R19, R49, R50, R51, R82, R83, R84: value 0.36 -> 10; device jonnew:R_0805T -> jonnew:R_0402T
- R31, R32, R33, R64, R65, R66, R87, R88: value 47k -> 0.36; device jonnew:R_0402T -> jonnew:R_0805T
- R7: value 0.36 -> 10k; device jonnew:R_0805T -> jonnew:R_0402T
- U3: value UCC27517DBVR -> LTC1693-5; device jonnew:UCC27517_SOT -> jonnew:LTC1693_MSOP
Connections:
- new net N$22: R82.1, U7.OUT
- new net N$24: R50.1, U4.OUT
- new net N$25: Q2.G, R18.2
- new net N$26: R19.1, U2.OUT
- new net N$27: Q5.G, R51.2
- new net N$28: R83.1, U8.OUT
- new net N$42: R84.1, U9.OUT
- new net N$46: C11.1, C14.1, J1.10, J1.11, J1.2, J1.3, J1.4, J1.5, J1.6, J1.7, J1.8, J1.9, Q1.S, U3.PHA, U3.VCC
- new net N$5: R49.1, U6.OUT
- new net N$51: Q1.D, TP1.TP
- new net N$66: Q1.G, U3.OUT
- net +12V: now also C100.1, C101.1, C102.1, C16.2, C25.+, C28.+, C29.+, C30.+, C31.2, C32.2, C33.2, C67.2, C68.2, C69.2, C82.2, C83.2, C84.2, C85.2, C86.2, C97.1, C98.1, C99.1, D104.A, D107.A, D110.A, D113.A, D116.A, D119.A, D16.A, D19.A, D22.A, D26.A, D29.A, D32.A, D35.A, D38.A, D41.A, D44.A, D62.A, D65.A, D68.A, D71.A, D74.A, D77.A, D80.A, D83.A, D86.A, D89.A, TP2.TP; no longer C11.2, C14.2, C16.1, C25.1, C28.1, C29.1, C3.2, C30.1, C4.2, C40.2, C41.2, C42.2, C7.2, C76.2, C77.2, C78.2, C8.2, C82.1, C83.1, C84.1, C85.1, C86.1, D100.A, D11.A, D12.A, D14.A, D15.A, D2.A, D3.A, D46.A, D48.A, D49.A, D5.A, D51.A, D52.A, D54.A, D55.A, D57.A, D58.A, D6.A, D60.A, D8.A, D9.A, D93.A, D94.A, D96.A, D97.A, D99.A, J1.10, J1.11, J1.2, J1.3, J1.4, J1.5, J1.6, J1.7, J1.8, J1.9
- net +5V0: now also C3.1, C4.1, C40.1, C41.1, C42.1, C7.1, C76.1, C77.1, C78.1, C8.1, D25.A, U9.VDD; no longer C100.1, C31.1, C32.1, C33.1, C67.1, C68.1, C69.1, C97.1, C98.1, C99.1, D91.A, U3.VDD
- net BLUE_C: now also D25.CB; no longer D91.CB
- net GND: now also C101.2, C102.2, C11.2, C14.2, C16.1, C25.-, C28.-, C29.-, C3.2, C30.-, C31.1, C32.1, C33.1, C4.2, C40.2, C41.2, C42.2, C67.1, C68.1, C69.1, C7.2, C76.2, C77.2, C78.2, C8.2, C82.1, C83.1, C84.1, C85.1, C86.1, Q9.S, R7.1, U9.GND, U9.IN-; no longer C11.1, C14.1, C16.2, C25.2, C28.2, C29.2, C3.1, C30.2, C31.2, C32.2, C33.2, C4.1, C40.1, C41.1, C42.1, C67.2, C68.2, C69.2, C7.1, C76.1, C77.1, C78.1, C8.1, C82.2, C83.2, C84.2, C85.2, C86.2, Q1.S, R31.2, R32.2, R33.2, R64.2, R65.2, R66.2, R87.2, R88.2, U3.IN-
- net GREEN_C: now also D25.CG; no longer D91.CG
- net N$1: now also D76.C, R54.2, R57.2; no longer D116.C, R75.2, R76.2
- net N$10: now also D65.C, D66.A; no longer D105.A, D95.C
- net N$100: now also D104.C, D105.A; no longer D14.C, D29.A
- net N$101: now also D97.C, R70.2, R73.2; no longer D43.C, R25.2, R26.2
- net N$102: now also D96.C, D97.A; no longer D28.C, D43.A
- net N$103: now also D95.C, D96.A; no longer D13.C, D28.A
- net N$104: now also D88.C, R64.2, R67.2; no longer D42.C, R23.2, R24.2
- net N$105: now also D87.C, D88.A; no longer D27.C, D42.A
- net N$106: now also D86.C, D87.A; no longer D12.C, D27.A
- net N$107: now also D79.C, R58.2, R61.2; no longer D41.C, R21.2, R22.2
- net N$108: now also D78.C, D79.A; no longer D26.C, D41.A
- net N$109: now also D77.C, D78.A; no longer D11.C, D26.A
- net N$11: now also D31.C, R22.2, R24.2; no longer D80.C, R42.2, R43.2
- net N$110: now also Q7.G, R82.2; no longer Q3.G, R33.1, U3.OUT
- net N$116: now also D73.C, R56.2; no longer D85.C, R52.2
- net N$117: now also D72.C, D73.A; no longer D70.C, D85.A
- net N$118: now also D71.C, D72.A; no longer D55.C, D70.A
- net N$119: now also R26.1, R29.1, R32.1, R35.1, R38.1, R41.1, R56.1; no longer R45.1, R46.1, R48.1, R49.1, R50.1, R51.1, R52.1
- net N$12: now also D56.C, D57.A; no longer D104.A, D94.C
- net N$121: now also D64.C, R44.2, R47.2; no longer D84.C, R50.2, R51.2
- net N$122: now also D63.C, D64.A; no longer D69.C, D84.A
- net N$123: now also D62.C, D63.A; no longer D54.C, D69.A
- net N$124: now also D55.C, R38.2, R41.2; no longer D83.C, R48.2, R49.2
- net N$125: now also D54.C, D55.A; no longer D68.C, D83.A
- net N$126: now also D54.A; no longer D68.A
- net N$127: now also D46.C, R32.2, R35.2; no longer D82.C, R46.2, R47.2
- net N$128: now also D45.C, D46.A; no longer D67.C, D82.A
- net N$129: now also D44.C, D45.A; no longer D52.C, D67.A
- net N$13: now also D49.C, R33.2, R36.2; no longer D113.C, R69.2, R70.2
- net N$130: now also D37.C, R26.2, R29.2; no longer D81.C, R44.2, R45.2
- net N$131: now also D36.C, D37.A; no longer D66.C, D81.A
- net N$132: now also D35.C, D36.A; no longer D51.C, D66.A
- net N$133: now also R51.1; no longer Q5.G, R65.1
- net N$139: now also D118.C, R86.2, R89.2; no longer D90.C, R62.2, R63.2
- net N$14: now also D48.C, D49.A; no longer D103.C, D113.A
- net N$140: now also D117.C, D118.A; no longer D75.C, D90.A
- net N$141: now also D116.C, D117.A; no longer D60.C, D75.A
- net N$142: now also Q8.D, R65.1, R68.1, R71.1, R74.1, R77.1, R80.1, R86.1, R89.1; no longer Q6.D, R54.1, R55.1, R56.1, R57.1, R58.1, R60.1, R61.1, R63.1
- net N$144: now also D109.C, R77.2, R80.2; no longer D89.C, R60.2, R61.2
- net N$145: now also D108.C, D109.A; no longer D74.C, D89.A
- net N$146: now also D107.C, D108.A; no longer D59.C, D74.A
- net N$147: now also D100.C, R71.2, R74.2; no longer D88.C, R58.2, R59.2
- net N$148: now also D100.A, D99.C; no longer D73.C, D88.A
- net N$149: now also D98.C, D99.A; no longer D58.C, D73.A
- net N$15: now also D47.C, D48.A; no longer D103.A, D93.C
- net N$150: now also D91.C, R65.2, R68.2; no longer D87.C, R56.2, R57.2
- net N$151: now also D90.C, D91.A; no longer D72.C, D87.A
- net N$152: now also D89.C, D90.A; no longer D57.C, D72.A
- net N$153: now also D82.C, R59.2, R62.2; no longer D86.C, R54.2, R55.2
- net N$154: now also D81.C, D82.A; no longer D71.C, D86.A
- net N$155: now also D80.C, D81.A; no longer D56.C, D71.A
- net N$156: now also Q8.G, R83.2; no longer Q6.G, R66.1, U6.OUT
- net N$16: now also D40.C, R27.2, R30.2; no longer D112.C, R67.2, R68.2
- net N$162: now also R87.2, R90.2; no longer R85.2, R86.2
- net N$163: now also D120.C; no longer D111.C
- net N$164: now also D119.C, D120.A; no longer D101.C, D111.A
- net N$165: now also Q9.D, R60.1, R63.1, R66.1, R69.1, R72.1, R75.1, R87.1, R90.1; no longer Q8.D, R77.1, R79.1, R80.1, R82.1, R83.1, R84.1, R85.1, R86.1
- net N$167: now also D112.C, R78.2, R81.2; no longer D120.C, R83.2, R84.2
- net N$168: now also D111.C, D112.A; no longer D110.C, D120.A
- net N$169: now also D110.C, D111.A; no longer D100.C, D110.A
- net N$17: now also D39.C, D40.A; no longer D102.C, D112.A
- net N$170: now also D103.C, R72.2, R75.2; no longer D119.C, R81.2, R82.2
- net N$171: now also D102.C, D103.A; no longer D109.C, D119.A
- net N$172: now also D101.C, D102.A; no longer D109.A, D99.C
- net N$173: now also D94.C, R66.2, R69.2; no longer D118.C, R79.2, R80.2
- net N$174: now also D93.C, D94.A; no longer D108.C, D118.A
- net N$175: now also D92.C, D93.A; no longer D108.A, D98.C
- net N$176: now also D85.C, R60.2, R63.2; no longer D117.C, R77.2, R78.2
- net N$177: now also D84.C, D85.A; no longer D107.C, D117.A
- net N$178: now also D83.C, D84.A; no longer D107.A, D97.C
- net N$179: now also Q9.G, R84.2; no longer Q8.G, R88.1, U8.OUT
- net N$18: now also D38.C, D39.A; no longer D102.A, D92.C
- net N$19: now also D30.C, D31.A; no longer D65.C, D80.A
- net N$2: now also D75.C, D76.A; no longer D106.C, D116.A
- net N$20: now also D29.C, D30.A; no longer D50.C, D65.A
- net N$21: now also Q3.D, R11.1, R13.1, R15.1, R17.1, R2.1, R22.1, R24.1, R4.1, R6.1, R9.1; no longer Q4.D, R34.1, R35.1, R36.1, R37.1, R38.1, R39.1, R40.1, R41.1, R42.1, R43.1
- net N$23: now also Q6.G, R49.2; no longer Q7.G, R87.1, U7.OUT
- net N$29: now also D24.C, R15.2, R17.2; no longer D79.C, R40.2, R41.2
- net N$3: now also D74.C, D75.A; no longer D106.A, D96.C
- net N$30: now also D23.C, D24.A; no longer D64.C, D79.A
- net N$31: now also D22.C, D23.A; no longer D49.C, D64.A
- net N$32: now also D18.C, R11.2, R13.2; no longer D78.C, R38.2, R39.2
- net N$33: now also D17.C, D18.A; no longer D63.C, D78.A
- net N$34: now also D16.C, D17.A; no longer D48.C, D63.A
- net N$35: now also D12.C, R6.2, R9.2; no longer D77.C, R36.2, R37.2
- net N$36: now also D11.C, D12.A; no longer D62.C, D77.A
- net N$37: now also D10.C, D11.A; no longer D47.C, D62.A
- net N$38: now also D6.C, R2.2, R4.2; no longer D76.C, R34.2, R35.2
- net N$39: now also D5.C, D6.A; no longer D61.C, D76.A
- net N$4: now also Q6.D, R27.1, R30.1, R33.1, R36.1, R39.1, R42.1, R45.1, R48.1, R54.1, R57.1; no longer Q7.D, R67.1, R68.1, R69.1, R70.1, R71.1, R72.1, R73.1, R74.1, R75.1, R76.1
- net N$40: now also D4.C, D5.A; no longer D46.C, D61.A
- net N$41: now also Q3.G, R19.2; no longer Q4.G, R64.1, U4.OUT
- net N$47: now also D28.C, R21.2, R23.2; no longer D35.C, R10.2, R9.2
- net N$48: now also D27.C, D28.A; no longer D20.C, D35.A
- net N$49: now also D26.C, D27.A; no longer D20.A, D5.C
- net N$50: now also Q2.D, R12.1, R14.1, R16.1, R21.1, R23.1; no longer Q1.D, R2.1, R4.1, R6.1, R7.1, R9.1
- net N$52: now also D21.C, R14.2, R16.2; no longer D34.C, R7.2, R8.2
- net N$53: now also D20.C, D21.A; no longer D19.C, D34.A
- net N$54: now also D19.C, D20.A; no longer D19.A, D4.C
- net N$55: now also D15.C, R10.2, R12.2; no longer D33.C, R5.2, R6.2
- net N$56: now also D14.C, D15.A; no longer D18.C, D33.A
- net N$57: now also D13.C, D14.A; no longer D18.A, D3.C
- net N$58: now also D9.C, R5.2, R8.2; no longer D32.C, R3.2, R4.2
- net N$59: now also D8.C, D9.A; no longer D17.C, D32.A
- net N$6: now also D58.C, R39.2, R42.2; no longer D114.C, R71.2, R72.2
- net N$60: now also D7.C, D8.A; no longer D17.A, D2.C
- net N$61: now also D3.C, R3.2; no longer D31.C, R2.2
- net N$62: now also D2.C, D3.A; no longer D16.C, D31.A
- net N$63: now also D2.A; no longer D16.A
- net N$64: now also R18.1; no longer Q1.G, R31.1
- net N$7: now also D57.C, D58.A; no longer D104.C, D114.A
- net N$70: now also D70.C, R52.2, R55.2; no longer D40.C, R19.2, R20.2
- net N$71: now also D69.C, D70.A; no longer D25.C, D40.A
- net N$72: now also D68.C, D69.A; no longer D10.C, D25.A
- net N$73: now also Q4.D, R25.1, R28.1, R31.1, R34.1, R37.1, R40.1, R43.1, R46.1, R52.1, R55.1; no longer Q2.D, R11.1, R12.1, R13.1, R14.1, R15.1, R16.1, R17.1, R18.1, R19.1, R20.1
- net N$75: now also D61.C, R43.2, R46.2; no longer D39.C, R17.2, R18.2
- net N$76: now also D60.C, D61.A; no longer D24.C, D39.A
- net N$77: now also D59.C, D60.A; no longer D24.A, D9.C
- net N$78: now also D52.C, R37.2, R40.2; no longer D38.C, R15.2, R16.2
- net N$79: now also D51.C, D52.A; no longer D23.C, D38.A
- net N$8: now also D67.C, R45.2, R48.2; no longer D115.C, R73.2, R74.2
- net N$80: now also D50.C, D51.A; no longer D23.A, D8.C
- net N$81: now also D43.C, R31.2, R34.2; no longer D37.C, R13.2, R14.2
- net N$82: now also D42.C, D43.A; no longer D22.C, D37.A
- net N$83: now also D41.C, D42.A; no longer D22.A, D7.C
- net N$84: now also D34.C, R25.2, R28.2; no longer D36.C, R11.2, R12.2
- net N$85: now also D33.C, D34.A; no longer D21.C, D36.A
- net N$86: now also D32.C, D33.A; no longer D21.A, D6.C
- net N$87: now also Q4.G, R50.2; no longer Q2.G, R32.1, U2.OUT
- net N$9: now also D66.C, D67.A; no longer D105.C, D115.A
- net N$93: now also D115.C, R85.2, R88.2; no longer D45.C, R29.2, R30.2
- net N$94: now also D114.C, D115.A; no longer D30.C, D45.A
- net N$95: now also D113.C, D114.A; no longer D15.C, D30.A
- net N$96: now also Q7.D, R58.1, R61.1, R64.1, R67.1, R70.1, R73.1, R76.1, R79.1, R85.1, R88.1; no longer Q3.D, R21.1, R22.1, R23.1, R24.1, R25.1, R26.1, R27.1, R28.1, R29.1, R30.1
- net N$98: now also D106.C, R76.2, R79.2; no longer D44.C, R27.2, R28.2
- net N$99: now also D105.C, D106.A; no longer D29.C, D44.A
- net RED_C: now also D25.CR; no longer D91.CR
- net SYNC: now also R7.2, U3.IN, U9.IN+; no longer U3.IN+
Other:
- note added: "R20 0.1, 1W"
- moved on the sheet: C1, C10, C100, C11, C12, C13, C14, C15, C16, C17, C18, C19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

Commit message: Lighthouse booster rev. 1.2
- Added a monostable vibrator to the high-side power-switch trigger
circuit in order to prevent the system 12V from seeing any of the LED
circuit when the LEDs are active.
- This circuit re-triggers on every incoming sync pulse so that a
perfect envelope is formed to disconnected the system 12V from the LED
12V whenever a sync train is being applied
Parts:
- removed C102: 22uF, jonnew:C_0805T
- added R20: 10, jonnew:R_0402T
- added U10: UCC27517DBVR, jonnew:UCC27517_SOT
- C10, C33, C69: value 22uF -> 0.1uF; device jonnew:C_0805T -> jonnew:C_0402T
- C11: value 4.7uF -> 22uF; device jonnew:C_0603T -> jonnew:C_0805T
- C14, C36, C72: value 0.1uF -> 22uF; device jonnew:C_0402T -> jonnew:C_0805T
- C15: value 22uF -> 100pF; device jonnew:C_0805T -> jonnew:C_0402T
- C25, C30: value 2.2mF -> 22uF; device jonnew:C-POL_C5MMA-SMD -> jonnew:C_0805T
- C39, C75, C9: value 22uF -> 10nF; device jonnew:C_0805T -> jonnew:C_0402T
- C42, C7, C78: value 10nF -> 22uF; device jonnew:C_0402T -> jonnew:C_0805T
- C5: value 22uF -> 4.7uF; device jonnew:C_0805T -> jonnew:C_0603T
- D25: value LTST-C19HE1WT -> (none); device jonnew:LED-RGB_LTST -> jonnew:LED_LUXEON-3.7MM
- D31: value (none) -> LTST-C19HE1WT; device jonnew:LED_LUXEON-3.7MM -> jonnew:LED-RGB_LTST
- Q1: value Si7655ADN -> BSZ034N04LSATMA1; device jonnew:P-MOSFET_POWERPACK-1212-8 -> jonnew:N-MOSFET_TSDSON-8
- Q3: value BSZ034N04LSATMA1 -> Si7655ADN; device jonnew:N-MOSFET_TSDSON-8 -> jonnew:P-MOSFET_POWERPACK-1212-8
- R10, R5: value 0.36 -> 10k; device jonnew:R_0805T -> jonnew:R_0402T
- R18: value 10 -> 0.36; device jonnew:R_0402T -> jonnew:R_0805T
- R7: value 10k -> 0.36; device jonnew:R_0402T -> jonnew:R_0805T
- TP1, TP2: device jonnew:TPTP12R -> jonnew:TPTP18SQ
- U3: value LTC1693-5 -> SN74LVC1G123YZPR; device jonnew:LTC1693_MSOP -> jonnew:MONOSTABLE-MULTIVIBRATOR_DSBGA
- U4: value UCC27517DBVR -> LTC1693-5; device jonnew:UCC27517_SOT -> jonnew:LTC1693_MSOP
Connections:
- removed net N$19 (its old number): D30.C, D31.A
- removed net N$48 (its old number): D27.C, D28.A
- new net N$20: D28.C, D29.A
- new net N$43: C15.1, R10.2, U3.R/C
- new net N$44: U3.Q, U4.IN
- new net N$45: C15.2, U3.C
- new net N$49: D25.C, D26.A
- net +12V: now also C11.2, C14.2, C17.2, C25.1, C30.2, C36.2, C42.2, C51.1, C66.2, C7.2, C72.2, C78.2, C86.1, D25.A, D28.A; no longer C10.2, C102.1, C15.2, C17.1, C25.+, C30.+, C33.2, C39.2, C5.2, C51.2, C66.1, C69.2, C75.2, C86.2, C9.2, D26.A, D29.A
- net +5V0: now also C33.1, C39.1, C69.1, C75.1, C9.1, D31.A, R10.1, U10.VDD, U3.!CLR, U3.VCC; no longer C36.1, C42.1, C7.1, C72.1, C78.1, D25.A, U4.VDD
- net BLUE_C: now also D31.CB; no longer D25.CB
- net GND: now also C10.2, C11.1, C14.1, C17.1, C25.2, C30.1, C33.2, C36.1, C39.2, C42.1, C5.2, C51.2, C66.1, C69.2, C7.1, C72.1, C75.2, C78.1, C86.2, C9.2, Q1.S, R5.1, U10.GND, U10.IN-, U3.!A; no longer C10.1, C102.2, C11.2, C14.2, C15.1, C17.2, C25.-, C30.-, C33.1, C36.2, C39.1, C42.2, C5.1, C51.1, C66.2, C69.1, C7.2, C72.2, C75.1, C78.2, C86.1, C9.1, Q3.S, R7.1, U4.IN-
- net GREEN_C: now also D31.CG; no longer D25.CG
- net N$11: now also D30.C; no longer D31.C
- net N$133: now also U6.OUT; no longer U5.OUT
- net N$21: now also Q2.D, R12.1, R14.1, R16.1, R18.1, R7.1; no longer Q3.D, R11.1, R13.1, R15.1, R17.1, R6.1
- net N$22: now also U8.OUT; no longer U7.OUT
- net N$24: now also U3.B, U5.OUT; no longer U4.OUT
- net N$25: now also Q1.G, R19.2; no longer Q2.G, R18.2
- net N$26: now also R20.1; no longer R19.1
- net N$28: now also U9.OUT; no longer U8.OUT
- net N$29: now also R16.2, R18.2; no longer R15.2, R17.2
- net N$32: now also R12.2, R14.2; no longer R11.2, R13.2
- net N$35: now also R7.2; no longer R6.2
- net N$41: now also Q2.G, R20.2; no longer Q3.G, R19.2
- net N$42: now also U10.OUT; no longer U9.OUT
- net N$46: now also C10.1, C5.1, Q3.S, U4.PHA, U4.VCC; no longer C11.1, C14.1, Q1.S, U3.PHA, U3.VCC
- net N$47: now also D27.C; no longer D28.C
- net N$5: now also U7.OUT; no longer U6.OUT
- net N$50: now also Q1.D, R11.1, R13.1, R15.1, R17.1, R6.1; no longer Q2.D, R10.1, R12.1, R14.1, R16.1, R5.1
- net N$51: now also Q3.D; no longer Q1.D
- net N$52: now also R15.2, R17.2; no longer R14.2, R16.2
- net N$55: now also R11.2, R13.2; no longer R10.2, R12.2
- net N$58: now also R6.2; no longer R5.2
- net N$64: now also R19.1; no longer R18.1
- net N$66: now also Q3.G, U4.OUT; no longer Q1.G, U3.OUT
- net RED_C: now also D31.CR; no longer D25.CR
- net SYNC: now also R5.2, U10.IN+; no longer R7.2, U3.IN, U4.IN+
Other:
- note added: "CXX 6.8mF BZ05FB682ZSB Manually solder between two large pads on left side of bottom."
- note added: "R20 0.2, 1W"
- note removed: "R20 0.1, 1W"
- moved on the sheet: C10, C100, C101, C11, C12, C13, C14, C15, C16, C17, C18, C19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

Commit message: Added ferrites in line with LEDs in lighthouse booster
- Only 2 LEDs in series instead of 3 to prevent voltage drop
- Ferrites to prevent oscillation
Parts:
- removed D1, D10, D101, D104, D107, D110, D113, D116, D119, D13, D16, D19, D22, D25, D28, D32, D35, D38, D4, D41, D44, D47, D50, D53, D56, D59, D62, D65, D68, D7, D71, D74, D77, D80, D83, D86, D89, D92, D95, D98: (no value), jonnew:LED_LUXEON-3.7MM
- added L1, L10, L11, L12, L13, L14, L15, L16, L17, L18, L19, L2, L20, L21, L22, L23, L24, L25, L26, L27, L28, L29, L3, L30, L31, L32, L33, L34, L35, L36, L37, L38, L39, L4, L40, L5, L6, L7, L8, L9: (no value), jonnew:L_0805T
Connections:
- net +12V: now also L1.1, L10.1, L11.1, L12.1, L13.1, L14.1, L15.1, L16.1, L17.1, L18.1, L19.1, L2.1, L20.1, L21.1, L22.1, L23.1, L24.1, L25.1, L26.1, L27.1, L28.1, L29.1, L3.1, L30.1, L31.1, L32.1, L33.1, L34.1, L35.1, L36.1, L37.1, L38.1, L39.1, L4.1, L40.1, L5.1, L6.1, L7.1, L8.1, L9.1; no longer D1.A, D10.A, D101.A, D104.A, D107.A, D110.A, D113.A, D116.A, D119.A, D13.A, D16.A, D19.A, D22.A, D25.A, D28.A, D32.A, D35.A, D38.A, D4.A, D41.A, D44.A, D47.A, D50.A, D53.A, D56.A, D59.A, D62.A, D65.A, D68.A, D7.A, D71.A, D74.A, D77.A, D80.A, D83.A, D86.A, D89.A, D92.A, D95.A, D98.A
- net N$10: now also L34.2; no longer D65.C
- net N$100: now also L14.2; no longer D104.C
- net N$103: now also L13.2; no longer D95.C
- net N$106: now also L12.2; no longer D86.C
- net N$109: now also L11.2; no longer D77.C
- net N$118: now also L25.2; no longer D71.C
- net N$12: now also L33.2; no longer D56.C
- net N$123: now also L24.2; no longer D62.C
- net N$126: now also L23.2; no longer D53.C
- net N$129: now also L22.2; no longer D44.C
- net N$132: now also L21.2; no longer D35.C
- net N$141: now also L30.2; no longer D116.C
- net N$146: now also L29.2; no longer D107.C
- net N$149: now also L28.2; no longer D98.C
- net N$15: now also L32.2; no longer D47.C
- net N$152: now also L27.2; no longer D89.C
- net N$155: now also L26.2; no longer D80.C
- net N$164: now also L40.2; no longer D119.C
- net N$169: now also L39.2; no longer D110.C
- net N$172: now also L38.2; no longer D101.C
- net N$175: now also L37.2; no longer D92.C
- net N$178: now also L36.2; no longer D83.C
- net N$18: now also L31.2; no longer D38.C
- net N$20: now also L20.2; no longer D28.C
- net N$3: now also L35.2; no longer D74.C
- net N$31: now also L19.2; no longer D22.C
- net N$34: now also L18.2; no longer D16.C
- net N$37: now also L17.2; no longer D10.C
- net N$40: now also L16.2; no longer D4.C
- net N$49: now also L5.2; no longer D25.C
- net N$54: now also L4.2; no longer D19.C
- net N$57: now also L3.2; no longer D13.C
- net N$60: now also L2.2; no longer D7.C
- net N$63: now also L1.2; no longer D1.C
- net N$72: now also L10.2; no longer D68.C
- net N$77: now also L9.2; no longer D59.C
- net N$80: now also L8.2; no longer D50.C
- net N$83: now also L7.2; no longer D41.C
- net N$86: now also L6.2; no longer D32.C
- net N$95: now also L15.2; no longer D113.C
Other:
- note added: "R20 0.4, 1W"
- note removed: "R20 0.2, 1W"
- moved on the sheet: C1, C100, C101, C11, C12, C13, C14, C16, C17, C18, C19, C2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
