File: headstage-neuropix/headstage-neuropix_no-test-fixtures.sch (EAGLE design)
At the start: 134 parts, among them J3 FH23-45S-0.3SHW(05), J5 X.FL-R-SMT-1(02), J7 FH23-45S-0.3SHW(05), U1 10M08SAM15317G, U2 ASCO2-24.000MHZ-EK-T3, U25 TS4231, U27 TS4231, U3 TPS8268180, U4 TLV70712, U5 TLV70733, U6 BNO055, U7 DS90UB913A_WQFN, U8 500SJAE93M6000ACF, U9 PL133-27GC-R, X2 OE-LOGO_14X10

Commit message: headstage-neuropix rev 1.2
- Dual neuropixels probe support
- 2X HTC Vive receivers
- Many changes made for reliability of manufacturing
Parts:
- removed J1: (no value), jonnew:PINHD-2X5_IDC
- removed J2: (no value), jonnew:PINHD-2X8_THRU
- removed J4, J6: (no value), jonnew:JP2E_THRU-HOLE
- removed TP12, TP13: (no value), jonnew:TPTP20R
- removed X2: OE-LOGO_14X10, jonnew:OE-LOGO_14X10
Connections:
- net +3V3: no longer J1.4
- net DEBUG0: no longer J2.1
- net DEBUG1: no longer J2.3
- net DEBUG2: no longer J2.5
- net DEBUG3: no longer J2.7
- net DEBUG4: no longer J2.9
- net DEBUG5: no longer J2.11
- net DEBUG6: no longer J2.13
- net DEBUG7: no longer J2.15
- net GND: no longer J1.10, J1.2, J2.10, J2.12, J2.14, J2.16, J2.2, J2.4, J2.6, J2.8, J4.2, J6.1, J6.2, TP12.TP, TP13.TP
- net TCK: no longer J1.1
- net TDI: no longer J1.9
- net TDO: no longer J1.3
- net TMS: no longer J1.5
- net VCOAX: no longer J4.1
Other:
- note removed: "DEBUG"
- moved on the sheet: C30, C31, C32, C33, C36, C37, C38, C39, C40, C41, C43, C44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
