File: headstage-neuropix/headstage-neuropix.sch (EAGLE design)
At the start: 134 parts, among them J3 FH23-45S-0.3SHW(05), J5 X.FL-R-SMT-1(02), J7 FH23-45S-0.3SHW(05), U1 10M08SAM15317G, U2 ASCO2-24.000MHZ-EK-T3, U25 TS4231, U27 TS4231, U3 TPS8268180, U4 TLV70712, U5 TLV70733, U6 BNO055, U7 DS90UB913A_WQFN, U8 500SJAE93M6000ACF, U9 PL133-27GC-R, X2 OE-LOGO_14X10

Commit message: Revision 1.2 of headstage-neuropix
- Routed all GPIO from serializer to FPGA
- Inner layers are now 3 mil trace space
- via-reduce just like headstage-64
Parts:
- U7: value DS90UB913A_WQFN -> DS90UB933_WQFN
Connections:
- net DIN10 renamed SER_DIN10
- net DIN11 renamed SER_DIN11
- net DIN2 renamed SER_DIN2
- net DIN3 renamed SER_DIN3
- net DIN4 renamed SER_DIN4
- net DIN6 renamed SER_DIN6
- net DIN7 renamed SER_DIN7
- net DIN8 renamed SER_DIN8
- net DIN9 renamed SER_DIN9
- net HSYNC renamed SER_HSYNC
- net PCLK renamed SER_PCLK
- net SERDES_GPIO0 renamed SER_GPIO0
- net SERDES_GPIO1 renamed SER_GPIO1
- net SERDES_SCL renamed SER_SCL
- net SERDES_SDA renamed SER_SDA
- net VSYNC renamed SER_VSYNC
- removed net DIN0: U1G$9.DIFFIO_RX_T23N/A5, U7.DIN0
- removed net DIN1: U1G$9.DIFFIO_RX_T16N/DEV_CLRN/B8, U7.DIN1
- removed net DIN5: U1G$9.DIFFIO_RX_T19N/B11, U7.DIN5
- new net SER_DIN0: U1G$9.DIFFIO_RX_T16N/DEV_CLRN/B8, U7.DIN0
- new net SER_DIN1: U1G$9.DIFFIO_RX_T16P/C8, U7.DIN1
- new net SER_DIN5: U1G$9.DIFFIO_RX_T14N/D10, U7.DIN5
- new net SER_GPIO2: U1G$9.DIFFIO_RX_T15N/B14, U7.GPIO2/CLKOUT
- new net SER_GPIO3: U1G$9.DIFFIO_RX_T19P/B12, U7.GPO3/CLKIN
Other:
- moved on the sheet: TP10, TP11, TP8

Commit message: Final headstage-neuropix rev. 1.2
- BOM simplification while updating the google sheet
- Small PCB changes
Parts:
- removed C71: 0.1uF, jonnew:C_0201T
- removed C76: 1uF, jonnew:C_0201T
- removed D10: VEMD1160X01, jonnew:PHOTODIODE_0805PT
- removed R48: 9k, 0.1%, jonnew:R_0201T
- removed R51: 1k, 0.1%, jonnew:R_0201T
- added C42: 47nF, jonnew:C_0201T
- added C48: 4.7uF, jonnew:C_0402T
- added D5: SESD0402X1UN-0020-090, jonnew:Z-DIODE_0402T-DFN
- added R31: 100, jonnew:R_0201T
- added R34: 1k, jonnew:R_0201T
- C25, C33: value 10nF -> 10uF; device jonnew:C_0201T -> jonnew:C_0402TW
- C26: value 1uF -> 0.1uF; device jonnew:C_0402T -> jonnew:C_0201T
- C27: value 1uF -> 10uF; device jonnew:C_0402T -> jonnew:C_0402TW
- C30, C31: value 0.1uF -> 10nF
- C32, C38, C49: value 10nF -> 0.1uF
- C34: value 15uF -> 10uF
- C35: value 10uF -> 10nF; device jonnew:C_0402T -> jonnew:C_0201T
- C43: value 0.1uF -> 4.7uF; device jonnew:C_0201T -> jonnew:C_0402T
- C44: value 47nF -> 4.7uF; device jonnew:C_0201T -> jonnew:C_0402T
- C45: value 4.7uF -> 10uF; device jonnew:C_0402T -> jonnew:C_0402TW
- C46: value 4.7uF -> 10nF; device jonnew:C_0402T -> jonnew:C_0201T
- C47: value 15uF -> 10nF; device jonnew:C_0402TW -> jonnew:C_0201T
- C52: value 4.7uF -> 1uF; device jonnew:C_0402T -> jonnew:C_0201T; PARTNO (none) -> CL03A105MP3ZSNH
- C53: PARTNO (none) -> C0603X5R1C104K030BC
- D3: value SESD0402X1UN-0020-090 -> VEMD1160X01; device jonnew:Z-DIODE_0402T-DFN -> jonnew:PHOTODIODE_0805PT
- J4: value (none) -> X.FL-R-SMT-1(02); device jonnew:JP2E_THRU-HOLE -> jonnew:COAX_XFL
- J5: value X.FL-R-SMT-1(02) -> (none); device jonnew:COAX_XFL -> jonnew:JP2E_THRU-HOLE
- R1: value 2k -> 4.7k
- R11, R14, R15, R4: value 10k -> 4.7k
- R16: value 10k -> 9k, 0.1%
- R17: value 10k -> 1k, 0.1%
- R18: value 49.9 -> 10k
- R20: value 100k -> 10k
- R21: value 22 -> 10k
- R22: value 20k -> 10k
- R23: value 100 -> 49.9
- R24, R25: value 1k -> 10k
- R26: value 4.7k -> 100k
- R27, R9: value 4.7k -> 1k
- R28, R29: value 4.7k -> 22
- R3: value 4.7k -> 2k
- R30: value 22 -> 20k
- R7: value 1k -> 4.7k
- U6: value BNO055 -> DS90UB933_WQFN; device jonnew:BNO055 -> jonnew:DS90UB913A_WQFN
- U7: value DS90UB933_WQFN -> BNO055; device jonnew:DS90UB913A_WQFN -> jonnew:BNO055
- renumbered C72 to C51, C75 to C54, D9 to D4, R86 to R32, R90 to R33, U25 to U10, U27 to U11
Connections:
- net !IMU_BL: now also R24.2, U7.!BOOT_LOAD; no longer R16.2, U6.!BOOT_LOAD
- net !IMU_RESET: now also R21.1, U7.!RESET; no longer R15.1, U6.!RESET
- net +1V2: now also C33.1; no longer C34.1
- net +1V8: now also C28.1, C36.1, C39.1, C44.1, C46.2, C47.2, R10.2, R14.2, R25.1, R4.2, R7.2, U6.VDDD, U6.VDDT; no longer C25.2, C32.1, C37.1, C40.1, C46.1, C49.2, R19.1, R26.2, R27.2, R28.2, R29.2, U7.VDDD, U7.VDDT
- net +3V3: now also C25.1, C29.1, C34.1, C53.1, R1.2, R11.2, R18.1, R19.1, R20.1, R21.2, R22.1, R24.1, R3.1, U7.VDD; no longer C28.1, C33.1, C35.1, C71.1, R1.1, R10.2, R12.1, R14.1, R16.1, R17.1, R3.2, R4.1, R9.2, U6.VDD
- net BNO_SCL: now also R1.1, U7.COM1/SCL/RX; no longer R2.1, U6.COM1/SCL/RX
- net BNO_SDA: now also R2.1, U7.COM0/SDA/TX; no longer R3.1, U6.COM0/SDA/TX
- net CAL_1.3KHZ: now also R30.1; no longer R22.1
- net CAL_SIGNAL: now also R30.2, R31.1; no longer R22.2, R23.1
- net CONFIG_SEL: now also R12.1; no longer R11.1
- net CONF_DONE: now also R20.2; no longer R14.2
- net GND: now also C25.2, C29.2, C32.1, C43.2, C44.2, C46.1, C47.1, C48.2, C49.2, D5.A, R12.2, R17.1, R23.1, R26.2, R31.2, R9.2, U6.ID, U6.RES, U7.COM2, U7.COM3/ADDR, U7.GNDIO, U7.PS0, U7.PS1; no longer C25.1, C29.1, C32.2, C41.2, C46.2, C47.2, C49.1, C71.2, C76.2, D3.A, R11.2, R18.1, R20.2, R23.2, R51.1, R7.2, U6.COM2, U6.COM3/ADDR, U6.GNDIO, U6.PS0, U6.PS1, U7.ID, U7.RES
- net I2C_SCL_A: now also R14.1; no longer R27.1
- net I2C_SCL_B: now also R7.1; no longer R29.1
- net I2C_SDA_A: now also R10.1; no longer R26.1
- net I2C_SDA_B: now also R4.1; no longer R28.1
- net JTAGEN: now also R5.2; no longer R4.2
- net MIDFILT: now also R27.1, R34.2; no longer R24.1, R25.2
- net N$13: now also C48.1, C49.1, R27.2; no longer C52.1, C53.1, R24.2
- net N$2: now also R28.1; no longer R30.1
- net N$28: now also C41.2, U6.DOUT+; no longer C43.2, U7.DOUT+
- net N$3: now also R29.2; no longer R21.2
- net N$30: now also R22.2, U6.PDB; no longer R17.2, U7.PDB
- net N$31: now also C42.2, U6.DOUT-; no longer C44.2, U7.DOUT-
- net N$32: now also C42.1, R23.2; no longer C44.1, R18.2
- net N$33: now also R25.2, R26.1, U6.MODE; no longer R19.2, R20.1, U7.MODE
- net N$34: now also C35.1, C38.1, C43.1, U6.VDDPLL; no longer C36.1, C39.1, C45.1, U7.VDDPLL
- net N$35: now also C37.1, C40.1, C45.1, U6.VDDCML; no longer C38.1, C41.1, C47.1, U7.VDDCML
- net N$36: now also C52.1; no longer C76.1
- net N$5: now also R28.2; no longer R30.2
- net N$52: now also R16.2, R17.2; no longer R48.2, R51.2
- net N$6: now also R29.1; no longer R21.1
- net N$67: now also C32.2, U7.CAP; no longer C29.2, U6.CAP
- net N$7: now also D3.C; no longer D10.C
- net N$8: now also D3.A; no longer D10.A
- net N$93: now also R3.2; no longer R1.2
- net NCONFIG: now also R18.2; no longer R12.2
- net NSTATUS: now also R19.2; no longer R13.2
- net SER_DIN0: now also U6.DIN0; no longer U7.DIN0
- net SER_DIN1: now also U6.DIN1; no longer U7.DIN1
- net SER_DIN10: now also U6.DIN10; no longer U7.DIN10
- net SER_DIN11: now also U6.DIN11; no longer U7.DIN11
- net SER_DIN2: now also U6.DIN2; no longer U7.DIN2
- net SER_DIN3: now also U6.DIN3; no longer U7.DIN3
- net SER_DIN4: now also U6.DIN4; no longer U7.DIN4
- net SER_DIN5: now also U6.DIN5; no longer U7.DIN5
- net SER_DIN6: now also U6.DIN6; no longer U7.DIN6
- net SER_DIN7: now also U6.DIN7; no longer U7.DIN7
- net SER_DIN8: now also U6.DIN8; no longer U7.DIN8
- net SER_DIN9: now also U6.DIN9; no longer U7.DIN9
- net SER_GPIO0: now also U6.GPIO0; no longer U7.GPIO0
- net SER_GPIO1: now also U6.GPIO1; no longer U7.GPIO1
- net SER_GPIO2: now also U6.GPIO2/CLKOUT; no longer U7.GPIO2/CLKOUT
- net SER_GPIO3: now also U6.GPO3/CLKIN; no longer U7.GPO3/CLKIN
- net SER_HSYNC: now also U6.HSYNC; no longer U7.HSYNC
- net SER_PCLK: now also U6.PCLK1; no longer U7.PCLK1
- net SER_SCL: now also R11.1, U6.SCL; no longer R9.1, U7.SCL
- net SER_SDA: now also R15.1, U6.SDA; no longer R10.1, U7.SDA
- net SER_VSYNC: now also U6.VSYNC; no longer U7.VSYNC
- net SIGOUT: now also C41.1, D5.C, J4.1, R34.1; no longer C43.1, D3.C, J5.1, R25.1
- net TCK: now also R9.1; no longer R7.1
- net TDI: now also R13.2; no longer R8.2
- net TMS: now also R8.2; no longer R5.2
- net VCOAX: now also J5.1, R16.1; no longer J4.1, R48.1
Other:
- moved on the sheet: C25, C26, C28, C29, C30, C31, C32, C33, C34, C35, C36, C37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

Commit message: Added third lighthouse receiver to headstage-neuropix
- I'm now sending this to speedy for a quote
Parts:
- removed C49: 0.1uF, jonnew:C_0201T
- removed L10: CIG21L4R7MNE, jonnew:L_0805T
- removed R34: 1k, jonnew:R_0201T
- added C55: 1uF, jonnew:C_0201T
- added C56, C57: 0.1uF, jonnew:C_0201T
- added D6: VEMD1160X01, jonnew:PHOTODIODE_0805PT
- added L11: BLM15HD102SN1D, jonnew:L_0402T
- added R35: 15k, jonnew:R_0201T
- added U12: TS4231, jonnew:TS4231
- C48: value 4.7uF -> 10uF
- L9: value CBC3225T101MR -> ADL3225V-470MT-TL000
- R27: value 1k -> 2k
Connections:
- new net LH_DATA0: U11.D/CFGDATA, U1G$3.DIFFIO_RX_L3P/ADCIN4/G5
- new net LH_ENV0: U11.E/CFGCLK, U1G$3.DIFFIO_RX_L3N/ADCIN3/F5
- new net N$26: D6.C, U12.IIN-
- new net N$27: D6.A, U12.IIN+
- new net N$29: R35.2, U12.RBIAS
- new net N$37: C55.1, U12.AVDD
- net +3V3: now also C56.1, U12.DVDD
- net GND: now also C55.2, C56.2, C57.2, R35.1, U12.AVSS, U12.AVSS2; no longer C49.2
- net LH_DATA2: now also U12.D/CFGDATA, U1G$9.DIFFIO_RX_T19N/B11; no longer U11.D/CFGDATA, U1G$3.DIFFIO_RX_L3P/ADCIN4/G5
- net LH_ENV2: now also U12.E/CFGCLK, U1G$9.DIFFIO_RX_T17P/B13; no longer U11.E/CFGCLK, U1G$3.DIFFIO_RX_L3N/ADCIN3/F5
- net MIDFILT: now also L11.2; no longer L10.2, R34.2
- net N$13: no longer C49.1
- net N$52: now also C57.1
- net SIGOUT: now also L11.1; no longer L10.1, R34.1
Other:
- note added: "3D TRACKING"
- note removed: "TRACKING"
- moved on the sheet: C28, C29, C30, C31, C35, C36, C37, C38, C39, C40, C41, C42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

Commit message: Minor improvements to headstage-neuropix rev 1.2
- Final changes before production
- Minor BOM simplification
Parts:
- removed C57: 0.1uF, jonnew:C_0201T
- removed L11: BLM15HD102SN1D, jonnew:L_0402T
- added C49: 10nF, jonnew:C_0201T
- added L10: MPZ1608S102ATA00, jonnew:L_0603T
- added R34: 15k, jonnew:R_0201T
- C16: PARTNO (none) -> C0603X5R1C104K030BC
- C20: value 10uF -> 0.1uF; device jonnew:C_0402T -> jonnew:C_0201T
- C24: value 0.1uF -> 10uF; device jonnew:C_0201T -> jonnew:C_0402T
- C25, C27, C33: value 10uF -> 0.1uF; device jonnew:C_0402TW -> jonnew:C_0201T
- C26, C28: value 0.1uF -> 10uF; device jonnew:C_0201T -> jonnew:C_0402TW
- C30: value 10nF -> 0.1uF
- C32, C38: value 0.1uF -> 10nF
- C35, C46: value 10nF -> 10uF; device jonnew:C_0201T -> jonnew:C_0402TW
- C42: value 47nF -> 0.1uF
- C43: value 4.7uF -> 47nF; device jonnew:C_0402T -> jonnew:C_0201T
- C45: value 10uF -> 4.7uF; device jonnew:C_0402TW -> jonnew:C_0402T
- C53: value 0.1uF -> 1uF; PARTNO C0603X5R1C104K030BC -> CL03A105MP3ZSNH
- C55: value 1uF -> 0.1uF; PARTNO CL03A105MP3ZSNH -> C0603X5R1C104K030BC
- D3: value VEMD1160X01 -> SESD0402X1UN-0020-090; device jonnew:PHOTODIODE_0805PT -> jonnew:Z-DIODE_0402T-DFN
- D5: value SESD0402X1UN-0020-090 -> VEMD1160X01; device jonnew:Z-DIODE_0402T-DFN -> jonnew:PHOTODIODE_0805PT
- J2: value (none) -> X.FL-R-SMT-1(02); device jonnew:PINHD-2X8_THRU -> jonnew:COAX_XFL
- J4: value X.FL-R-SMT-1(02) -> (none); device jonnew:COAX_XFL -> jonnew:PINHD-2X8_THRU
- J6: value (none) -> FH23-45S-0.3SHW(05); device jonnew:JP2E_THRU-HOLE -> jonnew:PINHD-1X45_FH23
- J7: value FH23-45S-0.3SHW(05) -> (none); device jonnew:PINHD-1X45_FH23 -> jonnew:JP2E_THRU-HOLE
- R30: value 20k -> 10k
- R35: value 15k -> 10k
Connections:
- new net N$38: R30.1, R35.2
- net +1V2: now also C34.1, J6.P$38, J6.P$39, J6.P$7, J6.P$8; no longer C33.1, J7.P$38, J7.P$39, J7.P$7, J7.P$8
- net +1V8: now also C29.1, C31.1, C37.1, C40.1, C45.1, C49.2, J6.P$3, J6.P$4, J6.P$42, J6.P$43; no longer C28.1, C30.1, C36.1, C39.1, C44.1, C46.2, J7.P$3, J7.P$4, J7.P$42, J7.P$43
- net +3V3: now also C27.1, C30.1, C32.1, C35.1, C55.1; no longer C24.1, C29.1, C31.1, C34.1, C53.1
- net CAL_1.3KHZ: now also R35.1; no longer R30.1
- net CAL_SIGNAL: now also J6.P$11; no longer J7.P$11
- net DEBUG0: now also J4.1; no longer J2.1
- net DEBUG1: now also J4.3; no longer J2.3
- net DEBUG2: now also J4.5; no longer J2.5
- net DEBUG3: now also J4.7; no longer J2.7
- net DEBUG4: now also J4.9; no longer J2.9
- net DEBUG5: now also J4.11; no longer J2.11
- net DEBUG6: now also J4.13; no longer J2.13
- net DEBUG7: now also J4.15; no longer J2.15
- net GND: now also C32.2, C33.1, C41.2, C46.2, C49.1, D3.A, J4.10, J4.12, J4.14, J4.16, J4.4, J4.6, J4.8, J6.P$1, J6.P$10, J6.P$13, J6.P$14, J6.P$17, J6.P$2, J6.P$20, J6.P$23, J6.P$26, J6.P$29, J6.P$32, J6.P$34, J6.P$36, J6.P$37, J6.P$41, J6.P$44, J6.P$45, J6.P$5, J6.P$6, J6.P$9, J7.1, J7.2, R34.1; no longer C32.1, C33.2, C43.2, C46.1, C57.2, D5.A, J2.10, J2.12, J2.14, J2.16, J2.4, J2.6, J2.8, J6.1, J6.2, J7.P$1, J7.P$10, J7.P$13, J7.P$14, J7.P$17, J7.P$2, J7.P$20, J7.P$23, J7.P$26, J7.P$29, J7.P$32, J7.P$34, J7.P$36, J7.P$37, J7.P$41, J7.P$44, J7.P$45, J7.P$5, J7.P$6, J7.P$9, R35.1
- net I2C_SCL_B: now also J6.P$19; no longer J7.P$19
- net I2C_SDA_B: now also J6.P$18; no longer J7.P$18
- net MIDFILT: now also L10.2; no longer L11.2
- net N$14: now also D5.C; no longer D4.C
- net N$15: now also D5.A; no longer D4.A
- net N$28: now also C42.2; no longer C41.2
- net N$29: now also R34.2; no longer R35.2
- net N$31: now also C43.2; no longer C42.2
- net N$32: now also C43.1; no longer C42.1
- net N$34: now also C36.1, C39.1, C44.1; no longer C35.1, C38.1, C43.1
- net N$35: now also C38.1, C41.1, C46.1; no longer C37.1, C40.1, C45.1
- net N$37: now also C53.1; no longer C55.1
- net N$4: now also C18.1, C21.1; no longer C17.1, C20.1
- net N$5: now also J6.P$35; no longer J7.P$35
- net N$52: now also C16.1; no longer C57.1
- net N$67: now also C33.2; no longer C32.2
- net N$7: now also D4.C; no longer D3.C
- net N$8: now also D4.A; no longer D3.A
- net NRST_B: now also J6.P$15; no longer J7.P$15
- net OSC_PDOWN_N_B: now also J6.P$12; no longer J7.P$12
- net PSB_CLK_B: now also J6.P$33; no longer J7.P$33
- net PSB_DATA_0_B: now also J6.P$31; no longer J7.P$31
- net PSB_DATA_1_B: now also J6.P$30; no longer J7.P$30
- net PSB_DATA_2_B: now also J6.P$28; no longer J7.P$28
- net PSB_DATA_3_B: now also J6.P$27; no longer J7.P$27
- net PSB_DATA_4_B: now also J6.P$25; no longer J7.P$25
- net PSB_DATA_5_B: now also J6.P$24; no longer J7.P$24
- net PSB_DATA_6_B: now also J6.P$22; no longer J7.P$22
- net PSB_SYNC_B: now also J6.P$21; no longer J7.P$21
- net REC_NRST_B: now also J6.P$16; no longer J7.P$16
- net SIGOUT: now also C42.1, D3.C, J2.1, L10.1; no longer C41.1, D5.C, J4.1, L11.1
- net VCCIO: now also C20.1, C23.1; no longer C19.1, C22.1
- net VCCIO2: now also C19.1, C22.1; no longer C18.1, C21.1
- net VCCIOA: now also C17.1, C24.1; no longer C16.1, C23.1
- net VCOAX: now also C28.1; no longer C27.1
Other:
- moved on the sheet: C16, C17, C18, C19, C20, C21, C22, C23, C24, C25, C26, C27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

Commit message: More updates to headstage-neuropix after review from Speedy
- Many bottom side pads moved apart to allow solder mask in between and
to prevent shorts
Parts:
- J1: value (none) -> 302-S101
- J4: value (none) -> 68602-116HLF
- J5, J7: value (none) -> 77311-118-02LF
- U5: value TLV70733 -> NCP161BMX330
Other:
- note added: "NB: programmed to 93.6 MHz"
- note added: "NB:CLK0 drives PLL1."
- note removed: "NB: LVPECL with V_cm = 1.8V. 500 Mbps ≤ DMAX ≤ 700 Mbps for bothclock inputs. CLK0 drives PLL1."
- note removed: "NB:VCCIO = 2.5 for LVPECL"
Changed lines of the file:
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@@
 <parts>
 <part name="U6" library="jonnew" deviceset="DS90UB913A" device="_WQFN" value="DS90UB933_WQFN"/>
-<part name="U5" library="jonnew" deviceset="TLV707" device="" value="TLV70733"/>
+<part name="U5" library="jonnew" deviceset="TLV707" device="" value="NCP161BMX330"/>
 <part name="U4" library="jonnew" deviceset="TLV707" device="" value="TLV70712"/>
 <part name="C28" library="jonnew" deviceset="C" device="_0402TW" value="10uF"/>
@@
 <part name="C11" library="jonnew" deviceset="C" device="_0201T" value="10nF"/>
 <part name="J3" library="jonnew" deviceset="PINHD-1X45" device="_FH23" value="FH23-45S-0.3SHW(05)"/>
-<part name="J1" library="jonnew" deviceset="PINHD-2X5" device="_IDC"/>
+<part name="J1" library="jonnew" deviceset="PINHD-2X5" device="_IDC" value="302-S101"/>
 <part name="SUPPLY16" library="jonnew" deviceset="GND" device=""/>
 <part name="P23" library="jonnew" deviceset="+3V3" device=""/>
@@
 <part name="TP10" library="jonnew" deviceset="TP" device="TP09R"/>
 <part name="TP11" library="jonnew" deviceset="TP" device="TP09R"/>
-<part name="J5" library="jonnew" deviceset="JP2E" device="_THRU-HOLE"/>
+<part name="J5" library="jonnew" deviceset="JP2E" device="_THRU-HOLE" value="77311-118-02LF"/>
 <part name="P58" library="jonnew" deviceset="+VCOAX" device=""/>
 <part name="SUPPLY56" library="jonnew" deviceset="GND" device=""/>
-<part name="J4" library="jonnew" deviceset="PINHD-2X8" device="_THRU"/>
+<part name="J4" library="jonnew" deviceset="PINHD-2X8" device="_THRU" value="68602-116HLF"/>
 <part name="SUPPLY54" library="jonnew" deviceset="GND" device=""/>
 <part name="TP13" library="jonnew" deviceset="TP" device="TP20R"/>
@@
 <part name="P9" library="jonnew" deviceset="+1V8" device=""/>
 <part name="P12" library="jonnew" deviceset="+1V8" device=""/>
-<part name="J7" library="jonnew" deviceset="JP2E" device="_THRU-HOLE"/>
+<part name="J7" library="jonnew" deviceset="JP2E" device="_THRU-HOLE" value="77311-118-02LF"/>
 <part name="SUPPLY57" library="jonnew" deviceset="GND" device=""/>
 <part name="P29" library="jonnew" deviceset="+3V3" device=""/>
@@
 max voltage. Use
 3.3V.</text>
-<text x="30.48" y="591.82" size="1.778" layer="97" rot="R90">NB: VCCIO = 1.8V for the neuropix interface.</text>
+<text x="33.02" y="629.92" size="1.778" layer="97" rot="R90">NB: VCCIO = 1.8V for the neuropix interface.</text>
 <text x="116.84" y="810.26" size="10.16" layer="97">FPGA</text>
 <text x="38.1" y="528.32" size="1.778" layer="97">South-East</text>
@@
 <text x="182.88" y="739.14" size="1.778" layer="97">NB: Programming interface</text>
 <text x="106.68" y="363.22" size="1.778" layer="97">NB: 0.1 is not needed.</text>
-<text x="30.48" y="668.02" size="1.27" layer="97" rot="R90">NB:VCCIO = 2.5 for LVPECL</text>
-<text x="88.9" y="695.96" size="1.27" layer="97">NB: LVPECL with V_cm = 1.8V.
-500 Mbps ≤ DMAX ≤ 700 Mbps
-for bothclock inputs. CLK0 drives PLL1.</text>
+<text x="88.9" y="693.42" size="1.27" layer="97">NB:CLK0 drives PLL1.</text>
 <text x="337.82" y="591.82" size="10.16" layer="97">IMU</text>
 <text x="337.82" y="558.8" size="1.778" layer="97">I2C Selected</text>
@@
 <wire x1="591.82" y1="393.7" x2="718.82" y2="393.7" width="0.508" layer="94" style="longdash"/>
 <wire x1="591.82" y1="393.7" x2="591.82" y2="261.62" width="0.508" layer="94" style="longdash"/>
+<text x="439.42" y="668.02" size="1.778" layer="97">NB: programmed to 93.6 MHz</text>
 </plain>
 <instances>
