File: headstage-neuropix/headstage-neuropix.sch (EAGLE design)
At the start: 139 parts, among them J1 302-S101, J2 X.FL-R-SMT-1(02), J3 FH23-45S-0.3SHW(05), J4 68602-116HLF, J5 77311-118-02LF, J6 FH23-45S-0.3SHW(05), J7 77311-118-02LF, U1 10M08SAM15317G, U10 TS4231, U11 TS4231, U12 TS4231, U2 ASCO2-24.000MHZ-EK-T3, U3 TPS8268180, U4 TLV70712, U5 NCP161BMX330, U6 DS90UB933_WQFN, U7 BNO055, U8 500SJAE93M6000ACF, U9 PL133-27GC-R, X2 OE-LOGO_14X10

Commit message: headstage-neuropix rev. 1.3
- Fixes several issues found during testing or revision 1.2
- Analog power to neurpixels probe is now isolated using LC filter from
digital power
- 93.6 MHz osc gets power from 1.8V instead of 3.3. Footprint fixed.
- Vcoax has more bulk capacitance now
- Serializer has capacitance on its PDN pin as recormmended to get POR
sequence correct
- I added a UVLO OVLO circuit between the DC filter on coax input and
all the regulators powering the board. The headstage will only operate
in a ~4.1-6.5 volt window.
Parts:
- removed R35: 10k, jonnew:R_0201T
- added C57, C58, C59, C60: 0.1uF, jonnew:C_0201T
- added L11, L12: BLM15PX601SN1D, jonnew:L_0402T
- added U13: TS4231, jonnew:TS4231
- C16: PARTNO C0603X5R1C104K030BC -> (none)
- C20: value 0.1uF -> 10uF; device jonnew:C_0201T -> jonnew:C_0402T
- C24: value 10uF -> 0.1uF; device jonnew:C_0402T -> jonnew:C_0201T
- C25, C27, C33, C41, C42: value 0.1uF -> 10uF; device jonnew:C_0201T -> jonnew:C_0402TW
- C26, C28, C34: value 10uF -> 0.1uF; device jonnew:C_0402TW -> jonnew:C_0201T
- C30: value 0.1uF -> 10nF
- C32, C47: value 10nF -> 10uF; device jonnew:C_0201T -> jonnew:C_0402TW
- C35: value 10uF -> 10nF; device jonnew:C_0402TW -> jonnew:C_0201T
- C38: value 10nF -> 0.1uF
- C43: value 47nF -> 0.1uF
- C44: value 4.7uF -> 47nF; device jonnew:C_0402T -> jonnew:C_0201T
- C46: device jonnew:C_0402TW -> jonnew:C_0402T
- C48: value 10uF -> 1uF; device jonnew:C_0402T -> jonnew:C_0201T
- C50: value 0.33nF -> 0.1uF
- C51: value 1uF -> 10uF; device jonnew:C_0201T -> jonnew:C_0402T; PARTNO CL03A105MP3ZSNH -> (none)
- C52: value 1uF -> 10nF; PARTNO CL03A105MP3ZSNH -> (none)
- C54, C55: value 0.1uF -> 1uF; PARTNO C0603X5R1C104K030BC -> CL03A105MP3ZSNH
- D4, D5, D6: device jonnew:PHOTODIODE_0805PT -> jonnew:PHOTODIODE0805PT-NOSILK
- R16: value 9k, 0.1% -> 10k
- R17: value 1k, 0.1% -> 10k
- R21: value 10k -> 49.9
- R23: value 49.9 -> 10k
- R24: value 10k -> 100k
- R25: value 10k -> 2k
- R26: value 100k -> 22
- R27: value 2k -> 22
- R28: value 22 -> 20k
- R29: value 22 -> 100
- R30: value 10k -> 15k
- R31: value 100 -> 15k
- R33: value 15k -> 20k
- R34: value 15k -> 100
- U10: value TS4231 -> PL133-27GC-R; device jonnew:TS4231 -> jonnew:CLKBUF2_DFN_2X1.3_PAD
- U3: value TPS8268180 -> MAX4944ELA+T; device jonnew:TPS8268X -> jonnew:MAX494X
- U4: value TLV70712 -> DS90UB933_WQFN; device jonnew:TLV707 -> jonnew:DS90UB913A_WQFN
- U6: value DS90UB933_WQFN -> TPS8268180; device jonnew:DS90UB913A_WQFN -> jonnew:TPS8268X
- U7: value BNO055 -> TLV70712; device jonnew:BNO055 -> jonnew:TLV707
- U8: value 500SJAE93M6000ACF -> BNO055; device jonnew:CRYSTAL-OSC_SIT8008BCA7-18E -> jonnew:BNO055
- U9: value PL133-27GC-R -> DSC6102MI2A-093.6000; device jonnew:CLKBUF2_DFN_2X1.3_PAD -> jonnew:CRYSTAL-OSC_VFLGA4-2X1.6
Connections:
- removed net CAL_1.3KHZ: R35.1, U1G$7.DIFFIO_TX_RX_B9P/N8
- removed net CAL_SIGNAL: C50.2, J3.P$11, J6.P$11, R30.2, R31.1
- removed net N$52: C16.1, R16.2, R17.2, U1G$1.ANAIN1/D4
- new net 1V2A: C56.1, J3.P$7, J3.P$8, J6.P$7, J6.P$8, L11.1
- new net 1V8A: C60.1, J3.P$3, J3.P$4, J6.P$3, J6.P$4, L12.1
- new net CAL_A_1.3KHZ: R28.1, U1G$7.DIFFIO_TX_RX_B9P/N8
- new net CAL_B_1.3KHZ: R33.1, U1G$7.DIFFIO_TX_RX_B16N/P14
- new net CAL_SIGNAL_A: J3.P$11, R28.2, R29.1
- new net CAL_SIGNAL_A1: J6.P$11, R33.2, R34.1
- net !IMU_BL: now also R22.2, U8.!BOOT_LOAD; no longer R24.2, U7.!BOOT_LOAD
- net !IMU_RESET: now also R19.1, U8.!RESET; no longer R21.1, U7.!RESET
- net +1V2: now also C42.1, L11.2, U7.OUT; no longer C34.1, J3.P$7, J3.P$8, J6.P$7, J6.P$8, U4.OUT
- net +1V8: now also C11.2, C28.1, C30.1, C36.1, C39.1, C46.1, C52.2, L12.2, R23.1, U10.VCC, U2.EN, U2.VCC, U4.VDDD, U4.VDDT, U6.VOUT, U9.EN; no longer C29.1, C31.1, C37.1, C40.1, C45.1, C47.2, J3.P$3, J3.P$4, J6.P$3, J6.P$4, R25.1, U3.VOUT, U6.VDDD, U6.VDDT, U8.EN, U8.VCC
- net +3V3: now also C24.1, C29.1, C31.1, C33.1, C41.1, C57.1, C58.1, C59.1, R16.1, R17.1, R19.2, U13.DVDD, U4.VDDIO, U7.EN, U7.IN, U8.VDD, U8.VDDIO; no longer C11.2, C25.1, C27.1, C30.1, C32.1, C35.1, C54.1, C55.1, C56.1, R19.1, R21.2, R24.1, U10.DVDD, U2.EN, U2.VCC, U4.EN, U4.IN, U6.VDDIO, U7.VDD, U7.VDDIO
- net BNO_SCL: now also U8.COM1/SCL/RX; no longer U7.COM1/SCL/RX
- net BNO_SDA: now also U8.COM0/SDA/TX; no longer U7.COM0/SDA/TX
- net CONF_DONE: now also R18.2; no longer R20.2
- net GND: now also C33.2, C34.1, C42.2, C47.2, C50.2, C52.1, C57.2, C58.2, C59.2, C60.2, R21.1, R24.2, R29.2, R30.1, R31.1, R34.2, U10.GND, U13.AVSS, U13.AVSS2, U1G$1.ANAIN1/D4, U4.ID, U4.RES, U8.COM2, U8.COM3/ADDR, U8.GNDIO, U8.PS0, U8.PS1; no longer C33.1, C34.2, C44.2, C47.1, C50.1, C52.2, R17.1, R23.1, R26.2, R31.2, R33.1, R34.1, U10.AVSS, U10.AVSS2, U6.ID, U6.RES, U7.COM2, U7.COM3/ADDR, U7.GNDIO, U7.PS0, U7.PS1
- net LH_DATA0: now also U12.D/CFGDATA; no longer U11.D/CFGDATA
- net LH_DATA1: now also U11.D/CFGDATA; no longer U10.D/CFGDATA
- net LH_DATA2: now also U13.D/CFGDATA; no longer U12.D/CFGDATA
- net LH_ENV0: now also U12.E/CFGCLK; no longer U11.E/CFGCLK
- net LH_ENV1: now also U11.E/CFGCLK; no longer U10.E/CFGCLK
- net LH_ENV2: now also U13.E/CFGCLK; no longer U12.E/CFGCLK
- net MIDFILT: now also R25.1; no longer R27.1
- net N$1: now also U10.EN, U10.IN, U9.OUT; no longer U8.OUT, U9.EN, U9.IN
- net N$12: now also C53.1, U11.AVDD; no longer C51.1, U10.AVDD
- net N$13: now also C51.1, R25.2; no longer C48.1, R27.2
- net N$14: now also U12.IIN-; no longer U11.IIN-
- net N$15: now also U12.IIN+; no longer U11.IIN+
- net N$16: now also R31.2, U12.RBIAS; no longer R33.2, U11.RBIAS
- net N$2: now also R26.1, U10.CLK0; no longer R28.1, U9.CLK0
- net N$26: now also U13.IIN-; no longer U12.IIN-
- net N$27: now also U13.IIN+; no longer U12.IIN+
- net N$28: now also C43.2, U4.DOUT+; no longer C42.2, U6.DOUT+
- net N$29: now also R32.2, U13.RBIAS; no longer R34.2, U12.RBIAS
- net N$3: now also R27.2; no longer R29.2
- net N$30: now also C48.1, R20.2, U4.PDB; no longer R22.2, U6.PDB
- net N$31: now also C44.2, U4.DOUT-; no longer C43.2, U6.DOUT-
- net N$32: now also C44.1, R21.2; no longer C43.1, R23.2
- net N$33: now also C50.1, R23.2, R24.1, U4.MODE; no longer R25.2, R26.1, U6.MODE
- net N$34: now also C35.1, C38.1, C45.1, U4.VDDPLL; no longer C36.1, C39.1, C44.1, U6.VDDPLL
- net N$35: now also C37.1, C40.1, C47.1, U4.VDDCML; no longer C38.1, C41.1, C46.1, U6.VDDCML
- net N$36: now also C54.1, U12.AVDD; no longer C52.1, U11.AVDD
- net N$37: now also C55.1, U13.AVDD; no longer C53.1, U12.AVDD
- net N$38: now also C25.1, C27.1, C32.1, U3.OUT, U5.EN, U5.IN, U6.EN, U6.MODE, U6.VIN; no longer R30.1, R35.2
- net N$4: now also C17.1, C20.1; no longer C18.1, C21.1
- net N$5: now also R26.2; no longer R28.2
- net N$6: now also R27.1, U10.CLK1; no longer R29.1, U9.CLK1
- net N$67: now also C34.2, U8.CAP; no longer C33.2, U7.CAP
- net N$7: now also U11.IIN-; no longer U10.IIN-
- net N$8: now also U11.IIN+; no longer U10.IIN+
- net N$9: now also R30.2, U11.RBIAS; no longer R32.2, U10.RBIAS
- net NCONFIG: now also R16.2; no longer R18.2
- net NSTATUS: now also R17.2; no longer R19.2
- net PSB_DATA_0_B: now also U1G$7.DIFFIO_TX_RX_B3P/L7; no longer U1G$7.DIFFIO_TX_RX_B7P/M7
- net PSB_DATA_6_B: now also U1G$7.DIFFIO_TX_RX_B7P/M7; no longer U1G$7.DIFFIO_TX_RX_B3P/L7
- net SER_DIN0: now also U4.DIN0; no longer U6.DIN0
- net SER_DIN1: now also U4.DIN1; no longer U6.DIN1
- net SER_DIN10: now also U4.DIN10; no longer U6.DIN10
- net SER_DIN11: now also U4.DIN11; no longer U6.DIN11
- net SER_DIN2: now also U4.DIN2; no longer U6.DIN2
- net SER_DIN3: now also U4.DIN3; no longer U6.DIN3
- net SER_DIN4: now also U4.DIN4; no longer U6.DIN4
- net SER_DIN5: now also U4.DIN5; no longer U6.DIN5
- net SER_DIN6: now also U4.DIN6; no longer U6.DIN6
- net SER_DIN7: now also U4.DIN7; no longer U6.DIN7
- net SER_DIN8: now also U4.DIN8; no longer U6.DIN8
- net SER_DIN9: now also U4.DIN9; no longer U6.DIN9
- net SER_GPIO0: now also U4.GPIO0; no longer U6.GPIO0
- net SER_GPIO1: now also U4.GPIO1; no longer U6.GPIO1
- net SER_GPIO2: now also U4.GPIO2/CLKOUT; no longer U6.GPIO2/CLKOUT
- net SER_GPIO3: now also U4.GPO3/CLKIN; no longer U6.GPO3/CLKIN
- net SER_HSYNC: now also U4.HSYNC; no longer U6.HSYNC
- net SER_PCLK: now also U4.PCLK1; no longer U6.PCLK1
- net SER_SCL: now also U4.SCL; no longer U6.SCL
- net SER_SDA: now also U4.SDA; no longer U6.SDA
- net SER_VSYNC: now also U4.VSYNC; no longer U6.VSYNC
- net SIGOUT: now also C43.1; no longer C42.1
- net VCCIO: now also C19.1, C22.1; no longer C20.1, C23.1
- net VCCIO2: now also C18.1, C21.1; no longer C19.1, C22.1
- net VCCIOA: now also C16.1, C23.1; no longer C17.1, C24.1
- net VCOAX: now also U3.IN; no longer C28.1, R16.1, U3.EN, U3.MODE, U3.VIN, U5.EN, U5.IN
Other:
- moved on the sheet: C16, C17, C18, C19, C20, C21, C22, C23, C24, C25, C26, C27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

Commit message: headstage-neuropix rev. 1.3
- Addresses several more issues encountered during extensive testing of
rev.  1.2
- Analog rails of probes provided by dedicated LDOs that respect the
complex POR sequence required by the probes
- The clock enable for the dual clock buffer for each probe is tied high
instead of being driven by the clock input (!)
- Each probe has a dedicated calibration signal
Parts:
- removed C56, C60: 0.1uF, jonnew:C_0201T
- removed J4: 68602-116HLF, jonnew:PINHD-2X8_THRU
- removed J7: 77311-118-02LF, jonnew:JP2E_THRU-HOLE
- removed L11, L12: BLM15PX601SN1D, jonnew:L_0402T
- removed TP11: (no value), jonnew:TPTP09R
- removed TP12: (no value), jonnew:TPTP20R
- removed TP8: (no value), jonnew:TPTP11R
- added C61, C67: 1uF, jonnew:C_0201T
- added C62, C63: 1nF, jonnew:C_0201T
- added C64, C65, C66: 10uF, jonnew:C_0402TW
- added R35: 6.6k, jonnew:R_0201T
- added R36: 10k, jonnew:R_0201T
- added U14, U15: (no value), jonnew:LDO_ADJUST-EN-SS_WLCSP-ADP7112
- U3: value MAX4944ELA+T -> MAX4945AELA+T
Connections:
- net CAL_A_1.3KHZ renamed CAL_A_1KHZ
- net CAL_B_1.3KHZ renamed CAL_B_1KHZ
- removed net DEBUG0: J4.1, U1G$8.E14
- removed net DEBUG1: J4.3, U1G$8.VREFB6N0/E15
- removed net DEBUG2: J4.5, U1G$8.DIFFIO_RX_R18N/G15
- removed net DEBUG3: J4.7, U1G$6.DIFFIO_RX_R11N/J14
- removed net DEBUG4: J4.9, U1G$8.DIFFIO_RX_R18P/J15
- removed net DEBUG5: J4.11, U1G$6.DIFFIO_RX_R11P/K14
- removed net DEBUG6: J4.13, U1G$6.VREFB5N0/L15
- removed net DEBUG7: J4.15, U1G$6.DIFFIO_RX_R2P/N15
- removed net NRST_A: J3.P$15, U1G$7.DIFFIO_RX_B6P/P8
- removed net NRST_B: J6.P$15, U1G$7.DIFFIO_TX_RX_B10P/P15
- new net N$39: C62.1, U14.SS
- new net N$40: C63.1, U15.SS
- new net N$41: C67.1, R35.1, U15.EN
- new net NP_OSC_EN: U1G$7.DIFFIO_RX_B6P/P8, U9.EN
- new net NRST: J3.P$15, J6.P$15, R35.2, U14.EN, U1G$7.DIFFIO_TX_RX_B10P/P15
- net +1V2: no longer L11.2
- net +1V8: now also U10.EN; no longer L12.2, U9.EN
- net +3V3: now also C65.1, U14.VI, U15.VI
- net 1V2A: now also C66.1, U15.ADJ, U15.VO; no longer C56.1, L11.1
- net 1V8A: now also C64.1, U14.ADJ, U14.VO; no longer C60.1, L12.1
- net GND: now also C61.2, C62.2, C63.2, C64.2, C65.2, C66.2, C67.2, R36.2, U14.GND, U15.GND; no longer C56.2, C60.2, J4.10, J4.12, J4.14, J4.16, J4.2, J4.4, J4.6, J4.8, J7.1, J7.2, TP12.TP, TP8.TP
- net N$1: no longer U10.EN
- net PSB_DATA_1_A: now also U1G$7.DIFFIO_TX_RX_B5P/P7; no longer U1G$7.DIFFIO_RX_B6N/R7
- net PSB_DATA_5_A: now also U1G$7.DIFFIO_RX_B6N/R7; no longer U1G$7.DIFFIO_TX_RX_B5P/P7
- net SER_GPIO0: no longer TP11.TP
- net SER_GPIO2: now also R36.1
- net VCOAX: now also C61.1
Other:
- note added: "NB: 1.8 msec delay"
- note added: "NB: Input cap serves both LDOs"
- note added: "NB: Needed on POR to get LOCK"
- note added: "NP POR Sequence 1. Digital 1.8V and 1.2V on 2. Wait 10 msec (handled by Osc EN kinda: it takes 1.3 msec) 3. Enable MCLK 4. Wait 10 MCLK cycles 5. NRST = 1 for 10 periods 6. NRSET = 0 to reset 7. Wait 200 msec 8. Power on 1.8 analog 9. Wait 1.8 ms 10. Power on 1.2 analog"
- moved on the sheet: C24, C25, C26, C27, C32, C33, C34, C41, C42, C49, C52, J5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
