File: headstage-64/headstage-64-coax-adapter.sch (EAGLE design)
At the start: 125 parts, among them J1 X.FL-R-SMT-1(02), J11 X.FL-R-SMT-1(02), J13 X.FL-R-SMT-1(02), J15 X.FL-R-SMT-1(02), J17 X.FL-R-SMT-1(02), J21 X.FL-R-SMT-1(02), J25 X.FL-R-SMT-1(02), J29 X.FL-R-SMT-1(02), J33 X.FL-R-SMT-1(02), J37 X.FL-R-SMT-1(02), J41 X.FL-R-SMT-1(02), J45 X.FL-R-SMT-1(02), J49 X.FL-R-SMT-1(02), J5 X.FL-R-SMT-1(02), J53 X.FL-R-SMT-1(02), J57 X.FL-R-SMT-1(02), J61 X.FL-R-SMT-1(02), J65 X.FL-R-SMT-1(02), J69 X.FL-R-SMT-1(02), J7 X.FL-R-SMT-1(02), J73 X.FL-R-SMT-1(02), J77 X.FL-R-SMT-1(02), J81 X.FL-R-SMT-1(02), J85 X.FL-R-SMT-1(02), J9 X.FL-R-SMT-1(02)

Commit message: Update headstage-64 and headstage-256 schematics
- I did this while double checking the BOM for Filipe
- Divide functional blocks into labeled sections
- Add images of schematics to the READMEs
Parts:
- removed D27, D31, D35, D37, D39, D43: SESD0402X1UN-0020-090, jonnew:Z-DIODE_0402T-DFN
- removed J53, J57, J65, J69, J73, J77, J85: X.FL-R-SMT-1(02), jonnew:COAX_XFL
- removed J54, J62, J70, J74, J78, J86: (no value), jonnew:PINHD-1X4HEADSTAGE64-DAUGHTER-CARD-CASTELLATED
- removed L27, L31, L35, L37, L39, L43: CIG21L4R7MNE, jonnew:L_0805T
- removed R27, R31, R37, R39, R43: 1k, jonnew:R_0201T
- added D10, D14, D18, D2, D20, D24: SESD0402X1UN-0020-090, jonnew:Z-DIODE_0402T-DFN
- added J19, J20, J28, J39, J40, J48: (no value), jonnew:PINHD-1X4HEADSTAGE64-DAUGHTER-CARD-CASTELLATED
- added J23, J24, J3, J35, J4, J43, J44: X.FL-R-SMT-1(02), jonnew:COAX_XFL
- added L10, L14, L18, L2, L20, L24: CIG21L4R7MNE, jonnew:L_0805T
- added R10, R14, R18, R20, R24: 1k, jonnew:R_0201T
- J12, J14, J2, J22, J34, J42: value (none) -> X.FL-R-SMT-1(02); device jonnew:PINHD-1X4HEADSTAGE64-DAUGHTER-CARD-CASTELLATED -> jonnew:COAX_XFL
- J17, J29, J37, J49, J7, J9: value X.FL-R-SMT-1(02) -> (none); device jonnew:COAX_XFL -> jonnew:PINHD-1X4HEADSTAGE64-DAUGHTER-CARD-CASTELLATED
- renumbered D29 to D12, D33 to D22, D41 to D16, J58 to J27, J61 to J32, J66 to J47, J81 to J31, J82 to J36, L29 to L12, L33 to L22, L41 to L16, R29 to R12, R33 to R22, R35 to R1, R41 to R16
Connections:
- removed net N$15 (its old number): J18.1, L9.2, R9.2
- removed net N$48 (its old number): J2.1, L1.2, R3.2
- new net N$27: J8.1, L3.2, R3.2
- new net N$47: J7.1, L2.2, R2.2
- net GND: now also D10.A, D14.A, D18.A, D2.A, D20.A, D24.A, J17.4, J19.2, J19.4, J20.2, J20.4, J23.2, J24.2, J28.2, J28.4, J29.4, J3.2, J35.2, J37.4, J39.2, J39.4, J4.2, J40.2, J40.4, J43.2, J44.2, J48.2, J48.4, J49.4, J7.4, J9.4; no longer D27.A, D31.A, D35.A, D37.A, D39.A, D43.A, J12.4, J14.4, J2.4, J22.4, J34.4, J42.4, J53.2, J54.2, J54.4, J57.2, J62.2, J62.4, J65.2, J69.2, J70.2, J70.4, J73.2, J74.2, J74.4, J77.2, J78.2, J78.4, J85.2, J86.2, J86.4
- net N$11: now also J40.1, L20.2, R20.2; no longer J14.1, L7.2, R7.2
- net N$13: now also J19.1, L9.2, R9.2; no longer J16.1, L8.2, R8.2
- net N$19: now also J39.1, L19.2, R19.2; no longer J22.1, L11.2, R11.2
- net N$23: now also J49.1, L24.2, R24.2; no longer J26.1, L13.2, R13.2
- net N$3: now also J20.1, L10.2, R10.2; no longer J6.1, L3.2, R2.2
- net N$31: now also J18.1, L8.2, R8.2; no longer J34.1, L17.2, R17.2
- net N$35: now also J28.1, L13.2, R13.2; no longer J38.1, L19.2, R19.2
- net N$39: now also J38.1, L18.2, R18.2; no longer J42.1, L21.2, R21.2
- net N$43: now also J48.1; no longer J46.1
- net N$5: now also J9.1; no longer J8.1
- net N$53: now also J17.1, L7.2, R7.2; no longer J54.1, L27.2, R27.2
- net N$61: now also J37.1, L17.2, R17.2; no longer J62.1, L31.2, R31.2
- net N$69: now also J6.1, L1.2; no longer J70.1, L35.2
- net N$73: now also J16.1, L6.2, R6.2; no longer J74.1, L37.2, R37.2
- net N$77: now also J26.1, L11.2, R11.2; no longer J78.1, L39.2, R39.2
- net N$85: now also J46.1, L21.2, R21.2; no longer J86.1, L43.2, R43.2
- net N$9: now also J29.1, L14.2, R14.2; no longer J12.1, L6.2, R6.2
- net _SIGOUT1: now also D5.C, J10.3, J5.1, L5.1, R5.1; no longer D1.C, J1.1, J2.3, L1.1, R3.1
- net _SIGOUT11: now also D19.C, J34.1, J39.3, L19.1, R19.1; no longer D11.C, J21.1, J22.3, L11.1, R11.1
- net _SIGOUT13: now also D24.C, J44.1, J49.3, L24.1, R24.1; no longer D13.C, J25.1, J26.3, L13.1, R13.1
- net _SIGOUT15: now also D3.C, J3.1, J8.3, L3.1, R3.1; no longer D15.C, J29.1, J30.3, L15.1, R15.1
- net _SIGOUT17: now also D8.C, J13.1, J18.3, L8.1, R8.1; no longer D17.C, J33.1, J34.3, L17.1, R17.1
- net _SIGOUT19: now also D13.C, J23.1, J28.3, L13.1, R13.1; no longer D19.C, J37.1, J38.3, L19.1, R19.1
- net _SIGOUT21: now also D18.C, J33.1, J38.3, L18.1, R18.1; no longer D21.C, J41.1, J42.3, L21.1, R21.1
- net _SIGOUT23: now also J43.1, J48.3; no longer J45.1, J46.3
- net _SIGOUT25: now also D2.C, J2.1, J7.3, L2.1, R2.1; no longer D25.C, J49.1, J50.3, L25.1, R25.1
- net _SIGOUT27: now also D7.C, J12.1, J17.3, L7.1, R7.1; no longer D27.C, J53.1, J54.3, L27.1, R27.1
- net _SIGOUT29: now also J22.1; no longer J57.1
- net _SIGOUT3: now also D10.C, J15.1, J20.3, L10.1, R10.1; no longer D3.C, J5.1, J6.3, L3.1, R2.1
- net _SIGOUT31: now also D17.C, J37.3, L17.1, R17.1; no longer D31.C, J62.3, L31.1, R31.1
- net _SIGOUT33: now also J42.1; no longer J65.1
- net _SIGOUT35: now also D1.C, J1.1, J6.3, L1.1; no longer D35.C, J69.1, J70.3, L35.1
- net _SIGOUT37: now also D6.C, J11.1, J16.3, L6.1, R6.1; no longer D37.C, J73.1, J74.3, L37.1, R37.1
- net _SIGOUT39: now also D11.C, J21.1, J26.3, L11.1, R11.1; no longer D39.C, J77.1, J78.3, L39.1, R39.1
- net _SIGOUT4: now also J4.1, J9.3; no longer J7.1, J8.3
- net _SIGOUT43: now also D21.C, J41.1, J46.3, L21.1, R21.1; no longer D43.C, J85.1, J86.3, L43.1, R43.1
- net _SIGOUT5: now also D15.C, J25.1, J30.3, L15.1, R15.1; no longer D5.C, J10.3, J9.1, L5.1, R5.1
- net _SIGOUT6: now also D14.C, J24.1, J29.3, L14.1, R14.1; no longer D6.C, J11.1, J12.3, L6.1, R6.1
- net _SIGOUT7: now also D20.C, J35.1, J40.3, L20.1, R20.1; no longer D7.C, J13.1, J14.3, L7.1, R7.1
- net _SIGOUT8: now also D9.C, J14.1, J19.3, L9.1, R9.1; no longer D8.C, J15.1, J16.3, L8.1, R8.1
- net _SIGOUT9: now also D25.C, J45.1, J50.3, L25.1, R25.1; no longer D9.C, J17.1, J18.3, L9.1, R9.1
Other:
- moved on the sheet: D1, D11, D13, D15, D17, D19, D21, D25, D3, D5, D6, D7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

Commit message: headstage-64 rev. 1.4 along with all dependencies
- This is headstage-64 revision 1.4. Because it involves a change in the
bottom analog connector, a lot of other boards had to be changed to
match the new pinout. That is why there are so many files in this
commit. Changes in revision 1.4 and affects on other boards are as
follows:

1. The coaxial adapter board has been improved to allow a regulator to
sit on the daughter board. To do this, the filtered vcoax had to brought
back to the daughter board and then out again after regulation. Of
course this regulation can be bypassed simply by connecting these
contacts

2. Vcoax decoupling has been greatly improved to lower impedance of
power input. There is now 70 uF of decoupling capacitance on the
post-regulated vcoax.

3. The JTAG interface was changed to allow it to be enabled and disabled
by the programmer. This means that these pins are nominally used for
extra IO. The programmer now contains a jumper that allows it operate in
this new mode (closed) or legacy mode (open) for headstage-64 rev 1.3.

4. All of the serializers GPIO lines are now all routed to the FPGA.

5. The opto and estim circuits no longer share SPI lines so they can be
operated independently.

6. The analog routing to the intan chip has been changed such that the
electrode lines are shielded from vcoax, which was polluting the anlog
signals, by a ground pin. This means that eibs etc. need to respect this
new pinout. This is why eib-64, eib-64-large, nanoz-adapter,
omnetics-adapter-64, and test-board-64 have been changed.

7. The serializer on headstage-64 has been upgraded to DS90UB933-Q1
which has reduced back channel latencies, increased forward channel
bandwidth, and improved performance with
imperfect cabling.

8. There is a solder jumper on the bottom of headstage-64 to allow the
addition of an external resistor to AUXIN3 on the intan to allow it to
operate at lower bandwidths. This comes at the cost of not being able to
measure istim unless t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
Parts:
- removed D10, D11, D12, D13, D14, D15, D16, D17, D18, D19, D2, D20, D21, D22, D23, D24, D25, D3, D4, D5, D6, D7, D8, D9: SESD0402X1UN-0020-090, jonnew:Z-DIODE_0402T-DFN
- removed J10, J16, J17, J18, J19, J20, J26, J27, J28, J29, J30, J36, J37, J38, J39, J40, J46, J47, J48, J49, J50, J6, J7, J8, J9: (no value), jonnew:PINHD-1X4HEADSTAGE64-DAUGHTER-CARD-CASTELLATED
- removed J11, J12, J13, J14, J15, J21, J22, J23, J24, J25, J3, J31, J32, J33, J34, J35, J4, J41, J42, J43, J44, J45, J5: X.FL-R-SMT-1(02), jonnew:COAX_XFL
- removed L10, L11, L12, L13, L14, L15, L16, L17, L18, L19, L2, L20, L21, L22, L23, L24, L25, L3, L4, L5, L6, L7, L8, L9: CIG21L4R7MNE, jonnew:L_0805T
- removed R10, R11, R12, R13, R14, R15, R16, R17, R18, R19, R20, R21, R22, R23, R24, R25, R4, R5, R6, R7, R8, R9: 1k, jonnew:R_0201T
- added C1, C2: 10uF, jonnew:C_0402T
- added U1: TPS82085, jonnew:TPS8208X
- J2: value X.FL-R-SMT-1(02) -> (none); device jonnew:COAX_XFL -> jonnew:PINHD-1X5_HEADSTAGE-64-REV1.4-DAUGHTER-CARD-CASTELLATED
- R2: value 1k -> 143k
- R3: value 1k -> 24k
Connections:
- removed net N$11: J40.1, L20.2, R20.2
- removed net N$13: J19.1, L9.2, R9.2
- removed net N$15: J50.1, L25.2, R25.2
- removed net N$19: J39.1, L19.2, R19.2
- removed net N$23: J49.1, L24.2, R24.2
- removed net N$27: J8.1, L3.2, R3.2
- removed net N$3: J20.1, L10.2, R10.2
- removed net N$31: J18.1, L8.2, R8.2
- removed net N$35: J28.1, L13.2, R13.2
- removed net N$39: J38.1, L18.2, R18.2
- removed net N$43: J48.1, L23.2, R23.2
- removed net N$47: J7.1, L2.2, R2.2
- removed net N$5: J9.1, L4.2, R4.2
- removed net N$53: J17.1, L7.2, R7.2
- removed net N$57: J27.1, L12.2, R12.2
- removed net N$61: J37.1, L17.2, R17.2
- removed net N$65: J47.1, L22.2, R22.2
- removed net N$69: J6.1, L1.2, R1.2
- removed net N$7: J30.1, L15.2, R15.2
- removed net N$73: J16.1, L6.2, R6.2
- removed net N$77: J26.1, L11.2, R11.2
- removed net N$81: J36.1, L16.2, R16.2
- removed net N$85: J46.1, L21.2, R21.2
- removed net N$9: J29.1, L14.2, R14.2
- removed net _SIGOUT1: D5.C, J10.3, J5.1, L5.1, R5.1
- removed net _SIGOUT11: D19.C, J34.1, J39.3, L19.1, R19.1
- removed net _SIGOUT13: D24.C, J44.1, J49.3, L24.1, R24.1
- removed net _SIGOUT15: D3.C, J3.1, J8.3, L3.1, R3.1
- removed net _SIGOUT17: D8.C, J13.1, J18.3, L8.1, R8.1
- removed net _SIGOUT19: D13.C, J23.1, J28.3, L13.1, R13.1
- removed net _SIGOUT21: D18.C, J33.1, J38.3, L18.1, R18.1
- removed net _SIGOUT23: D23.C, J43.1, J48.3, L23.1, R23.1
- removed net _SIGOUT25: D2.C, J2.1, J7.3, L2.1, R2.1
- removed net _SIGOUT27: D7.C, J12.1, J17.3, L7.1, R7.1
- removed net _SIGOUT29: D12.C, J22.1, J27.3, L12.1, R12.1
- removed net _SIGOUT3: D10.C, J15.1, J20.3, L10.1, R10.1
- removed net _SIGOUT31: D17.C, J32.1, J37.3, L17.1, R17.1
- removed net _SIGOUT33: D22.C, J42.1, J47.3, L22.1, R22.1
- removed net _SIGOUT35: D1.C, J1.1, J6.3, L1.1, R1.1
- removed net _SIGOUT37: D6.C, J11.1, J16.3, L6.1, R6.1
- removed net _SIGOUT39: D11.C, J21.1, J26.3, L11.1, R11.1
- removed net _SIGOUT4: D4.C, J4.1, J9.3, L4.1, R4.1
- removed net _SIGOUT41: D16.C, J31.1, J36.3, L16.1, R16.1
- removed net _SIGOUT43: D21.C, J41.1, J46.3, L21.1, R21.1
- removed net _SIGOUT5: D15.C, J25.1, J30.3, L15.1, R15.1
- removed net _SIGOUT6: D14.C, J24.1, J29.3, L14.1, R14.1
- removed net _SIGOUT7: D20.C, J35.1, J40.3, L20.1, R20.1
- removed net _SIGOUT8: D9.C, J14.1, J19.3, L9.1, R9.1
- removed net _SIGOUT9: D25.C, J45.1, J50.3, L25.1, R25.1
- new net N$2: R2.1, R3.2, U1.ADJ
- new net SIGOUT: D1.C, J1.1, J2.4, L1.1, R1.1
- new net VCOAX: C2.1, J2.3, R2.2, U1.VOUT
- new net VRAW: C1.1, J2.2, U1.EN, U1.VIN
- net GND: now also C1.2, C2.2, J2.5, R3.1, U1.GND; no longer D10.A, D11.A, D12.A, D13.A, D14.A, D15.A, D16.A, D17.A, D18.A, D19.A, D2.A, D20.A, D21.A, D22.A, D23.A, D24.A, D25.A, D3.A, D4.A, D5.A, D6.A, D7.A, D8.A, D9.A, J10.2, J10.4, J11.2, J12.2, J13.2, J14.2, J15.2, J16.2, J16.4, J17.2, J17.4, J18.2, J18.4, J19.2, J19.4, J2.2, J20.2, J20.4, J21.2, J22.2, J23.2, J24.2, J25.2, J26.2, J26.4, J27.2, J27.4, J28.2, J28.4, J29.2, J29.4, J3.2, J30.2, J30.4, J31.2, J32.2, J33.2, J34.2, J35.2, J36.2, J36.4, J37.2, J37.4, J38.2, J38.4, J39.2, J39.4, J4.2, J40.2, J40.4, J41.2, J42.2, J43.2, J44.2, J45.2, J46.2, J46.4, J47.2, J47.4, J48.2, J48.4, J49.2, J49.4, J5.2, J50.2, J50.4, J6.2, J6.4, J7.2, J7.4, J8.2, J8.4, J9.2, J9.4
- net N$48: now also J2.1, L1.2, R1.2; no longer J10.1, L5.2, R5.2
Other:
- moved on the sheet: D1, J1, L1, R1, R2, R3
