File: fmc-host/fmc-host.sch (EAGLE design)
At the start: 325 parts, among them J9 FMC_SINGLE_WIDTH_MODULE, Q1 SI1012R, Q2 SI1012R, Q3 SI1012R, Q4 SI1012R, U1 NC7WZ07P6X, U10 DS90UB914A-Q1, U11 DS90UB914A-Q1, U12 DS91M040, U13 AD5766BCPZ-RL7, U14 MCP47FEB02A0-E/ST, U15 LM4132AMF-2.5/NOPBCT-ND, U16 AD7617BSTZ, U17 AD5142, U18 LTM4622A, U19 TPS7A49, U2 SN65LVDS9638DGN, U20 TPS7A49, U21 TPS7A30, U22 24AA64ST, U23 LTM8049_BGA, U3 FIN1032MTCX, U4 LTC2875_DFN, U5 ADCMP600, U6 ADCMP600, U7 ADG1434YCPZ, U8 ADG1434YCPZ, U9 ADG1434YCPZ, X2 OE-LOGO_7X5, X3 OE-LOGO_7X5

Commit message: Replace SMD MMCX with thru hole on fmc-host
- Less likely to rip off
- Also, got rid of redundant ground vias around these connectors
Parts:
- CLKI0, CLKI1, CLKO, LINKA, LINKB: device jonnew:COAX_MMCX-RA -> jonnew:COAX_MMCX-THRU
- D10, D11: value (none) -> APFA3011-AK13/F
- J10: value (none) -> ASP-134488-01
- Q1, Q2: device jonnew:N-MOSFET_SOT23-GSD -> jonnew:N-MOSFET_SC75-GSD
- S3: value (none) -> CHS-02TB
- U17: value AD5142 -> AD5142BCPZ10
Changed lines of the file:
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@@
 </classes>
 <parts>
-<part name="CLKI0" library="jonnew" deviceset="COAX" device="_MMCX-RA" value="SMA002"/>
-<part name="CLKO" library="jonnew" deviceset="COAX" device="_MMCX-RA" value="SMA002"/>
+<part name="CLKI0" library="jonnew" deviceset="COAX" device="_MMCX-THRU" value="SMA002"/>
+<part name="CLKO" library="jonnew" deviceset="COAX" device="_MMCX-THRU" value="SMA002"/>
 <part name="C127" library="jonnew" deviceset="C" device="_0402" value="0.1uF"/>
 <part name="C128" library="jonnew" deviceset="C" device="_0402" value="0.1uF"/>
@@
 <part name="R24" library="jonnew" deviceset="R" device="_0402" value="10k"/>
 <part name="C16" library="jonnew" deviceset="C" device="_0402" value="0.1uF"/>
-<part name="CLKI1" library="jonnew" deviceset="COAX" device="_MMCX-RA" value="SMA002"/>
+<part name="CLKI1" library="jonnew" deviceset="COAX" device="_MMCX-THRU" value="SMA002"/>
 <part name="F2" library="jonnew" deviceset="FUSE" device="_1812" value="C014F-2"/>
 <part name="R15" library="jonnew" deviceset="R" device="_0603" value="150,0.25W"/>
@@
 <part name="R72" library="jonnew" deviceset="R" device="_0402" value="2k"/>
 <part name="R73" library="jonnew" deviceset="R" device="_0402" value="2k"/>
-<part name="LINKA" library="jonnew" deviceset="COAX" device="_MMCX-RA" value="SMA002"/>
+<part name="LINKA" library="jonnew" deviceset="COAX" device="_MMCX-THRU" value="SMA002"/>
 <part name="C74" library="jonnew" deviceset="C" device="_0402" value="10nF"/>
 <part name="C77" library="jonnew" deviceset="C" device="_0402" value="0.1uF"/>
@@
 <part name="SUPPLY37" library="jonnew" deviceset="GND" device=""/>
 <part name="SUPPLY50" library="jonnew" deviceset="GND" device=""/>
-<part name="GND1" library="supply1" deviceset="GND" device=""/>
+<part name="GND1" library="jonnew" deviceset="GND" device=""/>
 <part name="SUPPLY51" library="jonnew" deviceset="GND" device=""/>
 <part name="SUPPLY57" library="jonnew" deviceset="GND" device=""/>
@@
 <part name="R27" library="jonnew" deviceset="R" device="_0402" value="1k"/>
 <part name="R11" library="jonnew" deviceset="R" device="_0402" value="1k"/>
-<part name="Q2" library="jonnew" deviceset="N-MOSFET" device="_SOT23-GSD" value="SI1012R"/>
+<part name="Q2" library="jonnew" deviceset="N-MOSFET" device="_SC75-GSD" value="SI1012R"/>
 <part name="R13" library="jonnew" deviceset="R" device="_0402" value="165k"/>
 <part name="D5" library="jonnew" deviceset="Z-DIODE" device="_0402P-DFN" value="SESD0402X1UN-0020-090"/>
@@
 <part name="SUPPLY106" library="jonnew" deviceset="AGND" device=""/>
 <part name="SUPPLY99" library="jonnew" deviceset="AGND" device=""/>
-<part name="J10" library="jonnew" deviceset="FMC_HPC_400_PIN" device="_MALE"/>
+<part name="J10" library="jonnew" deviceset="FMC_HPC_400_PIN" device="_MALE" value="ASP-134488-01"/>
 <part name="SUPPLY155" library="jonnew" deviceset="GND" device=""/>
 <part name="SUPPLY173" library="jonnew" deviceset="GND" device=""/>
 <part name="P44" library="jonnew" deviceset="+3V3" device=""/>
 <part name="SUPPLY151" library="jonnew" deviceset="+12V" device=""/>
-<part name="U17" library="jonnew" deviceset="AD51X2" device="_QFN" value="AD5142"/>
+<part name="U17" library="jonnew" deviceset="AD51X2" device="_QFN" value="AD5142BCPZ10"/>
 <part name="SUPPLY121" library="jonnew" deviceset="GND" device=""/>
 <part name="P41" library="jonnew" deviceset="+3V3" device=""/>
@@
 <part name="SUPPLY74" library="jonnew" deviceset="GND" device=""/>
 <part name="P30" library="jonnew" deviceset="+1V8" device=""/>
-<part name="LINKB" library="jonnew" deviceset="COAX" device="_MMCX-RA" value="SMA002"/>
+<part name="LINKB" library="jonnew" deviceset="COAX" device="_MMCX-THRU" value="SMA002"/>
 <part name="C73" library="jonnew" deviceset="C" device="_0402" value="10nF"/>
 <part name="C76" library="jonnew" deviceset="C" device="_0402" value="0.1uF"/>
@@
 <part name="C55" library="jonnew" deviceset="C" device="_0402" value="10nF"/>
 <part name="R10" library="jonnew" deviceset="R" device="_0402" value="1k"/>
-<part name="Q1" library="jonnew" deviceset="N-MOSFET" device="_SOT23-GSD" value="SI1012R"/>
+<part name="Q1" library="jonnew" deviceset="N-MOSFET" device="_SC75-GSD" value="SI1012R"/>
 <part name="R12" library="jonnew" deviceset="R" device="_0402" value="165k"/>
 <part name="D4" library="jonnew" deviceset="Z-DIODE" device="_0402P-DFN" value="SESD0402X1UN-0020-090"/>
@@
 <part name="C64" library="jonnew" deviceset="C" device="_0402" value="0.1uF"/>
 <part name="SUPPLY101" library="jonnew" deviceset="GND" device=""/>
-<part name="S3" library="jonnew" deviceset="DIPSW-002" device=""/>
+<part name="S3" library="jonnew" deviceset="DIPSW-002" device="" value="CHS-02TB"/>
 <part name="SUPPLY171" library="jonnew" deviceset="GND" device=""/>
 <part name="R95" library="jonnew" deviceset="R" device="_0402" value="10k"/>
@@
 <part name="P50" library="jonnew" deviceset="+3V3" device=""/>
 <part name="P52" library="jonnew" deviceset="+3V3" device=""/>
-<part name="D11" library="jonnew" deviceset="LED_3X" device="_SMD-6"/>
+<part name="D11" library="jonnew" deviceset="LED_3X" device="_SMD-6" value="APFA3011-AK13/F"/>
 <part name="R67" library="jonnew" deviceset="R" device="_0402" value="1k"/>
 <part name="SUPPLY94" library="jonnew" deviceset="GND" device=""/>
 <part name="R66" library="jonnew" deviceset="R" device="_0402" value="1k"/>
-<part name="D10" library="jonnew" deviceset="LED_3X" device="_SMD-6"/>
+<part name="D10" library="jonnew" deviceset="LED_3X" device="_SMD-6" value="APFA3011-AK13/F"/>
 <part name="SUPPLY93" library="jonnew" deviceset="GND" device=""/>
 <part name="SJ1" library="jonnew" deviceset="SJ2" device="_0201"/>
@@
 <instance part="SUPPLY37" gate="PE" x="167.64" y="764.54"/>
 <instance part="SUPPLY50" gate="PE" x="190.5" y="764.54"/>
-<instance part="GND1" gate="1" x="205.74" y="787.4"/>
+<instance part="GND1" gate="PE" x="205.74" y="787.4"/>
 <instance part="SUPPLY51" gate="PE" x="190.5" y="675.64"/>
 <instance part="SUPPLY57" gate="PE" x="205.74" y="701.04"/>
@@
 <wire x1="203.2" y1="795.02" x2="205.74" y2="795.02" width="0.1524" layer="91"/>
 <wire x1="205.74" y1="795.02" x2="205.74" y2="789.94" width="0.1524" layer="91"/>
-<pinref part="GND1" gate="1" pin="GND"/>
-</segment>
-<segment>
+<pinref part="GND1" gate="PE" pin="GND"/>
+</segment>
+<segment>

Commit message: FMC host board rev. 1.3
- Some minor changes after building revision 1.2 and implementing FPGA
design
- DES_A_PCLK moved to positive pin
- Swapped DES_B_D[1] and DES_B_D[2]
- Minor fixes to packages
- BOM simplification
Parts:
- C120, C121, C126, C129, C84, C89: value 22uF -> 47uF
- C29, C30: value 1nF -> 4.7nF
- R52, R54, R57, R59: value 10k -> DNP
- R87, R89: value 15k -> 43k
- S3: device jonnew:DIPSW-002 -> jonnew:DIPSW-002_CHS-02TB
Connections:
- removed net N$70: D3.A, R3.2
- new net N$36: D3.C, R3.1
- net -13V_AN: now also R3.2; no longer D3.C
- net AGND: now also D3.A; no longer R3.1
- net DES_A_PCLK: now also J10G$5.HB06_P_CC; no longer J10G$5.HB06_N_CC
- net DES_B_D1: now also J10G$4.LA24_P; no longer J10G$4.LA25_N
- net DES_B_D2: now also J10G$4.LA25_N; no longer J10G$4.LA24_P
Other:
- moved on the sheet: D3, R3
Changed lines of the file:
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@@
 <attribute name="DESIGN_NAME" value="FMC DESERIALIZER"/>
 <attribute name="LICENSE" value="CERN OHL v1.2"/>
-<attribute name="REVISION" value="1.1"/>
+<attribute name="REVISION" value="1.3"/>
 </attributes>
 <variantdefs>
@@
 <part name="C2" library="jonnew" deviceset="C" device="_0805" value="10uF"/>
 <part name="R7" library="jonnew" deviceset="R" device="_0402" value="10k"/>
-<part name="R54" library="jonnew" deviceset="R" device="_0402" value="10k"/>
-<part name="R59" library="jonnew" deviceset="R" device="_0402" value="10k"/>
+<part name="R54" library="jonnew" deviceset="R" device="_0402" value="DNP"/>
+<part name="R59" library="jonnew" deviceset="R" device="_0402" value="DNP"/>
 <part name="R30" library="jonnew" deviceset="R" device="_0402" value="10k"/>
 <part name="R55" library="jonnew" deviceset="R" device="_0402" value="0"/>
@@
 <part name="R76" library="jonnew" deviceset="R" device="_0402" value="3.16k"/>
 <part name="R75" library="jonnew" deviceset="R" device="_0402" value="3.16k"/>
-<part name="C84" library="jonnew" deviceset="C" device="_1210" value="22uF"/>
-<part name="C89" library="jonnew" deviceset="C" device="_1210" value="22uF"/>
+<part name="C84" library="jonnew" deviceset="C" device="_1210" value="47uF"/>
+<part name="C89" library="jonnew" deviceset="C" device="_1210" value="47uF"/>
 <part name="C56" library="jonnew" deviceset="C" device="_0402" value="10nF"/>
 <part name="P33" library="jonnew" deviceset="+3V3" device=""/>
@@
 <part name="SUPPLY124" library="jonnew" deviceset="GND" device=""/>
 <part name="SUPPLY181" library="jonnew" deviceset="GND" device=""/>
-<part name="C121" library="jonnew" deviceset="C" device="_1210" value="22uF"/>
+<part name="C121" library="jonnew" deviceset="C" device="_1210" value="47uF"/>
 <part name="C122" library="jonnew" deviceset="C" device="_1210" value="47uF"/>
 <part name="R93" library="jonnew" deviceset="R" device="_0402" value="165k"/>
@@
 <part name="C47" library="jonnew" deviceset="C" device="_0805" value="10uF"/>
 <part name="C80" library="jonnew" deviceset="C" device="_0402" value="0.1uF"/>
-<part name="C126" library="jonnew" deviceset="C" device="_1210" value="22uF"/>
-<part name="C120" library="jonnew" deviceset="C" device="_1210" value="22uF"/>
+<part name="C126" library="jonnew" deviceset="C" device="_1210" value="47uF"/>
+<part name="C120" library="jonnew" deviceset="C" device="_1210" value="47uF"/>
 <part name="SUPPLY111" library="jonnew" deviceset="AGND" device=""/>
 <part name="SUPPLY87" library="jonnew" deviceset="AGND" device=""/>
@@
 <part name="C115" library="jonnew" deviceset="C" device="_0402" value="10nF"/>
 <part name="SUPPLY146" library="jonnew" deviceset="GND" device=""/>
-<part name="R87" library="jonnew" deviceset="R" device="_0402" value="15k"/>
+<part name="R87" library="jonnew" deviceset="R" device="_0402" value="43k"/>
 <part name="R88" library="jonnew" deviceset="R" device="_0402" value="4.7k"/>
 <part name="SUPPLY140" library="jonnew" deviceset="GND" device=""/>
@@
 <part name="C116" library="jonnew" deviceset="C" device="_0402" value="10nF"/>
 <part name="SUPPLY147" library="jonnew" deviceset="GND" device=""/>
-<part name="R89" library="jonnew" deviceset="R" device="_0402" value="15k"/>
+<part name="R89" library="jonnew" deviceset="R" device="_0402" value="43k"/>
 <part name="R90" library="jonnew" deviceset="R" device="_0402" value="4.7k"/>
 <part name="SUPPLY141" library="jonnew" deviceset="GND" device=""/>
@@
 <part name="C1" library="jonnew" deviceset="C" device="_0805" value="10uF"/>
 <part name="R6" library="jonnew" deviceset="R" device="_0402" value="10k"/>
-<part name="R52" library="jonnew" deviceset="R" device="_0402" value="10k"/>
-<part name="R57" library="jonnew" deviceset="R" device="_0402" value="10k"/>
+<part name="R52" library="jonnew" deviceset="R" device="_0402" value="DNP"/>
+<part name="R57" library="jonnew" deviceset="R" device="_0402" value="DNP"/>
 <part name="R28" library="jonnew" deviceset="R" device="_0402" value="10k"/>
 <part name="R53" library="jonnew" deviceset="R" device="_0402" value="0"/>
@@
 <part name="C64" library="jonnew" deviceset="C" device="_0402" value="0.1uF"/>
 <part name="SUPPLY101" library="jonnew" deviceset="GND" device=""/>
-<part name="S3" library="jonnew" deviceset="DIPSW-002" device="" value="CHS-02TB"/>
+<part name="S3" library="jonnew" deviceset="DIPSW-002" device="_CHS-02TB" value="CHS-02TB"/>
 <part name="SUPPLY171" library="jonnew" deviceset="GND" device=""/>
 <part name="R95" library="jonnew" deviceset="R" device="_0402" value="10k"/>
@@
 <part name="SUPPLY180" library="jonnew" deviceset="GND" device=""/>
 <part name="SUPPLY178" library="jonnew" deviceset="GND" device=""/>
-<part name="C129" library="jonnew" deviceset="C" device="_1210" value="22uF"/>
+<part name="C129" library="jonnew" deviceset="C" device="_1210" value="47uF"/>
 <part name="P51" library="jonnew" deviceset="+1V8" device=""/>
 <part name="P54" library="jonnew" deviceset="+3V3" device=""/>
@@
 <part name="U3" library="jonnew" deviceset="LVDS_RECEIVER_QUAD" device="_TSSOP" value="FIN1032MTCX"/>
 <part name="U2" library="jonnew" deviceset="LVDS_DRIVER_DUAL" device="_MSOP" value="SN65LVDS9638DGN"/>
-<part name="C30" library="jonnew" deviceset="C" device="_0402" value="1nF"/>
-<part name="C29" library="jonnew" deviceset="C" device="_0402" value="1nF"/>
+<part name="C30" library="jonnew" deviceset="C" device="_0402" value="4.7nF"/>
+<part name="C29" library="jonnew" deviceset="C" device="_0402" value="4.7nF"/>
 <part name="C35" library="jonnew" deviceset="C" device="_0402" value="0.1uF"/>
 <part name="C36" library="jonnew" deviceset="C" device="_0402" value="0.1uF"/>
@@
 <instance part="D2" gate="G$1" x="76.2" y="1211.58"/>
 <instance part="R2" gate="R" x="76.2" y="1224.28" rot="MR90"/>
-<instance part="D3" gate="G$1" x="76.2" y="1170.94"/>
-<instance part="R3" gate="R" x="76.2" y="1181.1" rot="MR270"/>
+<instance part="D3" gate="G$1" x="76.2" y="1186.18"/>
+<instance part="R3" gate="R" x="76.2" y="1170.94" rot="MR270"/>
 <instance part="TP1" gate="G$1" x="48.26" y="1234.44"/>
 <instance part="TP2" gate="G$1" x="88.9" y="1234.44"/>
@@
 <wire x1="76.2" y1="1206.5" x2="76.2" y2="1196.34" width="0.1524" layer="91"/>
 <wire x1="76.2" y1="1196.34" x2="88.9" y2="1196.34" width="0.1524" layer="91"/>
-<wire x1="76.2" y1="1186.18" x2="76.2" y2="1196.34" width="0.1524" layer="91"/>
-<junction x="76.2" y="1196.34"/>
-<pinref part="R3" gate="R" pin="1"/>
 <pinref part="TP3" gate="G$1" pin="TP"/>
 <pinref part="SUPPLY11" gate="G$1" pin="AGND"/>
 <wire x1="88.9" y1="1193.8" x2="88.9" y2="1196.34" width="0.1524" layer="91"/>
 <junction x="88.9" y="1196.34"/>
+<pinref part="D3" gate="G$1" pin="A"/>
+<wire x1="76.2" y1="1196.34" x2="76.2" y2="1188.72" width="0.1524" layer="91"/>
+<junction x="76.2" y="1196.34"/>
 </segment>
 <segment>
@@
 </segment>
 <segment>
-<wire x1="76.2" y1="1165.86" x2="76.2" y2="1163.32" width="0.1524" layer="91"/>
 <label x="76.2" y="1158.24" size="1.27" layer="95" rot="R270" xref="yes"/>
-<pinref part="D3" gate="G$1" pin="C"/>
 <pinref part="TP4" gate="G$1" pin="TP"/>
 <wire x1="76.2" y1="1163.32" x2="76.2" y2="1158.24" width="0.1524" layer="91"/>
 <wire x1="88.9" y1="1163.32" x2="76.2" y2="1163.32" width="0.1524" layer="91"/>
+<pinref part="R3" gate="R" pin="2"/>
+<wire x1="76.2" y1="1165.86" x2="76.2" y2="1163.32" width="0.1524" layer="91"/>
 <junction x="76.2" y="1163.32"/>
 </segment>
@@
 </segment>
 </net>
-<net name="N$70" class="0">
-<segment>
-<pinref part="R3" gate="R" pin="2"/>
-<pinref part="D3" gate="G$1" pin="A"/>
-<wire x1="76.2" y1="1176.02" x2="76.2" y2="1173.48" width="0.1524" layer="91"/>
-</segment>
-</net>
 <net name="DEBUG1" class="0">
 <segment>
@@
 </segment>
 <segment>
-<label x="805.18" y="266.7" size="1.27" layer="95" xref="yes"/>
-<wire x1="805.18" y1="266.7" x2="795.02" y2="266.7" width="0.1524" layer="91"/>
-<pinref part="J10" gate="G$5" pin="HB06_N_CC"/>
+<label x="805.18" y="269.24" size="1.27" layer="95" xref="yes"/>
+<pinref part="J10" gate="G$5" pin="HB06_P_CC"/>
+<wire x1="795.02" y1="269.24" x2="805.18" y2="269.24" width="0.1524" layer="91"/>
 </segment>
 </net>
@@
 </segment>
 <segment>
-<label x="716.28" y="434.34" size="1.27" layer="95" rot="MR0" xref="yes"/>
-<wire x1="716.28" y1="434.34" x2="726.44" y2="434.34" width="0.1524" layer="91"/>
-<pinref part="J10" gate="G$4" pin="LA25_N"/>
+<label x="805.18" y="434.34" size="1.27" layer="95" xref="yes"/>
+<wire x1="795.02" y1="434.34" x2="805.18" y2="434.34" width="0.1524" layer="91"/>
+<pinref part="J10" gate="G$4" pin="LA24_P"/>
 </segment>
 </net>
@@
 </segment>
 <segment>
-<label x="805.18" y="434.34" size="1.27" layer="95" xref="yes"/>
-<wire x1="795.02" y1="434.34" x2="805.18" y2="434.34" width="0.1524" layer="91"/>
-<pinref part="J10" gate="G$4" pin="LA24_P"/>
+<label x="716.28" y="434.34" size="1.27" layer="95" rot="MR0" xref="yes"/>
+<wire x1="716.28" y1="434.34" x2="726.44" y2="434.34" width="0.1524" layer="91"/>
+<pinref part="J10" gate="G$4" pin="LA25_N"/>
 </segment>
 </net>
@@
 </segment>
 </net>
+<net name="N$36" class="0">
+<segment>
+<pinref part="D3" gate="G$1" pin="C"/>
+<pinref part="R3" gate="R" pin="1"/>
+<wire x1="76.2" y1="1181.1" x2="76.2" y2="1176.02" width="0.1524" layer="91"/>
+</segment>
+</net>

Commit message: Updates to fmc-host board when testing revision 1.3
- This is starting revision 1.4
- Replaced SPDT analog switches for analog IO with SPST swiches inline
with the analog outpus. Inputs are always connected. This allows
loopback of analog output instead of wasting the analog input
capabilites when a line is selected to be an output
Parts:
- C106: value 100pF -> 0.1uF
- R75, R76: value 3.16k -> 3.48k
- U7, U8, U9: value ADG1434YCPZ -> DG1412E; device jonnew:ADG1434_QFN -> jonnew:DG141XE_QUAD_SPST_QFN
Connections:
- removed net !AIN_AOUT_EN: J10G$5.HA18_N, U7.!EN, U8.!EN, U9.!EN
- removed net AINA0: R68.C1, U9.S1A
- removed net AINA1: R68.C3, U9.S2A
- removed net AINA2: R68.C5, U9.S3A
- removed net AINA3: R68.C8, U9.S4A
- removed net AINA4: R69.C2, U8.S2A
- removed net AINA5: R69.C4, U8.S1A
- removed net AINB0: R70.C8, U7.S4A
- removed net AINB1: R70.C6, U7.S3A
- removed net AINB2: R70.C4, U7.S2A
- removed net AINB3: R70.C1, U7.S1A
- removed net AINB4: R71.C7, U8.S4A
- removed net AINB5: R71.C5, U8.S3A
- new net $N56: C106.1, R81.1, U16.!RESET
- net !ADC_RESET: no longer C106.1, U16.!RESET
- net +3V3: no longer R81.1
- net AIN_AOUT1: now also U7.IN4; no longer U7.IN2
- net AIN_AOUT10: now also J10G$2.LA05_P, U9.IN4; no longer J10G$3.HA13_P, U9.IN3
- net AIN_AOUT11: now also J10G$3.HA08_N, U9.IN1; no longer J10G$4.LA04_P, U9.IN4
- net AIN_AOUT2: now also J10G$5.HA18_P, U7.IN2; no longer J10G$4.LA15_N, U7.IN3
- net AIN_AOUT3: now also J10G$4.LA15_N, U7.IN3; no longer J10G$5.HA18_P, U7.IN4
- net AIN_AOUT4: now also J10G$3.HA15_N, U8.IN2; no longer J10G$3.HA20_P, U8.IN1
- net AIN_AOUT5: now also J10G$4.LA03_N, U8.IN3; no longer J10G$5.HA07_P, U8.IN2
- net AIN_AOUT6: now also J10G$5.HA07_P, U8.IN4; no longer J10G$4.LA03_N, U8.IN3
- net AIN_AOUT7: now also J10G$3.HA20_P, U8.IN1; no longer J10G$3.HA15_N, U8.IN4
- net AIN_AOUT8: now also J10G$4.LA04_P, U9.IN2; no longer J10G$3.HA08_N, U9.IN1
- net AIN_AOUT9: now also J10G$3.HA13_P, U9.IN3; no longer J10G$2.LA05_P, U9.IN2
- net AIO_0: now also R70.C1
- net AIO_1: now also R70.C4, U7.D4; no longer U7.D2
- net AIO_10: now also R68.C3, U9.D4; no longer U9.D2
- net AIO_11: now also R68.C1
- net AIO_2: now also R70.C8, U7.D2; no longer U7.D4
- net AIO_3: now also R70.C6
- net AIO_4: now also R71.C7, U8.D2; no longer U8.D4
- net AIO_5: now also R71.C5
- net AIO_6: now also R69.C2, U8.D4; no longer U8.D2
- net AIO_7: now also R69.C4
- net AIO_8: now also R68.C8, U9.D2; no longer U9.D4
- net AIO_9: now also R68.C5
- net AOUT0: now also U7.S1; no longer U7.S1B
- net AOUT1: now also U7.S4; no longer U7.S2B
- net AOUT10: now also U9.S4; no longer U9.S2B
- net AOUT11: now also U9.S1; no longer U9.S1B
- net AOUT2: now also U7.S3; no longer U7.S3B
- net AOUT3: now also U7.S2; no longer U7.S4B
- net AOUT4: now also U8.S1; no longer U8.S1B
- net AOUT5: now also U8.S4; no longer U8.S2B
- net AOUT6: now also U8.S2; no longer U8.S4B
- net AOUT7: now also U8.S3; no longer U8.S3B
- net AOUT8: now also U9.S3; no longer U9.S3B
- net AOUT9: now also U9.S2; no longer U9.S4B
Other:
- note added: "NB: 3.48k = 11V output."
- note added: "NB: Freq = 1.48 MHz"
- note added: "NB: VLINK adjust. - Max step down ratio: 1 - (45e-9 *1.48e6) = 0.933 - So max voltage = 11.19 - Linear mode selected - R_AW = 0 : VLINK = 11.0V - R_AW = 5k : VLINK = 5.0V - General: VLINK = 36.24k/(3.48k + R_AW) + 0.6"
- note added: "PIN ADC DAC -------------------------- AIO_0 3B 0 AIO_1 2B 3 AIO_2 0B 2 AIO_3 1B 1 AIO_4 4B 4 AIO_5 5B 6 AIO_6 4A 7 AIO_7 5A 5 AIO_8 3A 11 AIO_9 2A 9 AIO_10 1A 8 AIO_11 0A 10"
- note removed: "JLCPCB 6 layer stackup: 1. Top Copper 0.035 mm P. Prepreg (2313*1) 0.1 mm 2. Inner Copper 0.0175 mm C. Core (Copper) 0.565 mm 3. Inner Copper 0.0175 mm P. Prepeg (2116*1) 0.127 mm 4. Inner Copper 0.0175 mm C. Core (Copper) 0.565 mm 5. Inner Copper 0.0175 mm P. Prepreg (2313*1) 0.1 mm 6. Bottom Copper 0.0175 mm"
- note removed: "NB: 3.16k = 12V output."
- note removed: "NB: VLINK adjust. - Linear mode selected - R_AW = 0 : VLINK = 12V - R_AW = 5k : VLINK = 5.0V - General: VLINK = 36.24k/(3.16k + R_AW) + 0.6"
- moved on the sheet: C112, C113, C115, C116, C118, C119, C121, C122, C132, C133, L1, L14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

Commit message: headstage-neuropix rev 1.2
- Dual neuropixels probe support
- 2X HTC Vive receivers
- Many changes made for reliability of manufacturing
Connections:
- net N$30 renamed LVDS_DIN2_N/CAN_P
- net N$31 renamed LVDS_DIN2_P/CAN_N
- removed net $N56: C106.1, R81.1, U16.!RESET
- net !ADC_RESET: now also C106.1, R81.1, U16.!RESET; no longer R81.2
- net +3V3: now also R81.2
- net AIO_0: now also AUX.7, R68.C1, U9.D1; no longer AUX.25, R70.C1, U7.D1
- net AIO_1: now also AUX.20, R68.C3, U9.D4; no longer AUX.12, R70.C4, U7.D4
- net AIO_10: now also AUX.12, R70.C4, U7.D4; no longer AUX.20, R68.C3, U9.D4
- net AIO_11: now also AUX.25, R70.C1, U7.D1; no longer AUX.7, R68.C1, U9.D1
- net AIO_2: now also AUX.8, R68.C5, U9.D3; no longer AUX.24, R70.C8, U7.D2
- net AIO_3: now also AUX.21, R68.C8, U9.D2; no longer AUX.11, R70.C6, U7.D3
- net AIO_4: now also AUX.9, R69.C4, U8.D1; no longer AUX.23, R71.C7, U8.D2
- net AIO_5: now also AUX.22, R69.C2, U8.D4; no longer AUX.10, R71.C5, U8.D3
- net AIO_6: now also AUX.10, R71.C5, U8.D3; no longer AUX.22, R69.C2, U8.D4
- net AIO_7: now also AUX.23, R71.C7, U8.D2; no longer AUX.9, R69.C4, U8.D1
- net AIO_8: now also AUX.11, R70.C6, U7.D3; no longer AUX.21, R68.C8, U9.D2
- net AIO_9: now also AUX.24, R70.C8, U7.D2; no longer AUX.8, R68.C5, U9.D3
Other:
- note added: "PIN ADC DAC -------------------------- AIO_11 3B 0 AIO_10 2B 1 AIO_9 0B 3 AIO_8 1B 2 AIO_7 4B 6 AIO_6 5B 7 AIO_5 4A 5 AIO_4 5A 4 AIO_3 3A 9 AIO_2 2A 8 AIO_1 1A 10 AIO_0 0A 11"
- note removed: "PIN ADC DAC -------------------------- AIO_0 3B 0 AIO_1 2B 3 AIO_2 0B 2 AIO_3 1B 1 AIO_4 4B 4 AIO_5 5B 6 AIO_6 4A 7 AIO_7 5A 5 AIO_8 3A 11 AIO_9 2A 9 AIO_10 1A 8 AIO_11 0A 10"
- moved on the sheet: C106, R81
