File: fmc-host/fmc-host.sch (EAGLE design)
At the start: 325 parts, among them J10 ASP-134488-01, J9 FMC_SINGLE_WIDTH_MODULE, Q1 SI1012R, Q2 SI1012R, Q3 SI1012R, Q4 SI1012R, U1 NC7WZ07P6X, U10 DS90UB914A-Q1, U11 DS90UB914A-Q1, U12 DS91M040, U13 AD5766BCPZ-RL7, U14 MCP47FEB02A0-E/ST, U15 LM4132AMF-2.5/NOPBCT-ND, U16 AD7617BSTZ, U17 AD5142BCPZ10, U18 LTM4622A, U19 TPS7A49, U2 SN65LVDS9638DGN, U20 TPS7A49, U21 TPS7A30, U22 24AA64ST, U23 LTM8049_BGA, U3 FIN1032MTCX, U4 LTC2875_DFN, U5 ADCMP600, U6 ADCMP600, U7 DG1412E, U8 DG1412E, U9 DG1412E, X2 OE-LOGO_7X5, X3 OE-LOGO_7X5

Commit message: fmc-host board rev. 1.4
- Several small but significant changes to rev. 1.3
- DES LOCK and PASS lines have pull down resistors now to deal with the
fact that they are tri-stated when the DES is in PDN mode
- PDN pin directly driven by FPGA instead of unnecessary FET
Parts:
- removed C1, C2: 10uF, jonnew:C_0805
- removed Q1, Q2: SI1012R, jonnew:N-MOSFET_SC75-GSD
- R10, R11: value 1k -> 165k
Connections:
- removed net DES_A_PDN: J10G$3.HB16_N, R11.2
- removed net DES_B_PDN: J10G$4.LA31_P, R10.2
- removed net N$1: Q2.G, R11.1, R13.2
- removed net N$102: Q1.G, R10.1, R12.2
- removed net N$507: C2.2, Q2.D, R7.2, U11.PDN
- removed net N$600: C1.2, Q1.D, R6.2, U10.PDN
- new net DES_A_PDB: J10G$3.HB16_N, R7.2, U11.PDN
- new net DES_B_PDB: J10G$4.LA31_P, R6.2, U10.PDN
- net DES_A_LOCK: now also R12.2
- net DES_A_PASS: now also R13.2
- net DES_B_LOCK: now also R10.2
- net DES_B_PASS: now also R11.2
- net GND: now also R10.1, R11.1; no longer C1.1, C2.1, Q1.S, Q2.S
Other:
- moved on the sheet: R10, R11, R12, R13, R6, R7

Commit message: fmc-host rev. 1.3
- This revision of the fmc-host board addresses several issues
encountered during testing of revision 1.2
- The deserializers have been upgrated to DS90UB934-Q1s. This increases
the forward channel bandwidth to 14 x 100 MHz and reduces back channel
latency.
- The SPDT analog switches on rev. 1.2 have been replaced with SDST
switches. Analog inputs are perminently connected. So when the anlaog
outputs are selected, they are measured automatically.
- The top ground copper now has thermals to make assembly easier
Parts:
- removed AUX: 12226-8250-00FR, jonnew:PINHD-1X26_122
- removed CLKI0, CLKI1, CLKO: SMA002, jonnew:COAX_MMCX-THRU
- removed Q3, Q4: SI1012R, jonnew:N-MOSFET_SC75-GSD
- removed R89: 43k, jonnew:R_0402
- removed R90: 4.7k, jonnew:R_0402
- removed R91, R92: 2k, jonnew:R_0402
- removed R93: 165k, jonnew:R_0402
- removed R94: 178k, jonnew:R_0402
- removed R95, R96: 10k, jonnew:R_0402
- removed R97, R98: 73.2k, jonnew:R_0402
- added C1, C2: 10uF, jonnew:C_1206
- added C134, C136, C137: 0.1uF, jonnew:C_0402
- added C135: 47uF, jonnew:C_1210
- added C138, C139: 4.7uF, jonnew:C_1206
- added J3, J4, J5: SMA002, jonnew:COAX_MMCX-THRU
- added J7: 12226-8250-00FR, jonnew:PINHD-1X26_122
- added Q1, Q2: SI1012R, jonnew:N-MOSFET_SC75-GSD
- C10, C11, C133, C48, C49, C67, C8, C9: value 4.7uF -> 0.1uF; device jonnew:C_1206 -> jonnew:C_0402
- C102, C94: value 10uF -> 47uF; device jonnew:C_0805 -> jonnew:C_1210
- C103, C105, C108, C123, C124, C125, C64, C71, C77, C96: value 0.1uF -> 10uF; device jonnew:C_0402 -> jonnew:C_0805
- C109, C110, C111, C113, C47, C63, C85, C86, C99: value 10uF -> 0.1uF; device jonnew:C_0805 -> jonnew:C_0402
- C114, C3, C4, C50, C51, C55, C56, C58, C62, C68, C90: value 10nF -> 0.1uF
- C115, C116, C61: value 10nF -> 10uF; device jonnew:C_0402 -> jonnew:C_0805
- C12, C13, C21, C22, C53: value 0.1uF -> 10nF
- C120, C121, C122: value 47uF -> 10nF; device jonnew:C_1210 -> jonnew:C_0402
- C127, C128, C97, C98: value 0.1uF -> 47uF; device jonnew:C_0402 -> jonnew:C_1210
- C129, C84, C89: value 47uF -> 0.1uF; device jonnew:C_1210 -> jonnew:C_0402
- C132: value 4.7uF -> 47uF; device jonnew:C_1206 -> jonnew:C_1210
- C27, C28, C37, C38: value 4.7uF -> 10uF
- C35, C36, C6, C72, C79, C80, C92: value 0.1uF -> 10uF; device jonnew:C_0402 -> jonnew:C_1206
- C42, C44, C75, C76, C88: value 0.1uF -> 1uF; device jonnew:C_0402 -> jonnew:C_0805
- C5: value 0.1uF -> 4.7nF
- C52, C57: value 10uF -> 10nF; device jonnew:C_0805 -> jonnew:C_0402
- C60, C78: value 1uF -> 0.1uF; device jonnew:C_0805 -> jonnew:C_0402
- C69, C70: value 4.7uF -> 1uF
- C7: value 4.7nF -> 10uF; device jonnew:C_0402 -> jonnew:C_1206
- C73, C91: value 10nF -> 10uF; device jonnew:C_0402 -> jonnew:C_1206
- C74: value 10nF -> 1uF; device jonnew:C_0402 -> jonnew:C_0805
- C81: value 10nF -> 4.7uF; device jonnew:C_0402 -> jonnew:C_1206
- L10, L9: value MPZ2012S102AT000 -> BLM18KG601SN1D; device jonnew:L_0805 -> jonnew:L_0603
- L7, L8: value BLM18KG601SN1D -> MPZ2012S102AT000; device jonnew:L_0603 -> jonnew:L_0805
- R10, R11: value 165k -> 150,0.25W; device jonnew:R_0402 -> jonnew:R_0603
- R12, R13: value 165k -> 2k
- R16, R17: value 150,0.25W -> 165k; device jonnew:R_0603 -> jonnew:R_0402
- R18, R19, R65: value 1k -> 10k
- R20, R21: value 150,0.25W -> 1k; device jonnew:R_0603 -> jonnew:R_0402
- R22: value 165k -> 10k
- R23: value 165k -> 3k
- R24: value 10k -> 5.6k 1%
- R25: value 10k -> 21k 1%
- R26, R27: value 1k -> 60 1%
- R28: value 10k -> 49.9
- R29: value 3k -> 49.9
- R30: value 10k -> 100
- R31: value 3k -> 100
- R32: value 60 1% -> 100
- R33: value 60 1% -> 3k
- R36, R37, R38: value 100 -> 4.7k
- R39, R80: value 10k -> 4.7k
- R41, R43: value 10k -> 0
- R44: value 10k -> 3k
- R46: value 49.9 -> 4.7k
- R47: value 49.9 -> 1k
- R49: value 1k -> 4.7k
- R52: value DNP -> 1k
- R53: value 0 -> 1k
- R54: value DNP -> 0
- R55, R58: value 0 -> 165k
- R56: value 3k -> 165k
- R57: value DNP -> 165k
- R59: value DNP -> 2.2k; device jonnew:R_0402 -> jonnew:RN2X8_1506
- R6, R7, R81: value 10k -> 2k
- R60: value 0 -> 2.2k; device jonnew:R_0402 -> jonnew:RN2X8_1506
- R61: value 3k -> 2.2k; device jonnew:R_0402 -> jonnew:RN2X8_1506
- R62: value 1k -> 2.2k; device jonnew:R_0402 -> jonnew:RN2X8_1506
- R63, R64: value 1k -> 2k
- R66, R67: value 1k -> 3.48k
- R68: value 2.2k -> 649k; device jonnew:RN2X8_1506 -> jonnew:R_0402
- R69: value 2.2k -> 0; device jonnew:RN2X8_1506 -> jonnew:R_0402
- R70, R71: value 2.2k -> 10k; device jonnew:RN2X8_1506 -> jonnew:R_0402
- R72, R73: value 2k -> 10k
- R75: value 3.48k -> 15k
- R76: value 3.48k -> 4.7k
- R77: value 649k -> 43k
- R78: value 0 -> 4.7k
- R79: value 10k -> 43k
- R8, R9: value 1k -> 150,0.25W; device jonnew:R_0402 -> jonnew:R_0603
- R82: value 0 -> 2k
- R83: value 10k -> 165k
- R84: value 10k -> 178k
- R85: value 15k -> 10k
- R86: value 4.7k -> 10k
- R87: value 43k -> 73.2k
- R88: value 4.7k -> 73.2k
- U10, U11: value DS90UB914A-Q1 -> DS90UB934-Q1; device jonnew:DS90UB914A-Q1 -> jonnew:DS90UB934-Q1
- renumbered LINKA to J2, LINKB to J1
Connections:
- removed net N$101: R57.2, R58.1, U10.IDX1
- removed net N$400: R44.1, U11.OSS_SEL
- removed net N$401: R42.1, U11.OEN
- removed net N$405: R59.2, R60.1, U11.IDX1
- removed net N$601: R43.1, U10.OSS_SEL
- removed net N$602: R41.1, U10.OEN
- removed net VDDCML0_A: C26.2, C32.2, C38.2, L8.1, U11.VDDCML0
- removed net VDDCML0_B: C25.2, C31.2, C37.2, L7.1, U10.VDDCML0
- removed net VDDCML1_A: C10.2, C4.2, C6.2, L4.1, U11.VDDCML1
- removed net VDDCML1_B: C3.2, C5.2, C8.2, L3.1, U10.VDDCML1
- removed net VDDPLL_A: C49.2, C54.2, C59.2, L12.2, U11.VDDPLL
- removed net VDDPLL_B: C48.2, C53.2, C58.2, L11.2, U10.VDDPLL
- new net N$1: C60.2, C63.2, C70.2, L12.2, U11.VDDIO
- new net N$30: C37.2, C44.2, C49.2, U11.VDD11_D
- new net N$31: C38.2, C45.2, U11.VDD11_DVP
- new net N$45: C68.2, C76.2, C80.2, U11.VDD11_FPD
- new net N$46: C114.1, R72.1, U16.!RESET
- new net N$47: C58.2, C62.2, C69.2, L11.2, U10.VDDIO
- new net N$48: C35.2, C42.2, C48.2, U10.VDD11_D
- new net N$49: C36.2, C43.2, U10.VDD11_DVP
- new net N$50: C67.2, C75.2, C79.2, U10.VDD11_FPD
- new net VDD_FPDX_A: C13.2, C2.2, C22.2, C26.2, C4.2, L4.1, U11.VDD18_FPD0, U11.VDD18_FPD1
- new net VDD_FPDX_B: C1.2, C12.2, C21.2, C25.2, C3.2, L3.1, U10.VDD18_FPD0, U10.VDD18_FPD1
- new net VDD_PX_A: C51.2, C53.2, C56.2, C59.2, C66.2, C73.2, L10.2, U11.VDD18_P0, U11.VDD18_P1
- new net VDD_PX_B: C50.2, C52.2, C55.2, C57.2, C65.2, C72.2, L9.2, U10.VDD18_P0, U10.VDD18_P1
- net !ADC_RESET: now also R72.2; no longer C106.1, R81.1, U16.!RESET
- net $N1: now also R11.2, R29.1, R9.2; no longer R17.2, R21.2, R35.1
- net $N3: now also R10.2, R28.1, R8.2; no longer R16.2, R20.2, R34.1
- net +12V: now also C115.2, C126.2, C129.2, C130.2, J7.1, J7.26, R44.2, R45.2; no longer AUX.1, AUX.26, C109.2, C120.2, C123.2, C124.2, R56.2, R61.2
- net +13V_AN: now also C10.2, C104.2, C105.2, C8.2, C9.2; no longer C12.2, C13.2, C14.2, C98.2, C99.2
- net +15V: now also C127.2, R83.1; no longer C121.2, R93.1
- net +1V8: now also C135.2, C136.2, C137.2, C86.2, C92.2, L10.1, L9.1, R22.1, R24.1, R40.1, R42.1, U10.VDD18, U11.VDD18; no longer C129.2, C130.2, C131.2, C73.2, C74.2, C76.2, C77.2, C81.2, C82.2, C88.2, C90.2, C96.2, C97.2, L11.1, L12.1, L7.2, L8.2, R28.1, R30.1, R52.1, R54.1, R57.1, R59.1, U10.VDDD, U10.VDDR, U10.VDDSSCG, U11.VDDD, U11.VDDR, U11.VDDSSCG
- net +3V3: now also C11.2, C112.2, C113.2, C116.2, C132.2, C133.2, C134.2, C138.1, C139.1, C33.1, C34.1, C74.2, C78.2, C82.2, C89.2, C93.2, C96.2, L11.1, L12.1, R36.2, R37.2, R38.2, R39.2, R46.2, R63.2, R64.2, R69.1, R70.1, R71.1, R85.2, R86.2, U10.OEN, U10.OSS_SEL, U11.OEN, U11.OSS_SEL; no longer C104.2, C107.2, C108.2, C126.2, C127.2, C128.2, C132.1, C133.1, C15.2, C35.1, C36.1, C45.2, C46.2, C50.2, C51.2, C55.2, C56.2, C60.2, C61.2, C62.2, C64.2, C65.2, C66.2, C68.2, C69.2, C70.2, C79.2, C83.2, C86.2, R41.2, R42.2, R43.2, R44.2, R48.2, R50.2, R51.2, R6.1, R7.1, R72.2, R73.2, R78.1, R79.1, R80.1, R81.2, R95.2, R96.2, U10.VDDIO1, U10.VDDIO2, U10.VDDIO3, U11.VDDIO1, U11.VDDIO2, U11.VDDIO3
- net +5V_AN: now also C106.2, C107.2, C61.2, C64.2, C77.2, C81.1, C83.2, C84.2, C85.2, C90.2; no longer C100.2, C101.2, C47.2, C52.2, C57.2, C63.2, C67.1, C72.2, C75.2, C80.2
- net -13V_AN: now also C103.2, C18.2, C19.2, C99.2; no longer C21.2, C22.2, C92.2, C95.2
- net -15V: now also C128.1, R84.1; no longer C122.1, R94.1
- net ADDR0: now also R85.1; no longer R95.1
- net ADDR1: now also R86.1; no longer R96.1
- net AGND: now also C10.1, C103.1, C104.1, C105.1, C106.1, C107.1, C18.1, C19.1, C61.1, C64.1, C77.1, C8.1, C81.2, C83.1, C84.1, C88.1, C9.1, C90.1, J7.13, J7.14, R54.1, R59.C2, R59.C4, R59.C6, R59.C7, R60.C1, R60.C3, R60.C5, R60.C6, R60.C7, R60.C8, R61.C2, R61.C3, R61.C5, R61.C7, R62.C1, R62.C2, R62.C3, R62.C4, R62.C6, R62.C8; no longer AUX.13, AUX.14, C12.1, C13.1, C14.1, C21.1, C22.1, C47.1, C52.1, C57.1, C63.1, C67.2, C72.1, C75.1, C78.1, C80.1, C92.1, C93.1, C94.1, C98.1, R68.C2, R68.C4, R68.C6, R68.C7, R69.C1, R69.C3, R69.C5, R69.C6, R69.C7, R69.C8, R70.C2, R70.C3, R70.C5, R70.C7, R71.C1, R71.C2, R71.C3, R71.C4, R71.C6, R71.C8, R82.1
- net AIO_0: now also J7.7, R59.C1; no longer AUX.7, R68.C1
- net AIO_1: now also J7.20, R59.C3; no longer AUX.20, R68.C3
- net AIO_10: now also J7.12, R61.C4; no longer AUX.12, R70.C4
- net AIO_11: now also J7.25, R61.C1; no longer AUX.25, R70.C1
- net AIO_2: now also J7.8, R59.C5; no longer AUX.8, R68.C5
- net AIO_3: now also J7.21, R59.C8; no longer AUX.21, R68.C8
- net AIO_4: now also J7.9, R60.C4; no longer AUX.9, R69.C4
- net AIO_5: now also J7.22, R60.C2; no longer AUX.22, R69.C2
- net AIO_6: now also J7.10, R62.C5; no longer AUX.10, R71.C5
- net AIO_7: now also J7.23, R62.C7; no longer AUX.23, R71.C7
- net AIO_8: now also J7.11, R61.C6; no longer AUX.11, R70.C6
- net AIO_9: now also J7.24, R61.C8; no longer AUX.24, R70.C8
- net CAN_N: now also R27.2; no longer R33.2
- net CAN_P: now also R26.2; no longer R32.2
- net CLKIN_TERM0: now also R20.1; no longer R26.1
- net CLKIN_TERM1: now also R21.1; no longer R27.1
- net CLKIN_VBIAS_SCL: now also R64.1; no longer R73.1
- net CLKIN_VBIAS_SDA: now also R63.1; no longer R72.1
- net DES_A_GPIO3: now also R49.1, U11.GPIO3/INTB; no longer U11.GPIO3
- net DES_A_LEDG: now also R53.2; no longer R67.2
- net DES_A_LOCK: now also R48.2, R56.2; no longer R12.2, R63.2
- net DES_A_PASS: now also R51.2, R58.2; no longer R13.2, R65.2
- net DES_A_PDB: now also U11.PDB; no longer R7.2, U11.PDN
- net DES_A_SCL: now also R37.1; no longer R49.1
- net DES_A_SDA\: now also R39.1; no longer R51.1
- net DES_B_GPIO3: now also R46.1, U10.GPIO3/INTB; no longer U10.GPIO3
- net DES_B_LEDG: now also R52.2; no longer R66.2
- net DES_B_LOCK: now also R47.2, R55.2; no longer R10.2, R62.2
- net DES_B_PASS: now also R50.2, R57.2; no longer R11.2, R64.2
- net DES_B_PDB: now also U10.PDB; no longer R6.2, U10.PDN
- net DES_B_SCL: now also R36.1; no longer R48.1
- net DES_B_SDA: now also R38.1; no longer R50.1
- net DI_VBIAS0: now also R18.1; no longer R24.1
- net DI_VBIAS1: now also R19.1; no longer R25.1
- net DOUTP_F_A: now also C47.2, R7.2; no longer C43.2, R9.2
- net DOUTP_F_B: now also C46.2, R6.2; no longer C42.2, R8.2
- net GND: now also C1.1, C115.1, C116.1, C12.1, C120.2, C121.2, C128.2, C13.1, C132.1, C133.1, C134.1, C135.1, C136.1, C137.1, C138.2, C139.2, C14.2, C15.2, C2.1, C21.1, C22.1, C31.2, C32.2, C35.1, C36.1, C42.1, C43.1, C5.2, C52.1, C57.1, C63.1, C67.1, C7.1, C72.1, C75.1, C78.1, C80.1, C92.1, C93.1, C94.1, C98.1, J3.2, J4.2, J5.2, J7.PAD1, J7.PAD2, Q1.S, Q2.S, R16.1, R17.1, R23.2, R25.2, R33.1, R34.2, R35.2, R41.2, R43.2, R54.2, R55.1, R56.1, R57.1, R58.1, R68.2, R73.2, R74.2, R76.1, R78.1, R80.1, R87.2, R88.2, U10.GND, U10.RES1, U10.RES2, U11.GND, U11.RES1, U11.RES2; no longer AUX.PAD1, AUX.PAD2, C10.1, C103.1, C104.1, C105.1, C106.2, C107.1, C115.2, C116.2, C120.1, C121.1, C128.1, C132.2, C133.2, C15.1, C18.2, C19.2, C31.1, C32.1, C35.2, C36.2, C46.1, C5.1, C61.1, C64.1, C7.2, C77.1, C8.1, C81.1, C83.1, C84.1, C88.1, C9.1, C90.1, CLKI0.2, CLKI1.2, CLKO.2, Q3.S, Q4.S, R10.1, R11.1, R12.1, R13.1, R22.1, R23.1, R29.2, R31.2, R39.2, R40.2, R45.1, R46.2, R47.2, R53.2, R55.2, R58.2, R60.2, R77.2, R82.2, R83.2, R84.2, R86.1, R88.1, R90.1, R97.2, R98.2, U10.DAP, U10.RES, U10.TESTEN, U11.DAP, U11.RES, U11.TESTEN
- net LINK_A_PWR_EN: now also R74.1; no longer R84.1
- net LINK_B_PWR_EN: now also R73.1; no longer R83.1
- net LVDS_DIN0_N: now also J7.4, R30.1; no longer AUX.4, R36.1
- net LVDS_DIN0_P: now also J7.17, R30.2; no longer AUX.17, R36.2
- net LVDS_DIN1_N: now also J7.16, R31.1; no longer AUX.16, R37.1
- net LVDS_DIN1_P: now also J7.3, R31.2; no longer AUX.3, R37.2
- net LVDS_DIN2_N: now also R32.1; no longer R38.1
- net LVDS_DIN2_N/CAN_P: now also J7.2; no longer AUX.2
- net LVDS_DIN2_P: now also R32.2; no longer R38.2
- net LVDS_DIN2_P/CAN_N: now also J7.15; no longer AUX.15
- net LVDS_DOUT0_N: now also J7.19; no longer AUX.19
- net LVDS_DOUT0_P: now also J7.6; no longer AUX.6
- net LVDS_DOUT1_N: now also J7.18; no longer AUX.18
- net LVDS_DOUT1_P: now also J7.5; no longer AUX.5
- net N$10: now also R66.1; no longer R75.1
- net N$100: now also R40.2, R41.1, U10.IDX; no longer R52.2, R53.1, U10.IDX0
- net N$11: now also J3.1; no longer CLKI0.1
- net N$118: now also R47.1; no longer R62.1
- net N$119: now also R50.1; no longer R64.1
- net N$12: now also C111.2; no longer C105.2
- net N$122: now also R66.2; no longer R75.2
- net N$123: now also R67.2; no longer R76.2
- net N$13: now also R33.2; no longer R45.2
- net N$14: now also J5.1; no longer CLKO.1
- net N$145: now also R68.1; no longer R77.1
- net N$15: now also C123.2; no longer C117.2
- net N$16: now also R53.1; no longer R67.1
- net N$17: now also R87.1; no longer R97.1
- net N$18: now also C14.1, R18.2; no longer C16.1, R24.2
- net N$19: now also R29.2; no longer R35.2
- net N$2: now also Q1.D, R10.1, R8.1; no longer Q3.D, R16.1, R20.1
- net N$20: now also C15.1, R19.2; no longer C17.1, R25.2
- net N$21: now also R13.2, R7.1; no longer R19.2, R9.1
- net N$22: now also C17.1, C7.2, L8.2, R13.1; no longer C11.2, C19.1, L10.2, R19.1
- net N$23: now also R61.1; no longer R70.1
- net N$24: now also C16.1, C6.2, L7.2, R12.1; no longer C18.1, C9.2, L9.2, R18.1
- net N$25: now also R84.2; no longer R94.2
- net N$26: now also R52.1; no longer R66.1
- net N$27: now also C47.1; no longer C43.1
- net N$29: now also R83.2; no longer R93.2
- net N$3: now also R28.2; no longer R34.2
- net N$32: now also R35.1; no longer R47.1
- net N$33: now also C120.1; no longer C114.1
- net N$34: now also Q2.G, R17.2, R21.2; no longer Q4.G, R23.2, R27.2
- net N$37: now also Q1.G, R16.2, R20.2; no longer Q3.G, R22.2, R26.2
- net N$38: now also C46.1; no longer C42.1
- net N$39: now also R61.2; no longer R70.2
- net N$4: now also R12.2, R6.1; no longer R18.2, R8.1
- net N$40: now also R75.1, R76.2; no longer R85.1, R86.2
- net N$402: no longer R40.1
- net N$403: now also R24.2, R25.1; no longer R30.2, R31.1
- net N$404: now also R42.2, R43.1, U11.IDX; no longer R54.2, R55.1, U11.IDX0
- net N$41: now also C5.1, R26.1, R27.1; no longer C7.1, R32.1, R33.1
- net N$42: now also C124.2; no longer C118.2
- net N$43: now also C121.1; no longer C115.1
- net N$5: now also R67.1; no longer R76.1
- net N$500: now also C117.2, R75.2; no longer C111.2, R85.2
- net N$501: now also C118.2, R77.2; no longer C112.2, R87.2
- net N$502: now also C119.2, R79.2; no longer C113.2, R89.2
- net N$506: now also C100.2, R65.1; no longer C93.2, R74.1
- net N$53: now also R48.1; no longer R63.1
- net N$54: now also R51.1; no longer R65.1
- net N$56: now also R77.1, R78.2; no longer R87.1, R88.2
- net N$58: now also C125.2; no longer C119.2
- net N$59: now also C122.1; no longer C116.1
- net N$6: now also J4.1; no longer CLKI1.1
- net N$60: now also R79.1, R80.2; no longer R89.1, R90.2
- net N$603: no longer R39.1
- net N$604: now also R22.2, R23.1; no longer R28.2, R29.1
- net N$61: now also R71.2; no longer R80.2
- net N$62: now also R59.1; no longer R68.1
- net N$63: now also R70.2; no longer R79.2
- net N$64: now also C95.2; no longer C85.2
- net N$65: now also R59.2; no longer R68.2
- net N$67: now also C108.2; no longer C102.2
- net N$68: now also R61.8; no longer R70.8
- net N$69: now also C101.2; no longer C94.2
- net N$7: now also Q2.D, R11.1, R9.1; no longer Q4.D, R17.1, R21.1
- net N$71: now also R69.2; no longer R78.2
- net N$72: now also R62.7; no longer R71.7
- net N$73: now also R62.1; no longer R71.1
- net N$74: now also R61.7; no longer R70.7
- net N$75: now also R61.6; no longer R70.6
- net N$76: now also R61.5; no longer R70.5
- net N$77: now also R61.4; no longer R70.4
- net N$78: now also R61.3; no longer R70.3
- net N$79: now also R59.3; no longer R68.3
- net N$8: now also C109.2; no longer C103.2
- net N$80: now also R59.4; no longer R68.4
- net N$81: now also R59.5; no longer R68.5
- net N$82: now also R59.6; no longer R68.6
- net N$83: now also R59.8; no longer R68.8
- net N$84: now also R59.7; no longer R68.7
- net N$85: now also R60.2; no longer R69.2
- net N$86: now also R60.1; no longer R69.1
- net N$87: now also R60.4; no longer R69.4
- net N$88: now also R60.3; no longer R69.3
- net N$89: now also R60.5; no longer R69.5
- net N$9: now also R88.1; no longer R98.1
- net N$90: now also R60.6; no longer R69.6
- net N$91: now also R60.7; no longer R69.7
- net N$92: now also R60.8; no longer R69.8
- net N$93: now also R34.1; no longer R46.1
- net N$94: now also R62.8; no longer R71.8
- net N$95: now also R62.5; no longer R71.5
- net N$96: now also R62.6; no longer R71.6
- net N$97: now also R62.4; no longer R71.4
- net N$98: now also R62.3; no longer R71.3
- net N$99: now also R62.2; no longer R71.2
- net SCL: now also R81.1; no longer R91.1
- net SDA: now also R82.1; no longer R92.1
- net VAUX: now also C131.2, R81.2, R82.2; no longer C125.2, R91.2, R92.2
- net VLINK_A: now also C32.1, C94.2, C97.2, L8.1; no longer C34.1, C84.2, L10.1
- net VLINK_B: now also C102.2, C31.1, C98.2, L7.1; no longer C33.1, C89.2, L9.1
- net VREF: now also C88.2, R65.2; no longer C78.2, R74.2
- net V_PROTECT: now also C54.2, R44.1, R45.1; no longer C44.2, R56.1, R61.1
Other:
- moved on the sheet: C10, C100, C101, C102, C103, C104, C105, C106, C107, C108, C109, C11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

Commit message: Minor BOM simplifications to fmc-host rev. 1.3
Parts:
- removed J10: ASP-134488-01, jonnew:FMC_HPC_400_PIN_MALE
- added C140, C141: 10uF, jonnew:C_1206
- added X4: FMC_SINGLE_WIDTH_MODULE, jonnew:FMC_SINGLE_WIDTH_MODULE
- C138, C139, C81: value 4.7uF -> 10uF
- C69, C70: device jonnew:C_1206 -> jonnew:C_0805
- J9: value FMC_SINGLE_WIDTH_MODULE -> ASP-134488-01; device jonnew:FMC_SINGLE_WIDTH_MODULE -> jonnew:FMC_HPC_400_PIN_MALE
- R1: value 1.6k -> 2k
- R2, R3: value 3.9k -> 4.7k
Connections:
- removed net N$1: C60.2, C63.2, C70.2, L12.2, U11.VDDIO
- new net N$200: C140.2, C60.2, C63.2, C70.2, L12.2, U11.VDDIO
- net !ADC_CS: now also J9G$4.LA07_P; no longer J10G$4.LA07_P
- net !ADC_RESET: now also J9G$3.HA08_P; no longer J10G$3.HA08_P
- net !DAC_CS: now also J9G$5.HA14_N; no longer J10G$5.HA14_N
- net !DAC_RESET: now also J9G$3.HA12_N; no longer J10G$3.HA12_N
- net !LINK_PWR_ADJ_CS: now also J9G$3.HB20_N; no longer J10G$3.HB20_N
- net !LINK_PWR_ADJ_RESET: now also J9G$3.HB21_N; no longer J10G$3.HB21_N
- net +12V: now also J9G$2.12P0V1, J9G$2.12P0V2; no longer J10G$2.12P0V1, J10G$2.12P0V2
- net +1V8: now also J9G$3.VADJ@1, J9G$3.VADJ@2, J9G$4.VADJ@1, J9G$4.VADJ@2; no longer J10G$3.VADJ@1, J10G$3.VADJ@2, J10G$4.VADJ@1, J10G$4.VADJ@2
- net +3V3: now also J9G$2.3P3V1, J9G$2.3P3V2, J9G$2.3P3V3, J9G$2.3P3V4; no longer J10G$2.3P3V1, J10G$2.3P3V2, J10G$2.3P3V3, J10G$2.3P3V4
- net ADC_BUSY: now also J9G$5.HA11_P; no longer J10G$5.HA11_P
- net ADC_CONVST: now also J9G$5.HA10_P; no longer J10G$5.HA10_P
- net ADC_MISO_A: now also J9G$5.HA06_N; no longer J10G$5.HA06_N
- net ADC_MISO_B: now also J9G$5.HA07_N; no longer J10G$5.HA07_N
- net ADC_MOSI: now also J9G$5.HA06_P; no longer J10G$5.HA06_P
- net ADC_SCLK: now also J9G$5.HA11_N; no longer J10G$5.HA11_N
- net ADDR0: now also J9G$2.LA27_N; no longer J10G$2.LA27_N
- net ADDR1: now also J9G$2.LA27_P; no longer J10G$2.LA27_P
- net AIN_AOUT0: now also J9G$4.LA15_P; no longer J10G$4.LA15_P
- net AIN_AOUT1: now also J9G$4.LA16_N; no longer J10G$4.LA16_N
- net AIN_AOUT10: now also J9G$2.LA05_P; no longer J10G$2.LA05_P
- net AIN_AOUT11: now also J9G$3.HA08_N; no longer J10G$3.HA08_N
- net AIN_AOUT2: now also J9G$5.HA18_P; no longer J10G$5.HA18_P
- net AIN_AOUT3: now also J9G$4.LA15_N; no longer J10G$4.LA15_N
- net AIN_AOUT4: now also J9G$3.HA15_N; no longer J10G$3.HA15_N
- net AIN_AOUT5: now also J9G$4.LA03_N; no longer J10G$4.LA03_N
- net AIN_AOUT6: now also J9G$5.HA07_P; no longer J10G$5.HA07_P
- net AIN_AOUT7: now also J9G$3.HA20_P; no longer J10G$3.HA20_P
- net AIN_AOUT8: now also J9G$4.LA04_P; no longer J10G$4.LA04_P
- net AIN_AOUT9: now also J9G$3.HA13_P; no longer J10G$3.HA13_P
- net CAN_RX: now also J9G$5.HA02_N; no longer J10G$5.HA02_N
- net CAN_TX: now also J9G$5.HA02_P; no longer J10G$5.HA02_P
- net CLKIN0: now also J9G$2.LA17_N_CC; no longer J10G$2.LA17_N_CC
- net CLKIN1: now also J9G$3.HA20_N; no longer J10G$3.HA20_N
- net CLKIN_TERM0: now also J9G$5.HA21_P; no longer J10G$5.HA21_P
- net CLKIN_TERM1: now also J9G$5.HA17_N_CC; no longer J10G$5.HA17_N_CC
- net CLKIN_VBIAS_SCL: now also J9G$5.HA22_P; no longer J10G$5.HA22_P
- net CLKIN_VBIAS_SDA: now also J9G$5.HA21_N; no longer J10G$5.HA21_N
- net CLKOUT: now also J9G$2.LA17_P_CC; no longer J10G$2.LA17_P_CC
- net DAC_MISO: now also J9G$5.HA17_P_CC; no longer J10G$5.HA17_P_CC
- net DAC_MOSI: now also J9G$4.LA07_N; no longer J10G$4.LA07_N
- net DAC_SCLK: now also J9G$5.HA14_P; no longer J10G$5.HA14_P
- net DEBUG0: now also J9G$2.LA06_P; no longer J10G$2.LA06_P
- net DEBUG1: now also J9G$2.LA06_N; no longer J10G$2.LA06_N
- net DEBUG2: now also J9G$2.LA09_P; no longer J10G$2.LA09_P
- net DEBUG3: now also J9G$2.LA10_P; no longer J10G$2.LA10_P
- net DEBUG4: now also J9G$2.LA09_N; no longer J10G$2.LA09_N
- net DEBUG5: now also J9G$2.LA10_N; no longer J10G$2.LA10_N
- net DEBUG6: now also J9G$2.LA14_P; no longer J10G$2.LA14_P
- net DEBUG7: now also J9G$2.LA14_N; no longer J10G$2.LA14_N
- net DES_A_D0: now also J9G$3.HB16_P; no longer J10G$3.HB16_P
- net DES_A_D1: now also J9G$5.HB14_N; no longer J10G$5.HB14_N
- net DES_A_D10: now also J9G$5.HB11_N; no longer J10G$5.HB11_N
- net DES_A_D11: now also J9G$5.HB10_P; no longer J10G$5.HB10_P
- net DES_A_D2: now also J9G$5.HB15_N; no longer J10G$5.HB15_N
- net DES_A_D3: now also J9G$5.HB14_P; no longer J10G$5.HB14_P
- net DES_A_D4: now also J9G$3.HB19_P; no longer J10G$3.HB19_P
- net DES_A_D5: now also J9G$5.HB15_P; no longer J10G$5.HB15_P
- net DES_A_D6: now also J9G$3.HB12_N; no longer J10G$3.HB12_N
- net DES_A_D7: now also J9G$3.HB13_N; no longer J10G$3.HB13_N
- net DES_A_D8: now also J9G$5.HB10_N; no longer J10G$5.HB10_N
- net DES_A_D9: now also J9G$3.HB12_P; no longer J10G$3.HB12_P
- net DES_A_GPIO0: now also J9G$5.HB18_N; no longer J10G$5.HB18_N
- net DES_A_GPIO1: now also J9G$5.HB17_P_CC; no longer J10G$5.HB17_P_CC
- net DES_A_GPIO2: now also J9G$5.HB18_P; no longer J10G$5.HB18_P
- net DES_A_GPIO3: now also J9G$3.HB19_N; no longer J10G$3.HB19_N
- net DES_A_HSYNC: now also J9G$3.HB13_P; no longer J10G$3.HB13_P
- net DES_A_LEDG: now also J9G$3.HB08_P; no longer J10G$3.HB08_P
- net DES_A_LOCK: now also J9G$3.HB09_P; no longer J10G$3.HB09_P
- net DES_A_PASS: now also J9G$5.HB07_N; no longer J10G$5.HB07_N
- net DES_A_PCLK: now also J9G$5.HB06_P_CC; no longer J10G$5.HB06_P_CC
- net DES_A_PDB: now also J9G$3.HB16_N; no longer J10G$3.HB16_N
- net DES_A_SCL: now also J9G$3.HB08_N; no longer J10G$3.HB08_N
- net DES_A_SDA\: now also J9G$3.HB09_N; no longer J10G$3.HB09_N
- net DES_A_VSYNC: now also J9G$5.HB11_P; no longer J10G$5.HB11_P
- net DES_B_D0: now also J9G$4.LA24_N; no longer J10G$4.LA24_N
- net DES_B_D1: now also J9G$4.LA24_P; no longer J10G$4.LA24_P
- net DES_B_D10: now also J9G$4.LA22_P; no longer J10G$4.LA22_P
- net DES_B_D11: now also J9G$2.LA23_P; no longer J10G$2.LA23_P
- net DES_B_D2: now also J9G$4.LA25_N; no longer J10G$4.LA25_N
- net DES_B_D3: now also J9G$4.LA25_P; no longer J10G$4.LA25_P
- net DES_B_D4: now also J9G$2.LA26_N; no longer J10G$2.LA26_N
- net DES_B_D5: now also J9G$2.LA26_P; no longer J10G$2.LA26_P
- net DES_B_D6: now also J9G$4.LA21_N; no longer J10G$4.LA21_N
- net DES_B_D7: now also J9G$4.LA22_N; no longer J10G$4.LA22_N
- net DES_B_D8: now also J9G$4.LA21_P; no longer J10G$4.LA21_P
- net DES_B_D9: now also J9G$2.LA23_N; no longer J10G$2.LA23_N
- net DES_B_GPIO0: now also J9G$4.LA28_N; no longer J10G$4.LA28_N
- net DES_B_GPIO1: now also J9G$4.LA29_N; no longer J10G$4.LA29_N
- net DES_B_GPIO2: now also J9G$4.LA28_P; no longer J10G$4.LA28_P
- net DES_B_GPIO3: now also J9G$4.LA29_P; no longer J10G$4.LA29_P
- net DES_B_HSYNC\: now also J9G$4.LA19_N; no longer J10G$4.LA19_N
- net DES_B_LEDG: now also J9G$4.LA20_P; no longer J10G$4.LA20_P
- net DES_B_LOCK: now also J9G$5.HA22_N; no longer J10G$5.HA22_N
- net DES_B_PASS: now also J9G$5.HA23_P; no longer J10G$5.HA23_P
- net DES_B_PCLK: now also J9G$2.LA18_P_CC; no longer J10G$2.LA18_P_CC
- net DES_B_PDB: now also J9G$4.LA31_P; no longer J10G$4.LA31_P
- net DES_B_SCL: now also J9G$4.LA20_N; no longer J10G$4.LA20_N
- net DES_B_SDA: now also J9G$4.LA19_P; no longer J10G$4.LA19_P
- net DES_B_VSYNC: now also J9G$5.HA23_N; no longer J10G$5.HA23_N
- net GND: now also C140.1, C141.1, J9G$1.GND@1, J9G$1.GND@10, J9G$1.GND@11, J9G$1.GND@12, J9G$1.GND@13, J9G$1.GND@14, J9G$1.GND@15, J9G$1.GND@16, J9G$1.GND@17, J9G$1.GND@18, J9G$1.GND@19, J9G$1.GND@2, J9G$1.GND@20, J9G$1.GND@21, J9G$1.GND@22, J9G$1.GND@23, J9G$1.GND@24, J9G$1.GND@25, J9G$1.GND@26, J9G$1.GND@27, J9G$1.GND@28, J9G$1.GND@29, J9G$1.GND@3, J9G$1.GND@30, J9G$1.GND@31, J9G$1.GND@32, J9G$1.GND@33, J9G$1.GND@34, J9G$1.GND@35, J9G$1.GND@36, J9G$1.GND@37, J9G$1.GND@38, J9G$1.GND@39, J9G$1.GND@4, J9G$1.GND@40, J9G$1.GND@5, J9G$1.GND@6, J9G$1.GND@7, J9G$1.GND@8, J9G$1.GND@9, J9G$2.GA0, J9G$2.GA1, J9G$2.GND@1, J9G$2.GND@10, J9G$2.GND@11, J9G$2.GND@12, J9G$2.GND@13, J9G$2.GND@14, J9G$2.GND@15, J9G$2.GND@16, J9G$2.GND@17, J9G$2.GND@18, J9G$2.GND@19, J9G$2.GND@2, J9G$2.GND@20, J9G$2.GND@21, J9G$2.GND@23, J9G$2.GND@24, J9G$2.GND@25, J9G$2.GND@26, J9G$2.GND@27, J9G$2.GND@28, J9G$2.GND@29, J9G$2.GND@3, J9G$2.GND@30, J9G$2.GND@31, J9G$2.GND@33, J9G$2.GND@4, J9G$2.GND@5, J9G$2.GND@6, J9G$2.GND@7, J9G$2.GND@8, J9G$2.GND@9, J9G$3.GND@1, J9G$3.GND@10, J9G$3.GND@11, J9G$3.GND@12, J9G$3.GND@13, J9G$3.GND@14, J9G$3.GND@15, J9G$3.GND@16, J9G$3.GND@17, J9G$3.GND@18, J9G$3.GND@19, J9G$3.GND@21, J9G$3.GND@22, J9G$3.GND@23, J9G$3.GND@24, J9G$3.GND@25, J9G$3.GND@26, J9G$3.GND@27, J9G$3.GND@28, J9G$3.GND@29, J9G$3.GND@3, J9G$3.GND@4, J9G$3.GND@5, J9G$3.GND@6, J9G$3.GND@7, J9G$3.GND@8, J9G$3.GND@9, J9G$4.GND@1, J9G$4.GND@10, J9G$4.GND@11, J9G$4.GND@12, J9G$4.GND@13, J9G$4.GND@14, J9G$4.GND@15, J9G$4.GND@16, J9G$4.GND@17, J9G$4.GND@18, J9G$4.GND@19, J9G$4.GND@2, J9G$4.GND@20, J9G$4.GND@21, J9G$4.GND@22, J9G$4.GND@23, J9G$4.GND@24, J9G$4.GND@25, J9G$4.GND@26, J9G$4.GND@27, J9G$4.GND@28, J9G$4.GND@3, J9G$4.GND@4, J9G$4.GND@5, J9G$4.GND@6, J9G$4.GND@7, J9G$4.GND@8, J9G$4.GND@9, J9G$5.GND@1, J9G$5.GND@10, J9G$5.GND@11, J9G$5.GND@12, J9G$5.GND@13, J9G$5.GND@14, J9G$5.GND@15, J9G$5.GND@16, J9G$5.GND@17, J9G$5.GND@18, J9G$5.GND@19, J9G$5.GND@2, J9G$5.GND@20, J9G$5.GND@21, J9G$5.GND@22, J9G$5.GND@23, J9G$5.GND@24, J9G$5.GND@25, J9G$5.GND@26, J9G$5.GND@27, J9G$5.GND@28, J9G$5.GND@29, J9G$5.GND@3, J9G$5.GND@4, J9G$5.GND@5, J9G$5.GND@6, J9G$5.GND@7, J9G$5.GND@8, J9G$5.GND@9; no longer J10G$1.GND@1, J10G$1.GND@10, J10G$1.GND@11, J10G$1.GND@12, J10G$1.GND@13, J10G$1.GND@14, J10G$1.GND@15, J10G$1.GND@16, J10G$1.GND@17, J10G$1.GND@18, J10G$1.GND@19, J10G$1.GND@2, J10G$1.GND@20, J10G$1.GND@21, J10G$1.GND@22, J10G$1.GND@23, J10G$1.GND@24, J10G$1.GND@25, J10G$1.GND@26, J10G$1.GND@27, J10G$1.GND@28, J10G$1.GND@29, J10G$1.GND@3, J10G$1.GND@30, J10G$1.GND@31, J10G$1.GND@32, J10G$1.GND@33, J10G$1.GND@34, J10G$1.GND@35, J10G$1.GND@36, J10G$1.GND@37, J10G$1.GND@38, J10G$1.GND@39, J10G$1.GND@4, J10G$1.GND@40, J10G$1.GND@5, J10G$1.GND@6, J10G$1.GND@7, J10G$1.GND@8, J10G$1.GND@9, J10G$2.GA0, J10G$2.GA1, J10G$2.GND@1, J10G$2.GND@10, J10G$2.GND@11, J10G$2.GND@12, J10G$2.GND@13, J10G$2.GND@14, J10G$2.GND@15, J10G$2.GND@16, J10G$2.GND@17, J10G$2.GND@18, J10G$2.GND@19, J10G$2.GND@2, J10G$2.GND@20, J10G$2.GND@21, J10G$2.GND@23, J10G$2.GND@24, J10G$2.GND@25, J10G$2.GND@26, J10G$2.GND@27, J10G$2.GND@28, J10G$2.GND@29, J10G$2.GND@3, J10G$2.GND@30, J10G$2.GND@31, J10G$2.GND@33, J10G$2.GND@4, J10G$2.GND@5, J10G$2.GND@6, J10G$2.GND@7, J10G$2.GND@8, J10G$2.GND@9, J10G$3.GND@1, J10G$3.GND@10, J10G$3.GND@11, J10G$3.GND@12, J10G$3.GND@13, J10G$3.GND@14, J10G$3.GND@15, J10G$3.GND@16, J10G$3.GND@17, J10G$3.GND@18, J10G$3.GND@19, J10G$3.GND@21, J10G$3.GND@22, J10G$3.GND@23, J10G$3.GND@24, J10G$3.GND@25, J10G$3.GND@26, J10G$3.GND@27, J10G$3.GND@28, J10G$3.GND@29, J10G$3.GND@3, J10G$3.GND@4, J10G$3.GND@5, J10G$3.GND@6, J10G$3.GND@7, J10G$3.GND@8, J10G$3.GND@9, J10G$4.GND@1, J10G$4.GND@10, J10G$4.GND@11, J10G$4.GND@12, J10G$4.GND@13, J10G$4.GND@14, J10G$4.GND@15, J10G$4.GND@16, J10G$4.GND@17, J10G$4.GND@18, J10G$4.GND@19, J10G$4.GND@2, J10G$4.GND@20, J10G$4.GND@21, J10G$4.GND@22, J10G$4.GND@23, J10G$4.GND@24, J10G$4.GND@25, J10G$4.GND@26, J10G$4.GND@27, J10G$4.GND@28, J10G$4.GND@3, J10G$4.GND@4, J10G$4.GND@5, J10G$4.GND@6, J10G$4.GND@7, J10G$4.GND@8, J10G$4.GND@9, J10G$5.GND@1, J10G$5.GND@10, J10G$5.GND@11, J10G$5.GND@12, J10G$5.GND@13, J10G$5.GND@14, J10G$5.GND@15, J10G$5.GND@16, J10G$5.GND@17, J10G$5.GND@18, J10G$5.GND@19, J10G$5.GND@2, J10G$5.GND@20, J10G$5.GND@21, J10G$5.GND@22, J10G$5.GND@23, J10G$5.GND@24, J10G$5.GND@25, J10G$5.GND@26, J10G$5.GND@27, J10G$5.GND@28, J10G$5.GND@29, J10G$5.GND@3, J10G$5.GND@4, J10G$5.GND@5, J10G$5.GND@6, J10G$5.GND@7, J10G$5.GND@8, J10G$5.GND@9
- net LINK_A_PWR_EN: now also J9G$4.LA32_P; no longer J10G$4.LA32_P
- net LINK_B_PWR_EN: now also J9G$5.HB17_N_CC; no longer J10G$5.HB17_N_CC
- net LINK_PWR_ADJ_MISO: now also J9G$3.HB20_P; no longer J10G$3.HB20_P
- net LINK_PWR_ADJ_MOSI: now also J9G$3.HB21_P; no longer J10G$3.HB21_P
- net LINK_PWR_ADJ_SCLK: now also J9G$4.LA32_N; no longer J10G$4.LA32_N
- net LVDS_DIN0: now also J9G$5.CLK1_C2M_P; no longer J10G$5.CLK1_C2M_P
- net LVDS_DIN1: now also J9G$4.CLK0_M2C_N; no longer J10G$4.CLK0_M2C_N
- net LVDS_DIN2: now also J9G$4.CLK0_M2C_P; no longer J10G$4.CLK0_M2C_P
- net LVDS_DOUT0: now also J9G$5.CLK1_C2M_N; no longer J10G$5.CLK1_C2M_N
- net LVDS_DOUT1: now also J9G$5.CLK1_M2C_P; no longer J10G$5.CLK1_M2C_P
- net MLDVS_EN: now also J9G$4.LA02_N; no longer J10G$4.LA02_N
- net MLDVS_RO0: now also J9G$4.CLK0_C2M_P; no longer J10G$4.CLK0_C2M_P
- net MLDVS_RO1: now also J9G$3.HA01_N_CC; no longer J10G$3.HA01_N_CC
- net MLDVS_RO2: now also J9G$4.LA00_N_CC; no longer J10G$4.LA00_N_CC
- net MLDVS_RO3: now also J9G$3.HA00_P_CC; no longer J10G$3.HA00_P_CC
- net MLVDS_DE_!RE0: now also J9G$3.HA04_P; no longer J10G$3.HA04_P
- net MLVDS_DE_!RE1: now also J9G$3.HA05_N; no longer J10G$3.HA05_N
- net MLVDS_DE_!RE2: now also J9G$4.LA02_P; no longer J10G$4.LA02_P
- net MLVDS_DE_!RE3: now also J9G$3.HA04_N; no longer J10G$3.HA04_N
- net MLVDS_DI0: now also J9G$4.CLK0_C2M_N; no longer J10G$4.CLK0_C2M_N
- net MLVDS_DI1: now also J9G$3.HA01_P_CC; no longer J10G$3.HA01_P_CC
- net MLVDS_DI2: now also J9G$4.LA00_P_CC; no longer J10G$4.LA00_P_CC
- net MLVDS_DI3: now also J9G$3.HA00_N_CC; no longer J10G$3.HA00_N_CC
- net N$47: now also C141.2
- net SCL: now also J9G$2.SCL; no longer J10G$2.SCL
- net SDA: now also J9G$2.SDA; no longer J10G$2.SDA
- net TDI-TDO: now also J9G$2.TDI, J9G$2.TDO; no longer J10G$2.TDI, J10G$2.TDO
- net VAUX: now also J9G$2.3P3VAUX; no longer J10G$2.3P3VAUX
Other:
- moved on the sheet: C58, C60, C62, C63, C69, C70

Commit message: Address Filipe's suggestions prior to fabrication
- Use grid of cream bloks under QFN center pads instead of one large
one. Place vias between these blocks where possible
- Improve silk layer readability
- Move copper away from dimension in several areas
- Add SMD mount files
Parts:
- D1, D2, D3: value (none) -> HSMG-C280
- J6: value (none) -> ESHF-105-01-L-D-SM-K-TR
- J8: value (none) -> 95278-101A16LF
Connections:
- net DOUTP_F_A: now also J1.1; no longer J2.1
- net DOUTP_F_B: now also J2.1; no longer J1.1
Other:
- moved on the sheet: J1, J2
Changed lines of the file:
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@@
 <part name="R63" library="jonnew" deviceset="R" device="_0402" value="2k"/>
 <part name="R64" library="jonnew" deviceset="R" device="_0402" value="2k"/>
-<part name="J2" library="jonnew" deviceset="COAX" device="_MMCX-THRU" value="SMA002"/>
+<part name="J1" library="jonnew" deviceset="COAX" device="_MMCX-THRU" value="SMA002"/>
 <part name="C87" library="jonnew" deviceset="C" device="_0402" value="0.1uF"/>
 <part name="C49" library="jonnew" deviceset="C" device="_0402" value="0.1uF"/>
@@
 <part name="SUPPLY98" library="jonnew" deviceset="GND" device=""/>
 <part name="SUPPLY106" library="jonnew" deviceset="GND" device=""/>
-<part name="D1" library="jonnew" deviceset="LED" device="_0402"/>
+<part name="D1" library="jonnew" deviceset="LED" device="_0402" value="HSMG-C280"/>
 <part name="R1" library="jonnew" deviceset="R" device="_0402" value="2k"/>
-<part name="D2" library="jonnew" deviceset="LED" device="_0402"/>
+<part name="D2" library="jonnew" deviceset="LED" device="_0402" value="HSMG-C280"/>
 <part name="R2" library="jonnew" deviceset="R" device="_0402" value="4.7k"/>
-<part name="D3" library="jonnew" deviceset="LED" device="_0402"/>
+<part name="D3" library="jonnew" deviceset="LED" device="_0402" value="HSMG-C280"/>
 <part name="R3" library="jonnew" deviceset="R" device="_0402" value="4.7k"/>
 <part name="TP1" library="jonnew" deviceset="TP" device="B1,27"/>
@@
 <part name="TP6" library="jonnew" deviceset="TP" device="B1,27"/>
 <part name="TP7" library="jonnew" deviceset="TP" device="B1,27"/>
-<part name="J8" library="jonnew" deviceset="PINHD-2X8" device="_SMD"/>
+<part name="J8" library="jonnew" deviceset="PINHD-2X8" device="_SMD" value="95278-101A16LF"/>
 <part name="SUPPLY163" library="jonnew" deviceset="GND" device=""/>
 <part name="R65" library="jonnew" deviceset="R" device="_0402" value="10k"/>
@@
 <part name="SUPPLY36" library="jonnew" deviceset="GND" device=""/>
 <part name="SUPPLY85" library="jonnew" deviceset="GND" device=""/>
-<part name="J1" library="jonnew" deviceset="COAX" device="_MMCX-THRU" value="SMA002"/>
+<part name="J2" library="jonnew" deviceset="COAX" device="_MMCX-THRU" value="SMA002"/>
 <part name="C62" library="jonnew" deviceset="C" device="_0402" value="0.1uF"/>
 <part name="C69" library="jonnew" deviceset="C" device="_0805" value="1uF"/>
@@
 <part name="R26" library="jonnew" deviceset="R" device="_0402" value="60 1%"/>
 <part name="P14" library="jonnew" deviceset="+3V3" device=""/>
-<part name="J6" library="jonnew" deviceset="PINHD-2X5" device="_ESHF-SM"/>
+<part name="J6" library="jonnew" deviceset="PINHD-2X5" device="_ESHF-SM" value="ESHF-105-01-L-D-SM-K-TR"/>
 <part name="U12" library="jonnew" deviceset="DS91M040" device="_WQFN32" value="DS91M040"/>
 <part name="P24" library="jonnew" deviceset="+3V3" device=""/>
@@
 <instance part="R63" gate="R" x="421.64" y="779.78" rot="R90"/>
 <instance part="R64" gate="R" x="429.26" y="779.78" rot="R90"/>
-<instance part="J2" gate="G$1" x="45.72" y="78.74"/>
+<instance part="J1" gate="G$1" x="45.72" y="78.74"/>
 <instance part="C87" gate="C" x="403.86" y="259.08" rot="R180"/>
 <instance part="C49" gate="C" x="246.38" y="248.92" rot="R180"/>
@@
 <instance part="SUPPLY36" gate="PE" x="160.02" y="124.46" rot="MR0"/>
 <instance part="SUPPLY85" gate="PE" x="287.02" y="71.12"/>
-<instance part="J1" gate="G$1" x="45.72" y="312.42"/>
+<instance part="J2" gate="G$1" x="45.72" y="312.42"/>
 <instance part="C62" gate="C" x="330.2" y="365.76" rot="R180"/>
 <instance part="C69" gate="C" x="340.36" y="365.76" rot="R180"/>
@@
 <wire x1="48.26" y1="76.2" x2="58.42" y2="76.2" width="0.1524" layer="91"/>
 <wire x1="58.42" y1="76.2" x2="58.42" y2="60.96" width="0.1524" layer="91"/>
-<pinref part="J2" gate="G$1" pin="2"/>
+<pinref part="J1" gate="G$1" pin="2"/>
 <pinref part="SUPPLY2" gate="PE" pin="GND"/>
 </segment>
@@
 <wire x1="48.26" y1="309.88" x2="58.42" y2="309.88" width="0.1524" layer="91"/>
 <wire x1="58.42" y1="309.88" x2="58.42" y2="294.64" width="0.1524" layer="91"/>
-<pinref part="J1" gate="G$1" pin="2"/>
+<pinref part="J2" gate="G$1" pin="2"/>
 <pinref part="SUPPLY1" gate="PE" pin="GND"/>
 </segment>
@@
 <label x="63.5" y="96.52" size="1.27" layer="95" rot="MR270"/>
 <wire x1="233.68" y1="203.2" x2="60.96" y2="203.2" width="0.1524" layer="91"/>
-<pinref part="J2" gate="G$1" pin="1"/>
+<pinref part="J1" gate="G$1" pin="1"/>
 <wire x1="60.96" y1="78.74" x2="48.26" y2="78.74" width="0.1524" layer="91"/>
 <wire x1="60.96" y1="203.2" x2="60.96" y2="78.74" width="0.1524" layer="91"/>
@@
 <label x="63.5" y="332.74" size="1.27" layer="95" rot="MR270"/>
 <wire x1="233.68" y1="436.88" x2="60.96" y2="436.88" width="0.1524" layer="91"/>
-<pinref part="J1" gate="G$1" pin="1"/>
+<pinref part="J2" gate="G$1" pin="1"/>
 <wire x1="60.96" y1="312.42" x2="48.26" y2="312.42" width="0.1524" layer="91"/>
 <wire x1="60.96" y1="436.88" x2="60.96" y2="312.42" width="0.1524" layer="91"/>
